Commit message: Removing and fixing some URDFs

File: mara_description/urdf/common.gazebo.xacro (robot description, xacro)
@@ -2,25 +2,4 @@
 <robot xmlns:xacro="http://ros.org/wiki/xacro">
   <gazebo>
-    <plugin name="ros_control" filename="libgazebo_ros_control.so">
-      <!--robotNamespace>/</robotNamespace-->
-      <!--robotSimType>gazebo_ros_control/DefaultRobotHWSim</robotSimType-->
-      <legacyModeNS>true</legacyModeNS>
-      <robotNamespace>/</robotNamespace>
-      <robotSimType>gazebo_ros_control/DefaultRobotHWSim</robotSimType>
-    </plugin>
-<!--
-    <plugin name="gazebo_ros_power_monitor_controller" filename="libgazebo_ros_power_monitor.so">
-      <alwaysOn>true</alwaysOn>
-      <updateRate>1.0</updateRate>
-      <timeout>5</timeout>
-      <powerStateTopic>power_state</powerStateTopic>
-      <powerStateRate>10.0</powerStateRate>
-      <fullChargeCapacity>87.78</fullChargeCapacity>
-      <dischargeRate>-474</dischargeRate>
-      <chargeRate>525</chargeRate>
-      <dischargeVoltage>15.52</dischargeVoltage>
-      <chargeVoltage>16.41</chargeVoltage>
-    </plugin>
--->
   </gazebo>
 </robot>

File: mara_description/urdf/mara_robot_camera_top.urdf (robot description, URDF)
Before this commit: robot mara, 21 links, 20 joints
Links:
- removed link left_inner_finger
- removed link left_inner_knuckle
- removed link left_outer_finger
- removed link left_outer_knuckle
- removed link right_inner_finger
- removed link right_inner_knuckle
- removed link right_outer_finger
- removed link right_outer_knuckle
- removed link robotiq_arg2f_base_link
Joints:
- removed joint end_effector_adapter_to_robotiq
- removed joint left_inner_finger_joint
- removed joint left_inner_knuckle_joint
- removed joint left_outer_finger_joint
- removed joint left_outer_knuckle_joint
- removed joint right_inner_finger_joint
- removed joint right_inner_knuckle_joint
- removed joint right_outer_finger_joint
- removed joint right_outer_knuckle_joint

File: mara_description/urdf/mara_robot_camera_top.urdf.xacro (robot description, xacro)
@@ -8,17 +8,17 @@
   <!-- robotiq 140 gripper -->
   <xacro:include filename="$(find mara_description)/urdf/robotiq_gripper.urdf.xacro" />
-  <!-- <xacro:include filename="$(find mara_description)/urdf/camera_top.urdf.xacro" /> -->
+  <xacro:include filename="$(find mara_description)/urdf/camera_top.urdf.xacro" />
   <xacro:include filename="$(find mara_description)/urdf/table.urdf.xacro" />
   <!-- arm -->
   <xacro:mara_robot prefix="" joint_limited="false"/>
-  <xacro:robotiq_gripper prefix="" />
-  <!-- <xacro:mara_camera_top prefix="" /> -->
+  <!-- <xacro:robotiq_gripper prefix="" /> -->
+  <xacro:mara_camera_top prefix="" />
   <xacro:table prefix="" />
   <link name="world" />
-  <joint name="end_effector_adapter_to_robotiq" type="fixed">
+  <!-- <joint name="end_effector_adapter_to_robotiq" type="fixed">
     <origin rpy="0 0 0" xyz=" 0 0 0.05375"/>
     <parent link="motor6_link"/>
     <child link="robotiq_arg2f_base_link"/>
-  </joint>
+  </joint> -->
   <joint name="world_to_table_joint" type="fixed">
     <origin rpy="0 0 0" xyz="0 0 0.02"/>
