Commit message: Updating xacro model

File: mara_description/urdf/mara_robot_camera_top.urdf (robot description, URDF)
Before this commit: robot mara, 12 links, 11 joints
Links:
- added link left_inner_finger, mass 0.0104003125914103; collision mesh filename=package://robotiq_140_gripper_description/meshes/robotiq_ar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 scale=0.001 0.001 0.001; visual mesh filename=package://robotiq_140_gripper_description/meshes/robotiq_ar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 scale=0.001 0.001 0.001
- added link left_inner_knuckle, mass 0.0271177346495152; visual mesh filename=package://robotiq_140_gripper_description/meshes/robotiq_ar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
- added link left_outer_finger, mass 0.022614240507152; collision mesh filename=package://robotiq_140_gripper_description/meshes/robotiq_ar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; visual mesh filename=package://robotiq_140_gripper_description/meshes/robotiq_ar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
- added link left_outer_knuckle, mass 0.00853198276973456; collision mesh filename=package://robotiq_140_gripper_description/meshes/robotiq_ar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; visual mesh filename=package://robotiq_140_gripper_description/meshes/robotiq_ar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
- added link right_inner_finger, mass 0.0104003125914103; collision mesh filename=package://robotiq_140_gripper_description/meshes/robotiq_ar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 scale=0.001 0.001 0.001; visual mesh filename=package://robotiq_140_gripper_description/meshes/robotiq_ar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 scale=0.001 0.001 0.001
- added link right_inner_knuckle, mass 0.0271177346495152; visual mesh filename=package://robotiq_140_gripper_description/meshes/robotiq_ar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
- added link right_outer_finger, mass 0.022614240507152; collision mesh filename=package://robotiq_140_gripper_description/meshes/robotiq_ar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; visual mesh filename=package://robotiq_140_gripper_description/meshes/robotiq_ar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
- added link right_outer_knuckle, mass 0.00853198276973456; collision mesh filename=package://robotiq_140_gripper_description/meshes/robotiq_ar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; visual mesh filename=package://robotiq_140_gripper_description/meshes/robotiq_ar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
- added link robotiq_arg2f_base_link, mass 0.22652; collision mesh filename=package://robotiq_140_gripper_description/meshes/GRIPPER_ba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 scale=0.001 0.001 0.001; visual mesh filename=package://robotiq_140_gripper_description/meshes/GRIPPER_ba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 scale=0.001 0.001 0.001
Joints:
- added joint end_effector_adapter_to_robotiq: type fixed, parent motor6_link, child robotiq_arg2f_base_link, origin xyz= 0 0 0.05375 rpy=0 0 0
- added joint left_inner_finger_joint: type revolute, parent left_outer_finger, child left_inner_finger, origin xyz=0 0.0817554015893473 -0.0282203446692936 rpy=-.725 0 0, axis 1 0 0, limit lower=0 upper=0.8757 effort=1000 velocity=2.0
- added joint left_inner_knuckle_joint: type revolute, parent robotiq_arg2f_base_link, child left_inner_knuckle, origin xyz=0 -0.0127 0.06142 rpy=2.29579632679 0 0, axis -1 0 0, limit lower=0 upper=0.8757 effort=1000 velocity=2.0, mimic joint=left_outer_knuckle_joint multiplier=-1 offset=0
- added joint left_outer_finger_joint: type revolute, parent left_outer_knuckle, child left_outer_finger, origin xyz=0 0.01821998610742 0.0260018192872234 rpy=0 0 0, axis 1 0 0, limit lower=-2 upper=2 effort=1000 velocity=2.0
- added joint left_outer_knuckle_joint: type revolute, parent robotiq_arg2f_base_link, child left_outer_knuckle, origin xyz=0 -0.030601 0.054905 rpy=2.29579632679 0 0, axis -1 0 0, limit lower=0 upper=0.775 effort=1000 velocity=2.0
- added joint right_inner_finger_joint: type revolute, parent right_outer_finger, child right_inner_finger, origin xyz=0 0.0817554015893473 -0.0282203446692936 rpy=-.725 0 0, axis 1 0 0, limit lower=0 upper=0.8757 effort=1000 velocity=2.0
- added joint right_inner_knuckle_joint: type revolute, parent robotiq_arg2f_base_link, child right_inner_knuckle, origin xyz=0 0.0127 0.06142 rpy=2.29579632679 0  -3.14, axis -1 0 0, limit lower=0 upper=0.8757 effort=1000 velocity=2.0, mimic joint=right_outer_knuckle_joint multiplier=-1 offset=0
- added joint right_outer_finger_joint: type revolute, parent right_outer_knuckle, child right_outer_finger, origin xyz=0 0.01821998610742 0.0260018192872234 rpy=0 0 0, axis -1 0 0, limit lower=-2 upper=2 effort=1000 velocity=2.0
- added joint right_outer_knuckle_joint: type revolute, parent robotiq_arg2f_base_link, child right_outer_knuckle, origin xyz=0 0.030601 0.054905 rpy=2.29579632679 0 3.14, axis -1 0 0, limit lower=0 upper=0.775 effort=1000 velocity=2.0

File: mara_description/urdf/mara_robot_camera_top.urdf.xacro (robot description, xacro)
@@ -3,22 +3,22 @@
        name="mara" >
   <!-- common stuff -->
-  <xacro:include filename="$(find mara_description)/urdf/common.gazebo.xacro" />
+  <xacro:include filename="$(find mara_description)/urdf/mara_gazebo.urdf.xacro" />
   <!-- mara -->
   <xacro:include filename="$(find mara_description)/urdf/mara.urdf.xacro" />
   <!-- robotiq 140 gripper -->
-  <xacro:include filename="$(find mara_description)/urdf/robotiq_gripper.urdf.xacro" />
-  <xacro:include filename="$(find mara_description)/urdf/camera_top.urdf.xacro" />
+  <xacro:include filename="$(find robotiq_140_gripper_description)/urdf/robotiq_gripper.urdf.xacro" />
+  <!-- <xacro:include filename="$(find mara_description)/urdf/camera_top.urdf.xacro" /> -->
   <xacro:include filename="$(find mara_description)/urdf/table.urdf.xacro" />
   <!-- arm -->
   <xacro:mara_robot prefix="" joint_limited="false"/>
-  <!-- <xacro:robotiq_gripper prefix="" /> -->
-  <xacro:mara_camera_top prefix="" />
+  <xacro:robotiq_gripper prefix="" />
+  <!-- <xacro:mara_camera_top prefix="" /> -->
   <xacro:table prefix="" />
   <link name="world" />
-  <!-- <joint name="end_effector_adapter_to_robotiq" type="fixed">
+  <joint name="end_effector_adapter_to_robotiq" type="fixed">
     <origin rpy="0 0 0" xyz=" 0 0 0.05375"/>
     <parent link="motor6_link"/>
     <child link="robotiq_arg2f_base_link"/>
-  </joint> -->
+  </joint>
   <joint name="world_to_table_joint" type="fixed">
     <origin rpy="0 0 0" xyz="0 0 0.02"/>

Commit message: Fixing gripper issues

File: mara_description/urdf/mara_robot_camera_top.urdf (robot description, URDF)
Before this commit: robot mara, 21 links, 20 joints
Links:
- link table: mass .0 -> 0.00001
Joints:
- joint left_inner_finger_joint: limit lower=0 upper=0.8757 effort=1000 velocity=2.0 -> lower=-0.875 upper=0.8757 effort=1000 velocity=2.0
- joint left_outer_knuckle_joint: limit lower=0 upper=0.775 effort=1000 velocity=2.0 -> lower=-2 upper=2 effort=1000 velocity=2.0
- joint right_inner_finger_joint: limit lower=0 upper=0.8757 effort=1000 velocity=2.0 -> lower=-0.875 upper=0.8757 effort=1000 velocity=2.0
- joint right_outer_knuckle_joint: limit lower=0 upper=0.775 effort=1000 velocity=2.0 -> lower=-2 upper=2 effort=1000 velocity=2.0

File: robotiq_140_gripper_description/urdf/robotiq_gripper.urdf.xacro (robot description, xacro)
@@ -6,5 +6,5 @@
         <origin xyz="8.625E-08 -4.6583E-06 0.03145" rpy="0 0 0" />
         <mass value="0.22652" />
-        <inertia ixx="0.00020005" ixy="-4.2442E-10" ixz="-2.9069E-10" iyy="0.00017832" iyz="-3.4402E-08" izz="0.00013478" />
+        <inertia ixx="0.00020005" ixy="0" ixz="0" iyy="0.00017832" iyz="0" izz="0.00013478" />
       </inertial>
       <visual>
@@ -30,13 +30,13 @@
     <link name="left_outer_knuckle">
       <inertial>
-        <origin xyz="-0.000200000000003065 0.0199435877845359 0.0292245259211331" rpy="0 0 0" />
+        <!--<origin xyz="-0.000200000000003065 0.0199435877845359 0.0292245259211331" rpy="0 0 0" />-->
         <mass value="0.00853198276973456" />
         <inertia
-            ixx="2.89328108496468E-06"
-            ixy="-1.57935047237397E-19"
-            ixz="-1.93980378593255E-19"
-            iyy="1.86719750325683E-06"
-            iyz="-1.21858577871576E-06"
-            izz="1.21905238907251E-06" />
+            ixx="2.88840278e-09"
+            ixy="0"
+            ixz="0"
+            iyy="2.80689245e-10"
+            iyz="0"
+            izz="2.79961804e-09" />
       </inertial>
       <visual>
@@ -62,13 +62,13 @@
     <link name="right_outer_knuckle">
       <inertial>
-        <origin xyz="-0.000200000000003065 0.0199435877845359 0.0292245259211331" rpy="0 0 0" />
+        <origin xyz="0 0 0" rpy="0 0 0" />
         <mass value="0.00853198276973456" />
         <inertia
-            ixx="2.89328108496468E-06"
-            ixy="-1.57935047237397E-19"
-            ixz="-1.93980378593255E-19"
-            iyy="1.86719750325683E-06"
-            iyz="-1.21858577871576E-06"
-            izz="1.21905238907251E-06" />
+            ixx="2.88840278e-09"
+            ixy="0"
+            ixz="0"
+            iyy="2.80689245e-10"
+            iyz="0"
+            izz="2.79961804e-09" />
       </inertial>
       <visual>
@@ -94,12 +94,12 @@
     <link name="left_inner_knuckle">
       <inertial>
-        <origin xyz="0.000123011831763771 0.0507850843201817 0.00103968640075166" rpy="0 0 0" />
+        <origin xyz="0 0 0" rpy="0 0 0" />
         <mass value="0.0271177346495152" />
         <inertia
             ixx="2.61910379223783E-05"
-            ixy="-2.43616858946494E-07"
-            ixz="-6.37789906117123E-09"
+            ixy="0"
+            ixz="0"
             iyy="2.8270243746167E-06"
-            iyz="-5.37200748039765E-07"
+            iyz="0"
             izz="2.83695868220296E-05" />
       </inertial>
@@ -120,12 +120,12 @@
     <link name="right_inner_knuckle">
       <inertial>
-        <origin xyz="0.000123011831763771 0.0507850843201817 0.00103968640075166" rpy="0 0 0" />
+        <origin xyz="0 0 0" rpy="0 0 0" />
         <mass value="0.0271177346495152" />
         <inertia
             ixx="2.61910379223783E-05"
-            ixy="-2.43616858946494E-07"
-            ixz="-6.37789906117123E-09"
+            ixy="0"
+            ixz="0"
             iyy="2.8270243746167E-06"
-            iyz="-5.37200748039765E-07"
+            iyz="0"
             izz="2.83695868220296E-05" />
       </inertial>
@@ -146,12 +146,12 @@
     <link name="left_inner_finger">
       <inertial>
-        <origin xyz="0.000299999999999317 0.0160078233491243 -0.0136945669206257" rpy="0 0 0" />
+        <origin xyz="0 0 0" rpy="0 0 0" />
         <mass value="0.0104003125914103" />
         <inertia
             ixx="2.71909453810972E-06"
-            ixy="1.35402465472579E-21"
-            ixz="-7.1817349065269E-22"
+            ixy="0"
+            ixz="0"
             iyy="7.69100314106116E-07"
-            iyz="6.74715432769696E-07"
+            iyz="0"
             izz="2.30315190420171E-06" />
       </inertial>
@@ -174,17 +174,17 @@
     <gazebo reference="left_inner_finger">
       <material>Gazebo/Grey</material>
-      <selfCollide>False</selfCollide>
+      <selfCollide>True</selfCollide>
     </gazebo>
     <link name="right_inner_finger">
       <inertial>
-        <origin xyz="0.000299999999999317 0.0160078233491243 -0.0136945669206257" rpy="0 0 0" />
+        <origin xyz="0.0 0.031506174 -0.017648840" rpy="0 0 0" />
         <mass value="0.0104003125914103" />
         <inertia
-            ixx="2.71909453810972E-06"
-            ixy="1.35402465472579E-21"
-            ixz="-7.1817349065269E-22"
-            iyy="7.69100314106116E-07"
-            iyz="6.74715432769696E-07"
-            izz="2.30315190420171E-06" />
+            ixx="6.06863499e-06"
+            ixy="0"
+            ixz="0"
+            iyy="7.46305064e-07"
+            iyz="0"
+            izz="6.21796490e-06" />
       </inertial>
       <visual>
@@ -206,16 +206,16 @@
     <gazebo reference="right_inner_finger">
       <material>Gazebo/Grey</material>
-      <selfCollide>False</selfCollide>
+      <selfCollide>True</selfCollide>
     </gazebo>
     <link name="left_outer_finger">
       <inertial>
-        <origin xyz="0.00030115855001899 0.0373907951953854 -0.0208027427000385" rpy="0 0 0" />
+        <origin xyz="0 0 0" rpy="0 0 0" />
         <mass value="0.022614240507152" />
         <inertia
             ixx="1.52518312458174E-05"
-            ixy="9.76583423954399E-10"
-            ixz="-5.43838577022588E-10"
+            ixy="0"
+            ixz="0"
             iyy="6.17694243867776E-06"
-            iyz="6.78636130740228E-06"
+            iyz="0"
             izz="1.16494917907219E-05" />
       </inertial>
@@ -242,12 +242,12 @@
     <link name="right_outer_finger">
       <inertial>
-        <origin xyz="0.00030115855001899 0.0373907951953854 -0.0208027427000385" rpy="0 0 0" />
+        <origin xyz="-0.0002009,  0.0396149, -0.0161363" rpy="0 0 0" />
         <mass value="0.022614240507152" />
         <inertia
             ixx="1.52518312458174E-05"
-            ixy="9.76583423954399E-10"
-            ixz="-5.43838577022588E-10"
+            ixy="0"
+            ixz="0"
             iyy="6.17694243867776E-06"
-            iyz="6.78636130740228E-06"
+            iyz="0"
             izz="1.16494917907219E-05" />
       </inertial>
@@ -278,5 +278,5 @@
       <child link="left_outer_knuckle" />
       <axis xyz="-1 0 0" />
-      <limit lower="0" upper="0.775" velocity="2.0" effort="1000" />
+      <limit lower="-2" upper="2" velocity="2.0" effort="1000" />
     </joint>
 <!-- OK -->
@@ -286,5 +286,5 @@
       <child link="right_outer_knuckle" />
       <axis xyz="-1 0 0" />
-      <limit lower="0" upper="0.775" velocity="2.0" effort="1000" />
+      <limit lower="-2" upper="2" velocity="2.0" effort="1000" />
     </joint>
 <!-- OK -->
@@ -325,5 +325,5 @@
       <child link="left_inner_finger" />
       <axis xyz="1 0 0" />
-      <limit lower="0" upper="0.8757" velocity="2.0" effort="1000" />
+      <limit lower="-0.875" upper="0.8757" velocity="2.0" effort="1000" />
     </joint>
     <joint name="right_inner_finger_joint" type="revolute">
@@ -332,11 +332,11 @@
       <child link="right_inner_finger" />
       <axis xyz="1 0 0" />
-      <limit lower="0" upper="0.8757" velocity="2.0" effort="1000" />
+      <limit lower="-0.875" upper="0.8757" velocity="2.0" effort="1000" />
     </joint>
     <gazebo>
       <joint name="left_inner_finger_knuckle_joint" type="revolute">
         <pose frame="">0 0.006 -0.018 0 0 0</pose>
-        <parent>robot::left_inner_knuckle</parent>
-        <child>robot::left_inner_finger</child>
+        <parent>mara::left_inner_knuckle</parent>
+        <child>mara::left_inner_finger</child>
         <axis>
           <xyz>0 1 0</xyz>
@@ -351,6 +351,6 @@
       <joint name="right_inner_finger_knuckle_joint" type="revolute">
         <pose frame="">0 0.006 -0.018 0 0 0</pose>
-        <parent>robot::right_inner_knuckle</parent>
-        <child>robot::right_inner_finger</child>
+        <parent>mara::right_inner_knuckle</parent>
+        <child>mara::right_inner_finger</child>
         <axis>
           <xyz>0 1 0</xyz>

Commit message: Updating mara URDF

File: mara_description/urdf/mara_robot_camera_top.urdf (robot description, URDF)
Before this commit: robot mara, 21 links, 20 joints
Joints:
- joint left_inner_knuckle_joint: limit lower=0 upper=0.8757 effort=1000 velocity=2.0 -> lower=0 upper=0.87 effort=1000 velocity=2.0; origin xyz=0 -0.0127 0.06142 rpy=2.29579632679 0 0 -> xyz=0 -0.0127 0.06142 rpy=2.29 0 0
- joint left_outer_finger_joint: axis 1 0 0 -> -1 0 0; limit lower=-2 upper=2 effort=1000 velocity=2.0 -> lower=0.1 upper=0.875 effort=1000 velocity=2.0
- joint left_outer_knuckle_joint: limit lower=-2 upper=2 effort=1000 velocity=2.0 -> lower=0 upper=0.875 effort=1000 velocity=2.0; origin xyz=0 -0.030601 0.054905 rpy=2.29579632679 0 0 -> xyz=0 -0.030601 0.054905 rpy=2.31 0 0
- joint right_inner_knuckle_joint: limit lower=0 upper=0.8757 effort=1000 velocity=2.0 -> lower=0 upper=0.87 effort=1000 velocity=2.0; origin xyz=0 0.0127 0.06142 rpy=2.29579632679 0  -3.14 -> xyz=0 0.0127 0.06142 rpy=2.29 0 -3.1416
- joint right_outer_finger_joint: limit lower=-2 upper=2 effort=1000 velocity=2.0 -> lower=0.1 upper=0.875 effort=1000 velocity=2.0
- joint right_outer_knuckle_joint: limit lower=-2 upper=2 effort=1000 velocity=2.0 -> lower=0 upper=0.875 effort=1000 velocity=2.0; origin xyz=0 0.030601 0.054905 rpy=2.29579632679 0 3.14 -> xyz=0 0.030601 0.054905 rpy=2.31 0 3.1416

Commit message: update urdf model with 90º rotation

File: mara_description/urdf/mara_robot_camera_top.urdf (robot description, URDF)
Before this commit: robot mara, 24 links, 23 joints
Joints:
- joint table_to_base_joint: origin xyz=0 0 0.62 rpy=0 0 0 -> xyz=0 0 0.62 rpy=0 0 -1.57

Commit message: Change to make it work with OSX

File: mara_description/urdf/mara_robot_camera_top.urdf (robot description, URDF)
Before this commit: robot mara, 24 links, 23 joints
Links:
- link base_link: geometry collision mesh filename=package://ara_description/meshes/Base_plancha.stl scale=0.001 0.001 0.001; visual mesh filename=package://ara_description/meshes/Base_plancha.stl scale=0.001 0.001 0.001
- link base_robot: geometry collision mesh filename=package://ara_description/meshes/Base.stl scale=0.001 0.001 0.001; visual mesh filename=package://ara_description/meshes/Base.stl scale=0.001 0.001 0.001
- link motor1_cover: geometry collision mesh filename=package://ara_description/meshes/MARA_T49_Black.stl scale=0.001 0.001 0.001; visual mesh filename=package://ara_description/meshes/MARA_T49_Black.stl scale=0.001 0.001 0.001
- link motor1_link: geometry collision mesh filename=package://ara_description/meshes/MARA_T49.stl scale=0.001 0.001 0.001; visual mesh filename=package://ara_description/meshes/MARA_T49.stl scale=0.001 0.001 0.001
- link motor2_link: geometry collision mesh filename=package://ara_description/meshes/MARA_Link1.stl scale=0.001 0.001 0.001; visual mesh filename=package://ara_description/meshes/MARA_Link1.stl scale=0.001 0.001 0.001
- link motor3_cover: geometry collision mesh filename=package://ara_description/meshes/MARA_T30_Black.stl scale=0.001 0.001 0.001; visual mesh filename=package://ara_description/meshes/MARA_T30_Black.stl scale=0.001 0.001 0.001
- link motor3_link: geometry collision mesh filename=package://ara_description/meshes/MARA_T30.stl scale=0.001 0.001 0.001; visual mesh filename=package://ara_description/meshes/MARA_T30.stl scale=0.001 0.001 0.001
- link motor4_link: geometry collision mesh filename=package://ara_description/meshes/MARA_Link2.stl scale=0.001 0.001 0.001; visual mesh filename=package://ara_description/meshes/MARA_Link2.stl scale=0.001 0.001 0.001
- link motor5_cover: geometry collision mesh filename=package://ara_description/meshes/MARA_T5.4_black.stl scale=0.001 0.001 0.001; visual mesh filename=package://ara_description/meshes/MARA_T5.4_black.stl scale=0.001 0.001 0.001
- link motor5_link: geometry collision mesh filename=package://ara_description/meshes/MARA_T5.4.stl scale=0.001 0.001 0.001; visual mesh filename=package://ara_description/meshes/MARA_T5.4.stl scale=0.001 0.001 0.001
- link motor6_link: geometry collision mesh filename=package://ara_description/meshes/MARA_GripperAdapter.stl scale=0.001 0.001 0.001; visual mesh filename=package://ara_description/meshes/MARA_GripperAdapter.stl scale=0.001 0.001 0.001
- link table: geometry collision box size=1.5 1 0.05; visual mesh filename=package://ara_description/urdf/table.obj scale=0.1 0.1 0.58

Commit message: Removing texture field in the URDF

File: mara_description/urdf/mara_robot_camera_top.urdf (robot description, URDF)
Before this commit: robot mara, 25 links, 24 joints
Links:
- link table: geometry collision box size=1.5 1 0.05; visual mesh filename=package://mara_description/urdf/table.obj scale=0.1 0.1 0.58
