Commit message: Adapting textures to gzweb

File: mara_description/urdf/camera_side.urdf.xacro (robot description, xacro)
@@ -11,5 +11,5 @@
           <origin rpy="0 0 0" xyz="0 0 0"/>
           <geometry>
-            <mesh filename="package://mara_description/meshes/demo/AIR_WorkArea.stl" scale="0.001 0.001 0.001"/>
+            <mesh filename="model://mara_description/meshes/demo/AIR_WorkArea.stl" scale="0.001 0.001 0.001"/>
           </geometry>
           <material name="Gazebo/Wood">
@@ -20,5 +20,5 @@
           <origin rpy="0 0 0" xyz="0 0 0"/>
           <geometry>
-            <mesh filename="package://mara_description/meshes/demo/AIR_WorkArea.stl" scale="0.001 0.001 0.001"/>
+            <mesh filename="model://mara_description/meshes/demo/AIR_WorkArea.stl" scale="0.001 0.001 0.001"/>
           </geometry>
         </collision>
@@ -37,5 +37,5 @@
           <origin rpy="0 0 0" xyz="0 0 0"/>
           <geometry>
-            <mesh filename="package://mara_description/meshes/demo/side/side_camera_support.stl" scale="0.001 0.001 0.001"/>
+            <mesh filename="model://mara_description/meshes/demo/side/side_camera_support.stl" scale="0.001 0.001 0.001"/>
           </geometry>
           <material name="Gazebo/Wood">
@@ -46,5 +46,5 @@
           <origin rpy="0 0 0" xyz="0 0 0"/>
           <geometry>
-            <mesh filename="package://mara_description/meshes/demo/side/side_camera_support.stl" scale="0.001 0.001 0.001"/>
+            <mesh filename="model://mara_description/meshes/demo/side/side_camera_support.stl" scale="0.001 0.001 0.001"/>
           </geometry>
         </collision>
@@ -63,5 +63,5 @@
           <origin xyz="0 0 0" rpy="0 0 0" />
           <geometry>
-            <mesh scale="0.001 0.001 0.001" filename="package://mara_description/meshes/camera/SCARA_DepthSensor_SIDE.stl" />
+            <mesh scale="0.001 0.001 0.001" filename="model://mara_description/meshes/camera/SCARA_DepthSensor_SIDE.stl" />
           </geometry>
           <material name="Gazebo/Grey">

File: mara_description/urdf/camera_top.urdf.xacro (robot description, xacro)
@@ -11,5 +11,5 @@
           <origin rpy="0 0 0" xyz="0 0 0"/>
           <geometry>
-            <mesh filename="package://mara_description/meshes/demo/AIR_WorkArea.stl" scale="0.001 0.001 0.001"/>
+            <mesh filename="model://mara_description/meshes/demo/AIR_WorkArea.stl" scale="0.001 0.001 0.001"/>
           </geometry>
           <material name="Gazebo/Wood">
@@ -20,5 +20,5 @@
           <origin rpy="0 0 0" xyz="0 0 0"/>
           <geometry>
-            <mesh filename="package://mara_description/meshes/demo/AIR_WorkArea.stl" scale="0.001 0.001 0.001"/>
+            <mesh filename="model://mara_description/meshes/demo/AIR_WorkArea.stl" scale="0.001 0.001 0.001"/>
           </geometry>
         </collision>
@@ -37,5 +37,5 @@
           <origin rpy="0 0 0" xyz="0 0 0"/>
           <geometry>
-            <mesh filename="package://mara_description/meshes/demo/top/top_camera_support.stl" scale="0.001 0.001 0.001"/>
+            <mesh filename="model://mara_description/meshes/demo/top/top_camera_support.stl" scale="0.001 0.001 0.001"/>
           </geometry>
           <material name="Gazebo/Wood">
@@ -46,5 +46,5 @@
           <origin rpy="0 0 0" xyz="0 0 0"/>
           <geometry>
-            <mesh filename="package://mara_description/meshes/demo/top/top_camera_support.stl" scale="0.002 0.001 0.001"/>
+            <mesh filename="model://mara_description/meshes/demo/top/top_camera_support.stl" scale="0.002 0.001 0.001"/>
           </geometry>
         </collision>
@@ -63,5 +63,5 @@
           <origin xyz="0 0 0" rpy="0 0 0" />
           <geometry>
-            <mesh scale="0.001 0.001 0.001" filename="package://mara_description/meshes/depthSensor.stl" />
+            <mesh scale="0.001 0.001 0.001" filename="model://mara_description/meshes/depthSensor.stl" />
           </geometry>
           <material name="Gazebo/Grey">
@@ -72,5 +72,5 @@
           <origin rpy="0 0 0" xyz="0 0 0"/>
           <geometry>
-            <mesh filename="package://mara_description/meshes/depthSensor.stl" scale="0.002 0.002 0.002" />
+            <mesh filename="model://mara_description/meshes/depthSensor.stl" scale="0.002 0.002 0.002" />
           </geometry>
         </collision>

File: mara_description/urdf/mara.urdf.xacro (robot description, xacro)
@@ -16,5 +16,5 @@
         <origin rpy="0 0 0" xyz="0 0 0"/>
         <geometry>
-          <mesh filename="package://mara_description/meshes/Base_plancha.stl" scale="0.001 0.001 0.001"/>
+          <mesh filename="model://mara_description/meshes/Base_plancha.stl" scale="0.001 0.001 0.001"/>
         </geometry>
         <material name="Gazebo/Grey">
@@ -25,5 +25,5 @@
         <origin rpy="0 0 0" xyz="0 0 0"/>
         <geometry>
-          <mesh filename="package://mara_description/meshes/Base_plancha.stl" scale="0.001 0.001 0.001"/>
+          <mesh filename="model://mara_description/meshes/Base_plancha.stl" scale="0.001 0.001 0.001"/>
         </geometry>
       </collision>
@@ -42,5 +42,5 @@
         <origin rpy="0 0 0" xyz="0 0 0"/>
         <geometry>
-          <mesh filename="package://mara_description/meshes/Base.stl" scale="0.001 0.001 0.001"/>
+          <mesh filename="model://mara_description/meshes/Base.stl" scale="0.001 0.001 0.001"/>
         </geometry>
         <material name="Gazebo/Grey">
@@ -51,5 +51,5 @@
         <origin rpy="0 0 0" xyz="0 0 0"/>
         <geometry>
-          <mesh filename="package://mara_description/meshes/Base.stl" scale="0.001 0.001 0.001"/>
+          <mesh filename="model://mara_description/meshes/Base.stl" scale="0.001 0.001 0.001"/>
         </geometry>
       </collision>
@@ -68,5 +68,5 @@
         <origin rpy="0 0 0" xyz="0 0 0"/>
         <geometry>
-          <mesh filename="package://mara_description/meshes/MARA_T49.stl" scale="0.001 0.001 0.001"/>
+          <mesh filename="model://mara_description/meshes/MARA_T49.stl" scale="0.001 0.001 0.001"/>
         </geometry>
         <material name="Gazebo/White">
@@ -77,5 +77,5 @@
         <origin rpy="0 0 0" xyz="0 0 0"/>
         <geometry>
-          <mesh filename="package://mara_description/meshes/MARA_T49.stl" scale="0.001 0.001 0.001"/>
+          <mesh filename="model://mara_description/meshes/MARA_T49.stl" scale="0.001 0.001 0.001"/>
         </geometry>
       </collision>
@@ -94,14 +94,14 @@
         <origin rpy="0 0 0" xyz="0 0 0"/>
         <geometry>
-          <mesh filename="package://mara_description/meshes/MARA_T49_Black.stl" scale="0.001 0.001 0.001"/>
-        </geometry>
-        <material name="Gazebo/Black">
-          <color rgba="0. 0. 0. 1"/>
-        </material>
-      </visual>
-      <collision>
-        <origin rpy="0 0 0" xyz="0 0 0"/>
-        <geometry>
-          <mesh filename="package://mara_description/meshes/MARA_T49_Black.stl" scale="0.001 0.001 0.001"/>
+          <mesh filename="model://mara_description/meshes/MARA_T49_Black.stl" scale="0.001 0.001 0.001"/>
+        </geometry>
+        <material name="Gazebo/Black">
+          <color rgba="0. 0. 0. 1"/>
+        </material>
+      </visual>
+      <collision>
+        <origin rpy="0 0 0" xyz="0 0 0"/>
+        <geometry>
+          <mesh filename="model://mara_description/meshes/MARA_T49_Black.stl" scale="0.001 0.001 0.001"/>
         </geometry>
       </collision>
@@ -120,14 +120,14 @@
         <origin rpy="0 0 0" xyz="0 0 0"/>
         <geometry>
-          <mesh filename="package://mara_description/meshes/MARA_Link1.stl" scale="0.001 0.001 0.001"/>
-        </geometry>
-        <material name="Gazebo/Black">
-          <color rgba="0. 0. 0. 1"/>
-        </material>
-      </visual>
-      <collision>
-        <origin rpy="0 0 0" xyz="0 0 0"/>
-        <geometry>
-          <mesh filename="package://mara_description/meshes/MARA_Link1.stl" scale="0.001 0.001 0.001"/>
+          <mesh filename="model://mara_description/meshes/MARA_Link1.stl" scale="0.001 0.001 0.001"/>
+        </geometry>
+        <material name="Gazebo/Black">
+          <color rgba="0. 0. 0. 1"/>
+        </material>
+      </visual>
+      <collision>
+        <origin rpy="0 0 0" xyz="0 0 0"/>
+        <geometry>
+          <mesh filename="model://mara_description/meshes/MARA_Link1.stl" scale="0.001 0.001 0.001"/>
         </geometry>
       </collision>
@@ -146,5 +146,5 @@
         <origin rpy="0 0 0" xyz="0 0 0"/>
         <geometry>
-          <mesh filename="package://mara_description/meshes/MARA_T30.stl" scale="0.001 0.001 0.001"/>
+          <mesh filename="model://mara_description/meshes/MARA_T30.stl" scale="0.001 0.001 0.001"/>
         </geometry>
         <material name="Gazebo/White">
@@ -155,5 +155,5 @@
         <origin rpy="0 0 0" xyz="0 0 0"/>
         <geometry>
-          <mesh filename="package://mara_description/meshes/MARA_T30.stl" scale="0.001 0.001 0.001"/>
+          <mesh filename="model://mara_description/meshes/MARA_T30.stl" scale="0.001 0.001 0.001"/>
         </geometry>
       </collision>
@@ -172,14 +172,14 @@
         <origin rpy="0 0 0" xyz="0 0 0"/>
         <geometry>
-          <mesh filename="package://mara_description/meshes/MARA_T30_Black.stl" scale="0.001 0.001 0.001"/>
-        </geometry>
-        <material name="Gazebo/Black">
-          <color rgba="0. 0. 0. 1"/>
-        </material>
-      </visual>
-      <collision>
-        <origin rpy="0 0 0" xyz="0 0 0"/>
-        <geometry>
-          <mesh filename="package://mara_description/meshes/MARA_T30_Black.stl" scale="0.001 0.001 0.001"/>
+          <mesh filename="model://mara_description/meshes/MARA_T30_Black.stl" scale="0.001 0.001 0.001"/>
+        </geometry>
+        <material name="Gazebo/Black">
+          <color rgba="0. 0. 0. 1"/>
+        </material>
+      </visual>
+      <collision>
+        <origin rpy="0 0 0" xyz="0 0 0"/>
+        <geometry>
+          <mesh filename="model://mara_description/meshes/MARA_T30_Black.stl" scale="0.001 0.001 0.001"/>
         </geometry>
       </collision>
@@ -198,14 +198,14 @@
         <origin rpy="0 0 0" xyz="0 0 0"/>
         <geometry>
-          <mesh filename="package://mara_description/meshes/MARA_Link2.stl" scale="0.001 0.001 0.001"/>
-        </geometry>
-        <material name="Gazebo/Black">
-          <color rgba="0. 0. 0. 1"/>
-        </material>
-      </visual>
-      <collision>
-        <origin rpy="0 0 0" xyz="0 0 0"/>
-        <geometry>
-          <mesh filename="package://mara_description/meshes/MARA_Link2.stl" scale="0.001 0.001 0.001"/>
+          <mesh filename="model://mara_description/meshes/MARA_Link2.stl" scale="0.001 0.001 0.001"/>
+        </geometry>
+        <material name="Gazebo/Black">
+          <color rgba="0. 0. 0. 1"/>
+        </material>
+      </visual>
+      <collision>
+        <origin rpy="0 0 0" xyz="0 0 0"/>
+        <geometry>
+          <mesh filename="model://mara_description/meshes/MARA_Link2.stl" scale="0.001 0.001 0.001"/>
         </geometry>
       </collision>
@@ -224,5 +224,5 @@
         <origin rpy="0 0 0" xyz="0 0 0"/>
         <geometry>
-          <mesh filename="package://mara_description/meshes/MARA_T5.4.stl" scale="0.001 0.001 0.001"/>
+          <mesh filename="model://mara_description/meshes/MARA_T5.4.stl" scale="0.001 0.001 0.001"/>
         </geometry>
         <material name="Gazebo/White">
@@ -233,5 +233,5 @@
         <origin rpy="0 0 0" xyz="0 0 0"/>
         <geometry>
-          <mesh filename="package://mara_description/meshes/MARA_T5.4.stl" scale="0.001 0.001 0.001"/>
+          <mesh filename="model://mara_description/meshes/MARA_T5.4.stl" scale="0.001 0.001 0.001"/>
         </geometry>
       </collision>
@@ -250,14 +250,14 @@
         <origin rpy="0 0 0" xyz="0 0 0"/>
         <geometry>
-          <mesh filename="package://mara_description/meshes/MARA_T5.4_black.stl" scale="0.001 0.001 0.001"/>
-        </geometry>
-        <material name="Gazebo/Black">
-          <color rgba="0. 0. 0. 1"/>
-        </material>
-      </visual>
-      <collision>
-        <origin rpy="0 0 0" xyz="0 0 0"/>
-        <geometry>
-          <mesh filename="package://mara_description/meshes/MARA_T5.4_black.stl" scale="0.001 0.001 0.001"/>
+          <mesh filename="model://mara_description/meshes/MARA_T5.4_black.stl" scale="0.001 0.001 0.001"/>
+        </geometry>
+        <material name="Gazebo/Black">
+          <color rgba="0. 0. 0. 1"/>
+        </material>
+      </visual>
+      <collision>
+        <origin rpy="0 0 0" xyz="0 0 0"/>
+        <geometry>
+          <mesh filename="model://mara_description/meshes/MARA_T5.4_black.stl" scale="0.001 0.001 0.001"/>
         </geometry>
       </collision>
@@ -276,14 +276,14 @@
         <origin rpy="0 0 0" xyz="0 0 0"/>
         <geometry>
-          <mesh filename="package://mara_description/meshes/MARA_GripperAdapter.stl" scale="0.001 0.001 0.001"/>
-        </geometry>
-        <material name="Gazebo/Black">
-          <color rgba="0. 0. 0. 1"/>
-        </material>
-      </visual>
-      <collision>
-        <origin rpy="0 0 0" xyz="0 0 0"/>
-        <geometry>
-          <mesh filename="package://mara_description/meshes/MARA_GripperAdapter.stl" scale="0.001 0.001 0.001"/>
+          <mesh filename="model://mara_description/meshes/MARA_GripperAdapter.stl" scale="0.001 0.001 0.001"/>
+        </geometry>
+        <material name="Gazebo/Black">
+          <color rgba="0. 0. 0. 1"/>
+        </material>
+      </visual>
+      <collision>
+        <origin rpy="0 0 0" xyz="0 0 0"/>
+        <geometry>
+          <mesh filename="model://mara_description/meshes/MARA_GripperAdapter.stl" scale="0.001 0.001 0.001"/>
         </geometry>
       </collision>

File: mara_description/urdf/mara_robot_camera_top.urdf (robot description, URDF)
Before this commit: robot mara, 24 links, 23 joints
Links:
- link base_link: geometry collision mesh filename=model://mara_description/meshes/Base_plancha.stl scale=0.001 0.001 0.001; visual mesh filename=model://mara_description/meshes/Base_plancha.stl scale=0.001 0.001 0.001
- link base_robot: geometry collision mesh filename=model://mara_description/meshes/Base.stl scale=0.001 0.001 0.001; visual mesh filename=model://mara_description/meshes/Base.stl scale=0.001 0.001 0.001
- link motor1_cover: geometry collision mesh filename=model://mara_description/meshes/MARA_T49_Black.stl scale=0.001 0.001 0.001; visual mesh filename=model://mara_description/meshes/MARA_T49_Black.stl scale=0.001 0.001 0.001
- link motor1_link: geometry collision mesh filename=model://mara_description/meshes/MARA_T49.stl scale=0.001 0.001 0.001; visual mesh filename=model://mara_description/meshes/MARA_T49.stl scale=0.001 0.001 0.001
- link motor2_link: geometry collision mesh filename=model://mara_description/meshes/MARA_Link1.stl scale=0.001 0.001 0.001; visual mesh filename=model://mara_description/meshes/MARA_Link1.stl scale=0.001 0.001 0.001
- link motor3_cover: geometry collision mesh filename=model://mara_description/meshes/MARA_T30_Black.stl scale=0.001 0.001 0.001; visual mesh filename=model://mara_description/meshes/MARA_T30_Black.stl scale=0.001 0.001 0.001
- link motor3_link: geometry collision mesh filename=model://mara_description/meshes/MARA_T30.stl scale=0.001 0.001 0.001; visual mesh filename=model://mara_description/meshes/MARA_T30.stl scale=0.001 0.001 0.001
- link motor4_link: geometry collision mesh filename=model://mara_description/meshes/MARA_Link2.stl scale=0.001 0.001 0.001; visual mesh filename=model://mara_description/meshes/MARA_Link2.stl scale=0.001 0.001 0.001
- link motor5_cover: geometry collision mesh filename=model://mara_description/meshes/MARA_T5.4_black.stl scale=0.001 0.001 0.001; visual mesh filename=model://mara_description/meshes/MARA_T5.4_black.stl scale=0.001 0.001 0.001
- link motor5_link: geometry collision mesh filename=model://mara_description/meshes/MARA_T5.4.stl scale=0.001 0.001 0.001; visual mesh filename=model://mara_description/meshes/MARA_T5.4.stl scale=0.001 0.001 0.001
- link motor6_link: geometry collision mesh filename=model://mara_description/meshes/MARA_GripperAdapter.stl scale=0.001 0.001 0.001; visual mesh filename=model://mara_description/meshes/MARA_GripperAdapter.stl scale=0.001 0.001 0.001
- link table: geometry collision box size=1.5 1 0.05; visual mesh filename=model://mara_description/urdf/table.obj scale=0.1 0.1 0.58
Joints:
- joint table_to_base_joint: origin xyz=0 0 0.62 rpy=0 0 -1.57 -> xyz=0 0 0.62 rpy=0 0 1.57

File: mara_description/urdf/mara_robot_camera_top.urdf.xacro (robot description, xacro)
@@ -27,5 +27,5 @@
   </joint>
   <joint name="table_to_base_joint" type="fixed">
-    <origin rpy="0 0 -1.57" xyz="0 0 0.62"/>
+    <origin rpy="0 0 1.57" xyz="0 0 0.62"/>
     <parent link="table"/>
     <child link="base_link"/>

File: mara_description/urdf/table.urdf.xacro (robot description, xacro)
@@ -14,8 +14,9 @@
         <origin rpy="0 0 0" xyz="0 0 0.6"/>
         <geometry>
-  				<mesh filename="package://mara_description/urdf/table.obj" scale="1.5 1 0.05"/>
+  				<mesh filename="model://mara_description/urdf/table.obj" scale="1.5 1 0.05"/>
         </geometry>
-         <material name="white">
-          <color rgba="1 1 1 1"/>
+         <material name="brown">
+           <color rgba="0.63 0.16 0.16 1"/>
+          <texture filename="model://mara_description/material/gazebo.material" />
         </material>
       </visual>
@@ -29,5 +30,5 @@
         <origin rpy="0 0 0" xyz="-0.65 -0.4 0.29"/>
         <geometry>
-  	    <mesh filename="package://mara_description/urdf/table.obj" scale="0.1 0.1 0.58"/>
+  	    <mesh filename="model://mara_description/urdf/table.obj" scale="0.1 0.1 0.58"/>
         </geometry>
   	  <material name="framemat0"/>
@@ -36,5 +37,5 @@
         <origin rpy="0 0 0" xyz="-0.65 0.4 0.29"/>
         <geometry>
-          <mesh filename="package://mara_description/urdf/table.obj" scale="0.1 0.1 0.58"/>
+          <mesh filename="model://mara_description/urdf/table.obj" scale="0.1 0.1 0.58"/>
         </geometry>
   	  <material name="framemat0"/>
@@ -43,5 +44,5 @@
         <origin rpy="0 0 0" xyz="0.65 -0.4 0.29"/>
         <geometry>
-          <mesh filename="package://mara_description/urdf/table.obj" scale="0.1 0.1 0.58"/>
+          <mesh filename="model://mara_description/urdf/table.obj" scale="0.1 0.1 0.58"/>
         </geometry>
   	  <material name="framemat0"/>
@@ -50,8 +51,12 @@
         <origin rpy="0 0 0" xyz="0.65 0.4 0.29"/>
         <geometry>
-          <mesh filename="package://mara_description/urdf/table.obj" scale="0.1 0.1 0.58"/>
+          <mesh filename="model://mara_description/urdf/table.obj" scale="0.1 0.1 0.58"/>
         </geometry>
       </visual>
     </link>
+    <gazebo reference="table">
+      <material>Gazebo/Brown</material>
+      <selfCollide>True</selfCollide>
+    </gazebo>
   </xacro:macro>
 </robot>
