Commit message: using .dae instead of .stl

File: mara_description/urdf/camera_side.urdf.xacro (robot description, xacro)
@@ -11,5 +11,5 @@
           <origin rpy="0 0 0" xyz="0 0 0"/>
           <geometry>
-            <mesh filename="model://mara_description/meshes/demo/AIR_WorkArea.stl" scale="0.001 0.001 0.001"/>
+            <mesh filename="model://mara_description/meshes/demo/AIR_WorkArea.dae" scale="0.001 0.001 0.001"/>
           </geometry>
           <material name="Gazebo/Wood">
@@ -20,5 +20,5 @@
           <origin rpy="0 0 0" xyz="0 0 0"/>
           <geometry>
-            <mesh filename="model://mara_description/meshes/demo/AIR_WorkArea.stl" scale="0.001 0.001 0.001"/>
+            <mesh filename="model://mara_description/meshes/demo/AIR_WorkArea.dae" scale="0.001 0.001 0.001"/>
           </geometry>
         </collision>
@@ -37,5 +37,5 @@
           <origin rpy="0 0 0" xyz="0 0 0"/>
           <geometry>
-            <mesh filename="model://mara_description/meshes/demo/side/side_camera_support.stl" scale="0.001 0.001 0.001"/>
+            <mesh filename="model://mara_description/meshes/demo/side/side_camera_support.dae" scale="0.001 0.001 0.001"/>
           </geometry>
           <material name="Gazebo/Wood">
@@ -46,5 +46,5 @@
           <origin rpy="0 0 0" xyz="0 0 0"/>
           <geometry>
-            <mesh filename="model://mara_description/meshes/demo/side/side_camera_support.stl" scale="0.001 0.001 0.001"/>
+            <mesh filename="model://mara_description/meshes/demo/side/side_camera_support.dae" scale="0.001 0.001 0.001"/>
           </geometry>
         </collision>
@@ -63,5 +63,5 @@
           <origin xyz="0 0 0" rpy="0 0 0" />
           <geometry>
-            <mesh scale="0.001 0.001 0.001" filename="model://mara_description/meshes/camera/SCARA_DepthSensor_SIDE.stl" />
+            <mesh scale="0.001 0.001 0.001" filename="model://mara_description/meshes/camera/SCARA_DepthSensor_SIDE.dae" />
           </geometry>
           <material name="Gazebo/Grey">

File: mara_description/urdf/camera_top.urdf.xacro (robot description, xacro)
@@ -11,5 +11,5 @@
           <origin rpy="0 0 0" xyz="0 0 0"/>
           <geometry>
-            <mesh filename="model://mara_description/meshes/demo/AIR_WorkArea.stl" scale="0.001 0.001 0.001"/>
+            <mesh filename="model://mara_description/meshes/demo/AIR_WorkArea.dae" scale="0.001 0.001 0.001"/>
           </geometry>
           <material name="Gazebo/Wood">
@@ -20,5 +20,5 @@
           <origin rpy="0 0 0" xyz="0 0 0"/>
           <geometry>
-            <mesh filename="model://mara_description/meshes/demo/AIR_WorkArea.stl" scale="0.001 0.001 0.001"/>
+            <mesh filename="model://mara_description/meshes/demo/AIR_WorkArea.dae" scale="0.001 0.001 0.001"/>
           </geometry>
         </collision>
@@ -37,5 +37,5 @@
           <origin rpy="0 0 0" xyz="0 0 0"/>
           <geometry>
-            <mesh filename="model://mara_description/meshes/demo/top/top_camera_support.stl" scale="0.001 0.001 0.001"/>
+            <mesh filename="model://mara_description/meshes/demo/top/top_camera_support.dae" scale="0.001 0.001 0.001"/>
           </geometry>
           <material name="Gazebo/Wood">
@@ -46,5 +46,5 @@
           <origin rpy="0 0 0" xyz="0 0 0"/>
           <geometry>
-            <mesh filename="model://mara_description/meshes/demo/top/top_camera_support.stl" scale="0.002 0.001 0.001"/>
+            <mesh filename="model://mara_description/meshes/demo/top/top_camera_support.dae" scale="0.002 0.001 0.001"/>
           </geometry>
         </collision>
@@ -63,5 +63,5 @@
           <origin xyz="0 0 0" rpy="0 0 0" />
           <geometry>
-            <mesh scale="0.001 0.001 0.001" filename="model://mara_description/meshes/depthSensor.stl" />
+            <mesh scale="0.001 0.001 0.001" filename="model://mara_description/meshes/depthSensor.dae" />
           </geometry>
           <material name="Gazebo/Grey">
@@ -72,5 +72,5 @@
           <origin rpy="0 0 0" xyz="0 0 0"/>
           <geometry>
-            <mesh filename="model://mara_description/meshes/depthSensor.stl" scale="0.002 0.002 0.002" />
+            <mesh filename="model://mara_description/meshes/depthSensor.dae" scale="0.002 0.002 0.002" />
           </geometry>
         </collision>

File: mara_description/urdf/mara_robot_camera_top.urdf (robot description, URDF)
Before this commit: robot mara, 25 links, 24 joints
Links:
- removed link left_inner_finger
- removed link left_inner_knuckle
- removed link left_outer_finger
- removed link left_outer_knuckle
- removed link right_inner_finger
- removed link right_inner_knuckle
- removed link right_outer_finger
- removed link right_outer_knuckle
- removed link robotiq_adapter_link
- removed link robotiq_arg2f_base_link
- removed link table
Joints:
- removed joint base_adapter_to_base_robotiq_joint
- removed joint end_effector_adapter_to_robotiq
- removed joint left_inner_finger_joint
- removed joint left_inner_knuckle_joint
- removed joint left_outer_finger_joint
- removed joint left_outer_knuckle_joint
- removed joint right_inner_finger_joint
- removed joint right_inner_knuckle_joint
- removed joint right_outer_finger_joint
- removed joint right_outer_knuckle_joint
- removed joint world_to_table_joint
- joint table_to_base_joint: origin xyz=0 0 0.62 rpy=0 0 1.57 -> xyz=0 0 0.0 rpy=0 0 1.57; parent table -> world

File: mara_description/urdf/mara_robot_camera_top.urdf.xacro (robot description, xacro)
@@ -4,29 +4,17 @@
   <!-- common stuff -->
   <xacro:include filename="$(find mara_description)/urdf/mara_gazebo.urdf.xacro" />
-  <!-- mara -->
   <xacro:include filename="$(find mara_description)/urdf/mara.urdf.xacro" />
-  <!-- robotiq 140 gripper -->
-  <xacro:include filename="$(find robotiq_140_gripper_description)/urdf/robotiq_140.urdf.xacro" />
-  <!-- <xacro:include filename="$(find mara_description)/urdf/camera_top.urdf.xacro" /> -->
-  <xacro:include filename="$(find mara_description)/urdf/table.urdf.xacro" />
-  <!-- arm -->
-  <xacro:mara_robot prefix="" joint_limited="false"/>
-  <xacro:robotiq_gripper prefix="mara" />
-  <!-- <xacro:mara_camera_top prefix="" /> -->
-  <xacro:table prefix="" />
+  <!-- <xacro:include filename="$(find robotiq_140_gripper_description)/urdf/robotiq_140.urdf.xacro" /> -->
+  <xacro:mara_robot prefix="" ee_link_distance="0.24"/>
+  <!-- <xacro:robotiq_gripper prefix="mara" /> -->
   <link name="world" />
-  <joint name="end_effector_adapter_to_robotiq" type="fixed">
-    <origin rpy="0 0 1.57" xyz=" 0 0 0.04659"/>
+  <!-- <joint name="end_effector_adapter_to_robotiq" type="fixed">
+    <origin rpy="0 0 1.57" xyz=" 0 0 0.0353"/>
     <parent link="motor6_link"/>
-    <child link="robotiq_adapter_link"/>
-  </joint>
-  <joint name="world_to_table_joint" type="fixed">
-    <origin rpy="0 0 0" xyz="0 0 0.02"/>
+    <child link="robotiq_arg2f_base_link"/>
+  </joint> -->
+  <joint name="table_to_base_joint" type="fixed">
+    <origin rpy="0 0 1.57" xyz="0 0 0.0"/>
     <parent link="world"/>
-    <child link="table"/>
-  </joint>
-  <joint name="table_to_base_joint" type="fixed">
-    <origin rpy="0 0 1.57" xyz="0 0 0.62"/>
-    <parent link="table"/>
     <child link="base_link"/>
   </joint>

File: mara_description/urdf/module.urdf (robot description, URDF)
Before this commit: robot module17, 5 links, 4 joints
Links:
- link elfin_module_14: geometry collision mesh filename=model://mara_description/meshes/MARA_T49.dae scale=0.001 0.001 0.001; visual mesh filename=model://mara_description/meshes/MARA_T49.dae scale=0.001 0.001 0.001
- link motor_cover: geometry collision mesh filename=model://mara_description/meshes/MARA_T49_Black.dae scale=0.001 0.001 0.001; visual mesh filename=model://mara_description/meshes/MARA_T49_Black.dae scale=0.001 0.001 0.001

File: mara_description/urdf/module.urdf.xacro (robot description, xacro)
@@ -21,5 +21,5 @@
       <origin xyz="0 0 0" rpy="0 0 0" />
       <geometry>
-        <mesh filename="model://mara_description/meshes/MARA_T49.stl" scale="0.001 0.001 0.001"/>
+        <mesh filename="model://mara_description/meshes/MARA_T49.dae" scale="0.001 0.001 0.001"/>
       </geometry>
       <material name="metal"/>
@@ -28,5 +28,5 @@
       <origin xyz="0 0 0" rpy="0 0 0" />
       <geometry>
-        <mesh filename="model://mara_description/meshes/MARA_T49.stl" scale="0.001 0.001 0.001"/>
+        <mesh filename="model://mara_description/meshes/MARA_T49.dae" scale="0.001 0.001 0.001"/>
       </geometry>
     </collision>
@@ -41,5 +41,5 @@
       <origin rpy="0 0 0" xyz="0 0 0"/>
       <geometry>
-        <mesh filename="model://mara_description/meshes/MARA_T49_Black.stl" scale="0.001 0.001 0.001"/>
+        <mesh filename="model://mara_description/meshes/MARA_T49_Black.dae" scale="0.001 0.001 0.001"/>
       </geometry>
       <material name="Gazebo/Black">
@@ -50,5 +50,5 @@
       <origin rpy="0 0 0" xyz="0 0 0"/>
       <geometry>
-        <mesh filename="model://mara_description/meshes/MARA_T49_Black.stl" scale="0.001 0.001 0.001"/>
+        <mesh filename="model://mara_description/meshes/MARA_T49_Black.dae" scale="0.001 0.001 0.001"/>
       </geometry>
     </collision>
