Commit message: Updating model to be able to visualize the gripper in RVIZ

File: mara_description/urdf/mara_gazebo.urdf.xacro (robot description, xacro)
@@ -14,4 +14,12 @@
     		<joint_name>motor5</joint_name>
         <joint_name>motor6</joint_name>
+        <joint_name>left_inner_knuckle_joint</joint_name>
+        <joint_name>left_outer_knuckle_joint</joint_name>
+        <joint_name>left_outer_finger_joint</joint_name>
+        <joint_name>left_inner_finger_joint</joint_name>
+        <joint_name>right_inner_knuckle_joint</joint_name>
+        <joint_name>right_outer_knuckle_joint</joint_name>
+        <joint_name>right_outer_finger_joint</joint_name>
+        <joint_name>right_inner_finger_joint</joint_name>
     	</plugin>
       <plugin name="hros_actuation_servomotor_000000000001" filename="libmara_gazebo_joint_plugin.so">

File: mara_description/urdf/mara_robot_camera_top.urdf (robot description, URDF)
Before this commit: robot mara, 21 links, 20 joints
Links:
- link left_inner_finger: geometry collision mesh filename=package://robotiq_140_gripper_description/meshes/robotiq_14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 scale=0.001 0.001 0.001; visual mesh filename=package://robotiq_140_gripper_description/meshes/robotiq_14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 scale=0.001 0.001 0.001
- link left_inner_knuckle: geometry visual mesh filename=package://robotiq_140_gripper_description/meshes/robotiq_14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
- link left_outer_finger: geometry collision mesh filename=package://robotiq_140_gripper_description/meshes/robotiq_14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; visual mesh filename=package://robotiq_140_gripper_description/meshes/robotiq_14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
- link left_outer_knuckle: geometry collision mesh filename=package://robotiq_140_gripper_description/meshes/robotiq_14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; visual mesh filename=package://robotiq_140_gripper_description/meshes/robotiq_14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
- link right_inner_finger: geometry collision mesh filename=package://robotiq_140_gripper_description/meshes/robotiq_14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 scale=0.001 0.001 0.001; visual mesh filename=package://robotiq_140_gripper_description/meshes/robotiq_14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 scale=0.001 0.001 0.001
- link right_inner_knuckle: geometry visual mesh filename=package://robotiq_140_gripper_description/meshes/robotiq_14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
- link right_outer_finger: geometry collision mesh filename=package://robotiq_140_gripper_description/meshes/robotiq_14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; visual mesh filename=package://robotiq_140_gripper_description/meshes/robotiq_14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
- link right_outer_knuckle: geometry collision mesh filename=package://robotiq_140_gripper_description/meshes/robotiq_14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; visual mesh filename=package://robotiq_140_gripper_description/meshes/robotiq_14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

File: robotiq_140_gripper_description/urdf/robotiq_gripper.urdf.xacro (robot description, xacro)
@@ -30,5 +30,5 @@
     <link name="left_outer_knuckle">
       <inertial>
-        <!--<origin xyz="-0.000200000000003065 0.0199435877845359 0.0292245259211331" rpy="0 0 0" />-->
+        <origin xyz="0 0 0" rpy="0 0 0" />
         <mass value="0.00853198276973456" />
         <inertia
@@ -43,5 +43,5 @@
         <origin xyz="0 0 0" rpy="0 0 0" />
         <geometry>
-          <mesh filename="package://robotiq_140_gripper_description/meshes/robotiq_arg2f_140_outer_knuckle.stl" />
+          <mesh filename="package://robotiq_140_gripper_description/meshes/robotiq_140_left_outer_knuckle.stl" />
         </geometry>
         <material name="">
@@ -52,5 +52,5 @@
         <origin xyz="0 0 0" rpy="0 0 0" />
         <geometry>
-          <mesh filename="package://robotiq_140_gripper_description/meshes/robotiq_arg2f_140_outer_knuckle.stl" />
+          <mesh filename="package://robotiq_140_gripper_description/meshes/robotiq_140_left_outer_knuckle.stl" />
         </geometry>
       </collision>
@@ -75,5 +75,5 @@
         <origin xyz="0 0 0" rpy="0 0 0" />
         <geometry>
-          <mesh filename="package://robotiq_140_gripper_description/meshes/robotiq_arg2f_140_outer_knuckle.stl" />
+          <mesh filename="package://robotiq_140_gripper_description/meshes/robotiq_140_right_outer_knuckle.stl" />
         </geometry>
         <material name="">
@@ -84,5 +84,5 @@
         <origin xyz="0 0 0" rpy="0 0 0" />
         <geometry>
-          <mesh filename="package://robotiq_140_gripper_description/meshes/robotiq_arg2f_140_outer_knuckle.stl" />
+          <mesh filename="package://robotiq_140_gripper_description/meshes/robotiq_140_right_outer_knuckle.stl" />
         </geometry>
       </collision>
@@ -107,5 +107,5 @@
         <origin xyz="0 0 0" rpy="0 0 0" />
         <geometry>
-          <mesh filename="package://robotiq_140_gripper_description/meshes/robotiq_arg2f_140_inner_knuckle.stl" />
+          <mesh filename="package://robotiq_140_gripper_description/meshes/robotiq_140_left_inner_knuckle.stl" />
         </geometry>
         <material name="">
@@ -133,5 +133,5 @@
         <origin xyz="0 0 0" rpy="0 0 0" />
         <geometry>
-          <mesh filename="package://robotiq_140_gripper_description/meshes/robotiq_arg2f_140_inner_knuckle.stl" />
+          <mesh filename="package://robotiq_140_gripper_description/meshes/robotiq_140_right_inner_knuckle.stl" />
         </geometry>
         <material name="">
@@ -159,14 +159,14 @@
         <origin xyz="0 0 0" rpy="0 0 0" />
         <geometry>
-          <mesh filename="package://robotiq_140_gripper_description/meshes/robotiq_arg2f_140_inner_finger.stl" scale="0.001 0.001 0.001" />
-        </geometry>
-        <material name="">
-          <color rgba="0.1 0.1 0.1 1" />
-        </material>
-      </visual>
-      <collision>
-        <origin xyz="0 0 0" rpy="0 0 0" />
-        <geometry>
-          <mesh filename="package://robotiq_140_gripper_description/meshes/robotiq_arg2f_140_inner_finger.stl" scale="0.001 0.001 0.001" />
+          <mesh filename="package://robotiq_140_gripper_description/meshes/robotiq_140_left_inner_finger.stl" scale="0.001 0.001 0.001" />
+        </geometry>
+        <material name="">
+          <color rgba="0.1 0.1 0.1 1" />
+        </material>
+      </visual>
+      <collision>
+        <origin xyz="0 0 0" rpy="0 0 0" />
+        <geometry>
+          <mesh filename="package://robotiq_140_gripper_description/meshes/robotiq_140_left_inner_finger.stl" scale="0.001 0.001 0.001" />
         </geometry>
       </collision>
@@ -191,14 +191,14 @@
         <origin xyz="0 0 0" rpy="0 0 0" />
         <geometry>
-          <mesh filename="package://robotiq_140_gripper_description/meshes/robotiq_arg2f_140_inner_finger.stl" scale="0.001 0.001 0.001"/>
-        </geometry>
-        <material name="">
-          <color rgba="0.1 0.1 0.1 1" />
-        </material>
-      </visual>
-      <collision>
-        <origin xyz="0 0 0" rpy="0 0 0" />
-        <geometry>
-          <mesh filename="package://robotiq_140_gripper_description/meshes/robotiq_arg2f_140_inner_finger.stl" scale="0.001 0.001 0.001"/>
+          <mesh filename="package://robotiq_140_gripper_description/meshes/robotiq_140_right_inner_finger.stl" scale="0.001 0.001 0.001"/>
+        </geometry>
+        <material name="">
+          <color rgba="0.1 0.1 0.1 1" />
+        </material>
+      </visual>
+      <collision>
+        <origin xyz="0 0 0" rpy="0 0 0" />
+        <geometry>
+          <mesh filename="package://robotiq_140_gripper_description/meshes/robotiq_140_right_inner_finger.stl" scale="0.001 0.001 0.001"/>
         </geometry>
       </collision>
@@ -223,14 +223,14 @@
         <origin xyz="0 0 0" rpy="0 0 0" />
         <geometry>
-          <mesh filename="package://robotiq_140_gripper_description/meshes/robotiq_arg2f_140_outer_finger.stl" />
-        </geometry>
-        <material name="">
-          <color rgba="0.1 0.1 0.1 1" />
-        </material>
-      </visual>
-      <collision>
-        <origin xyz="0 0 0" rpy="0 0 0" />
-        <geometry>
-          <mesh filename="package://robotiq_140_gripper_description/meshes/robotiq_arg2f_140_outer_finger.stl" />
+          <mesh filename="package://robotiq_140_gripper_description/meshes/robotiq_140_left_outer_finger.stl" />
+        </geometry>
+        <material name="">
+          <color rgba="0.1 0.1 0.1 1" />
+        </material>
+      </visual>
+      <collision>
+        <origin xyz="0 0 0" rpy="0 0 0" />
+        <geometry>
+          <mesh filename="package://robotiq_140_gripper_description/meshes/robotiq_140_left_outer_finger.stl" />
         </geometry>
       </collision>
@@ -255,14 +255,14 @@
         <origin xyz="0 0 0" rpy="0 0 0" />
         <geometry>
-          <mesh filename="package://robotiq_140_gripper_description/meshes/robotiq_arg2f_140_outer_finger.stl" />
-        </geometry>
-        <material name="">
-          <color rgba="0.1 0.1 0.1 1" />
-        </material>
-      </visual>
-      <collision>
-        <origin xyz="0 0 0" rpy="0 0 0" />
-        <geometry>
-          <mesh filename="package://robotiq_140_gripper_description/meshes/robotiq_arg2f_140_outer_finger.stl" />
+          <mesh filename="package://robotiq_140_gripper_description/meshes/robotiq_140_right_outer_finger.stl" />
+        </geometry>
+        <material name="">
+          <color rgba="0.1 0.1 0.1 1" />
+        </material>
+      </visual>
+      <collision>
+        <origin xyz="0 0 0" rpy="0 0 0" />
+        <geometry>
+          <mesh filename="package://robotiq_140_gripper_description/meshes/robotiq_140_right_outer_finger.stl" />
         </geometry>
       </collision>

Commit message: Updating gripper

File: mara_description/urdf/mara_gazebo.urdf.xacro (robot description, xacro)
@@ -7,5 +7,5 @@
     			<argument>~/out:=joint_states</argument>
     		</ros>
-    		<update_rate>250</update_rate>
+    		<update_rate>25</update_rate>
     		<joint_name>motor1</joint_name>
     		<joint_name>motor2</joint_name>

File: mara_description/urdf/mara_robot_camera_top.urdf (robot description, URDF)
Before this commit: robot mara, 21 links, 20 joints
Joints:
- joint left_inner_knuckle_joint: mimic joint=left_outer_knuckle_joint multiplier=-1 offset=0 -> (none)
- joint right_inner_knuckle_joint: mimic joint=right_outer_knuckle_joint multiplier=-1 offset=0 -> (none); origin xyz=0 0.0127 0.06142 rpy=2.29 0 -3.1416 -> xyz=0 0.0127 0.06142 rpy=2.29 0 -3.14159265359
- joint right_outer_knuckle_joint: origin xyz=0 0.030601 0.054905 rpy=2.31 0 3.1416 -> xyz=0 0.030601 0.054905 rpy=2.31 0 3.14159265359

File: robotiq_140_gripper_description/urdf/robotiq_gripper.urdf.xacro (robot description, xacro)
@@ -33,10 +33,10 @@
         <mass value="0.00853198276973456" />
         <inertia
-            ixx="2.88840278e-09"
+            ixx="2.89328108496468E-06"
             ixy="0"
             ixz="0"
-            iyy="2.80689245e-10"
-            iyz="0"
-            izz="2.79961804e-09" />
+            iyy="1.86719750325683E-06"
+            iyz="-1.21858577871576E-06"
+            izz="1.21905238907251E-06" />
       </inertial>
       <visual>
@@ -58,5 +58,5 @@
     <gazebo reference="left_outer_knuckle">
       <material>Gazebo/Grey</material>
-      <selfCollide>False</selfCollide>
+      <selfCollide>True</selfCollide>
     </gazebo>
     <link name="right_outer_knuckle">
@@ -65,10 +65,10 @@
         <mass value="0.00853198276973456" />
         <inertia
-            ixx="2.88840278e-09"
+            ixx="2.89328108496468E-06"
             ixy="0"
             ixz="0"
-            iyy="2.80689245e-10"
-            iyz="0"
-            izz="2.79961804e-09" />
+            iyy="1.86719750325683E-06"
+            iyz="-1.21858577871576E-06"
+            izz="1.21905238907251E-06" />
       </inertial>
       <visual>
@@ -90,16 +90,16 @@
     <gazebo reference="right_outer_knuckle">
       <material>Gazebo/Grey</material>
-      <selfCollide>False</selfCollide>
+      <selfCollide>True</selfCollide>
     </gazebo>
     <link name="left_inner_knuckle">
       <inertial>
-        <origin xyz="0 0 0" rpy="0 0 0" />
+        <origin xyz="0.000123011831763771 0.0507850843201817 0.00103968640075166" rpy="0 0 0" />
         <mass value="0.0271177346495152" />
         <inertia
             ixx="2.61910379223783E-05"
-            ixy="0"
-            ixz="0"
+            ixy="-2.43616858946494E-07"
+            ixz="-6.37789906117123E-09"
             iyy="2.8270243746167E-06"
-            iyz="0"
+            iyz="-5.37200748039765E-07"
             izz="2.83695868220296E-05" />
       </inertial>
@@ -116,16 +116,16 @@
     <gazebo reference="left_inner_knuckle">
       <material>Gazebo/Grey</material>
-      <selfCollide>False</selfCollide>
+      <selfCollide>True</selfCollide>
     </gazebo>
     <link name="right_inner_knuckle">
       <inertial>
-        <origin xyz="0 0 0" rpy="0 0 0" />
+        <origin xyz="0.000123011831763771 0.0507850843201817 0.00103968640075166" rpy="0 0 0" />
         <mass value="0.0271177346495152" />
         <inertia
             ixx="2.61910379223783E-05"
-            ixy="0"
-            ixz="0"
+            ixy="-2.43616858946494E-07"
+            ixz="-6.37789906117123E-09"
             iyy="2.8270243746167E-06"
-            iyz="0"
+            iyz="-5.37200748039765E-07"
             izz="2.83695868220296E-05" />
       </inertial>
@@ -142,39 +142,7 @@
     <gazebo reference="right_inner_knuckle">
       <material>Gazebo/Grey</material>
-      <selfCollide>False</selfCollide>
+      <selfCollide>True</selfCollide>
     </gazebo>
     <link name="left_inner_finger">
-      <inertial>
-        <origin xyz="0 0 0" rpy="0 0 0" />
-        <mass value="0.0104003125914103" />
-        <inertia
-            ixx="2.71909453810972E-06"
-            ixy="0"
-            ixz="0"
-            iyy="7.69100314106116E-07"
-            iyz="0"
-            izz="2.30315190420171E-06" />
-      </inertial>
-      <visual>
-        <origin xyz="0 0 0" rpy="0 0 0" />
-        <geometry>
-          <mesh filename="package://robotiq_140_gripper_description/meshes/robotiq_140_left_inner_finger.stl" scale="0.001 0.001 0.001" />
-        </geometry>
-        <material name="">
-          <color rgba="0.1 0.1 0.1 1" />
-        </material>
-      </visual>
-      <collision>
-        <origin xyz="0 0 0" rpy="0 0 0" />
-        <geometry>
-          <mesh filename="package://robotiq_140_gripper_description/meshes/robotiq_140_left_inner_finger.stl" scale="0.001 0.001 0.001" />
-        </geometry>
-      </collision>
-    </link>
-    <gazebo reference="left_inner_finger">
-      <material>Gazebo/Grey</material>
-      <selfCollide>True</selfCollide>
-    </gazebo>
-    <link name="right_inner_finger">
       <inertial>
         <origin xyz="0.0 0.031506174 -0.017648840" rpy="0 0 0" />
@@ -191,31 +159,63 @@
         <origin xyz="0 0 0" rpy="0 0 0" />
         <geometry>
-          <mesh filename="package://robotiq_140_gripper_description/meshes/robotiq_140_right_inner_finger.stl" scale="0.001 0.001 0.001"/>
-        </geometry>
-        <material name="">
-          <color rgba="0.1 0.1 0.1 1" />
-        </material>
-      </visual>
-      <collision>
-        <origin xyz="0 0 0" rpy="0 0 0" />
-        <geometry>
-          <mesh filename="package://robotiq_140_gripper_description/meshes/robotiq_140_right_inner_finger.stl" scale="0.001 0.001 0.001"/>
-        </geometry>
-      </collision>
-    </link>
-    <gazebo reference="right_inner_finger">
-      <material>Gazebo/Grey</material>
-      <selfCollide>True</selfCollide>
-    </gazebo>
-    <link name="left_outer_finger">
-      <inertial>
-        <origin xyz="0 0 0" rpy="0 0 0" />
-        <mass value="0.022614240507152" />
-        <inertia
-            ixx="1.52518312458174E-05"
+          <mesh filename="package://robotiq_140_gripper_description/meshes/robotiq_140_left_inner_finger.stl" scale="0.001 0.001 0.001" />
+        </geometry>
+        <material name="">
+          <color rgba="0.1 0.1 0.1 1" />
+        </material>
+      </visual>
+      <collision>
+        <origin xyz="0 0 0" rpy="0 0 0" />
+        <geometry>
+          <mesh filename="package://robotiq_140_gripper_description/meshes/robotiq_140_left_inner_finger.stl" scale="0.001 0.001 0.001" />
+        </geometry>
+      </collision>
+    </link>
+    <gazebo reference="left_inner_finger">
+      <material>Gazebo/Grey</material>
+      <selfCollide>True</selfCollide>
+    </gazebo>
+    <link name="right_inner_finger">
+      <inertial>
+        <origin xyz="0.0 0.031506174 -0.017648840" rpy="0 0 0" />
+        <mass value="0.0104003125914103" />
+        <inertia
+            ixx="6.06863499e-06"
             ixy="0"
             ixz="0"
+            iyy="7.46305064e-07"
+            iyz="0"
+            izz="6.21796490e-06" />
+      </inertial>
+      <visual>
+        <origin xyz="0 0 0" rpy="0 0 0" />
+        <geometry>
+          <mesh filename="package://robotiq_140_gripper_description/meshes/robotiq_140_right_inner_finger.stl" scale="0.001 0.001 0.001"/>
+        </geometry>
+        <material name="">
+          <color rgba="0.1 0.1 0.1 1" />
+        </material>
+      </visual>
+      <collision>
+        <origin xyz="0 0 0" rpy="0 0 0" />
+        <geometry>
+          <mesh filename="package://robotiq_140_gripper_description/meshes/robotiq_140_right_inner_finger.stl" scale="0.001 0.001 0.001"/>
+        </geometry>
+      </collision>
+    </link>
+    <gazebo reference="right_inner_finger">
+      <material>Gazebo/Grey</material>
+      <selfCollide>True</selfCollide>
+    </gazebo>
+    <link name="left_outer_finger">
+      <inertial>
+        <origin xyz="0.00030115855001899 0.0373907951953854 -0.0208027427000385" rpy="0 0 0" />
+        <mass value="0.022614240507152" />
+        <inertia
+            ixx="1.52518312458174E-05"
+            ixy="9.76583423954399E-10"
+            ixz="-5.43838577022588E-10"
             iyy="6.17694243867776E-06"
-            iyz="0"
+            iyz="6.78636130740228E-06"
             izz="1.16494917907219E-05" />
       </inertial>
@@ -242,12 +242,12 @@
     <link name="right_outer_finger">
       <inertial>
-        <origin xyz="-0.0002009  0.0396149 -0.0161363" rpy="0 0 0" />
+        <origin xyz="0.00030115855001899 0.0373907951953854 -0.0208027427000385" rpy="0 0 0" />
         <mass value="0.022614240507152" />
         <inertia
             ixx="1.52518312458174E-05"
-            ixy="0"
-            ixz="0"
+            ixy="9.76583423954399E-10"
+            ixz="-5.43838577022588E-10"
             iyy="6.17694243867776E-06"
-            iyz="0"
+            iyz="6.78636130740228E-06"
             izz="1.16494917907219E-05" />
       </inertial>
@@ -280,5 +280,5 @@
     </joint>
     <joint name="right_outer_knuckle_joint" type="revolute">
-      <origin xyz="0 0.030601 0.054905" rpy="2.31 0 3.1416" />
+      <origin xyz="0 0.030601 0.054905" rpy="2.31 0 3.14159265359" />
       <parent link="robotiq_arg2f_base_link" />
       <child link="right_outer_knuckle" />
@@ -292,13 +292,11 @@
       <axis xyz="-1 0 0" />
       <limit lower="0" upper="0.87" velocity="2.0" effort="1000" />
-      <mimic joint="left_outer_knuckle_joint" multiplier="-1" offset="0" />
     </joint>
     <joint name="right_inner_knuckle_joint" type="revolute">
-      <origin xyz="0 0.0127 0.06142" rpy="2.29 0 -3.1416" />
+      <origin xyz="0 0.0127 0.06142" rpy="2.29 0 -3.14159265359" />
       <parent link="robotiq_arg2f_base_link" />
       <child link="right_inner_knuckle" />
       <axis xyz="-1 0 0" />
       <limit lower="0" upper="0.87" velocity="2.0" effort="1000" />
-      <mimic joint="right_outer_knuckle_joint" multiplier="-1" offset="0" />
     </joint>
     <joint name="left_outer_finger_joint" type="revolute">
@@ -338,6 +336,6 @@
           <xyz>1 0 0</xyz>
           <limit>
-            <lower>-0.6</lower>
-            <upper>0.6</upper>
+            <lower>-0.8</lower>
+            <upper>0.8</upper>
             <velocity>2.0</velocity>
             <effort>1000</effort>
@@ -352,6 +350,6 @@
           <xyz>-1 0 0</xyz>
           <limit>
-            <lower>-0.6</lower>
-            <upper>0.6</upper>
+            <lower>-0.8</lower>
+            <upper>0.8</upper>
             <velocity>2.0</velocity>
             <effort>1000</effort>
