Commit message: Add driver for running a traied nn

File: mara_description/urdf/mara_gazebo.urdf.xacro (robot description, xacro)
@@ -16,5 +16,5 @@
         <joint_name>joint_finger</joint_name>
     	</plugin>
-      <plugin name="hros_actuation_servomotor_000000000001" filename="libmara_gazebo_joint_plugin.so">
+      <plugin name="hros_actuation_servomotor_000000000001" filename="libmara_gazebo_joint_training_plugin.so">
         <ros></ros>
         <axis1>motor2</axis1>
@@ -22,5 +22,5 @@
         <type>series14</type>
       </plugin>
-      <plugin name="hros_actuation_servomotor_000000000002" filename="libmara_gazebo_joint_plugin.so">
+      <plugin name="hros_actuation_servomotor_000000000002" filename="libmara_gazebo_joint_training_plugin.so">
         <ros></ros>
         <axis1>motor3</axis1>
@@ -28,5 +28,5 @@
         <type>series17</type>
       </plugin>
-      <plugin name="hros_actuation_servomotor_000000000003" filename="libmara_gazebo_joint_plugin.so">
+      <plugin name="hros_actuation_servomotor_000000000003" filename="libmara_gazebo_joint_training_plugin.so">
         <ros></ros>
         <axis1>motor5</axis1>

File: mara_description/urdf/mara_robot_gripper_140_run.urdf (robot description, URDF)
Before this commit: robot mara, 18 links, 17 joints
Links:
- removed link finger1
- removed link finger2
- removed link robotiq_hande_base_link
- added link left_inner_finger, mass 0.0104003125914103; collision mesh filename=package://robotiq_140_gripper_description/meshes/robotiq_14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 scale=0.001 0.001 0.001; visual mesh filename=package://robotiq_140_gripper_description/meshes/robotiq_14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 scale=0.001 0.001 0.001
- added link left_inner_knuckle, mass 0.0271177346495152; visual mesh filename=package://robotiq_140_gripper_description/meshes/robotiq_14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
- added link left_outer_finger, mass 0.022614240507152; collision mesh filename=package://robotiq_140_gripper_description/meshes/robotiq_14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; visual mesh filename=package://robotiq_140_gripper_description/meshes/robotiq_14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
- added link left_outer_knuckle, mass 0.00853198276973456; collision mesh filename=package://robotiq_140_gripper_description/meshes/robotiq_14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; visual mesh filename=package://robotiq_140_gripper_description/meshes/robotiq_14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
- added link right_inner_finger, mass 0.0104003125914103; collision mesh filename=package://robotiq_140_gripper_description/meshes/robotiq_14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 scale=0.001 0.001 0.001; visual mesh filename=package://robotiq_140_gripper_description/meshes/robotiq_14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 scale=0.001 0.001 0.001
- added link right_inner_knuckle, mass 0.0271177346495152; visual mesh filename=package://robotiq_140_gripper_description/meshes/robotiq_14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
- added link right_outer_finger, mass 0.022614240507152; collision mesh filename=package://robotiq_140_gripper_description/meshes/robotiq_14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; visual mesh filename=package://robotiq_140_gripper_description/meshes/robotiq_14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
- added link right_outer_knuckle, mass 0.00853198276973456; collision mesh filename=package://robotiq_140_gripper_description/meshes/robotiq_14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; visual mesh filename=package://robotiq_140_gripper_description/meshes/robotiq_14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
- added link robotiq_arg2f_base_link, mass 0.22652; collision mesh filename=package://robotiq_140_gripper_description/meshes/GRIPPER_ba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 scale=0.001 0.001 0.001; visual mesh filename=package://robotiq_140_gripper_description/meshes/GRIPPER_ba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 scale=0.001 0.001 0.001
- link ee_link: geometry visual sphere radius=0.01
Joints:
- removed joint finger2_joint
- added joint left_inner_finger_joint: type revolute, parent left_outer_finger, child left_inner_finger, origin xyz=0 0.0817554015893473 -0.0282203446692936 rpy=-.725 0 0, axis 1 0 0, limit lower=0 upper=0.8757 effort=1000 velocity=2.0, mimic joint=joint_finger multiplier=1 offset=0
- added joint left_inner_knuckle_joint: type revolute, parent robotiq_arg2f_base_link, child left_inner_knuckle, origin xyz=0 -0.0127 0.06142 rpy=2.29 0 0, axis -1 0 0, limit lower=0 upper=0.78 effort=1000 velocity=2.0, mimic joint=joint_finger multiplier=1 offset=0
- added joint left_outer_finger_joint: type fixed, parent left_outer_knuckle, child left_outer_finger, origin xyz=0 0.01821998610742 0.0260018192872234 rpy=0 0 0
- added joint left_outer_knuckle_joint: type revolute, parent robotiq_arg2f_base_link, child left_outer_knuckle, origin xyz=0 -0.030601 0.054905 rpy=2.31 0 0, axis -1 0 0, limit lower=0 upper=0.775 effort=1000 velocity=2.0, mimic joint=joint_finger multiplier=1 offset=0
- added joint right_inner_finger_joint: type revolute, parent right_outer_finger, child right_inner_finger, origin xyz=0 0.0817554015893473 -0.0282203446692936 rpy=-.725 0 0, axis 1 0 0, limit lower=0 upper=0.8757 effort=1000 velocity=2.0, mimic joint=joint_finger multiplier=1 offset=0
- added joint right_inner_knuckle_joint: type revolute, parent robotiq_arg2f_base_link, child right_inner_knuckle, origin xyz=0 0.0127 0.06142 rpy=2.29 0 -3.14159265359, axis -1 0 0, limit lower=0 upper=0.78 effort=1000 velocity=2.0, mimic joint=joint_finger multiplier=1 offset=0
- added joint right_outer_finger_joint: type fixed, parent right_outer_knuckle, child right_outer_finger, origin xyz=0 0.01821998610742 0.0260018192872234 rpy=0 0 0
- joint ee_link: origin xyz=0 0.0 0.18 rpy=0 -1.57 0 -> xyz=0 0.0 0.24 rpy=0 0 0
- joint end_effector_adapter_to_robotiq: child robotiq_hande_base_link -> robotiq_arg2f_base_link; origin xyz= 0 0 0.13 rpy=0 1.57 0 -> xyz= 0 0 0.03653 rpy=0 0 1.57
- joint joint_finger: axis 0 0 -1 -> -1 0 0; child finger1 -> right_outer_knuckle; limit lower=0 upper=0.024858 effort=1000 velocity=2.0 -> lower=0 upper=0.775 effort=1000 velocity=2.0; origin xyz=0 0 0.0 rpy=0 0 0 -> xyz=0 0.030601 0.054905 rpy=2.31 0 3.14159265359; parent robotiq_hande_base_link -> robotiq_arg2f_base_link; type prismatic -> revolute
- joint motor6_link-tool0_fixed_joint: origin xyz=0 0.0 0.18 rpy=0 -1.57 0 -> xyz=0 0.0 0.24 rpy=0 0 0

File: mara_description/urdf/module.urdf.xacro (robot description, xacro)
@@ -118,5 +118,5 @@
   </joint>
   <gazebo>
-    <plugin name="hros_actuation_servomotor_000000000001" filename="libmara_gazebo_joint_plugin.so">
+    <plugin name="hros_actuation_servomotor_000000000001" filename="libmara_gazebo_joint_training_plugin.so">
       <ros></ros>
       <axis1>motor2</axis1>
