Commit message: Adding plugins to gripper

File: mara_description/urdf/mara_robot_gripper_140.urdf (robot description, URDF)
Before this commit: robot mara, 25 links, 24 joints
Links:
- removed link robotiq_adapter_link
Joints:
- removed joint base_adapter_to_base_robotiq_joint

File: robotiq_hande_gripper_description/urdf/robotiq_hande.urdf.xacro (robot description, xacro)
@@ -80,4 +80,10 @@
       <selfCollide>True</selfCollide>
     </gazebo>
+    <gazebo>
+      <plugin filename="librobotiq_linear_gripper_gazebo_plugin.so" name="robotiq_hande_gripper">
+        <left_joint>finger1_joint</left_joint>
+        <right_joint>finger2_joint</right_joint>
+      </plugin>
+    </gazebo>
     <joint name="finger1_joint" type="fixed">
       <origin rpy="0 0 0" xyz="0 0 0.0"/>

Commit message: update URDF robotiq 140

File: mara_description/urdf/mara_robot_gripper_140.urdf (robot description, URDF)
Before this commit: robot mara, 24 links, 23 joints
Links:
- link table: geometry collision box size=1.5 1 0.05; visual mesh filename=package://mara_description/urdf/table.obj scale=0.1 0.1 0.58
Joints:
- removed joint right_outer_knuckle_joint
- added joint joint_finger: type revolute, parent robotiq_arg2f_base_link, child right_outer_knuckle, origin xyz=0 0.030601 0.054905 rpy=2.31 0 3.14159265359, axis -1 0 0, limit lower=0 upper=0.775 effort=1000 velocity=2.0
- joint left_inner_finger_joint: limit lower=-0.875 upper=0.8757 effort=1000 velocity=2.0 -> lower=0 upper=0.8757 effort=1000 velocity=2.0; mimic (none) -> joint=joint_finger multiplier=1 offset=0
- joint left_inner_knuckle_joint: mimic (none) -> joint=joint_finger multiplier=1 offset=0
- joint left_outer_finger_joint: axis -1 0 0 -> (none); limit lower=-0.875 upper=-0.0075 effort=1000 velocity=2.0 -> (none); type revolute -> fixed
- joint left_outer_knuckle_joint: limit lower=0 upper=0.78 effort=1000 velocity=2.0 -> lower=0 upper=0.775 effort=1000 velocity=2.0; mimic (none) -> joint=joint_finger multiplier=1 offset=0
- joint right_inner_finger_joint: limit lower=-0.875 upper=0.8757 effort=1000 velocity=2.0 -> lower=0 upper=0.8757 effort=1000 velocity=2.0; mimic (none) -> joint=joint_finger multiplier=1 offset=0
- joint right_inner_knuckle_joint: mimic (none) -> joint=joint_finger multiplier=1 offset=0
- joint right_outer_finger_joint: axis -1 0 0 -> (none); limit lower=-0.875 upper=-0.0075 effort=1000 velocity=2.0 -> (none); type revolute -> fixed

Commit message: fix

File: mara_description/urdf/mara_robot_gripper_140.urdf (robot description, URDF)
Before this commit: robot mara, 24 links, 23 joints
Links:
- link ee_link: geometry visual sphere radius=0.01

Commit message: Updating URDFs robotiq: hande 85 and 140

File: mara_description/urdf/mara_robot_gripper_140.urdf (robot description, URDF)
Before this commit: robot mara, 24 links, 23 joints
Links:
- added link robotiq_adapter_link, mass 0.22652; collision mesh filename=package://robotiq_140_gripper_description/meshes/hros_robot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 scale=0.001 0.001 0.001; visual mesh filename=package://robotiq_140_gripper_description/meshes/hros_robot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 scale=0.001 0.001 0.001
Joints:
- added joint base_adapter_to_base_robotiq_joint: type fixed, parent robotiq_adapter_link, child robotiq_arg2f_base_link, origin xyz= 0 0 0.03653 rpy=0 0 0
- joint end_effector_adapter_to_robotiq: child robotiq_arg2f_base_link -> robotiq_adapter_link; origin xyz= 0 0 0.03653 rpy=0 0 1.57 -> xyz= 0 0 0.0 rpy=0 0 1.57

File: mara_description/urdf/mara_robot_gripper_140.urdf.xacro (robot description, xacro)
@@ -17,7 +17,7 @@
   <link name="world" />
   <joint name="end_effector_adapter_to_robotiq" type="fixed">
-    <origin rpy="0 0 1.57" xyz=" 0 0 0.03653"/>
+    <origin rpy="0 0 1.57" xyz=" 0 0 0.0"/>
     <parent link="motor6_link"/>
-    <child link="robotiq_arg2f_base_link"/>
+    <child link="robotiq_adapter_link"/>
   </joint>
   <joint name="world_to_table_joint" type="fixed">

File: mara_description/urdf/mara_robot_gripper_85.urdf (robot description, URDF)
Before this commit: robot mara, 24 links, 23 joints
Links:
- added link robotiq_adapter_link, mass 0.22652; collision mesh filename=package://robotiq_85_gripper_description/meshes/hros_roboti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 scale=0.001 0.001 0.001; visual mesh filename=package://robotiq_85_gripper_description/meshes/hros_roboti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 scale=0.001 0.001 0.001
Joints:
- added joint base_adapter_to_base_robotiq_joint: type fixed, parent robotiq_adapter_link, child robotiq_arg2f_base, origin xyz= 0 0 0.03653 rpy=0 0 0
- joint end_effector_adapter_to_robotiq: child robotiq_arg2f_base -> robotiq_adapter_link; origin xyz= 0 0 0.03653 rpy=0 0 0 -> xyz= 0 0 0.0 rpy=0 0 0

File: mara_description/urdf/mara_robot_gripper_hande.urdf (robot description, URDF)
Before this commit: robot mara, 18 links, 17 joints
Links:
- added link robotiq_adapter_link, mass 0.22652; collision mesh filename=package://robotiq_hande_gripper_description/meshes/hros_rob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 scale=0.001 0.001 0.001; visual mesh filename=package://robotiq_hande_gripper_description/meshes/hros_rob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 scale=0.001 0.001 0.001
Joints:
- added joint base_adapter_to_base_robotiq_joint: type fixed, parent robotiq_adapter_link, child robotiq_hande_base_link, origin xyz= 0 0 0.10653 rpy=0 1.57 0
- joint end_effector_adapter_to_robotiq: child robotiq_hande_base_link -> robotiq_adapter_link; origin xyz= 0 0 0.13 rpy=0 1.57 0 -> xyz= 0 0 0.0 rpy=0 0 0

Commit message: Fixing MARA axis

File: mara_description/urdf/mara_robot_gripper_140.urdf (robot description, URDF)
Before this commit: robot mara, 25 links, 24 joints
Joints:
- joint table_to_base_joint: origin xyz=0 0 0.62 rpy=0 0 1.57 -> xyz=0 0 0.62 rpy=0 0 0

File: mara_description/urdf/mara_robot_gripper_85.urdf (robot description, URDF)
Before this commit: robot mara, 25 links, 24 joints
Joints:
- joint table_to_base_joint: origin xyz=0 0 0.62 rpy=0 0 1.57 -> xyz=0 0 0.62 rpy=0 0 0

File: mara_description/urdf/mara_robot_gripper_hande.urdf (robot description, URDF)
Before this commit: robot mara, 19 links, 18 joints
Joints:
- joint table_to_base_joint: origin xyz=0 0 0.62 rpy=0 0 1.57 -> xyz=0 0 0.62 rpy=0 0 0

File: mara_description/urdf/mara_robot_gripper_ur_j.urdf (robot description, URDF)
Before this commit: robot mara, 18 links, 17 joints
Joints:
- joint table_to_base_joint: origin xyz=0 0 0.62 rpy=0 0 1.57 -> xyz=0 0 0.62 rpy=0 0 0

Commit message: update adapter in S140 models urdf

File: mara_description/urdf/mara_robot_gripper_140.urdf (robot description, URDF)
Before this commit: robot mara, 25 links, 24 joints
Links:
- added link gripper_adapter, mass 0.13969; collision mesh filename=package://mara_description/meshes/gripper_adapter.dae scale=0.001 0.001 0.001; visual mesh filename=package://mara_description/meshes/gripper_adapter.dae scale=0.001 0.001 0.001
- link left_inner_knuckle: geometry visual mesh filename=package://robotiq_140_gripper_description/meshes/robotiq_14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 scale=0.001 0.001 0.001
- link left_outer_finger: geometry collision mesh filename=package://robotiq_140_gripper_description/meshes/robotiq_14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 scale=0.001 0.001 0.001; visual mesh filename=package://robotiq_140_gripper_description/meshes/robotiq_14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 scale=0.001 0.001 0.001
- link left_outer_knuckle: geometry collision mesh filename=package://robotiq_140_gripper_description/meshes/robotiq_14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 scale=0.001 0.001 0.001; visual mesh filename=package://robotiq_140_gripper_description/meshes/robotiq_14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 scale=0.001 0.001 0.001
- link motor6_link: mass 0.14 -> 0.00001; geometry collision sphere radius=0; visual sphere radius=0
- link right_inner_knuckle: geometry visual mesh filename=package://robotiq_140_gripper_description/meshes/robotiq_14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 scale=0.001 0.001 0.001
- link right_outer_finger: geometry collision mesh filename=package://robotiq_140_gripper_description/meshes/robotiq_14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 scale=0.001 0.001 0.001; visual mesh filename=package://robotiq_140_gripper_description/meshes/robotiq_14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 scale=0.001 0.001 0.001
- link right_outer_knuckle: geometry collision mesh filename=package://robotiq_140_gripper_description/meshes/robotiq_14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 scale=0.001 0.001 0.001; visual mesh filename=package://robotiq_140_gripper_description/meshes/robotiq_14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 scale=0.001 0.001 0.001
- link robotiq_adapter_link: geometry collision mesh filename=package://mara_description/meshes/robotiq_adapter.dae scale=0.001 0.001 0.001; visual mesh filename=package://mara_description/meshes/robotiq_adapter.dae scale=0.001 0.001 0.001
Joints:
- removed joint base_adapter_to_base_robotiq_joint
- removed joint end_effector_adapter_to_robotiq
- removed joint left_inner_finger_joint
- removed joint left_inner_knuckle_joint
- removed joint left_outer_finger_joint
- removed joint left_outer_knuckle_joint
- removed joint right_inner_finger_joint
- removed joint right_inner_knuckle_joint
- removed joint right_outer_finger_joint
- removed joint table_to_base_joint
- removed joint world_to_table_joint
- added joint gripper_adapter_to_robotiq_adapter: type fixed, parent gripper_adapter, child robotiq_adapter_link, origin xyz= 0 0 0.05679 rpy=0 0 0
- added joint left_outer_finger_to_inner: type revolute, parent left_outer_finger, child left_inner_finger, origin xyz=0.03543 0 0.0789 rpy=0 0 0, axis 0 1 0, limit lower=0 upper=0.78574722925 effort=1000 velocity=2.0, mimic joint=joint_finger multiplier=1 offset=0
- added joint left_outer_knuckle_to_finger: type fixed, parent left_outer_knuckle, child left_outer_finger, origin xyz=0.03142 0 -0.00453 rpy=0 0 0
- added joint motor6_to_gripper_adapter: type fixed, parent motor6_link, child gripper_adapter, origin xyz= 0 0 -0.02026 rpy=0 0 0
- added joint right_outer_finger_to_inner: type revolute, parent right_outer_finger, child right_inner_finger, origin xyz=-0.03543 0 0.0789 rpy=0 0 0, axis 0 -1 0, limit lower=0 upper=0.78574722925 effort=1000 velocity=2.0, mimic joint=joint_finger multiplier=1 offset=0
- added joint right_outer_knuckle_to_finger: type fixed, parent right_outer_knuckle, child right_outer_finger, origin xyz=-0.03142 0 -0.00453 rpy=0 0 0
- added joint robotiq_adapter_to_arg2f_base: type fixed, parent robotiq_adapter_link, child robotiq_arg2f_base_link, origin xyz= 0 0 0 rpy=0 0 0
- added joint robotiq_arg2f_base_to_left_inner_knuckle: type revolute, parent robotiq_arg2f_base_link, child left_inner_knuckle, origin xyz=0.0127 0 0.06118 rpy=0 0 0, axis 0 -1 0, limit lower=0 upper=0.78574722925 effort=1000 velocity=2.0, mimic joint=joint_finger multiplier=1 offset=0
- added joint robotiq_arg2f_base_to_left_outer_knuckle: type revolute, parent robotiq_arg2f_base_link, child left_outer_knuckle, origin xyz=0.0306 0 0.05466 rpy=0 0 0, axis 0 -1 0, limit lower=0 upper=0.78574722925 effort=1000 velocity=2.0, mimic joint=joint_finger multiplier=1 offset=0
- added joint robotiq_arg2f_base_to_right_inner_knuckle: type revolute, parent robotiq_arg2f_base_link, child right_inner_knuckle, origin xyz=-0.0127 0 0.06118 rpy=0 0 0, axis 0 1 0, limit lower=0 upper=0.78574722925 effort=1000 velocity=2.0, mimic joint=joint_finger multiplier=1 offset=0
- added joint table_to_base: type fixed, parent table, child base_link, origin xyz=0 0 0.62 rpy=0 0 0
- added joint world_to_table: type fixed, parent world, child table, origin xyz=0 0 0 rpy=0 0 0
- joint ee_link: origin xyz=0 0.0 0.24 rpy=0 -1.57 0 -> xyz=0 0.0 0.24497 rpy=0 -1.57 0
- joint joint_finger: axis -1 0 0 -> 0 1 0; limit lower=0 upper=0.775 effort=1000 velocity=2.0 -> lower=0 upper=0.78574722925 effort=1000 velocity=2.0; origin xyz=0 0.030601 0.054905 rpy=2.31 0 3.14159265359 -> xyz=-0.0306 0 0.05466 rpy=0 0 0
- joint motor6_link-tool0_fixed_joint: origin xyz=0 0.0 0.24 rpy=0 -1.57 0 -> xyz=0 0.0 0.24497 rpy=0 -1.57 0

File: mara_description/urdf/mara_robot_gripper_140_no_table.urdf (robot description, URDF)
Before this commit: robot mara, 24 links, 23 joints
Links:
- added link gripper_adapter, mass 0.13969; collision mesh filename=package://mara_description/meshes/gripper_adapter.dae scale=0.001 0.001 0.001; visual mesh filename=package://mara_description/meshes/gripper_adapter.dae scale=0.001 0.001 0.001
- link left_inner_knuckle: geometry visual mesh filename=package://robotiq_140_gripper_description/meshes/robotiq_14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 scale=0.001 0.001 0.001
- link left_outer_finger: geometry collision mesh filename=package://robotiq_140_gripper_description/meshes/robotiq_14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 scale=0.001 0.001 0.001; visual mesh filename=package://robotiq_140_gripper_description/meshes/robotiq_14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 scale=0.001 0.001 0.001
- link left_outer_knuckle: geometry collision mesh filename=package://robotiq_140_gripper_description/meshes/robotiq_14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 scale=0.001 0.001 0.001; visual mesh filename=package://robotiq_140_gripper_description/meshes/robotiq_14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 scale=0.001 0.001 0.001
- link motor6_link: mass 0.14 -> 0.00001; geometry collision sphere radius=0; visual sphere radius=0
- link right_inner_knuckle: geometry visual mesh filename=package://robotiq_140_gripper_description/meshes/robotiq_14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 scale=0.001 0.001 0.001
- link right_outer_finger: geometry collision mesh filename=package://robotiq_140_gripper_description/meshes/robotiq_14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 scale=0.001 0.001 0.001; visual mesh filename=package://robotiq_140_gripper_description/meshes/robotiq_14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 scale=0.001 0.001 0.001
- link right_outer_knuckle: geometry collision mesh filename=package://robotiq_140_gripper_description/meshes/robotiq_14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 scale=0.001 0.001 0.001; visual mesh filename=package://robotiq_140_gripper_description/meshes/robotiq_14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 scale=0.001 0.001 0.001
- link robotiq_adapter_link: geometry collision mesh filename=package://mara_description/meshes/robotiq_adapter.dae scale=0.001 0.001 0.001; visual mesh filename=package://mara_description/meshes/robotiq_adapter.dae scale=0.001 0.001 0.001
Joints:
- removed joint base_adapter_to_base_robotiq_joint
- removed joint end_effector_adapter_to_robotiq
- removed joint left_inner_finger_joint
- removed joint left_inner_knuckle_joint
- removed joint left_outer_finger_joint
- removed joint left_outer_knuckle_joint
- removed joint right_inner_finger_joint
- removed joint right_inner_knuckle_joint
- removed joint right_outer_finger_joint
- removed joint world_to_base_joint
- added joint gripper_adapter_to_robotiq_adapter: type fixed, parent gripper_adapter, child robotiq_adapter_link, origin xyz= 0 0 0.05679 rpy=0 0 0
- added joint left_outer_finger_to_inner: type revolute, parent left_outer_finger, child left_inner_finger, origin xyz=0.03543 0 0.0789 rpy=0 0 0, axis 0 1 0, limit lower=0 upper=0.78574722925 effort=1000 velocity=2.0, mimic joint=joint_finger multiplier=1 offset=0
- added joint left_outer_knuckle_to_finger: type fixed, parent left_outer_knuckle, child left_outer_finger, origin xyz=0.03142 0 -0.00453 rpy=0 0 0
- added joint motor6_to_gripper_adapter: type fixed, parent motor6_link, child gripper_adapter, origin xyz= 0 0 -0.02026 rpy=0 0 0
- added joint right_outer_finger_to_inner: type revolute, parent right_outer_finger, child right_inner_finger, origin xyz=-0.03543 0 0.0789 rpy=0 0 0, axis 0 -1 0, limit lower=0 upper=0.78574722925 effort=1000 velocity=2.0, mimic joint=joint_finger multiplier=1 offset=0
- added joint right_outer_knuckle_to_finger: type fixed, parent right_outer_knuckle, child right_outer_finger, origin xyz=-0.03142 0 -0.00453 rpy=0 0 0
- added joint robotiq_adapter_to_arg2f_base: type fixed, parent robotiq_adapter_link, child robotiq_arg2f_base_link, origin xyz= 0 0 0 rpy=0 0 0
- added joint robotiq_arg2f_base_to_left_inner_knuckle: type revolute, parent robotiq_arg2f_base_link, child left_inner_knuckle, origin xyz=0.0127 0 0.06118 rpy=0 0 0, axis 0 -1 0, limit lower=0 upper=0.78574722925 effort=1000 velocity=2.0, mimic joint=joint_finger multiplier=1 offset=0
- added joint robotiq_arg2f_base_to_left_outer_knuckle: type revolute, parent robotiq_arg2f_base_link, child left_outer_knuckle, origin xyz=0.0306 0 0.05466 rpy=0 0 0, axis 0 -1 0, limit lower=0 upper=0.78574722925 effort=1000 velocity=2.0, mimic joint=joint_finger multiplier=1 offset=0
- added joint robotiq_arg2f_base_to_right_inner_knuckle: type revolute, parent robotiq_arg2f_base_link, child right_inner_knuckle, origin xyz=-0.0127 0 0.06118 rpy=0 0 0, axis 0 1 0, limit lower=0 upper=0.78574722925 effort=1000 velocity=2.0, mimic joint=joint_finger multiplier=1 offset=0
- added joint world_to_table: type fixed, parent world, child base_link, origin xyz=0 0 0 rpy=0 0 0
- joint ee_link: origin xyz=0 0.0 0.24 rpy=0 -1.57 0 -> xyz=0 0.0 0.24497 rpy=0 -1.57 0
- joint joint_finger: axis -1 0 0 -> 0 1 0; limit lower=0 upper=0.775 effort=1000 velocity=2.0 -> lower=0 upper=0.78574722925 effort=1000 velocity=2.0; origin xyz=0 0.030601 0.054905 rpy=2.31 0 3.14159265359 -> xyz=-0.0306 0 0.05466 rpy=0 0 0
- joint motor6_link-tool0_fixed_joint: origin xyz=0 0.0 0.24 rpy=0 -1.57 0 -> xyz=0 0.0 0.24497 rpy=0 -1.57 0
