Commit message: fix inertia and mass of the camera

File: mara_description/urdf/camera_gripper_support.urdf.xacro (robot description, xacro)
@@ -6,5 +6,5 @@
         <origin rpy="0 0 0" xyz="8.625E-08 -4.6583E-06 0.03145"/>
         <mass value="0.1"/>
-        <inertia ixx="0.00739172" ixy="-0.00001" ixz="0.0" iyy="0.00739172" iyz="0.0" izz="0.0147358995"/>
+        <inertia ixx="91283.23E-9" ixy="634.87E-9" ixz="-0.02E-9" iyy="97239.94E-9" iyz="93.72E-9" izz="175963.64E-9"/>
       </inertial>
       <visual>
@@ -31,6 +31,6 @@
       <inertial>
         <origin rpy="0 0 0" xyz="8.625E-08 -4.6583E-06 0.03145"/>
-        <mass value="0.1"/>
-        <inertia ixx="0.00739172" ixy="-0.00001" ixz="0.0" iyy="0.00739172" iyz="0.0" izz="0.0147358995"/>
+        <mass value="0.00361"/>
+        <inertia ixx="266.47E-9" ixy="0.0" ixz="0.0" iyy="115.40E-9" iyz="-0.40E-9" izz="233.53E-9"/>
       </inertial>
       <visual>
@@ -57,6 +57,6 @@
       <inertial>
         <origin rpy="0 0 0" xyz="8.625E-08 -4.6583E-06 0.03145"/>
-        <mass value="0.1"/>
-        <inertia ixx="0.00739172" ixy="-0.00001" ixz="0.0" iyy="0.00739172" iyz="0.0" izz="0.0147358995"/>
+        <mass value="0.00676"/>
+        <inertia ixx="584.80E-9" ixy="28.57E-9" ixz="-2.42E-9" iyy="1930.29E-9" iyz="-140.62E-9" izz="2077.50E-9"/>
       </inertial>
       <visual>

File: mara_description/urdf/reinforcement_learning/mara_robot_gripper_140_camera_run.urdf (robot description, URDF)
Before this commit: robot mara, 32 links, 31 joints
Links:
- link camera_link: mass 0.564 -> 0.07397
- link mara_camera_support1_link: mass 0.1 -> 0.00361
- link mara_camera_support2_link: mass 0.1 -> 0.00676

File: mara_description/urdf/reinforcement_learning/mara_robot_gripper_140_camera_train.urdf (robot description, URDF)
Before this commit: robot mara, 32 links, 31 joints
Links:
- link camera_link: mass 0.564 -> 0.07397
- link mara_camera_support1_link: mass 0.1 -> 0.00361
- link mara_camera_support2_link: mass 0.1 -> 0.00676

File: mara_description/urdf/rs_d435.urdf.xacro (robot description, xacro)
@@ -5,6 +5,6 @@
       <inertial>
         <origin rpy="0 0 0" xyz="8.625E-08 -4.6583E-06 0.03145"/>
-        <mass value="0.564"/>
-        <inertia ixx="0.003881243" ixy="0.0" ixz="0.0" iyy="0.000498940" iyz="0.0" izz="0.003879257" />
+        <mass value="0.07397"/>
+        <inertia ixx="6975.32E-9" ixy="287.18E-9" ixz="25.68E-9" iyy="47975.37E-9" iyz="-25.58E-9" izz="48114.25E-9" />
       </inertial>
       <visual>

Commit message: update mara_gripper_adapter mass value

File: mara_description/urdf/camera_gripper_support.urdf.xacro (robot description, xacro)
@@ -5,5 +5,5 @@
       <inertial>
         <origin rpy="0 0 0" xyz="8.625E-08 -4.6583E-06 0.03145"/>
-        <mass value="0.1"/>
+        <mass value="0.13969"/>
         <inertia ixx="91283.23E-9" ixy="634.87E-9" ixz="-0.02E-9" iyy="97239.94E-9" iyz="93.72E-9" izz="175963.64E-9"/>
       </inertial>

File: mara_description/urdf/reinforcement_learning/mara_robot_gripper_140_camera_run.urdf (robot description, URDF)
Before this commit: robot mara, 32 links, 31 joints
Links:
- link mara_gripper_adapter: mass 0.1 -> 0.13969

File: mara_description/urdf/reinforcement_learning/mara_robot_gripper_140_camera_train.urdf (robot description, URDF)
Before this commit: robot mara, 32 links, 31 joints
Links:
- link mara_gripper_adapter: mass 0.1 -> 0.13969

Commit message: remove tool0 and mara naming from camera

File: mara_description/urdf/camera_gripper_support.urdf.xacro (robot description, xacro)
@@ -1,6 +1,6 @@
 <?xml version="1.0"?>
 <robot xmlns:xacro="http://ros.org/wiki/xacro">
-  <xacro:macro name="mara_camera_gripper_support" params="prefix">
-    <link name="${prefix}mara_gripper_adapter">
+  <xacro:macro name="camera_gripper_support" params="prefix">
+    <link name="${prefix}gripper_adapter">
       <inertial>
         <origin rpy="0 0 0" xyz="8.625E-08 -4.6583E-06 0.03145"/>
@@ -24,9 +24,9 @@
       </collision>
     </link>
-    <gazebo reference="${prefix}mara_gripper_adapter">
+    <gazebo reference="${prefix}gripper_adapter">
       <material>Gazebo/Black</material>
       <selfCollide>True</selfCollide>
     </gazebo>
-    <link name="${prefix}mara_camera_support1_link">
+    <link name="${prefix}camera_support1_link">
       <inertial>
         <origin rpy="0 0 0" xyz="8.625E-08 -4.6583E-06 0.03145"/>
@@ -50,9 +50,9 @@
       </collision>
     </link>
-    <gazebo reference="${prefix}mara_camera_support1_link">
+    <gazebo reference="${prefix}camera_support1_link">
       <material>Gazebo/Black</material>
       <selfCollide>True</selfCollide>
     </gazebo>
-    <link name="${prefix}mara_camera_support2_link">
+    <link name="${prefix}camera_support2_link">
       <inertial>
         <origin rpy="0 0 0" xyz="8.625E-08 -4.6583E-06 0.03145"/>
@@ -76,5 +76,5 @@
       </collision>
     </link>
-    <gazebo reference="${prefix}mara_camera_support2_link">
+    <gazebo reference="${prefix}camera_support2_link">
       <material>Gazebo/Black</material>
       <selfCollide>True</selfCollide>
@@ -82,11 +82,11 @@
     <joint name="${prefix}gripper_adapter_to_camera_support1" type="fixed">
       <origin rpy="0 0 0" xyz="0 0.03956 -0.0213"/>
-      <parent link="${prefix}mara_gripper_adapter"/>
-      <child link="${prefix}mara_camera_support1_link"/>
+      <parent link="${prefix}gripper_adapter"/>
+      <child link="${prefix}camera_support1_link"/>
     </joint>
     <joint name="${prefix}camera_support1_to_support2" type="fixed">
       <origin rpy="0 0 0" xyz="0 0.01029 -0.0128"/>
-      <parent link="${prefix}mara_camera_support1_link"/>
-      <child link="${prefix}mara_camera_support2_link"/>
+      <parent link="${prefix}camera_support1_link"/>
+      <child link="${prefix}camera_support2_link"/>
     </joint>
   </xacro:macro>

File: mara_description/urdf/reinforcement_learning/mara_robot_gripper_140_camera_run.urdf (robot description, URDF)
Before this commit: robot mara, 31 links, 30 joints
Links:
- removed link mara_camera_support1_link
- removed link mara_camera_support2_link
- removed link mara_gripper_adapter
- removed link tool0
- added link camera_support1_link, mass 0.00361; collision mesh filename=package://mara_description/meshes/Camera_Support_1.dae scale=0.001 0.001 0.001; visual mesh filename=package://mara_description/meshes/Camera_Support_1.dae scale=0.001 0.001 0.001
- added link camera_support2_link, mass 0.00676; collision mesh filename=package://mara_description/meshes/Camera_Support_2.dae scale=0.001 0.001 0.001; visual mesh filename=package://mara_description/meshes/Camera_Support_2.dae scale=0.001 0.001 0.001
- added link gripper_adapter, mass 0.13969; collision mesh filename=package://mara_description/meshes/ROBOTIQ_Gripper_Adapter.d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 scale=0.001 0.001 0.001; visual mesh filename=package://mara_description/meshes/ROBOTIQ_Gripper_Adapter.d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 scale=0.001 0.001 0.001
Joints:
- removed joint mara_camera_gripper_support_to_robotiq_adapter
- removed joint motor6_link-tool0_fixed_joint
- removed joint motor6_to_mara_camera_gripper_support
- added joint camera_gripper_support_to_robotiq_adapter: type fixed, parent gripper_adapter, child robotiq_adapter_link, origin xyz= 0 0 0 rpy=0 0 1.57
- added joint motor6_to_camera_gripper_support: type fixed, parent motor6_link, child gripper_adapter, origin xyz=0 0 0 rpy=0 0 0
- joint camera_support1_to_support2: child mara_camera_support2_link -> camera_support2_link; parent mara_camera_support1_link -> camera_support1_link
- joint camera_support2_to_camera: parent mara_camera_support2_link -> camera_support2_link
- joint gripper_adapter_to_camera_support1: child mara_camera_support1_link -> camera_support1_link; parent mara_gripper_adapter -> gripper_adapter

File: mara_description/urdf/reinforcement_learning/mara_robot_gripper_140_camera_run.urdf.xacro (robot description, xacro)
@@ -11,5 +11,5 @@
   <!-- arm -->
   <xacro:mara_robot_run prefix="" ee_link_distance="0.2"/>
-  <xacro:mara_camera_gripper_support prefix="" />
+  <xacro:camera_gripper_support prefix="" />
   <xacro:rs_d435_camera prefix="" />
   <xacro:robotiq_gripper prefix="mara" />
@@ -80,17 +80,17 @@
     <dynamics damping="0" friction="0"/>
   </joint>
-  <joint name="motor6_to_mara_camera_gripper_support" type="fixed">
+  <joint name="motor6_to_camera_gripper_support" type="fixed">
     <origin rpy="0 0 0" xyz="0 0 0"/>
     <parent link="motor6_link"/>
-    <child link="mara_gripper_adapter"/>
+    <child link="gripper_adapter"/>
   </joint>
   <joint name="camera_support2_to_camera" type="fixed">
     <origin rpy="0 0 0" xyz="0 0.018 0.012"/>
-    <parent link="mara_camera_support2_link"/>
+    <parent link="camera_support2_link"/>
     <child link="camera_link"/>
   </joint>
-  <joint name="mara_camera_gripper_support_to_robotiq_adapter" type="fixed">
+  <joint name="camera_gripper_support_to_robotiq_adapter" type="fixed">
     <origin rpy="0 0 1.57" xyz=" 0 0 0"/>
-    <parent link="mara_gripper_adapter"/>
+    <parent link="gripper_adapter"/>
     <child link="robotiq_adapter_link"/>
   </joint>

File: mara_description/urdf/reinforcement_learning/mara_robot_gripper_140_camera_train.urdf (robot description, URDF)
Before this commit: robot mara, 31 links, 30 joints
Links:
- removed link mara_camera_support1_link
- removed link mara_camera_support2_link
- removed link mara_gripper_adapter
- removed link tool0
- added link camera_support1_link, mass 0.00361; collision mesh filename=package://mara_description/meshes/Camera_Support_1.dae scale=0.001 0.001 0.001; visual mesh filename=package://mara_description/meshes/Camera_Support_1.dae scale=0.001 0.001 0.001
- added link camera_support2_link, mass 0.00676; collision mesh filename=package://mara_description/meshes/Camera_Support_2.dae scale=0.001 0.001 0.001; visual mesh filename=package://mara_description/meshes/Camera_Support_2.dae scale=0.001 0.001 0.001
- added link gripper_adapter, mass 0.13969; collision mesh filename=package://mara_description/meshes/ROBOTIQ_Gripper_Adapter.d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 scale=0.001 0.001 0.001; visual mesh filename=package://mara_description/meshes/ROBOTIQ_Gripper_Adapter.d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 scale=0.001 0.001 0.001
Joints:
- removed joint mara_camera_gripper_support_to_robotiq_adapter
- removed joint motor6_link-tool0_fixed_joint
- removed joint motor6_to_mara_camera_gripper_support
- added joint camera_gripper_support_to_robotiq_adapter: type fixed, parent gripper_adapter, child robotiq_adapter_link, origin xyz= 0 0 0 rpy=0 0 1.57
- added joint motor6_to_camera_gripper_support: type fixed, parent motor6_link, child gripper_adapter, origin xyz=0 0 0 rpy=0 0 0
- joint camera_support1_to_support2: child mara_camera_support2_link -> camera_support2_link; parent mara_camera_support1_link -> camera_support1_link
- joint camera_support2_to_camera: parent mara_camera_support2_link -> camera_support2_link
- joint gripper_adapter_to_camera_support1: child mara_camera_support1_link -> camera_support1_link; parent mara_gripper_adapter -> gripper_adapter

File: mara_description/urdf/reinforcement_learning/mara_robot_gripper_140_camera_train.urdf.xacro (robot description, xacro)
@@ -11,5 +11,5 @@
   <!-- arm -->
   <xacro:mara_robot_train prefix="" ee_link_distance="0.2"/>
-  <xacro:mara_camera_gripper_support prefix="" />
+  <xacro:camera_gripper_support prefix="" />
   <xacro:rs_d435_camera prefix="" />
   <xacro:robotiq_gripper prefix="mara" />
@@ -80,17 +80,17 @@
     <dynamics damping="0" friction="0"/>
   </joint>
-  <joint name="motor6_to_mara_camera_gripper_support" type="fixed">
+  <joint name="motor6_to_camera_gripper_support" type="fixed">
     <origin rpy="0 0 0" xyz="0 0 0"/>
     <parent link="motor6_link"/>
-    <child link="mara_gripper_adapter"/>
+    <child link="gripper_adapter"/>
   </joint>
   <joint name="camera_support2_to_camera" type="fixed">
     <origin rpy="0 0 0" xyz="0 0.018 0.012"/>
-    <parent link="mara_camera_support2_link"/>
+    <parent link="camera_support2_link"/>
     <child link="camera_link"/>
   </joint>
-  <joint name="mara_camera_gripper_support_to_robotiq_adapter" type="fixed">
+  <joint name="camera_gripper_support_to_robotiq_adapter" type="fixed">
     <origin rpy="0 0 1.57" xyz=" 0 0 0"/>
-    <parent link="mara_gripper_adapter"/>
+    <parent link="gripper_adapter"/>
     <child link="robotiq_adapter_link"/>
   </joint>

File: mara_description/urdf/reinforcement_learning/mara_robot_run.urdf (robot description, URDF)
Before this commit: robot mara, 13 links, 12 joints
Links:
- removed link tool0
Joints:
- removed joint motor6_link-tool0_fixed_joint

File: mara_description/urdf/reinforcement_learning/mara_robot_train.urdf (robot description, URDF)
Before this commit: robot mara, 13 links, 12 joints
Links:
- removed link tool0
Joints:
- removed joint motor6_link-tool0_fixed_joint

File: mara_description/urdf/reinforcement_learning/mara_run.urdf.xacro (robot description, xacro)
@@ -306,10 +306,4 @@
       <child link="${prefix}ee_link"/>
     </joint>
-    <link name="${prefix}tool0"/>
-    <joint name="${prefix}${prefix}motor6_link-tool0_fixed_joint" type="fixed">
-      <origin rpy="0 0 0" xyz="0 0.0 ${ee_link_distance}"/>
-      <parent link="${prefix}${prefix}motor6_link"/>
-      <child link="${prefix}tool0"/>
-    </joint>
     <xacro:mara_transmission prefix="${prefix}"/>
     <xacro:mara_gazebo_run prefix="${prefix}"/>

File: mara_description/urdf/reinforcement_learning/mara_train.urdf.xacro (robot description, xacro)
@@ -306,10 +306,4 @@
       <child link="${prefix}ee_link"/>
     </joint>
-    <link name="${prefix}tool0"/>
-    <joint name="${prefix}${prefix}motor6_link-tool0_fixed_joint" type="fixed">
-      <origin rpy="0 0 0" xyz="0 0.0 ${ee_link_distance}"/>
-      <parent link="${prefix}${prefix}motor6_link"/>
-      <child link="${prefix}tool0"/>
-    </joint>
     <xacro:mara_transmission prefix="${prefix}"/>
     <xacro:mara_gazebo_train prefix="${prefix}"/>
