Commit message: update adapter dae files and its dependencies

File: mara_description/urdf/camera_gripper_support.urdf.xacro (robot description, xacro)
@@ -11,5 +11,5 @@
         <origin rpy="0 0 0" xyz="0 0 0"/>
         <geometry>
-          <mesh filename="package://mara_description/meshes/ROBOTIQ_Gripper_Adapter.dae" scale="0.001 0.001 0.001"/>
+          <mesh filename="package://mara_description/meshes/gripper_adapter.dae" scale="0.001 0.001 0.001"/>
         </geometry>
         <material name="Gazebo/Wood">
@@ -20,5 +20,5 @@
         <origin rpy="0 0 0" xyz="0 0 0"/>
         <geometry>
-          <mesh filename="package://mara_description/meshes/ROBOTIQ_Gripper_Adapter.dae" scale="0.001 0.001 0.001"/>
+          <mesh filename="package://mara_description/meshes/gripper_adapter.dae" scale="0.001 0.001 0.001"/>
         </geometry>
       </collision>
@@ -81,10 +81,10 @@
     </gazebo>
     <joint name="${prefix}gripper_adapter_to_camera_support1" type="fixed">
-      <origin rpy="0 0 0" xyz="0 0.03956 -0.0213"/>
+      <origin rpy="0 0 0" xyz="0 0.03956 -0.00213"/>
       <parent link="${prefix}gripper_adapter"/>
       <child link="${prefix}camera_support1_link"/>
     </joint>
     <joint name="${prefix}camera_support1_to_support2" type="fixed">
-      <origin rpy="0 0 0" xyz="0 0.01029 -0.0128"/>
+      <origin rpy="0 0 0" xyz="0 0.01029 -0.00128"/>
       <parent link="${prefix}camera_support1_link"/>
       <child link="${prefix}camera_support2_link"/>

File: mara_description/urdf/reinforcement_learning/mara_robot_gripper_140_camera_run.urdf (robot description, URDF)
Before this commit: robot mara, 30 links, 29 joints
Links:
- link gripper_adapter: geometry collision mesh filename=package://mara_description/meshes/gripper_adapter.dae scale=0.001 0.001 0.001; visual mesh filename=package://mara_description/meshes/gripper_adapter.dae scale=0.001 0.001 0.001
- link robotiq_adapter_link: geometry collision mesh filename=package://mara_description/meshes/robotiq_adapter.dae scale=0.001 0.001 0.001; visual mesh filename=package://mara_description/meshes/robotiq_adapter.dae scale=0.001 0.001 0.001
Joints:
- removed joint camera_gripper_support_to_robotiq_adapter
- removed joint motor6_to_camera_gripper_support
- added joint gripper_adapter_to_robotiq_adapter: type fixed, parent gripper_adapter, child robotiq_adapter_link, origin xyz=0 0 0.05679 rpy=0 0 0
- added joint motor6_to_gripper_adapter: type fixed, parent motor6_link, child gripper_adapter, origin xyz=0 0 -0.02026 rpy=0 0 0
- joint camera_support1_to_support2: origin xyz=0 0.01029 -0.0128 rpy=0 0 0 -> xyz=0 0.01029 -0.00128 rpy=0 0 0
- joint ee_link: origin xyz=0 0.0 0.2 rpy=0 0 0 -> xyz=0 0.0 0.24 rpy=0 0 0
- joint gripper_adapter_to_camera_support1: origin xyz=0 0.03956 -0.0213 rpy=0 0 0 -> xyz=0 0.03956 -0.00213 rpy=0 0 0
- joint robotiq_adapter_link_to_robotiq_arg2f_base_link: origin xyz= 0 0 0 rpy=0 0 1.57 -> xyz= 0 0 0 rpy=0 0 0

File: mara_description/urdf/reinforcement_learning/mara_robot_gripper_140_camera_run.urdf.xacro (robot description, xacro)
@@ -10,5 +10,5 @@
   <xacro:include filename="$(find robotiq_140_gripper_description)/urdf/robotiq_140.urdf.xacro" />
   <!-- arm -->
-  <xacro:mara_robot_run prefix="" ee_link_distance="0.2"/>
+  <xacro:mara_robot_run prefix="" ee_link_distance="0.24"/>
   <xacro:camera_gripper_support prefix="" />
   <xacro:rs_d435_camera prefix="" />
@@ -48,7 +48,7 @@
     </inertial>
     <visual>
-      <origin xyz="0 0 0" rpy="0 0 1.57" />
+      <origin xyz="0 0 0" rpy="0 0 0" />
       <geometry>
-        <mesh filename="package://robotiq_140_gripper_description/meshes/hros_robotiq_adapter.dae" scale="0.001 0.001 0.001"/>
+        <mesh filename="package://mara_description/meshes/robotiq_adapter.dae" scale="0.001 0.001 0.001"/>
       </geometry>
       <material name="Gazebo/Black">
@@ -57,7 +57,7 @@
     </visual>
     <collision>
-      <origin xyz="0 0 0" rpy="0 0 1.57" />
+      <origin xyz="0 0 0" rpy="0 0 0" />
       <geometry>
-        <mesh filename="package://robotiq_140_gripper_description/meshes/hros_robotiq_adapter.dae" scale="0.001 0.001 0.001"/>
+        <mesh filename="package://mara_description/meshes/robotiq_adapter.dae" scale="0.001 0.001 0.001"/>
       </geometry>
     </collision>
@@ -80,8 +80,13 @@
     <dynamics damping="0" friction="0"/>
   </joint>
-  <joint name="motor6_to_camera_gripper_support" type="fixed">
-    <origin rpy="0 0 0" xyz="0 0 0"/>
+  <joint name="motor6_to_gripper_adapter" type="fixed">
+    <origin rpy="0 0 0" xyz="0 0 -0.02026"/>
     <parent link="motor6_link"/>
     <child link="gripper_adapter"/>
+  </joint>
+  <joint name="gripper_adapter_to_robotiq_adapter" type="fixed">
+    <origin rpy="0 0 0" xyz="0 0 0.05679"/>
+    <parent link="gripper_adapter"/>
+    <child link="robotiq_adapter_link"/>
   </joint>
   <joint name="camera_support2_to_camera" type="fixed">
@@ -90,11 +95,6 @@
     <child link="camera_link"/>
   </joint>
-  <joint name="camera_gripper_support_to_robotiq_adapter" type="fixed">
-    <origin rpy="0 0 1.57" xyz=" 0 0 0"/>
-    <parent link="gripper_adapter"/>
-    <child link="robotiq_adapter_link"/>
-  </joint>
   <joint name="robotiq_adapter_link_to_robotiq_arg2f_base_link" type="fixed">
-    <origin rpy="0 0 1.57" xyz=" 0 0 0"/>
+    <origin rpy="0 0 0" xyz=" 0 0 0"/>
     <parent link="robotiq_adapter_link"/>
     <child link="robotiq_arg2f_base_link"/>

File: mara_description/urdf/reinforcement_learning/mara_robot_gripper_140_camera_train.urdf (robot description, URDF)
Before this commit: robot mara, 30 links, 29 joints
Links:
- link gripper_adapter: geometry collision mesh filename=package://mara_description/meshes/gripper_adapter.dae scale=0.001 0.001 0.001; visual mesh filename=package://mara_description/meshes/gripper_adapter.dae scale=0.001 0.001 0.001
- link robotiq_adapter_link: geometry collision mesh filename=package://mara_description/meshes/robotiq_adapter.dae scale=0.001 0.001 0.001; visual mesh filename=package://mara_description/meshes/robotiq_adapter.dae scale=0.001 0.001 0.001
Joints:
- removed joint camera_gripper_support_to_robotiq_adapter
- removed joint motor6_to_camera_gripper_support
- added joint gripper_adapter_to_robotiq_adapter: type fixed, parent gripper_adapter, child robotiq_adapter_link, origin xyz=0 0 0.05679 rpy=0 0 0
- added joint motor6_to_gripper_adapter: type fixed, parent motor6_link, child gripper_adapter, origin xyz=0 0 -0.02026 rpy=0 0 0
- joint camera_support1_to_support2: origin xyz=0 0.01029 -0.0128 rpy=0 0 0 -> xyz=0 0.01029 -0.00128 rpy=0 0 0
- joint ee_link: origin xyz=0 0.0 0.2 rpy=0 0 0 -> xyz=0 0.0 0.24 rpy=0 0 0
- joint gripper_adapter_to_camera_support1: origin xyz=0 0.03956 -0.0213 rpy=0 0 0 -> xyz=0 0.03956 -0.00213 rpy=0 0 0
- joint robotiq_adapter_link_to_robotiq_arg2f_base_link: origin xyz= 0 0 0 rpy=0 0 1.57 -> xyz= 0 0 0 rpy=0 0 0

File: mara_description/urdf/reinforcement_learning/mara_robot_gripper_140_camera_train.urdf.xacro (robot description, xacro)
@@ -10,5 +10,5 @@
   <xacro:include filename="$(find robotiq_140_gripper_description)/urdf/robotiq_140.urdf.xacro" />
   <!-- arm -->
-  <xacro:mara_robot_train prefix="" ee_link_distance="0.2"/>
+  <xacro:mara_robot_train prefix="" ee_link_distance="0.24"/>
   <xacro:camera_gripper_support prefix="" />
   <xacro:rs_d435_camera prefix="" />
@@ -48,7 +48,7 @@
     </inertial>
     <visual>
-      <origin xyz="0 0 0" rpy="0 0 1.57" />
+      <origin xyz="0 0 0" rpy="0 0 0" />
       <geometry>
-        <mesh filename="package://robotiq_140_gripper_description/meshes/hros_robotiq_adapter.dae" scale="0.001 0.001 0.001"/>
+        <mesh filename="package://mara_description/meshes/robotiq_adapter.dae" scale="0.001 0.001 0.001"/>
       </geometry>
       <material name="Gazebo/Black">
@@ -57,7 +57,7 @@
     </visual>
     <collision>
-      <origin xyz="0 0 0" rpy="0 0 1.57" />
+      <origin xyz="0 0 0" rpy="0 0 0" />
       <geometry>
-        <mesh filename="package://robotiq_140_gripper_description/meshes/hros_robotiq_adapter.dae" scale="0.001 0.001 0.001"/>
+        <mesh filename="package://mara_description/meshes/robotiq_adapter.dae" scale="0.001 0.001 0.001"/>
       </geometry>
     </collision>
@@ -80,8 +80,13 @@
     <dynamics damping="0" friction="0"/>
   </joint>
-  <joint name="motor6_to_camera_gripper_support" type="fixed">
-    <origin rpy="0 0 0" xyz="0 0 0"/>
+  <joint name="motor6_to_gripper_adapter" type="fixed">
+    <origin rpy="0 0 0" xyz="0 0 -0.02026"/>
     <parent link="motor6_link"/>
     <child link="gripper_adapter"/>
+  </joint>
+  <joint name="gripper_adapter_to_robotiq_adapter" type="fixed">
+    <origin rpy="0 0 0" xyz="0 0 0.05679"/>
+    <parent link="gripper_adapter"/>
+    <child link="robotiq_adapter_link"/>
   </joint>
   <joint name="camera_support2_to_camera" type="fixed">
@@ -90,11 +95,6 @@
     <child link="camera_link"/>
   </joint>
-  <joint name="camera_gripper_support_to_robotiq_adapter" type="fixed">
-    <origin rpy="0 0 1.57" xyz=" 0 0 0"/>
-    <parent link="gripper_adapter"/>
-    <child link="robotiq_adapter_link"/>
-  </joint>
   <joint name="robotiq_adapter_link_to_robotiq_arg2f_base_link" type="fixed">
-    <origin rpy="0 0 1.57" xyz=" 0 0 0"/>
+    <origin rpy="0 0 0" xyz=" 0 0 0"/>
     <parent link="robotiq_adapter_link"/>
     <child link="robotiq_arg2f_base_link"/>
