Commit message: fix inertial values of the adapters

File: mara_description/urdf/camera_gripper_support.urdf.xacro (robot description, xacro)
@@ -4,7 +4,7 @@
     <link name="${prefix}gripper_adapter">
       <inertial>
-        <origin rpy="0 0 0" xyz="8.625E-08 -4.6583E-06 0.03145"/>
-        <mass value="0.13969"/>
-        <inertia ixx="91283.23E-9" ixy="634.87E-9" ixz="-0.02E-9" iyy="97239.94E-9" iyz="93.72E-9" izz="175963.64E-9"/>
+        <origin rpy="0 0 0" xyz="0 0 0.0173"/>
+        <mass value="0.14"/>
+        <inertia ixx="0.0001" ixy="0" ixz="0" iyy="0.0001" iyz="0" izz="0.0002"/>
       </inertial>
       <visual>

File: mara_description/urdf/mara_robot_gripper_140.urdf (robot description, URDF)
Before this commit: robot mara, 26 links, 25 joints
Links:
- link gripper_adapter: mass 0.13969 -> 0.14
- link left_inner_finger: mass 0.0104003125914103 -> 0.045
- link left_inner_knuckle: mass 0.0271177346495152 -> 0.04476; geometry collision mesh filename=package://robotiq_140_gripper_description/meshes/robotiq_14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 scale=0.001 0.001 0.001; visual mesh filename=package://robotiq_140_gripper_description/meshes/robotiq_14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 scale=0.001 0.001 0.001
- link left_outer_finger: mass 0.022614240507152 -> 0.07637
- link left_outer_knuckle: mass 0.00853198276973456 -> 0.0131
- link right_inner_finger: mass 0.0104003125914103 -> 0.045
- link right_inner_knuckle: mass 0.0271177346495152 -> 0.04476; geometry collision mesh filename=package://robotiq_140_gripper_description/meshes/robotiq_14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 scale=0.001 0.001 0.001; visual mesh filename=package://robotiq_140_gripper_description/meshes/robotiq_14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 scale=0.001 0.001 0.001
- link right_outer_finger: mass 0.022614240507152 -> 0.07637
- link right_outer_knuckle: mass 0.00853198276973456 -> 0.0131
- link robotiq_adapter_link: mass 0.22652 -> 0.317
- link robotiq_arg2f_base_link: mass 0.22652 -> 0.52954
Joints:
- joint joint_finger: limit lower=0 upper=0.78574722925 effort=1000 velocity=2.0 -> lower=0 upper=0.78574722925 effort=18.65 velocity=3.54
- joint left_outer_finger_to_inner: limit lower=0 upper=0.78574722925 effort=1000 velocity=2.0 -> lower=0 upper=0.78574722925 effort=18.65 velocity=3.54
- joint right_outer_finger_to_inner: limit lower=0 upper=0.78574722925 effort=1000 velocity=2.0 -> lower=0 upper=0.78574722925 effort=18.65 velocity=3.54
- joint robotiq_arg2f_base_to_left_inner_knuckle: limit lower=0 upper=0.78574722925 effort=1000 velocity=2.0 -> lower=0 upper=0.78574722925 effort=18.65 velocity=3.54
- joint robotiq_arg2f_base_to_left_outer_knuckle: limit lower=0 upper=0.78574722925 effort=1000 velocity=2.0 -> lower=0 upper=0.78574722925 effort=18.65 velocity=2.0
- joint robotiq_arg2f_base_to_right_inner_knuckle: limit lower=0 upper=0.78574722925 effort=1000 velocity=2.0 -> lower=0 upper=0.78574722925 effort=18.65 velocity=3.54

File: mara_description/urdf/mara_robot_gripper_140.urdf.xacro (robot description, xacro)
@@ -15,7 +15,7 @@
   <link name="gripper_adapter">
     <inertial>
-      <origin rpy="0 0 0" xyz="8.625E-08 -4.6583E-06 0.03145"/>
-      <mass value="0.13969"/>
-      <inertia ixx="91283.23E-9" ixy="634.87E-9" ixz="-0.02E-9" iyy="97239.94E-9" iyz="93.72E-9" izz="175963.64E-9"/>
+      <origin rpy="0 0 0" xyz="0 0 0.0173"/>
+      <mass value="0.14"/>
+      <inertia ixx="0.0001" ixy="0" ixz="0" iyy="0.0001" iyz="0" izz="0.0002"/>
     </inertial>
     <visual>
@@ -41,7 +41,7 @@
   <link name="robotiq_adapter_link">
     <inertial>
-      <origin xyz="8.625E-08 -4.6583E-06 0.03145" rpy="0 0 0" />
-      <mass value="0.22652" />
-      <inertia ixx="0.00020005" ixy="0" ixz="0" iyy="0.00017832" iyz="0" izz="0.00013478" />
+      <origin xyz="0 0 -0.0253" rpy="0 0 0" />
+      <mass value="0.317" />
+      <inertia ixx="298526E-9" ixy="3928E-9" ixz="-926E-9" iyy="354661E-9" iyz="42E-9" izz="415572E-9" />
     </inertial>
     <visual>

File: mara_description/urdf/mara_robot_gripper_140_no_table.urdf (robot description, URDF)
Before this commit: robot mara, 25 links, 24 joints
Links:
- link gripper_adapter: mass 0.13969 -> 0.14
- link left_inner_finger: mass 0.0104003125914103 -> 0.045
- link left_inner_knuckle: mass 0.0271177346495152 -> 0.04476; geometry collision mesh filename=package://robotiq_140_gripper_description/meshes/robotiq_14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 scale=0.001 0.001 0.001; visual mesh filename=package://robotiq_140_gripper_description/meshes/robotiq_14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 scale=0.001 0.001 0.001
- link left_outer_finger: mass 0.022614240507152 -> 0.07637
- link left_outer_knuckle: mass 0.00853198276973456 -> 0.0131
- link right_inner_finger: mass 0.0104003125914103 -> 0.045
- link right_inner_knuckle: mass 0.0271177346495152 -> 0.04476; geometry collision mesh filename=package://robotiq_140_gripper_description/meshes/robotiq_14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 scale=0.001 0.001 0.001; visual mesh filename=package://robotiq_140_gripper_description/meshes/robotiq_14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 scale=0.001 0.001 0.001
- link right_outer_finger: mass 0.022614240507152 -> 0.07637
- link right_outer_knuckle: mass 0.00853198276973456 -> 0.0131
- link robotiq_adapter_link: mass 0.22652 -> 0.317
- link robotiq_arg2f_base_link: mass 0.22652 -> 0.52954
Joints:
- joint joint_finger: limit lower=0 upper=0.78574722925 effort=1000 velocity=2.0 -> lower=0 upper=0.78574722925 effort=18.65 velocity=3.54
- joint left_outer_finger_to_inner: limit lower=0 upper=0.78574722925 effort=1000 velocity=2.0 -> lower=0 upper=0.78574722925 effort=18.65 velocity=3.54
- joint right_outer_finger_to_inner: limit lower=0 upper=0.78574722925 effort=1000 velocity=2.0 -> lower=0 upper=0.78574722925 effort=18.65 velocity=3.54
- joint robotiq_arg2f_base_to_left_inner_knuckle: limit lower=0 upper=0.78574722925 effort=1000 velocity=2.0 -> lower=0 upper=0.78574722925 effort=18.65 velocity=3.54
- joint robotiq_arg2f_base_to_left_outer_knuckle: limit lower=0 upper=0.78574722925 effort=1000 velocity=2.0 -> lower=0 upper=0.78574722925 effort=18.65 velocity=2.0
- joint robotiq_arg2f_base_to_right_inner_knuckle: limit lower=0 upper=0.78574722925 effort=1000 velocity=2.0 -> lower=0 upper=0.78574722925 effort=18.65 velocity=3.54

File: mara_description/urdf/mara_robot_gripper_140_no_table.urdf.xacro (robot description, xacro)
@@ -13,7 +13,7 @@
   <link name="gripper_adapter">
     <inertial>
-      <origin rpy="0 0 0" xyz="8.625E-08 -4.6583E-06 0.03145"/>
-      <mass value="0.13969"/>
-      <inertia ixx="91283.23E-9" ixy="634.87E-9" ixz="-0.02E-9" iyy="97239.94E-9" iyz="93.72E-9" izz="175963.64E-9"/>
+      <origin rpy="0 0 0" xyz="0 0 0.0173"/>
+      <mass value="0.14"/>
+      <inertia ixx="0.0001" ixy="0" ixz="0" iyy="0.0001" iyz="0" izz="0.0002"/>
     </inertial>
     <visual>
@@ -39,7 +39,7 @@
   <link name="robotiq_adapter_link">
     <inertial>
-      <origin xyz="8.625E-08 -4.6583E-06 0.03145" rpy="0 0 0" />
-      <mass value="0.22652" />
-      <inertia ixx="0.00020005" ixy="0" ixz="0" iyy="0.00017832" iyz="0" izz="0.00013478" />
+      <origin xyz="0 0 -0.0253" rpy="0 0 0" />
+      <mass value="0.317" />
+      <inertia ixx="298526E-9" ixy="3928E-9" ixz="-926E-9" iyy="354661E-9" iyz="42E-9" izz="415572E-9" />
     </inertial>
     <visual>

File: mara_description/urdf/mara_robot_gripper_85.urdf (robot description, URDF)
Before this commit: robot mara, 26 links, 25 joints
Links:
- link gripper_adapter: mass 0.13969 -> 0.14
- link left_inner_finger: mass 0.22652 -> 0.037
- link left_inner_knuckle: mass 0.22652 -> 0.02731
- link left_outer_finger: mass 0.22652 -> 0.03848
- link left_outer_knuckle: mass 0.22652 -> 0.01252
- link right_inner_finger: mass 0.22652 -> 0.037
- link right_inner_knuckle: mass 0.22652 -> 0.02731
- link right_outer_finger: mass 0.22652 -> 0.03848
- link right_outer_knuckle: mass 0.22652 -> 0.01252
- link robotiq_adapter_link: mass 0.22652 -> 0.317
- link robotiq_arg2f_base_link: mass 0.22652 -> 0.55938
Joints:
- joint joint_finger: limit lower=0 upper=0.78 effort=1000 velocity=2.0 -> lower=0 upper=0.82589 effort=21.03 velocity=3.87
- joint left_outer_finger_to_inner: limit lower=0 upper=0.775 effort=1000 velocity=2.0 -> lower=0 upper=0.82589 effort=21.03 velocity=3.87
- joint right_outer_finger_to_inner: limit lower=0 upper=0.775 effort=1000 velocity=2.0 -> lower=0 upper=0.82589 effort=21.03 velocity=3.87
- joint robotiq_arg2f_base_link_to_left_inner_knuckle: limit lower=0 upper=0.8757 effort=1000 velocity=2.0 -> lower=0 upper=0.82589 effort=21.03 velocity=3.87
- joint robotiq_arg2f_base_link_to_left_outer_knuckle: limit lower=0.0 upper=0.78 effort=1000 velocity=2.0 -> lower=0 upper=0.82589 effort=21.03 velocity=3.87
- joint robotiq_arg2f_base_link_to_right_inner_knuckle: limit lower=0 upper=0.8757 effort=1000 velocity=2.0 -> lower=0 upper=0.82589 effort=21.03 velocity=3.87

File: mara_description/urdf/mara_robot_gripper_85.urdf.xacro (robot description, xacro)
@@ -15,7 +15,7 @@
   <link name="gripper_adapter">
     <inertial>
-      <origin rpy="0 0 0" xyz="8.625E-08 -4.6583E-06 0.03145"/>
-      <mass value="0.13969"/>
-      <inertia ixx="91283.23E-9" ixy="634.87E-9" ixz="-0.02E-9" iyy="97239.94E-9" iyz="93.72E-9" izz="175963.64E-9"/>
+      <origin rpy="0 0 0" xyz="0 0 0.0173"/>
+      <mass value="0.14"/>
+      <inertia ixx="0.0001" ixy="0" ixz="0" iyy="0.0001" iyz="0" izz="0.0002"/>
     </inertial>
     <visual>
@@ -41,7 +41,7 @@
   <link name="robotiq_adapter_link">
     <inertial>
-      <origin xyz="8.625E-08 -4.6583E-06 0.03145" rpy="0 0 0" />
-      <mass value="0.22652" />
-      <inertia ixx="0.00020005" ixy="0" ixz="0" iyy="0.00017832" iyz="0" izz="0.00013478" />
+      <origin xyz="0 0 -0.0253" rpy="0 0 0" />
+      <mass value="0.317" />
+      <inertia ixx="298526E-9" ixy="3928E-9" ixz="-926E-9" iyy="354661E-9" iyz="42E-9" izz="415572E-9" />
     </inertial>
     <visual>

File: mara_description/urdf/mara_robot_gripper_hande.urdf (robot description, URDF)
Before this commit: robot mara, 20 links, 19 joints
Links:
- link gripper_adapter: mass 0.13969 -> 0.14
- link robotiq_adapter_link: mass 0.22652 -> 0.317

File: mara_description/urdf/mara_robot_gripper_hande.urdf.xacro (robot description, xacro)
@@ -15,7 +15,7 @@
   <link name="gripper_adapter">
     <inertial>
-      <origin rpy="0 0 0" xyz="8.625E-08 -4.6583E-06 0.03145"/>
-      <mass value="0.13969"/>
-      <inertia ixx="91283.23E-9" ixy="634.87E-9" ixz="-0.02E-9" iyy="97239.94E-9" iyz="93.72E-9" izz="175963.64E-9"/>
+      <origin rpy="0 0 0" xyz="0 0 0.0173"/>
+      <mass value="0.14"/>
+      <inertia ixx="0.0001" ixy="0" ixz="0" iyy="0.0001" iyz="0" izz="0.0002"/>
     </inertial>
     <visual>
@@ -41,7 +41,7 @@
   <link name="robotiq_adapter_link">
     <inertial>
-      <origin xyz="8.625E-08 -4.6583E-06 0.03145" rpy="0 0 0" />
-      <mass value="0.22652" />
-      <inertia ixx="0.00020005" ixy="0" ixz="0" iyy="0.00017832" iyz="0" izz="0.00013478" />
+      <origin xyz="0 0 -0.0253" rpy="0 0 0" />
+      <mass value="0.317" />
+      <inertia ixx="298526E-9" ixy="3928E-9" ixz="-926E-9" iyy="354661E-9" iyz="42E-9" izz="415572E-9" />
     </inertial>
     <visual>

File: mara_description/urdf/reinforcement_learning/mara_robot_gripper_140_camera_run.urdf (robot description, URDF)
Before this commit: robot mara, 30 links, 29 joints
Links:
- link gripper_adapter: mass 0.13969 -> 0.14
- link left_inner_finger: mass 0.0104003125914103 -> 0.045
- link left_inner_knuckle: mass 0.0271177346495152 -> 0.04476; geometry collision mesh filename=package://robotiq_140_gripper_description/meshes/robotiq_14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 scale=0.001 0.001 0.001; visual mesh filename=package://robotiq_140_gripper_description/meshes/robotiq_14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 scale=0.001 0.001 0.001
- link left_outer_finger: mass 0.022614240507152 -> 0.07637
- link left_outer_knuckle: mass 0.00853198276973456 -> 0.0131
- link right_inner_finger: mass 0.0104003125914103 -> 0.045
- link right_inner_knuckle: mass 0.0271177346495152 -> 0.04476; geometry collision mesh filename=package://robotiq_140_gripper_description/meshes/robotiq_14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 scale=0.001 0.001 0.001; visual mesh filename=package://robotiq_140_gripper_description/meshes/robotiq_14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 scale=0.001 0.001 0.001
- link right_outer_finger: mass 0.022614240507152 -> 0.07637
- link right_outer_knuckle: mass 0.00853198276973456 -> 0.0131
- link robotiq_adapter_link: mass 0.22652 -> 0.317
- link robotiq_arg2f_base_link: mass 0.22652 -> 0.52954
Joints:
- joint joint_finger: limit lower=0 upper=0.78574722925 effort=1000 velocity=2.0 -> lower=0 upper=0.78574722925 effort=18.65 velocity=3.54
- joint left_outer_finger_to_inner: limit lower=0 upper=0.78574722925 effort=1000 velocity=2.0 -> lower=0 upper=0.78574722925 effort=18.65 velocity=3.54
- joint right_outer_finger_to_inner: limit lower=0 upper=0.78574722925 effort=1000 velocity=2.0 -> lower=0 upper=0.78574722925 effort=18.65 velocity=3.54
- joint robotiq_arg2f_base_to_left_inner_knuckle: limit lower=0 upper=0.78574722925 effort=1000 velocity=2.0 -> lower=0 upper=0.78574722925 effort=18.65 velocity=3.54
- joint robotiq_arg2f_base_to_left_outer_knuckle: limit lower=0 upper=0.78574722925 effort=1000 velocity=2.0 -> lower=0 upper=0.78574722925 effort=18.65 velocity=2.0
- joint robotiq_arg2f_base_to_right_inner_knuckle: limit lower=0 upper=0.78574722925 effort=1000 velocity=2.0 -> lower=0 upper=0.78574722925 effort=18.65 velocity=3.54

File: mara_description/urdf/reinforcement_learning/mara_robot_gripper_140_camera_run.urdf.xacro (robot description, xacro)
@@ -43,7 +43,7 @@
   <link name="robotiq_adapter_link">
     <inertial>
-      <origin xyz="8.625E-08 -4.6583E-06 0.03145" rpy="0 0 0" />
-      <mass value="0.22652" />
-      <inertia ixx="0.00020005" ixy="0" ixz="0" iyy="0.00017832" iyz="0" izz="0.00013478" />
+      <origin xyz="0 0 -0.0253" rpy="0 0 0" />
+      <mass value="0.317" />
+      <inertia ixx="298526E-9" ixy="3928E-9" ixz="-926E-9" iyy="354661E-9" iyz="42E-9" izz="415572E-9" />
     </inertial>
     <visual>

File: mara_description/urdf/reinforcement_learning/mara_robot_gripper_140_camera_train.urdf (robot description, URDF)
Before this commit: robot mara, 30 links, 29 joints
Links:
- link gripper_adapter: mass 0.13969 -> 0.14
- link left_inner_finger: mass 0.0104003125914103 -> 0.045
- link left_inner_knuckle: mass 0.0271177346495152 -> 0.04476; geometry collision mesh filename=package://robotiq_140_gripper_description/meshes/robotiq_14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 scale=0.001 0.001 0.001; visual mesh filename=package://robotiq_140_gripper_description/meshes/robotiq_14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 scale=0.001 0.001 0.001
- link left_outer_finger: mass 0.022614240507152 -> 0.07637
- link left_outer_knuckle: mass 0.00853198276973456 -> 0.0131
- link right_inner_finger: mass 0.0104003125914103 -> 0.045
- link right_inner_knuckle: mass 0.0271177346495152 -> 0.04476; geometry collision mesh filename=package://robotiq_140_gripper_description/meshes/robotiq_14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 scale=0.001 0.001 0.001; visual mesh filename=package://robotiq_140_gripper_description/meshes/robotiq_14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 scale=0.001 0.001 0.001
- link right_outer_finger: mass 0.022614240507152 -> 0.07637
- link right_outer_knuckle: mass 0.00853198276973456 -> 0.0131
- link robotiq_adapter_link: mass 0.22652 -> 0.317
- link robotiq_arg2f_base_link: mass 0.22652 -> 0.52954
Joints:
- joint joint_finger: limit lower=0 upper=0.78574722925 effort=1000 velocity=2.0 -> lower=0 upper=0.78574722925 effort=18.65 velocity=3.54
- joint left_outer_finger_to_inner: limit lower=0 upper=0.78574722925 effort=1000 velocity=2.0 -> lower=0 upper=0.78574722925 effort=18.65 velocity=3.54
- joint right_outer_finger_to_inner: limit lower=0 upper=0.78574722925 effort=1000 velocity=2.0 -> lower=0 upper=0.78574722925 effort=18.65 velocity=3.54
- joint robotiq_arg2f_base_to_left_inner_knuckle: limit lower=0 upper=0.78574722925 effort=1000 velocity=2.0 -> lower=0 upper=0.78574722925 effort=18.65 velocity=3.54
- joint robotiq_arg2f_base_to_left_outer_knuckle: limit lower=0 upper=0.78574722925 effort=1000 velocity=2.0 -> lower=0 upper=0.78574722925 effort=18.65 velocity=2.0
- joint robotiq_arg2f_base_to_right_inner_knuckle: limit lower=0 upper=0.78574722925 effort=1000 velocity=2.0 -> lower=0 upper=0.78574722925 effort=18.65 velocity=3.54

File: mara_description/urdf/reinforcement_learning/mara_robot_gripper_140_camera_train.urdf.xacro (robot description, xacro)
@@ -43,7 +43,7 @@
   <link name="robotiq_adapter_link">
     <inertial>
-      <origin xyz="8.625E-08 -4.6583E-06 0.03145" rpy="0 0 0" />
-      <mass value="0.22652" />
-      <inertia ixx="0.00020005" ixy="0" ixz="0" iyy="0.00017832" iyz="0" izz="0.00013478" />
+      <origin xyz="0 0 -0.0253" rpy="0 0 0" />
+      <mass value="0.317" />
+      <inertia ixx="298526E-9" ixy="3928E-9" ixz="-926E-9" iyy="354661E-9" iyz="42E-9" izz="415572E-9" />
     </inertial>
     <visual>

Commit message: stuff for AI demo

File: mara_description/urdf/camera_gripper_support.urdf.xacro (robot description, xacro)
@@ -11,5 +11,5 @@
         <origin rpy="0 0 0" xyz="0 0 0"/>
         <geometry>
-          <mesh filename="package://mara_description/meshes/ROBOTIQ_Gripper_Adapter.dae" scale="0.001 0.001 0.001"/>
+          <mesh filename="package://mara_description/meshes/gripper_adapter.dae" scale="0.001 0.001 0.001"/>
         </geometry>
         <material name="Gazebo/Wood">
@@ -20,5 +20,5 @@
         <origin rpy="0 0 0" xyz="0 0 0"/>
         <geometry>
-          <mesh filename="package://mara_description/meshes/ROBOTIQ_Gripper_Adapter.dae" scale="0.001 0.001 0.001"/>
+          <mesh filename="package://mara_description/meshes/gripper_adapter.dae" scale="0.001 0.001 0.001"/>
         </geometry>
       </collision>
@@ -81,10 +81,10 @@
     </gazebo>
     <joint name="${prefix}gripper_adapter_to_camera_support1" type="fixed">
-      <origin rpy="0 0 0" xyz="0 0.03956 -0.0213"/>
+      <origin rpy="0 0 0" xyz="0 0.03956 -0.00213"/>
       <parent link="${prefix}mara_gripper_adapter"/>
       <child link="${prefix}mara_camera_support1_link"/>
     </joint>
     <joint name="${prefix}camera_support1_to_support2" type="fixed">
-      <origin rpy="0 0 0" xyz="0 0.01029 -0.0128"/>
+      <origin rpy="0 0 0" xyz="0 0.01029 -0.00128"/>
       <parent link="${prefix}mara_camera_support1_link"/>
       <child link="${prefix}mara_camera_support2_link"/>

File: mara_description/urdf/mara.urdf.xacro (robot description, xacro)
@@ -269,28 +269,21 @@
     <link name="${prefix}motor6_link">
       <inertial>
-        <origin rpy="0 0 0" xyz="0.0 0.0 -0.0173"/>
-        <mass value="0.14"/>
-        <inertia ixx="9.22e-05" ixy="6.35e-7" ixz="2.00e-11" iyy="9.73e-5" iyz="2.36e-9" izz="1.77e-4"/>
-      </inertial>
-      <visual>
-        <origin rpy="0 0 0" xyz="0 0 0"/>
-        <geometry>
-          <mesh filename="package://mara_description/meshes/MARA_GripperAdapter.dae" scale="0.001 0.001 0.001"/>
-        </geometry>
-        <material name="Gazebo/Black">
-          <color rgba="0. 0. 0. 1"/>
-        </material>
-      </visual>
-      <collision>
-        <origin rpy="0 0 0" xyz="0 0 0"/>
-        <geometry>
-          <mesh filename="package://mara_description/meshes/MARA_GripperAdapter.dae" scale="0.001 0.001 0.001"/>
-        </geometry>
-      </collision>
-    </link>
-    <gazebo reference="${prefix}motor6_link">
-      <material>Gazebo/Black</material>
-      <selfCollide>True</selfCollide>
-    </gazebo>
+        <origin rpy="0 0 0" xyz="0 0 0"/>
+        <mass value="0.00001"/>
+        <inertia ixx="0" ixy="0" ixz="0" iyy="0" iyz="0" izz="0"/>
+      </inertial>
+      <visual>
+        <origin rpy="0 0 0" xyz="0 0 0"/>
+        <geometry>
+          <sphere radius="0"/>
+        </geometry>
+      </visual>
+      <collision>
+        <origin rpy="0 0 0" xyz="0 0 0"/>
+        <geometry>
+          <sphere radius="0"/>
+        </geometry>
+      </collision>
+    </link>
     <link name="${prefix}ee_link">
     </link>

File: mara_description/urdf/mara_robot_camera.urdf (robot description, URDF)
Before this commit: robot mara, 14 links, 13 joints
Links:
- added link camera_color
- added link camera_ir_projector
- added link camera_left_depth
- added link camera_link, mass 0.07397; collision mesh filename=package://mara_description/meshes/Intel_RealSense_Depth_Cam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 scale=0.001 0.001 0.001; visual mesh filename=package://mara_description/meshes/Intel_RealSense_Depth_Cam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 scale=0.001 0.001 0.001
- added link camera_right_depth
- added link mara_camera_support1_link, mass 0.00361; collision mesh filename=package://mara_description/meshes/Camera_Support_1.dae scale=0.001 0.001 0.001; visual mesh filename=package://mara_description/meshes/Camera_Support_1.dae scale=0.001 0.001 0.001
- added link mara_camera_support2_link, mass 0.00676; collision mesh filename=package://mara_description/meshes/Camera_Support_2.dae scale=0.001 0.001 0.001; visual mesh filename=package://mara_description/meshes/Camera_Support_2.dae scale=0.001 0.001 0.001
- added link mara_gripper_adapter, mass 0.13969; collision mesh filename=package://mara_description/meshes/gripper_adapter.dae scale=0.001 0.001 0.001; visual mesh filename=package://mara_description/meshes/gripper_adapter.dae scale=0.001 0.001 0.001
Joints:
- added joint camera_support1_to_support2: type fixed, parent mara_camera_support1_link, child mara_camera_support2_link, origin xyz=0 0.01029 -0.00128 rpy=0 0 0
- added joint camera_support2_to_camera: type fixed, parent mara_camera_support2_link, child camera_link, origin xyz=0 0.018 0.012 rpy=0 0 0
- added joint camera_to_color: type fixed, parent camera_link, child camera_color, origin xyz=-0.0325 0.0214 0.0 rpy=0.0 0.0 1.57
- added joint camera_to_ir_projector: type fixed, parent camera_link, child camera_ir_projector, origin xyz=0.0115 0.0214 0.0 rpy=0 0 0
- added joint camera_to_left_depth: type fixed, parent camera_link, child camera_left_depth, origin xyz=-0.0175 0.024 0.0 rpy=0 0 0
- added joint camera_to_right_depth: type fixed, parent camera_link, child camera_right_depth, origin xyz=0.0325 0.024 0.0 rpy=0 0 0
- added joint gripper_adapter_to_camera_support1: type fixed, parent mara_gripper_adapter, child mara_camera_support1_link, origin xyz=0 0.03956 -0.00213 rpy=0 0 0
- added joint motor6_to_gripper_adapter: type fixed, parent motor6_link, child mara_gripper_adapter, origin xyz=0 0 -0.02026 rpy=0 0 0
- joint ee_link: origin xyz=0 0.0 0.24 rpy=0 -1.57 0 -> xyz=0 0.0 0.0 rpy=0 -1.57 0
