Commit message: Fixing joint type

File: mara_description/urdf/mara_robot_gripper_hande.urdf (robot description, URDF)
Before this commit: robot mara, 18 links, 17 joints
Joints:
- joint finger1_joint: axis (none) -> 0 0 -1; limit (none) -> lower=0 upper=0.024858 effort=1000 velocity=2.0; type fixed -> prismatic
- joint finger2_joint: axis (none) -> 0 0 1; limit (none) -> lower=0 upper=0.024858 effort=1000 velocity=2.0; type fixed -> prismatic

Commit message: updating hande URDF

File: mara_description/urdf/mara_robot_gripper_hande.urdf (robot description, URDF)
Before this commit: robot mara, 18 links, 17 joints
Links:
- link table: geometry collision box size=1.5 1 0.05; visual mesh filename=package://mara_description/urdf/table.obj scale=0.1 0.1 0.58
Joints:
- removed joint finger1_joint
- added joint joint_finger: type prismatic, parent robotiq_hande_base_link, child finger1, origin xyz=0 0 0.0 rpy=0 0 0, axis 0 0 -1, limit lower=0 upper=0.024858 effort=1000 velocity=2.0
- joint finger2_joint: mimic (none) -> joint=joint_finger multiplier=1 offset=0

Commit message: update adapters in hande gripper

File: mara_description/urdf/mara_robot_gripper_hande.urdf (robot description, URDF)
Before this commit: robot mara, 19 links, 18 joints
Links:
- removed link finger1
- removed link finger2
- added link gripper_adapter, mass 0.13969; collision mesh filename=package://mara_description/meshes/gripper_adapter.dae scale=0.001 0.001 0.001; visual mesh filename=package://mara_description/meshes/gripper_adapter.dae scale=0.001 0.001 0.001
- added link left_finger, mass 0.03804; collision mesh filename=package://robotiq_hande_gripper_description/meshes/finger_1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 scale=0.001 0.001 0.001; visual mesh filename=package://robotiq_hande_gripper_description/meshes/finger_1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 scale=0.001 0.001 0.001
- added link right_finger, mass 0.03804; collision mesh filename=package://robotiq_hande_gripper_description/meshes/finger_2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 scale=0.001 0.001 0.001; visual mesh filename=package://robotiq_hande_gripper_description/meshes/finger_2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 scale=0.001 0.001 0.001
- link motor6_link: mass 0.14 -> 0.00001; geometry collision sphere radius=0; visual sphere radius=0
- link robotiq_adapter_link: geometry collision mesh filename=package://mara_description/meshes/robotiq_adapter.dae scale=0.001 0.001 0.001; visual mesh filename=package://mara_description/meshes/robotiq_adapter.dae scale=0.001 0.001 0.001
- link robotiq_hande_base_link: mass 0.22652 -> 0.86387
Joints:
- removed joint base_adapter_to_base_robotiq_joint
- removed joint end_effector_adapter_to_robotiq
- removed joint finger2_joint
- added joint gripper_adapter_to_robotiq_adapter: type fixed, parent gripper_adapter, child robotiq_adapter_link, origin xyz= 0 0 0.0 rpy=0 0 0
- added joint motor6_to_gripper_adapter: type fixed, parent motor6_link, child gripper_adapter, origin xyz= 0 0 0.0 rpy=0 0 0
- added joint robotiq_adapter_to_hande_base: type fixed, parent robotiq_adapter_link, child robotiq_hande_base_link, origin xyz= 0 0 0 rpy=0 0 0
- added joint robotiq_hande_base_to_right_finger: type prismatic, parent robotiq_hande_base_link, child right_finger, origin xyz=0 0 0.099 rpy=0 0 0, axis 1 0 0, limit lower=0 upper=0.025 effort=130 velocity=0.15, mimic joint=joint_finger multiplier=1 offset=0
- joint ee_link: origin xyz=0 0.0 0.18 rpy=0 -1.57 0 -> xyz=0 0.0 0.18253 rpy=0 -1.57 0
- joint joint_finger: axis 0 0 -1 -> -1 0 0; child finger1 -> left_finger; limit lower=0 upper=0.024858 effort=1000 velocity=2.0 -> lower=0 upper=0.025 effort=130 velocity=0.15; origin xyz=0 0 0.0 rpy=0 0 0 -> xyz=0 0 0.099 rpy=0 0 0
- joint motor6_link-tool0_fixed_joint: origin xyz=0 0.0 0.18 rpy=0 -1.57 0 -> xyz=0 0.0 0.18253 rpy=0 -1.57 0

Commit message: fix hande adapters joint origin values

File: mara_description/urdf/mara_robot_gripper_hande.urdf (robot description, URDF)
Before this commit: robot mara, 20 links, 19 joints
Joints:
- joint gripper_adapter_to_robotiq_adapter: origin xyz= 0 0 0.0 rpy=0 0 0 -> xyz= 0 0 0.05679 rpy=0 0 0
- joint motor6_to_gripper_adapter: origin xyz= 0 0 0.0 rpy=0 0 0 -> xyz= 0 0 -0.02026 rpy=0 0 0

File: mara_description/urdf/mara_robot_gripper_hande.urdf.xacro (robot description, xacro)
@@ -76,10 +76,10 @@
   </joint>
   <joint name="motor6_to_gripper_adapter" type="fixed">
-    <origin rpy="0 0 0" xyz=" 0 0 0.0"/>
+    <origin rpy="0 0 0" xyz=" 0 0 -0.02026"/>
     <parent link="motor6_link"/>
     <child link="gripper_adapter"/>
   </joint>
   <joint name="gripper_adapter_to_robotiq_adapter" type="fixed">
-    <origin rpy="0 0 0" xyz=" 0 0 0.0"/>
+    <origin rpy="0 0 0" xyz=" 0 0 0.05679"/>
     <parent link="gripper_adapter"/>
     <child link="robotiq_adapter_link"/>
