Commit message: updating MARA gripper 85 URDF

File: mara_description/urdf/mara_robot_gripper_85.urdf (robot description, URDF)
Before this commit: robot mara, 24 links, 23 joints
Links:
- removed link robotiq_85_base_link
- removed link robotiq_85_left_finger_link
- removed link robotiq_85_left_inner_finger_link
- removed link robotiq_85_left_inner_knuckle_link
- removed link robotiq_85_left_outer_knuckle_link
- removed link robotiq_85_right_finger_link
- removed link robotiq_85_right_inner_finger_link
- removed link robotiq_85_right_inner_knuckle_link
- removed link robotiq_85_right_outer_knuckle_link
- added link left_inner_finger, mass 0.22652; collision mesh filename=package://robotiq_85_gripper_description/meshes/2-F-85_4_l.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 scale=0.001 0.001 0.001; visual mesh filename=package://robotiq_85_gripper_description/meshes/2-F-85_4_l.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 scale=0.001 0.001 0.001
- added link left_inner_knuckle, mass 0.22652; collision mesh filename=package://robotiq_85_gripper_description/meshes/2-F-85_2_l.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 scale=0.001 0.001 0.001; visual mesh filename=package://robotiq_85_gripper_description/meshes/2-F-85_2_l.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 scale=0.001 0.001 0.001
- added link left_outer_finger, mass 0.22652; collision mesh filename=package://robotiq_85_gripper_description/meshes/2-F-85_3_l.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 scale=0.001 0.001 0.001; visual mesh filename=package://robotiq_85_gripper_description/meshes/2-F-85_3_l.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 scale=0.001 0.001 0.001
- added link left_outer_knuckle, mass 0.22652; collision mesh filename=package://robotiq_85_gripper_description/meshes/2-F-85_1_l.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 scale=0.001 0.001 0.001; visual mesh filename=package://robotiq_85_gripper_description/meshes/2-F-85_1_l.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 scale=0.001 0.001 0.001
- added link right_inner_finger, mass 0.22652; collision mesh filename=package://robotiq_85_gripper_description/meshes/2-F-85_4_r.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 scale=0.001 0.001 0.001; visual mesh filename=package://robotiq_85_gripper_description/meshes/2-F-85_4_r.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 scale=0.001 0.001 0.001
- added link right_inner_knuckle, mass 0.22652; collision mesh filename=package://robotiq_85_gripper_description/meshes/2-F-85_2_r.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 scale=0.001 0.001 0.001; visual mesh filename=package://robotiq_85_gripper_description/meshes/2-F-85_2_r.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 scale=0.001 0.001 0.001
- added link right_outer_finger, mass 0.22652; collision mesh filename=package://robotiq_85_gripper_description/meshes/2-F-85_3_r.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 scale=0.001 0.001 0.001; visual mesh filename=package://robotiq_85_gripper_description/meshes/2-F-85_3_r.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 scale=0.001 0.001 0.001
- added link right_outer_knuckle, mass 0.22652; collision mesh filename=package://robotiq_85_gripper_description/meshes/2-F-85_1_r.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 scale=0.001 0.001 0.001; visual mesh filename=package://robotiq_85_gripper_description/meshes/2-F-85_1_r.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 scale=0.001 0.001 0.001
- added link robotiq_arg2f_base, mass 0.22652; collision mesh filename=package://robotiq_85_gripper_description/meshes/base_grippe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 scale=0.001 0.001 0.001; visual mesh filename=package://robotiq_85_gripper_description/meshes/base_grippe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 scale=0.001 0.001 0.001
- link table: geometry collision box size=1.5 1 0.05; visual mesh filename=package://mara_description/urdf/table.obj scale=0.1 0.1 0.58
Joints:
- removed joint left_finger_joint
- removed joint right_finger_joint
- removed joint right_outer_knuckle_joint
- added joint joint_finger: type revolute, parent robotiq_arg2f_base, child right_outer_knuckle, origin xyz=0.0306 0 0.05490 rpy=0 0 3.1416, axis 0 1 0, limit lower=0 upper=0.78 effort=1000 velocity=2.0
- added joint left_outer_finger_joint: type fixed, parent left_outer_knuckle, child left_outer_finger, origin xyz=-0.03156 0 -0.003758 rpy=0 0 0
- added joint right_outer_finger_joint: type fixed, parent right_outer_knuckle, child right_outer_finger, origin xyz=-0.03156 0 -0.003758 rpy=0 0 0
- joint end_effector_adapter_to_robotiq: child robotiq_85_base_link -> robotiq_arg2f_base
- joint left_inner_finger_joint: axis 0 1 0 -> 0 -1 0; child robotiq_85_left_inner_finger_link -> left_inner_finger; limit lower=0 upper=0.8757 effort=1000 velocity=2.0 -> lower=0 upper=0.775 effort=1000 velocity=2.0; mimic (none) -> joint=joint_finger multiplier=1 offset=0; origin xyz=-0.0127 0 0.06142 rpy=0 0 0 -> xyz=-0.005625 0 0.04718 rpy=0 0.0 0; parent robotiq_85_base_link -> left_outer_finger
- joint left_inner_knuckle_joint: child robotiq_85_left_inner_knuckle_link -> left_inner_knuckle; limit lower=0.0 upper=0.794 effort=1000 velocity=2.0 -> lower=0 upper=0.8757 effort=1000 velocity=2.0; mimic (none) -> joint=joint_finger multiplier=1 offset=0; origin xyz=-0.0306 0 0.05490 rpy=0 0 0 -> xyz=-0.0127 0 0.06142 rpy=0 0 0; parent robotiq_85_base_link -> robotiq_arg2f_base
- joint left_outer_knuckle_joint: axis 0 -1 0 -> 0 1 0; child robotiq_85_left_outer_knuckle_link -> left_outer_knuckle; limit lower=0 upper=0.8757 effort=1000 velocity=2.0 -> lower=0.0 upper=0.78 effort=1000 velocity=2.0; mimic (none) -> joint=joint_finger multiplier=1 offset=0; origin xyz=-0.03156 0 -0.003758 rpy=0 0 0 -> xyz=-0.0306 0 0.05490 rpy=0 0 0; parent robotiq_85_left_inner_knuckle_link -> robotiq_arg2f_base
- joint right_inner_finger_joint: axis 0 1 0 -> 0 -1 0; child robotiq_85_right_inner_finger_link -> right_inner_finger; limit lower=0 upper=0.8757 effort=1000 velocity=2.0 -> lower=0 upper=0.775 effort=1000 velocity=2.0; mimic (none) -> joint=joint_finger multiplier=1 offset=0; origin xyz=0.0127 0 0.06142 rpy=0 0 3.1416 -> xyz=-0.005625 0 0.04718 rpy=0 0 0; parent robotiq_85_base_link -> right_outer_finger
- joint right_inner_knuckle_joint: child robotiq_85_right_inner_knuckle_link -> right_inner_knuckle; limit lower=0 upper=0.794 effort=1000 velocity=2.0 -> lower=0 upper=0.8757 effort=1000 velocity=2.0; mimic (none) -> joint=joint_finger multiplier=1 offset=0; origin xyz=0.0306 0 0.05490 rpy=0 0 3.1416 -> xyz=0.0127 0 0.06142 rpy=0 0 3.1416; parent robotiq_85_base_link -> robotiq_arg2f_base

File: mara_description/urdf/mara_robot_gripper_85.urdf.xacro (robot description, xacro)
@@ -17,5 +17,5 @@
     <origin rpy="0 0 0" xyz=" 0 0 0.03653"/>
     <parent link="motor6_link"/>
-    <child link="robotiq_85_base_link"/>
+    <child link="robotiq_arg2f_base"/>
   </joint>
   <joint name="world_to_table_joint" type="fixed">

Commit message: update adapters in mara_robot_gripper_85.urdf

File: mara_description/urdf/mara_robot_gripper_85.urdf (robot description, URDF)
Before this commit: robot mara, 25 links, 24 joints
Links:
- removed link robotiq_arg2f_base
- added link gripper_adapter, mass 0.13969; collision mesh filename=package://mara_description/meshes/gripper_adapter.dae scale=0.001 0.001 0.001; visual mesh filename=package://mara_description/meshes/gripper_adapter.dae scale=0.001 0.001 0.001
- added link robotiq_arg2f_base_link, mass 0.22652; collision mesh filename=package://robotiq_85_gripper_description/meshes/base_grippe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 scale=0.001 0.001 0.001; visual mesh filename=package://robotiq_85_gripper_description/meshes/base_grippe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 scale=0.001 0.001 0.001
- link motor6_link: mass 0.14 -> 0.00001; geometry collision sphere radius=0; visual sphere radius=0
- link robotiq_adapter_link: geometry collision mesh filename=package://mara_description/meshes/robotiq_adapter.dae scale=0.001 0.001 0.001; visual mesh filename=package://mara_description/meshes/robotiq_adapter.dae scale=0.001 0.001 0.001
Joints:
- removed joint base_adapter_to_base_robotiq_joint
- removed joint end_effector_adapter_to_robotiq
- removed joint left_inner_finger_joint
- removed joint left_inner_knuckle_joint
- removed joint left_outer_finger_joint
- removed joint left_outer_knuckle_joint
- removed joint right_inner_finger_joint
- removed joint right_inner_knuckle_joint
- removed joint right_outer_finger_joint
- removed joint table_to_base_joint
- removed joint world_to_table_joint
- added joint gripper_adapter_to_robotiq_adapter: type fixed, parent gripper_adapter, child robotiq_adapter_link, origin xyz= 0 0 0.05679 rpy=0 0 0
- added joint left_outer_finger_to_inner: type revolute, parent left_outer_finger, child left_inner_finger, origin xyz=0.00678 0 0.04703 rpy=0 0 0, axis 0 1 0, limit lower=0 upper=0.775 effort=1000 velocity=2.0, mimic joint=joint_finger multiplier=1 offset=0
- added joint left_outer_knuckle_to_finger: type fixed, parent left_outer_knuckle, child left_outer_finger, origin xyz=0.03142 0 -0.00453 rpy=0 0 0
- added joint motor6_to_gripper_adapter: type fixed, parent motor6_link, child gripper_adapter, origin xyz= 0 0 -0.02026 rpy=0 0 0
- added joint right_outer_finger_to_inner: type revolute, parent right_outer_finger, child right_inner_finger, origin xyz=-0.00678 0 0.04703 rpy=0 0 0, axis 0 -1 0, limit lower=0 upper=0.775 effort=1000 velocity=2.0, mimic joint=joint_finger multiplier=1 offset=0
- added joint right_outer_knuckle_to_finger: type fixed, parent right_outer_knuckle, child right_outer_finger, origin xyz=-0.03142 0 -0.00453 rpy=0 0 0
- added joint robotiq_adapter_to_arg2f_base: type fixed, parent robotiq_adapter_link, child robotiq_arg2f_base_link, origin xyz= 0 0 0 rpy=0 0 0
- added joint robotiq_arg2f_base_link_to_left_inner_knuckle: type revolute, parent robotiq_arg2f_base_link, child left_inner_knuckle, origin xyz=0.0127 0 0.06118 rpy=0 0 0, axis 0 -1 0, limit lower=0 upper=0.8757 effort=1000 velocity=2.0, mimic joint=joint_finger multiplier=1 offset=0
- added joint robotiq_arg2f_base_link_to_left_outer_knuckle: type revolute, parent robotiq_arg2f_base_link, child left_outer_knuckle, origin xyz=0.0306 0 0.05466 rpy=0 0 0, axis 0 -1 0, limit lower=0.0 upper=0.78 effort=1000 velocity=2.0, mimic joint=joint_finger multiplier=1 offset=0
- added joint robotiq_arg2f_base_link_to_right_inner_knuckle: type revolute, parent robotiq_arg2f_base_link, child right_inner_knuckle, origin xyz=-0.0127 0 0.06118 rpy=0 0 0, axis 0 1 0, limit lower=0 upper=0.8757 effort=1000 velocity=2.0, mimic joint=joint_finger multiplier=1 offset=0
- added joint table_to_base: type fixed, parent table, child base_link, origin xyz=0 0 0.62 rpy=0 0 0
- added joint world_to_table: type fixed, parent world, child table, origin xyz=0 0 0 rpy=0 0 0
- joint ee_link: origin xyz=0 0.0 0.165 rpy=0 -1.57 0 -> xyz=0 0.0 0.18491 rpy=0 -1.57 0
- joint joint_finger: origin xyz=0.0306 0 0.05490 rpy=0 0 3.1416 -> xyz=-0.0306 0 0.05466 rpy=0 0 0; parent robotiq_arg2f_base -> robotiq_arg2f_base_link
- joint motor6_link-tool0_fixed_joint: origin xyz=0 0.0 0.165 rpy=0 -1.57 0 -> xyz=0 0.0 0.18491 rpy=0 -1.57 0

Commit message: regenerate mara_robot_gripper_85.urdf

File: mara_description/urdf/mara_robot_gripper_85.urdf (robot description, URDF)
Before this commit: robot mara, 26 links, 25 joints
Links:
- removed link left_inner_finger
- removed link left_inner_knuckle
- removed link left_outer_finger
- removed link left_outer_knuckle
- removed link right_inner_finger
- removed link right_inner_knuckle
- removed link right_outer_finger
- removed link right_outer_knuckle
- removed link robotiq_arg2f_base_link
- added link left_finger, mass 0.03804; collision mesh filename=package://robotiq_hande_gripper_description/meshes/finger_1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 scale=0.001 0.001 0.001; visual mesh filename=package://robotiq_hande_gripper_description/meshes/finger_1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 scale=0.001 0.001 0.001
- added link right_finger, mass 0.03804; collision mesh filename=package://robotiq_hande_gripper_description/meshes/finger_2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 scale=0.001 0.001 0.001; visual mesh filename=package://robotiq_hande_gripper_description/meshes/finger_2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 scale=0.001 0.001 0.001
- added link robotiq_hande_base_link, mass 0.86387; collision mesh filename=package://robotiq_hande_gripper_description/meshes/hand-e.d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 scale=0.001 0.001 0.001; visual mesh filename=package://robotiq_hande_gripper_description/meshes/hand-e.d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 scale=0.001 0.001 0.001
Joints:
- removed joint left_outer_finger_to_inner
- removed joint left_outer_knuckle_to_finger
- removed joint right_outer_finger_to_inner
- removed joint right_outer_knuckle_to_finger
- removed joint robotiq_adapter_to_arg2f_base
- removed joint robotiq_arg2f_base_link_to_left_inner_knuckle
- removed joint robotiq_arg2f_base_link_to_left_outer_knuckle
- removed joint robotiq_arg2f_base_link_to_right_inner_knuckle
- removed joint table_to_base
- removed joint world_to_table
- added joint robotiq_adapter_to_hande_base: type fixed, parent robotiq_adapter_link, child robotiq_hande_base_link, origin xyz= 0 0 0 rpy=0 0 0
- added joint robotiq_hande_base_to_right_finger: type prismatic, parent robotiq_hande_base_link, child right_finger, origin xyz=0 0 0.099 rpy=0 0 0, axis 1 0 0, limit lower=0 upper=0.025 effort=130 velocity=0.15, mimic joint=joint_finger multiplier=1 offset=0
- added joint table_to_base_joint: type fixed, parent table, child base_link, origin xyz=0 0 0.62 rpy=0 0 0
- added joint world_to_table_joint: type fixed, parent world, child table, origin xyz=0 0 0.02 rpy=0 0 0
- joint ee_link: origin xyz=0 0.0 0.18491 rpy=0 -1.57 0 -> xyz=0 0.0 0.18253 rpy=0 -1.57 0
- joint joint_finger: axis 0 1 0 -> -1 0 0; child right_outer_knuckle -> left_finger; limit lower=0 upper=0.82589 effort=21.03 velocity=3.87 -> lower=0 upper=0.025 effort=130 velocity=0.15; origin xyz=-0.0306 0 0.05466 rpy=0 0 0 -> xyz=0 0 0.099 rpy=0 0 0; parent robotiq_arg2f_base_link -> robotiq_hande_base_link; type revolute -> prismatic
- joint motor6_link-tool0_fixed_joint: origin xyz=0 0.0 0.18491 rpy=0 -1.57 0 -> xyz=0 0.0 0.18253 rpy=0 -1.57 0

Commit message: regenerate necessary urdfs to fix PID values

File: mara_description/urdf/mara_robot_gripper_85.urdf (robot description, URDF)
Before this commit: robot mara, 20 links, 19 joints
Links:
- removed link left_finger
- removed link right_finger
- removed link robotiq_hande_base_link
- added link left_inner_finger, mass 0.037; collision mesh filename=package://robotiq_85_gripper_description/meshes/2-F-85_4_l.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 scale=0.001 0.001 0.001; visual mesh filename=package://robotiq_85_gripper_description/meshes/2-F-85_4_l.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 scale=0.001 0.001 0.001
- added link left_inner_knuckle, mass 0.02731; collision mesh filename=package://robotiq_85_gripper_description/meshes/2-F-85_2_l.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 scale=0.001 0.001 0.001; visual mesh filename=package://robotiq_85_gripper_description/meshes/2-F-85_2_l.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 scale=0.001 0.001 0.001
- added link left_outer_finger, mass 0.03848; collision mesh filename=package://robotiq_85_gripper_description/meshes/2-F-85_3_l.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 scale=0.001 0.001 0.001; visual mesh filename=package://robotiq_85_gripper_description/meshes/2-F-85_3_l.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 scale=0.001 0.001 0.001
- added link left_outer_knuckle, mass 0.01252; collision mesh filename=package://robotiq_85_gripper_description/meshes/2-F-85_1_l.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 scale=0.001 0.001 0.001; visual mesh filename=package://robotiq_85_gripper_description/meshes/2-F-85_1_l.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 scale=0.001 0.001 0.001
- added link right_inner_finger, mass 0.037; collision mesh filename=package://robotiq_85_gripper_description/meshes/2-F-85_4_r.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 scale=0.001 0.001 0.001; visual mesh filename=package://robotiq_85_gripper_description/meshes/2-F-85_4_r.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 scale=0.001 0.001 0.001
- added link right_inner_knuckle, mass 0.02731; collision mesh filename=package://robotiq_85_gripper_description/meshes/2-F-85_2_r.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 scale=0.001 0.001 0.001; visual mesh filename=package://robotiq_85_gripper_description/meshes/2-F-85_2_r.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 scale=0.001 0.001 0.001
- added link right_outer_finger, mass 0.03848; collision mesh filename=package://robotiq_85_gripper_description/meshes/2-F-85_3_r.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 scale=0.001 0.001 0.001; visual mesh filename=package://robotiq_85_gripper_description/meshes/2-F-85_3_r.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 scale=0.001 0.001 0.001
- added link right_outer_knuckle, mass 0.01252; collision mesh filename=package://robotiq_85_gripper_description/meshes/2-F-85_1_r.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 scale=0.001 0.001 0.001; visual mesh filename=package://robotiq_85_gripper_description/meshes/2-F-85_1_r.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 scale=0.001 0.001 0.001
- added link robotiq_arg2f_base_link, mass 0.55938; collision mesh filename=package://robotiq_85_gripper_description/meshes/base_grippe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 scale=0.001 0.001 0.001; visual mesh filename=package://robotiq_85_gripper_description/meshes/base_grippe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 scale=0.001 0.001 0.001
Joints:
- removed joint robotiq_adapter_to_hande_base
- removed joint robotiq_hande_base_to_right_finger
- removed joint table_to_base_joint
- removed joint world_to_table_joint
- added joint left_outer_finger_to_inner: type revolute, parent left_outer_finger, child left_inner_finger, origin xyz=0.00678 0 0.04703 rpy=0 0 0, axis 0 1 0, limit lower=0 upper=0.82589 effort=21.03 velocity=3.87, mimic joint=joint_finger multiplier=1 offset=0
- added joint left_outer_knuckle_to_finger: type fixed, parent left_outer_knuckle, child left_outer_finger, origin xyz=0.03142 0 -0.00453 rpy=0 0 0
- added joint right_outer_finger_to_inner: type revolute, parent right_outer_finger, child right_inner_finger, origin xyz=-0.00678 0 0.04703 rpy=0 0 0, axis 0 -1 0, limit lower=0 upper=0.82589 effort=21.03 velocity=3.87, mimic joint=joint_finger multiplier=1 offset=0
- added joint right_outer_knuckle_to_finger: type fixed, parent right_outer_knuckle, child right_outer_finger, origin xyz=-0.03142 0 -0.00453 rpy=0 0 0
- added joint robotiq_adapter_to_arg2f_base: type fixed, parent robotiq_adapter_link, child robotiq_arg2f_base_link, origin xyz= 0 0 0 rpy=0 0 0
- added joint robotiq_arg2f_base_link_to_left_inner_knuckle: type revolute, parent robotiq_arg2f_base_link, child left_inner_knuckle, origin xyz=0.0127 0 0.06118 rpy=0 0 0, axis 0 -1 0, limit lower=0 upper=0.82589 effort=21.03 velocity=3.87, mimic joint=joint_finger multiplier=1 offset=0
- added joint robotiq_arg2f_base_link_to_left_outer_knuckle: type revolute, parent robotiq_arg2f_base_link, child left_outer_knuckle, origin xyz=0.0306 0 0.05466 rpy=0 0 0, axis 0 -1 0, limit lower=0 upper=0.82589 effort=21.03 velocity=3.87, mimic joint=joint_finger multiplier=1 offset=0
- added joint robotiq_arg2f_base_link_to_right_inner_knuckle: type revolute, parent robotiq_arg2f_base_link, child right_inner_knuckle, origin xyz=-0.0127 0 0.06118 rpy=0 0 0, axis 0 1 0, limit lower=0 upper=0.82589 effort=21.03 velocity=3.87, mimic joint=joint_finger multiplier=1 offset=0
- added joint table_to_base: type fixed, parent table, child base_link, origin xyz=0 0 0.62 rpy=0 0 0
- added joint world_to_table: type fixed, parent world, child table, origin xyz=0 0 0 rpy=0 0 0
- joint ee_link: origin xyz=0 0.0 0.18253 rpy=0 -1.57 0 -> xyz=0 0.0 0.18491 rpy=0 -1.57 0
- joint joint_finger: axis -1 0 0 -> 0 1 0; child left_finger -> right_outer_knuckle; limit lower=0 upper=0.025 effort=130 velocity=0.15 -> lower=0 upper=0.82589 effort=21.03 velocity=3.87; origin xyz=0 0 0.099 rpy=0 0 0 -> xyz=-0.0306 0 0.05466 rpy=0 0 0; parent robotiq_hande_base_link -> robotiq_arg2f_base_link; type prismatic -> revolute
- joint motor6_link-tool0_fixed_joint: origin xyz=0 0.0 0.18253 rpy=0 -1.57 0 -> xyz=0 0.0 0.18491 rpy=0 -1.57 0
