Commit message: Updating mara description

File: mara_description/urdf/mara.urdf.xacro (robot description, xacro)
@@ -5,5 +5,5 @@
 -->
   <xacro:include filename="$(find mara_description)/urdf/mara.transmission.xacro" />
-  <xacro:include filename="$(find mara_description)/urdf/mara.gazebo.xacro" />
+  <xacro:include filename="$(find mara_description)/urdf/mara_gazebo.urdf.xacro" />
   <xacro:macro name="mara_robot"  params="prefix joint_limited">
     <link name="${prefix}base_link">

File: mara_description/urdf/mara_gazebo.urdf.xacro (robot description, xacro)
@@ -1,39 +1,34 @@
 <?xml version="1.0"?>
 <robot xmlns:xacro="http://ros.org/wiki/xacro">
-  <gazebo>
-    <plugin name="mara_joint_state" filename="libgazebo_ros_joint_state_publisher.so">
-  		<ros>
-  			<!-- <namespace>/mara</namespace> -->
-  			<argument>~/out:=joint_states</argument>
-  		</ros>
-  		<update_rate>250</update_rate>
-  		<joint_name>motor1</joint_name>
-  		<joint_name>motor2</joint_name>
-  		<joint_name>motor3</joint_name>
-  		<joint_name>motor4</joint_name>
-  		<joint_name>motor5</joint_name>
-      <joint_name>motor6</joint_name>
-  	</plugin>
-    <plugin name="hros_actuation_servomotor_000000000001" filename="libmara_gazebo_joint_plugin.so">
-      <ros>
-        <!-- <namespace>/tb3</namespace> -->
-      </ros>
-      <axis1>motor2</axis1>
-      <axis2>motor1</axis2>
-    </plugin>
-    <plugin name="hros_actuation_servomotor_000000000002" filename="libmara_gazebo_joint_plugin.so">
-      <ros>
-        <!-- <namespace>/tb3</namespace> -->
-      </ros>
-      <axis1>motor3</axis1>
-      <axis2>motor4</axis2>
-    </plugin>
-    <plugin name="hros_actuation_servomotor_000000000003" filename="libmara_gazebo_joint_plugin.so">
-      <ros>
-        <!-- <namespace>/tb3</namespace> -->
-      </ros>
-      <axis1>motor5</axis1>
-      <axis2>motor6</axis2>
-    </plugin>
-  </gazebo>
+  <xacro:macro name="mara_gazebo" params="prefix">
+    <gazebo>
+      <plugin name="mara_joint_state" filename="libgazebo_ros_joint_state_publisher.so">
+    		<ros>
+    			<argument>~/out:=joint_states</argument>
+    		</ros>
+    		<update_rate>250</update_rate>
+    		<joint_name>motor1</joint_name>
+    		<joint_name>motor2</joint_name>
+    		<joint_name>motor3</joint_name>
+    		<joint_name>motor4</joint_name>
+    		<joint_name>motor5</joint_name>
+        <joint_name>motor6</joint_name>
+    	</plugin>
+      <plugin name="hros_actuation_servomotor_000000000001" filename="libmara_gazebo_joint_plugin.so">
+        <ros></ros>
+        <axis1>motor2</axis1>
+        <axis2>motor1</axis2>
+      </plugin>
+      <plugin name="hros_actuation_servomotor_000000000002" filename="libmara_gazebo_joint_plugin.so">
+        <ros></ros>
+        <axis1>motor3</axis1>
+        <axis2>motor4</axis2>
+      </plugin>
+      <plugin name="hros_actuation_servomotor_000000000003" filename="libmara_gazebo_joint_plugin.so">
+        <ros></ros>
+        <axis1>motor5</axis1>
+        <axis2>motor6</axis2>
+      </plugin>
+    </gazebo>
+  </xacro:macro>
 </robot>
