Commit message: updating MARA model

File: mara_description/urdf/mara.urdf.xacro (robot description, xacro)
@@ -16,5 +16,5 @@
         <origin rpy="0 0 0" xyz="0 0 0"/>
         <geometry>
-          <mesh filename="package://mara_description/meshes/H-ROS_Robot_BASE.stl" scale="0.001 0.001 0.001"/>
+          <mesh filename="package://mara_description/meshes/Base_plancha.stl" scale="0.001 0.001 0.001"/>
         </geometry>
         <material name="Gazebo/Grey">
@@ -25,5 +25,5 @@
         <origin rpy="0 0 0" xyz="0 0 0"/>
         <geometry>
-          <mesh filename="package://mara_description/meshes/H-ROS_Robot_BASE.stl" scale="0.001 0.001 0.001"/>
+          <mesh filename="package://mara_description/meshes/Base_plancha.stl" scale="0.001 0.001 0.001"/>
         </geometry>
       </collision>
@@ -33,14 +33,40 @@
       <selfCollide>True</selfCollide>
     </gazebo>
+    <link name="${prefix}base_robot">
+      <inertial>
+        <origin rpy="0 0 0" xyz="8.625E-08 -4.6583E-06 0.03145"/>
+        <mass value="7.033"/>
+        <inertia ixx="0.1478344" ixy="-0.00001" ixz="0.0" iyy="0.14782335" iyz="0.0" izz="0.29471799"/>
+      </inertial>
+      <visual>
+        <origin rpy="0 0 0" xyz="0 0 0"/>
+        <geometry>
+          <mesh filename="package://mara_description/meshes/Base.stl" scale="0.001 0.001 0.001"/>
+        </geometry>
+        <material name="Gazebo/Grey">
+          <color rgba="0. 0. 0. 1"/>
+        </material>
+      </visual>
+      <collision>
+        <origin rpy="0 0 0" xyz="0 0 0"/>
+        <geometry>
+          <mesh filename="package://mara_description/meshes/Base.stl" scale="0.001 0.001 0.001"/>
+        </geometry>
+      </collision>
+    </link>
+    <gazebo reference="${prefix}base_robot">
+      <material>Gazebo/Grey</material>
+      <selfCollide>True</selfCollide>
+    </gazebo>
     <link name="${prefix}motor1_link">
       <inertial>
         <origin rpy="0 0 0" xyz="8.625E-08 -4.6583E-06 0.03145"/>
-        <mass value="5.8"/>
-        <inertia ixx="0.10105893" ixy="0.000211" ixz="-0.004" iyy="0.09386624" iyz="-0.01698537" izz="0.01449937"/>
-      </inertial>
-      <visual>
-        <origin rpy="0 0 0" xyz="0 0 0"/>
-        <geometry>
-          <mesh filename="package://mara_description/meshes/H-ROS_Robot_mara1.stl" scale="0.001 0.001 0.001"/>
+        <mass value="7.033"/>
+        <inertia ixx="0.1478344" ixy="-0.00001" ixz="0.0" iyy="0.14782335" iyz="0.0" izz="0.29471799"/>
+      </inertial>
+      <visual>
+        <origin rpy="0 0 0" xyz="0 0 0"/>
+        <geometry>
+          <mesh filename="package://mara_description/meshes/MARA_T49.stl" scale="0.001 0.001 0.001"/>
         </geometry>
         <material name="Gazebo/White">
@@ -51,5 +77,5 @@
         <origin rpy="0 0 0" xyz="0 0 0"/>
         <geometry>
-          <mesh filename="package://mara_description/meshes/H-ROS_Robot_mara1.stl" scale="0.001 0.001 0.001"/>
+          <mesh filename="package://mara_description/meshes/MARA_T49.stl" scale="0.001 0.001 0.001"/>
         </geometry>
       </collision>
@@ -59,23 +85,49 @@
       <selfCollide>True</selfCollide>
     </gazebo>
+    <link name="${prefix}motor1_cover">
+      <inertial>
+        <origin rpy="0 0 0" xyz="8.625E-08 -4.6583E-06 0.03145"/>
+        <mass value="7.033"/>
+        <inertia ixx="0.1478344" ixy="-0.00001" ixz="0.0" iyy="0.14782335" iyz="0.0" izz="0.29471799"/>
+      </inertial>
+      <visual>
+        <origin rpy="0 0 0" xyz="0 0 0"/>
+        <geometry>
+          <mesh filename="package://mara_description/meshes/MARA_T49_Black.stl" scale="0.001 0.001 0.001"/>
+        </geometry>
+        <material name="Gazebo/Black">
+          <color rgba="0. 0. 0. 1"/>
+        </material>
+      </visual>
+      <collision>
+        <origin rpy="0 0 0" xyz="0 0 0"/>
+        <geometry>
+          <mesh filename="package://mara_description/meshes/MARA_T49_Black.stl" scale="0.001 0.001 0.001"/>
+        </geometry>
+      </collision>
+    </link>
+    <gazebo reference="${prefix}motor1_cover">
+      <material>Gazebo/Black</material>
+      <selfCollide>True</selfCollide>
+    </gazebo>
     <link name="${prefix}motor2_link">
       <inertial>
         <origin rpy="0 0 0" xyz="8.625E-08 -4.6583E-06 0.03145"/>
-        <mass value="1.03237"/>
-        <inertia ixx="0.014865226" ixy="0.0" ixz="0.0" iyy="0.01557" iyz="0.00071" izz="0.00092"/>
-      </inertial>
-      <visual>
-        <origin rpy="0 0 0" xyz="0 0 0"/>
-        <geometry>
-          <mesh filename="package://mara_description/meshes/H-ROS_Robot_LINK1.stl" scale="0.001 0.001 0.001"/>
-        </geometry>
-        <material name="Gazebo/Black">
-          <color rgba="0. 0. 0. 1"/>
-        </material>
-      </visual>
-      <collision>
-        <origin rpy="0 0 0" xyz="0 0 0"/>
-        <geometry>
-          <mesh filename="package://mara_description/meshes/H-ROS_Robot_LINK1.stl" scale="0.001 0.001 0.001"/>
+        <mass value="7.033"/>
+        <inertia ixx="0.1478344" ixy="-0.00001" ixz="0.0" iyy="0.14782335" iyz="0.0" izz="0.29471799"/>
+      </inertial>
+      <visual>
+        <origin rpy="0 0 0" xyz="0 0 0"/>
+        <geometry>
+          <mesh filename="package://mara_description/meshes/MARA_Link1.stl" scale="0.001 0.001 0.001"/>
+        </geometry>
+        <material name="Gazebo/Black">
+          <color rgba="0. 0. 0. 1"/>
+        </material>
+      </visual>
+      <collision>
+        <origin rpy="0 0 0" xyz="0 0 0"/>
+        <geometry>
+          <mesh filename="package://mara_description/meshes/MARA_Link1.stl" scale="0.001 0.001 0.001"/>
         </geometry>
       </collision>
@@ -88,11 +140,11 @@
       <inertial>
         <origin rpy="0 0 0" xyz="8.625E-08 -4.6583E-06 0.03145"/>
-        <mass value="3.8"/>
-        <inertia ixx="0.04517" ixy="0.00002" ixz="0.0" iyy="0.01587" iyz="0.01444" izz="0.03303"/>
-      </inertial>
-      <visual>
-        <origin rpy="0 0 0" xyz="0 0 0"/>
-        <geometry>
-          <mesh filename="package://mara_description/meshes/H-ROS_Robot_mara2.stl" scale="0.001 0.001 0.001"/>
+        <mass value="7.033"/>
+        <inertia ixx="0.1478344" ixy="-0.00001" ixz="0.0" iyy="0.14782335" iyz="0.0" izz="0.29471799"/>
+      </inertial>
+      <visual>
+        <origin rpy="0 0 0" xyz="0 0 0"/>
+        <geometry>
+          <mesh filename="package://mara_description/meshes/MARA_T30.stl" scale="0.001 0.001 0.001"/>
         </geometry>
         <material name="Gazebo/White">
@@ -103,5 +155,5 @@
         <origin rpy="0 0 0" xyz="0 0 0"/>
         <geometry>
-          <mesh filename="package://mara_description/meshes/H-ROS_Robot_mara2.stl" scale="0.001 0.001 0.001"/>
+          <mesh filename="package://mara_description/meshes/MARA_T30.stl" scale="0.001 0.001 0.001"/>
         </geometry>
       </collision>
@@ -111,23 +163,49 @@
       <selfCollide>True</selfCollide>
     </gazebo>
+    <link name="${prefix}motor3_cover">
+      <inertial>
+        <origin rpy="0 0 0" xyz="8.625E-08 -4.6583E-06 0.03145"/>
+        <mass value="7.033"/>
+        <inertia ixx="0.1478344" ixy="-0.00001" ixz="0.0" iyy="0.14782335" iyz="0.0" izz="0.29471799"/>
+      </inertial>
+      <visual>
+        <origin rpy="0 0 0" xyz="0 0 0"/>
+        <geometry>
+          <mesh filename="package://mara_description/meshes/MARA_T30_Black.stl" scale="0.001 0.001 0.001"/>
+        </geometry>
+        <material name="Gazebo/Black">
+          <color rgba="0. 0. 0. 1"/>
+        </material>
+      </visual>
+      <collision>
+        <origin rpy="0 0 0" xyz="0 0 0"/>
+        <geometry>
+          <mesh filename="package://mara_description/meshes/MARA_T30_Black.stl" scale="0.001 0.001 0.001"/>
+        </geometry>
+      </collision>
+    </link>
+    <gazebo reference="${prefix}motor3_cover">
+      <material>Gazebo/Black</material>
+      <selfCollide>True</selfCollide>
+    </gazebo>
     <link name="${prefix}motor4_link">
       <inertial>
         <origin rpy="0 0 0" xyz="8.625E-08 -4.6583E-06 0.03145"/>
-        <mass value="1.1"/>
-        <inertia ixx="0.01464" ixy="0.0" ixz="0.0" iyy="0.00895" iyz="-0.00631" izz="0.00725"/>
-      </inertial>
-      <visual>
-        <origin rpy="0 0 0" xyz="0 0 0"/>
-        <geometry>
-          <mesh filename="package://mara_description/meshes/H-ROS_Robot_LINK2.stl" scale="0.001 0.001 0.001"/>
-        </geometry>
-        <material name="Gazebo/Black">
-          <color rgba="0. 0. 0. 1"/>
-        </material>
-      </visual>
-      <collision>
-        <origin rpy="0 0 0" xyz="0 0 0"/>
-        <geometry>
-          <mesh filename="package://mara_description/meshes/H-ROS_Robot_LINK2.stl" scale="0.001 0.001 0.001"/>
+        <mass value="7.033"/>
+        <inertia ixx="0.1478344" ixy="-0.00001" ixz="0.0" iyy="0.14782335" iyz="0.0" izz="0.29471799"/>
+      </inertial>
+      <visual>
+        <origin rpy="0 0 0" xyz="0 0 0"/>
+        <geometry>
+          <mesh filename="package://mara_description/meshes/MARA_Link2.stl" scale="0.001 0.001 0.001"/>
+        </geometry>
+        <material name="Gazebo/Black">
+          <color rgba="0. 0. 0. 1"/>
+        </material>
+      </visual>
+      <collision>
+        <origin rpy="0 0 0" xyz="0 0 0"/>
+        <geometry>
+          <mesh filename="package://mara_description/meshes/MARA_Link2.stl" scale="0.001 0.001 0.001"/>
         </geometry>
       </collision>
@@ -140,11 +218,11 @@
       <inertial>
         <origin rpy="0 0 0" xyz="8.625E-08 -4.6583E-06 0.03145"/>
-        <mass value="2.9"/>
-        <inertia ixx="0.03406" ixy="0.0" ixz="0.0" iyy="0.01066" iyz="0.00989" izz="0.02563"/>
-      </inertial>
-      <visual>
-        <origin rpy="0 0 0" xyz="0 0 0"/>
-        <geometry>
-          <mesh filename="package://mara_description/meshes/H-ROS_Robot_mara3.stl" scale="0.001 0.001 0.001"/>
+        <mass value="7.033"/>
+        <inertia ixx="0.1478344" ixy="-0.00001" ixz="0.0" iyy="0.14782335" iyz="0.0" izz="0.29471799"/>
+      </inertial>
+      <visual>
+        <origin rpy="0 0 0" xyz="0 0 0"/>
+        <geometry>
+          <mesh filename="package://mara_description/meshes/MARA_T5.4.stl" scale="0.001 0.001 0.001"/>
         </geometry>
         <material name="Gazebo/White">
@@ -155,5 +233,5 @@
         <origin rpy="0 0 0" xyz="0 0 0"/>
         <geometry>
-          <mesh filename="package://mara_description/meshes/H-ROS_Robot_mara3.stl" scale="0.001 0.001 0.001"/>
+          <mesh filename="package://mara_description/meshes/MARA_T5.4.stl" scale="0.001 0.001 0.001"/>
         </geometry>
       </collision>
@@ -163,23 +241,49 @@
       <selfCollide>True</selfCollide>
     </gazebo>
+    <link name="${prefix}motor5_cover">
+      <inertial>
+        <origin rpy="0 0 0" xyz="8.625E-08 -4.6583E-06 0.03145"/>
+        <mass value="7.033"/>
+        <inertia ixx="0.1478344" ixy="-0.00001" ixz="0.0" iyy="0.14782335" iyz="0.0" izz="0.29471799"/>
+      </inertial>
+      <visual>
+        <origin rpy="0 0 0" xyz="0 0 0"/>
+        <geometry>
+          <mesh filename="package://mara_description/meshes/MARA_T5.4_black.stl" scale="0.001 0.001 0.001"/>
+        </geometry>
+        <material name="Gazebo/Black">
+          <color rgba="0. 0. 0. 1"/>
+        </material>
+      </visual>
+      <collision>
+        <origin rpy="0 0 0" xyz="0 0 0"/>
+        <geometry>
+          <mesh filename="package://mara_description/meshes/MARA_T5.4_black.stl" scale="0.001 0.001 0.001"/>
+        </geometry>
+      </collision>
+    </link>
+    <gazebo reference="${prefix}motor5_cover">
+      <material>Gazebo/Black</material>
+      <selfCollide>True</selfCollide>
+    </gazebo>
     <link name="${prefix}motor6_link">
       <inertial>
         <origin rpy="0 0 0" xyz="8.625E-08 -4.6583E-06 0.03145"/>
-        <mass value="2.9"/>
-        <inertia ixx="0.0005" ixy="0.0" ixz="0.0" iyy="0.0005" iyz="0.0000" izz="0.0003"/>
-      </inertial>
-      <visual>
-        <origin rpy="0 0 ${60*3.14/180}" xyz="0 0 0"/>
-        <geometry>
-          <mesh filename="package://mara_description/meshes/gripper_support.stl" scale="0.001 0.001 0.001"/>
-        </geometry>
-        <material name="Gazebo/Black">
-          <color rgba="0. 0. 0. 1"/>
-        </material>
-      </visual>
-      <collision>
-        <origin rpy="0 0 ${60*3.14/180}" xyz="0 0 0"/>
-        <geometry>
-          <mesh filename="package://mara_description/meshes/gripper_support.stl" scale="0.001 0.001 0.001"/>
+        <mass value="7.033"/>
+        <inertia ixx="0.1478344" ixy="-0.00001" ixz="0.0" iyy="0.14782335" iyz="0.0" izz="0.29471799"/>
+      </inertial>
+      <visual>
+        <origin rpy="0 0 0" xyz="0 0 0"/>
+        <geometry>
+          <mesh filename="package://mara_description/meshes/MARA_GripperAdapter.stl" scale="0.001 0.001 0.001"/>
+        </geometry>
+        <material name="Gazebo/Black">
+          <color rgba="0. 0. 0. 1"/>
+        </material>
+      </visual>
+      <collision>
+        <origin rpy="0 0 0" xyz="0 0 0"/>
+        <geometry>
+          <mesh filename="package://mara_description/meshes/MARA_GripperAdapter.stl" scale="0.001 0.001 0.001"/>
         </geometry>
       </collision>
@@ -195,7 +299,12 @@
       <selfCollide>False</selfCollide>
     </gazebo>
+    <joint name="${prefix}joint_bases" type="fixed">
+      <origin rpy="0 0 0" xyz="0 0 0.04"/>
+      <parent link="${prefix}base_link"/>
+      <child link="${prefix}base_robot"/>
+    </joint>
     <joint name="${prefix}motor1" type="revolute">
-      <origin rpy="0 0 0" xyz="0 0 0.00625"/>
-      <parent link="${prefix}base_link"/>
+      <origin rpy="0 0 0" xyz="0 0 0.05122"/>
+      <parent link="${prefix}base_robot"/>
       <child link="${prefix}motor1_link"/>
       <axis xyz="0 0 -1"/>
@@ -203,42 +312,57 @@
       <dynamics damping="0" friction="0"/>
     </joint>
+    <joint name="${prefix}motor1_cover_joint" type="fixed">
+      <origin rpy="0 0 0" xyz="0 0 0.0"/>
+      <parent link="${prefix}motor1_link"/>
+      <child link="${prefix}motor1_cover"/>
+    </joint>
     <joint name="${prefix}motor2" type="revolute">
-      <origin rpy="0 0 0" xyz="0 -0.100499999 0.1545"/>
+      <origin rpy="0 0 0" xyz="0.118 0 0.1637"/>
       <parent link="${prefix}motor1_link"/>
       <child link="${prefix}motor2_link"/>
-      <axis xyz="0 1 0"/>
-      <limit effort="330.0" lower="-3.13" upper="3.13" velocity="3.1416"/>
+      <axis xyz="1 0 0"/>
+      <limit effort="330.0" lower="-2.3562" upper="2.3562" velocity="3.1416"/>
       <dynamics damping="0" friction="0"/>
     </joint>
     <joint name="${prefix}motor3" type="revolute">
-      <origin rpy="0 0 0" xyz="0 -0.000499999 0.2"/>
+      <origin rpy="0 0 0" xyz="-0.009 0 0.2"/>
       <parent link="${prefix}motor2_link"/>
       <child link="${prefix}motor3_link"/>
-      <axis xyz="0 -1 0"/>
-      <limit effort="330" lower="-3.13" upper="3.13" velocity="3.1416"/>
-      <dynamics damping="0" friction="0"/>
+      <axis xyz="1 0 0"/>
+      <limit effort="330.0" lower="-2.3562" upper="2.3562" velocity="3.1416"/>
+      <dynamics damping="0" friction="0"/>
+    </joint>
+    <joint name="${prefix}motor3_cover_joint" type="fixed">
+      <origin rpy="0 0 0" xyz="0 0 0.0"/>
+      <parent link="${prefix}motor3_link"/>
+      <child link="${prefix}motor3_cover"/>
     </joint>
     <joint name="${prefix}motor4" type="revolute">
-      <origin rpy="0 0 0" xyz="0 0.09999 0.12999997"/>
+      <origin rpy="0 0 0" xyz="-0.109255 0 0.149255"/>
       <parent link="${prefix}motor3_link"/>
       <child link="${prefix}motor4_link"/>
-      <axis xyz="0 0 -1"/>
-      <limit effort="330" lower="-3.13" upper="3.13" velocity="3.1416"/>
+      <axis xyz="0 0 1"/>
+      <limit effort="330.0" lower="-2.3562" upper="2.3562" velocity="3.1416"/>
       <dynamics damping="0" friction="0"/>
     </joint>
     <joint name="${prefix}motor5" type="revolute">
-      <origin rpy="0 0 0" xyz="0 -0.096999 0.15906"/>
+      <origin rpy="0 0 0" xyz="0.1054570 0 0.16074"/>
       <parent link="${prefix}motor4_link"/>
       <child link="${prefix}motor5_link"/>
-      <axis xyz="0 -1 0"/>
-      <limit effort="330" lower="-3.13" upper="3.13" velocity="3.1416"/>
-      <dynamics damping="0" friction="0"/>
+      <axis xyz="1 0 0"/>
+      <limit effort="330.0" lower="-2.3562" upper="2.3562" velocity="3.1416"/>
+      <dynamics damping="0" friction="0"/>
+    </joint>
+    <joint name="${prefix}motor5_cover_joint" type="fixed">
+      <origin rpy="0 0 0" xyz="0 0 0.0"/>
+      <parent link="${prefix}motor5_link"/>
+      <child link="${prefix}motor5_cover"/>
     </joint>
     <joint name="${prefix}motor6" type="revolute">
-      <origin rpy="0 0 0" xyz="0 0.0969999 0.1265"/>
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
File: mara_description/urdf/mara_robot_camera_top.urdf (robot description, URDF)
Before this commit: robot mara, 21 links, 20 joints
Links:
- removed link base
- added link base_robot, mass 7.033; collision mesh filename=package://mara_description/meshes/Base.stl scale=0.001 0.001 0.001; visual mesh filename=package://mara_description/meshes/Base.stl scale=0.001 0.001 0.001
- added link motor1_cover, mass 7.033; collision mesh filename=package://mara_description/meshes/MARA_T49_Black.stl scale=0.001 0.001 0.001; visual mesh filename=package://mara_description/meshes/MARA_T49_Black.stl scale=0.001 0.001 0.001
- added link motor3_cover, mass 7.033; collision mesh filename=package://mara_description/meshes/MARA_T30_Black.stl scale=0.001 0.001 0.001; visual mesh filename=package://mara_description/meshes/MARA_T30_Black.stl scale=0.001 0.001 0.001
- added link motor5_cover, mass 7.033; collision mesh filename=package://mara_description/meshes/MARA_T5.4_black.stl scale=0.001 0.001 0.001; visual mesh filename=package://mara_description/meshes/MARA_T5.4_black.stl scale=0.001 0.001 0.001
- link base_link: geometry collision mesh filename=package://mara_description/meshes/Base_plancha.stl scale=0.001 0.001 0.001; visual mesh filename=package://mara_description/meshes/Base_plancha.stl scale=0.001 0.001 0.001
- link motor1_link: mass 5.8 -> 7.033; geometry collision mesh filename=package://mara_description/meshes/MARA_T49.stl scale=0.001 0.001 0.001; visual mesh filename=package://mara_description/meshes/MARA_T49.stl scale=0.001 0.001 0.001
- link motor2_link: mass 1.03237 -> 7.033; geometry collision mesh filename=package://mara_description/meshes/MARA_Link1.stl scale=0.001 0.001 0.001; visual mesh filename=package://mara_description/meshes/MARA_Link1.stl scale=0.001 0.001 0.001
- link motor3_link: mass 3.8 -> 7.033; geometry collision mesh filename=package://mara_description/meshes/MARA_T30.stl scale=0.001 0.001 0.001; visual mesh filename=package://mara_description/meshes/MARA_T30.stl scale=0.001 0.001 0.001
- link motor4_link: mass 1.1 -> 7.033; geometry collision mesh filename=package://mara_description/meshes/MARA_Link2.stl scale=0.001 0.001 0.001; visual mesh filename=package://mara_description/meshes/MARA_Link2.stl scale=0.001 0.001 0.001
- link motor5_link: mass 2.9 -> 7.033; geometry collision mesh filename=package://mara_description/meshes/MARA_T5.4.stl scale=0.001 0.001 0.001; visual mesh filename=package://mara_description/meshes/MARA_T5.4.stl scale=0.001 0.001 0.001
- link motor6_link: mass 2.9 -> 7.033; geometry collision mesh filename=package://mara_description/meshes/MARA_GripperAdapter.stl scale=0.001 0.001 0.001; visual mesh filename=package://mara_description/meshes/MARA_GripperAdapter.stl scale=0.001 0.001 0.001
Joints:
- removed joint base_link-base_fixed_joint
- added joint joint_bases: type fixed, parent base_link, child base_robot, origin xyz=0 0 0.04 rpy=0 0 0
- added joint motor1_cover_joint: type fixed, parent motor1_link, child motor1_cover, origin xyz=0 0 0.0 rpy=0 0 0
- added joint motor3_cover_joint: type fixed, parent motor3_link, child motor3_cover, origin xyz=0 0 0.0 rpy=0 0 0
- added joint motor5_cover_joint: type fixed, parent motor5_link, child motor5_cover, origin xyz=0 0 0.0 rpy=0 0 0
- joint end_effector_adapter_to_robotiq: origin xyz= 0 0 0.05375 rpy=0 0 0 -> xyz= 0 0 0.04659 rpy=0 0 1.57
- joint motor1: origin xyz=0 0 0.00625 rpy=0 0 0 -> xyz=0 0 0.05122 rpy=0 0 0; parent base_link -> base_robot
- joint motor2: axis 0 1 0 -> 1 0 0; limit lower=-3.13 upper=3.13 effort=330.0 velocity=3.1416 -> lower=-2.3562 upper=2.3562 effort=330.0 velocity=3.1416; origin xyz=0 -0.100499999 0.1545 rpy=0 0 0 -> xyz=0.118 0 0.1637 rpy=0 0 0
- joint motor3: axis 0 -1 0 -> 1 0 0; limit lower=-3.13 upper=3.13 effort=330 velocity=3.1416 -> lower=-2.3562 upper=2.3562 effort=330.0 velocity=3.1416; origin xyz=0 -0.000499999 0.2 rpy=0 0 0 -> xyz=-0.009 0 0.2 rpy=0 0 0
- joint motor4: axis 0 0 -1 -> 0 0 1; limit lower=-3.13 upper=3.13 effort=330 velocity=3.1416 -> lower=-2.3562 upper=2.3562 effort=330.0 velocity=3.1416; origin xyz=0 0.09999 0.12999997 rpy=0 0 0 -> xyz=-0.109255 0 0.149255 rpy=0 0 0
- joint motor5: axis 0 -1 0 -> 1 0 0; limit lower=-3.13 upper=3.13 effort=330 velocity=3.1416 -> lower=-2.3562 upper=2.3562 effort=330.0 velocity=3.1416; origin xyz=0 -0.096999 0.15906 rpy=0 0 0 -> xyz=0.1054570 0 0.16074 rpy=0 0 0
- joint motor6: axis 0 0 -1 -> 0 0 1; limit lower=-3.13 upper=3.13 effort=330 velocity=3.1416 -> lower=-2.3562 upper=2.3562 effort=330.0 velocity=3.1416; origin xyz=0 0.0969999 0.1265 rpy=0 0 0 -> xyz=-0.10625569 0 0.14675569 rpy=0 0 0
- joint table_to_base_joint: origin xyz=0 0 0.65 rpy=0 0 0 -> xyz=0 0 0.62 rpy=0 0 0

File: mara_description/urdf/mara_robot_camera_top.urdf.xacro (robot description, xacro)
@@ -17,5 +17,5 @@
   <link name="world" />
   <joint name="end_effector_adapter_to_robotiq" type="fixed">
-    <origin rpy="0 0 0" xyz=" 0 0 0.05375"/>
+    <origin rpy="0 0 1.57" xyz=" 0 0 0.04659"/>
     <parent link="motor6_link"/>
     <child link="robotiq_arg2f_base_link"/>
@@ -27,5 +27,5 @@
   </joint>
   <joint name="table_to_base_joint" type="fixed">
-    <origin rpy="0 0 0" xyz="0 0 0.65"/>
+    <origin rpy="0 0 0" xyz="0 0 0.62"/>
     <parent link="table"/>
     <child link="base_link"/>
