Commit message: Update MARA inertias

File: mara_description/urdf/mara.urdf.xacro (robot description, xacro)
@@ -62,6 +62,6 @@
       <inertial>
         <origin rpy="0 0 0" xyz="8.625E-08 -4.6583E-06 0.03145"/>
-        <mass value="7.033"/>
-        <inertia ixx="0.1478344" ixy="-0.00001" ixz="0.0" iyy="0.14782335" iyz="0.0" izz="0.29471799"/>
+        <mass value="5.8"/>
+        <inertia ixx="0.10105893" ixy="0.000211" ixz="-0.004" iyy="0.09386624" iyz="-0.01698537" izz="0.01449937"/>
       </inertial>
       <visual>
@@ -88,6 +88,6 @@
       <inertial>
         <origin rpy="0 0 0" xyz="8.625E-08 -4.6583E-06 0.03145"/>
-        <mass value="7.033"/>
-        <inertia ixx="0.1478344" ixy="-0.00001" ixz="0.0" iyy="0.14782335" iyz="0.0" izz="0.29471799"/>
+        <mass value="5.8"/>
+        <inertia ixx="0.10105893" ixy="0.000211" ixz="-0.004" iyy="0.09386624" iyz="-0.01698537" izz="0.01449937"/>
       </inertial>
       <visual>
@@ -114,6 +114,6 @@
       <inertial>
         <origin rpy="0 0 0" xyz="8.625E-08 -4.6583E-06 0.03145"/>
-        <mass value="7.033"/>
-        <inertia ixx="0.1478344" ixy="-0.00001" ixz="0.0" iyy="0.14782335" iyz="0.0" izz="0.29471799"/>
+        <mass value="1.03237"/>
+        <inertia ixx="0.014865226" ixy="0.0" ixz="0.0" iyy="0.01557" iyz="0.00071" izz="0.00092"/>
       </inertial>
       <visual>
@@ -140,6 +140,6 @@
       <inertial>
         <origin rpy="0 0 0" xyz="8.625E-08 -4.6583E-06 0.03145"/>
-        <mass value="7.033"/>
-        <inertia ixx="0.1478344" ixy="-0.00001" ixz="0.0" iyy="0.14782335" iyz="0.0" izz="0.29471799"/>
+        <mass value="3.8"/>
+        <inertia ixx="0.04517" ixy="0.00002" ixz="0.0" iyy="0.01587" iyz="0.01444" izz="0.03303"/>
       </inertial>
       <visual>
@@ -166,6 +166,6 @@
       <inertial>
         <origin rpy="0 0 0" xyz="8.625E-08 -4.6583E-06 0.03145"/>
-        <mass value="7.033"/>
-        <inertia ixx="0.1478344" ixy="-0.00001" ixz="0.0" iyy="0.14782335" iyz="0.0" izz="0.29471799"/>
+        <mass value="3.8"/>
+        <inertia ixx="0.04517" ixy="0.00002" ixz="0.0" iyy="0.01587" iyz="0.01444" izz="0.03303"/>
       </inertial>
       <visual>
@@ -192,6 +192,6 @@
       <inertial>
         <origin rpy="0 0 0" xyz="8.625E-08 -4.6583E-06 0.03145"/>
-        <mass value="7.033"/>
-        <inertia ixx="0.1478344" ixy="-0.00001" ixz="0.0" iyy="0.14782335" iyz="0.0" izz="0.29471799"/>
+        <mass value="1.1"/>
+        <inertia ixx="0.01464" ixy="0.0" ixz="0.0" iyy="0.00895" iyz="-0.00631" izz="0.00725"/>
       </inertial>
       <visual>
@@ -218,6 +218,6 @@
       <inertial>
         <origin rpy="0 0 0" xyz="8.625E-08 -4.6583E-06 0.03145"/>
-        <mass value="7.033"/>
-        <inertia ixx="0.1478344" ixy="-0.00001" ixz="0.0" iyy="0.14782335" iyz="0.0" izz="0.29471799"/>
+        <mass value="2.9"/>
+        <inertia ixx="0.03406" ixy="0.0" ixz="0.0" iyy="0.01066" iyz="0.00989" izz="0.02563"/>
       </inertial>
       <visual>
@@ -244,6 +244,6 @@
       <inertial>
         <origin rpy="0 0 0" xyz="8.625E-08 -4.6583E-06 0.03145"/>
-        <mass value="7.033"/>
-        <inertia ixx="0.1478344" ixy="-0.00001" ixz="0.0" iyy="0.14782335" iyz="0.0" izz="0.29471799"/>
+        <mass value="2.9"/>
+        <inertia ixx="0.03406" ixy="0.0" ixz="0.0" iyy="0.01066" iyz="0.00989" izz="0.02563"/>
       </inertial>
       <visual>
@@ -270,6 +270,6 @@
       <inertial>
         <origin rpy="0 0 0" xyz="8.625E-08 -4.6583E-06 0.03145"/>
-        <mass value="7.033"/>
-        <inertia ixx="0.1478344" ixy="-0.00001" ixz="0.0" iyy="0.14782335" iyz="0.0" izz="0.29471799"/>
+        <mass value="2.9"/>
+        <inertia ixx="0.0005" ixy="0.0" ixz="0.0" iyy="0.0005" iyz="0.0000" izz="0.0003"/>
       </inertial>
       <visual>

File: mara_description/urdf/mara_robot_camera_top.urdf (robot description, URDF)
Before this commit: robot mara, 24 links, 23 joints
Links:
- link motor1_cover: mass 7.033 -> 5.8
- link motor1_link: mass 7.033 -> 5.8
- link motor2_link: mass 7.033 -> 1.03237
- link motor3_cover: mass 7.033 -> 3.8
- link motor3_link: mass 7.033 -> 3.8
- link motor4_link: mass 7.033 -> 1.1
- link motor5_cover: mass 7.033 -> 2.9
- link motor5_link: mass 7.033 -> 2.9
- link motor6_link: mass 7.033 -> 2.9

Commit message: Adding textures in all materials

File: mara_description/urdf/mara.urdf.xacro (robot description, xacro)
@@ -20,4 +20,5 @@
         <material name="Gazebo/Grey">
           <color rgba="0. 0. 0. 1"/>
+          <texture filename="model://mara_description/material/gazebo.material" />
         </material>
       </visual>
@@ -46,5 +47,6 @@
         <material name="Gazebo/Grey">
           <color rgba="0. 0. 0. 1"/>
-        </material>
+          <texture filename="model://mara_description/material/gazebo.material" />
+      </material>
       </visual>
       <collision>
@@ -72,4 +74,5 @@
         <material name="Gazebo/White">
           <color rgba="0. 0. 0. 1"/>
+          <texture filename="model://mara_description/material/gazebo.material" />
         </material>
       </visual>
@@ -98,4 +101,5 @@
         <material name="Gazebo/Black">
           <color rgba="0. 0. 0. 1"/>
+          <texture filename="model://mara_description/material/gazebo.material" />
         </material>
       </visual>
@@ -124,4 +128,5 @@
         <material name="Gazebo/Black">
           <color rgba="0. 0. 0. 1"/>
+          <texture filename="model://mara_description/material/gazebo.material" />
         </material>
       </visual>
@@ -150,4 +155,5 @@
         <material name="Gazebo/White">
           <color rgba="0. 0. 0. 1"/>
+          <texture filename="model://mara_description/material/gazebo.material" />
         </material>
       </visual>
@@ -176,4 +182,5 @@
         <material name="Gazebo/Black">
           <color rgba="0. 0. 0. 1"/>
+          <texture filename="model://mara_description/material/gazebo.material" />
         </material>
       </visual>
@@ -202,4 +209,5 @@
         <material name="Gazebo/Black">
           <color rgba="0. 0. 0. 1"/>
+          <texture filename="model://mara_description/material/gazebo.material" />
         </material>
       </visual>
@@ -228,4 +236,5 @@
         <material name="Gazebo/White">
           <color rgba="0. 0. 0. 1"/>
+          <texture filename="model://mara_description/material/gazebo.material" />
         </material>
       </visual>
@@ -254,4 +263,5 @@
         <material name="Gazebo/Black">
           <color rgba="0. 0. 0. 1"/>
+          <texture filename="model://mara_description/material/gazebo.material" />
         </material>
       </visual>
@@ -280,5 +290,6 @@
         <material name="Gazebo/Black">
           <color rgba="0. 0. 0. 1"/>
-        </material>
+          <texture filename="model://mara_description/material/gazebo.material" />
+      </material>
       </visual>
       <collision>

Commit message: fixing orientation

File: mara_description/urdf/mara.urdf.xacro (robot description, xacro)
@@ -332,5 +332,5 @@
       <parent link="${prefix}motor1_link"/>
       <child link="${prefix}motor2_link"/>
-      <axis xyz="1 0 0"/>
+      <axis xyz="-1 0 0"/>
       <limit effort="330.0" lower="-2.3562" upper="2.3562" velocity="3.1416"/>
       <dynamics damping="0" friction="0"/>
@@ -353,5 +353,5 @@
       <parent link="${prefix}motor3_link"/>
       <child link="${prefix}motor4_link"/>
-      <axis xyz="0 0 1"/>
+      <axis xyz="0 0 -1"/>
       <limit effort="330.0" lower="-2.3562" upper="2.3562" velocity="3.1416"/>
       <dynamics damping="0" friction="0"/>
@@ -374,5 +374,5 @@
       <parent link="${prefix}motor5_link"/>
       <child link="${prefix}motor6_link"/>
-      <axis xyz="0 0 1"/>
+      <axis xyz="0 0 -1"/>
       <limit effort="330.0" lower="-2.3562" upper="2.3562" velocity="3.1416"/>
       <dynamics damping="0" friction="0"/>

File: mara_description/urdf/mara_robot_camera_top.urdf (robot description, URDF)
Before this commit: robot mara, 24 links, 23 joints
Joints:
- joint motor2: axis 1 0 0 -> -1 0 0
- joint motor4: axis 0 0 1 -> 0 0 -1
- joint motor6: axis 0 0 1 -> 0 0 -1

Commit message: Allow the gripper to move +-3.14

File: mara_description/urdf/mara.urdf.xacro (robot description, xacro)
@@ -375,5 +375,5 @@
       <child link="${prefix}motor6_link"/>
       <axis xyz="0 0 -1"/>
-      <limit effort="330.0" lower="-2.3562" upper="2.3562" velocity="3.1416"/>
+      <limit effort="330.0" lower="-3.1416" upper="3.1416" velocity="3.1416"/>
       <dynamics damping="0" friction="0"/>
     </joint>

File: mara_description/urdf/mara_robot_camera_top.urdf (robot description, URDF)
Before this commit: robot mara, 24 links, 23 joints
Joints:
- joint motor6: limit lower=-2.3562 upper=2.3562 effort=330.0 velocity=3.1416 -> lower=-3.1416 upper=3.1416 effort=330.0 velocity=3.1416

Commit message: Increasing mara limits

File: mara_description/urdf/mara.urdf.xacro (robot description, xacro)
@@ -320,5 +320,5 @@
       <child link="${prefix}motor1_link"/>
       <axis xyz="0 0 -1"/>
-      <limit effort="330.0" lower="-2.3562" upper="2.3562" velocity="3.1416"/>
+      <limit effort="330.0" lower="-3.1416" upper="3.1416" velocity="3.1416"/>
       <dynamics damping="0" friction="0"/>
     </joint>
@@ -333,5 +333,5 @@
       <child link="${prefix}motor2_link"/>
       <axis xyz="-1 0 0"/>
-      <limit effort="330.0" lower="-2.3562" upper="2.3562" velocity="3.1416"/>
+      <limit effort="330.0" lower="-3.1416" upper="3.1416" velocity="3.1416"/>
       <dynamics damping="0" friction="0"/>
     </joint>
@@ -341,5 +341,5 @@
       <child link="${prefix}motor3_link"/>
       <axis xyz="1 0 0"/>
-      <limit effort="330.0" lower="-2.3562" upper="2.3562" velocity="3.1416"/>
+      <limit effort="330.0" lower="-3.1416" upper="3.1416" velocity="3.1416"/>
       <dynamics damping="0" friction="0"/>
     </joint>
@@ -354,5 +354,5 @@
       <child link="${prefix}motor4_link"/>
       <axis xyz="0 0 -1"/>
-      <limit effort="330.0" lower="-2.3562" upper="2.3562" velocity="3.1416"/>
+      <limit effort="330.0" lower="-3.1416" upper="3.1416" velocity="3.1416"/>
       <dynamics damping="0" friction="0"/>
     </joint>
@@ -362,5 +362,5 @@
       <child link="${prefix}motor5_link"/>
       <axis xyz="1 0 0"/>
-      <limit effort="330.0" lower="-2.3562" upper="2.3562" velocity="3.1416"/>
+      <limit effort="330.0" lower="-3.1416" upper="3.1416" velocity="3.1416"/>
       <dynamics damping="0" friction="0"/>
     </joint>

File: mara_description/urdf/mara_robot_camera_top.urdf (robot description, URDF)
Before this commit: robot mara, 24 links, 23 joints
Joints:
- joint motor1: limit lower=-2.3562 upper=2.3562 effort=330.0 velocity=3.1416 -> lower=-3.1416 upper=3.1416 effort=330.0 velocity=3.1416
- joint motor2: limit lower=-2.3562 upper=2.3562 effort=330.0 velocity=3.1416 -> lower=-3.1416 upper=3.1416 effort=330.0 velocity=3.1416
- joint motor3: limit lower=-2.3562 upper=2.3562 effort=330.0 velocity=3.1416 -> lower=-3.1416 upper=3.1416 effort=330.0 velocity=3.1416
- joint motor4: limit lower=-2.3562 upper=2.3562 effort=330.0 velocity=3.1416 -> lower=-3.1416 upper=3.1416 effort=330.0 velocity=3.1416
- joint motor5: limit lower=-2.3562 upper=2.3562 effort=330.0 velocity=3.1416 -> lower=-3.1416 upper=3.1416 effort=330.0 velocity=3.1416
