Commit message: Change stl to dae to visualize everything in RVIZ2

File: mara_description/urdf/mara.urdf.xacro (robot description, xacro)
@@ -16,15 +16,15 @@
         <origin rpy="0 0 0" xyz="0 0 0"/>
         <geometry>
-          <mesh filename="model://mara_description/meshes/Base_plancha.stl" scale="0.001 0.001 0.001"/>
+          <mesh filename="package://mara_description/meshes/Base_plancha.dae" scale="0.001 0.001 0.001"/>
         </geometry>
         <material name="Gazebo/Grey">
           <color rgba="0. 0. 0. 1"/>
-          <texture filename="model://mara_description/material/gazebo.material" />
-        </material>
-      </visual>
-      <collision>
-        <origin rpy="0 0 0" xyz="0 0 0"/>
-        <geometry>
-          <mesh filename="model://mara_description/meshes/Base_plancha.stl" scale="0.001 0.001 0.001"/>
+          <texture filename="package://mara_description/material/gazebo.material" />
+        </material>
+      </visual>
+      <collision>
+        <origin rpy="0 0 0" xyz="0 0 0"/>
+        <geometry>
+          <mesh filename="package://mara_description/meshes/Base_plancha.dae" scale="0.001 0.001 0.001"/>
         </geometry>
       </collision>
@@ -43,9 +43,9 @@
         <origin rpy="0 0 0" xyz="0 0 0"/>
         <geometry>
-          <mesh filename="model://mara_description/meshes/Base.stl" scale="0.001 0.001 0.001"/>
+          <mesh filename="package://mara_description/meshes/Base.dae" scale="0.001 0.001 0.001"/>
         </geometry>
         <material name="Gazebo/Grey">
           <color rgba="0. 0. 0. 1"/>
-          <texture filename="model://mara_description/material/gazebo.material" />
+          <texture filename="package://mara_description/material/gazebo.material" />
       </material>
       </visual>
@@ -53,5 +53,5 @@
         <origin rpy="0 0 0" xyz="0 0 0"/>
         <geometry>
-          <mesh filename="model://mara_description/meshes/Base.stl" scale="0.001 0.001 0.001"/>
+          <mesh filename="package://mara_description/meshes/Base.dae" scale="0.001 0.001 0.001"/>
         </geometry>
       </collision>
@@ -70,15 +70,15 @@
         <origin rpy="0 0 0" xyz="0 0 0"/>
         <geometry>
-          <mesh filename="model://mara_description/meshes/MARA_T49.stl" scale="0.001 0.001 0.001"/>
+          <mesh filename="package://mara_description/meshes/MARA_T49.dae" scale="0.001 0.001 0.001"/>
         </geometry>
         <material name="Gazebo/White">
           <color rgba="0. 0. 0. 1"/>
-          <texture filename="model://mara_description/material/gazebo.material" />
-        </material>
-      </visual>
-      <collision>
-        <origin rpy="0 0 0" xyz="0 0 0"/>
-        <geometry>
-          <mesh filename="model://mara_description/meshes/MARA_T49.stl" scale="0.001 0.001 0.001"/>
+          <texture filename="package://mara_description/material/gazebo.material" />
+        </material>
+      </visual>
+      <collision>
+        <origin rpy="0 0 0" xyz="0 0 0"/>
+        <geometry>
+          <mesh filename="package://mara_description/meshes/MARA_T49.dae" scale="0.001 0.001 0.001"/>
         </geometry>
       </collision>
@@ -97,15 +97,15 @@
         <origin rpy="0 0 0" xyz="0 0 0"/>
         <geometry>
-          <mesh filename="model://mara_description/meshes/MARA_T49_Black.stl" scale="0.001 0.001 0.001"/>
-        </geometry>
-        <material name="Gazebo/Black">
-          <color rgba="0. 0. 0. 1"/>
-          <texture filename="model://mara_description/material/gazebo.material" />
-        </material>
-      </visual>
-      <collision>
-        <origin rpy="0 0 0" xyz="0 0 0"/>
-        <geometry>
-          <mesh filename="model://mara_description/meshes/MARA_T49_Black.stl" scale="0.001 0.001 0.001"/>
+          <mesh filename="package://mara_description/meshes/MARA_T49_Black.dae" scale="0.001 0.001 0.001"/>
+        </geometry>
+        <material name="Gazebo/Black">
+          <color rgba="0. 0. 0. 1"/>
+          <texture filename="package://mara_description/material/gazebo.material" />
+        </material>
+      </visual>
+      <collision>
+        <origin rpy="0 0 0" xyz="0 0 0"/>
+        <geometry>
+          <mesh filename="package://mara_description/meshes/MARA_T49_Black.dae" scale="0.001 0.001 0.001"/>
         </geometry>
       </collision>
@@ -124,15 +124,15 @@
         <origin rpy="0 0 0" xyz="0 0 0"/>
         <geometry>
-          <mesh filename="model://mara_description/meshes/MARA_Link1.stl" scale="0.001 0.001 0.001"/>
-        </geometry>
-        <material name="Gazebo/Black">
-          <color rgba="0. 0. 0. 1"/>
-          <texture filename="model://mara_description/material/gazebo.material" />
-        </material>
-      </visual>
-      <collision>
-        <origin rpy="0 0 0" xyz="0 0 0"/>
-        <geometry>
-          <mesh filename="model://mara_description/meshes/MARA_Link1.stl" scale="0.001 0.001 0.001"/>
+          <mesh filename="package://mara_description/meshes/MARA_Link1.dae" scale="0.001 0.001 0.001"/>
+        </geometry>
+        <material name="Gazebo/Black">
+          <color rgba="0. 0. 0. 1"/>
+          <texture filename="package://mara_description/material/gazebo.material" />
+        </material>
+      </visual>
+      <collision>
+        <origin rpy="0 0 0" xyz="0 0 0"/>
+        <geometry>
+          <mesh filename="package://mara_description/meshes/MARA_Link1.dae" scale="0.001 0.001 0.001"/>
         </geometry>
       </collision>
@@ -151,15 +151,15 @@
         <origin rpy="0 0 0" xyz="0 0 0"/>
         <geometry>
-          <mesh filename="model://mara_description/meshes/MARA_T30.stl" scale="0.001 0.001 0.001"/>
+          <mesh filename="package://mara_description/meshes/MARA_T30.dae" scale="0.001 0.001 0.001"/>
         </geometry>
         <material name="Gazebo/White">
           <color rgba="0. 0. 0. 1"/>
-          <texture filename="model://mara_description/material/gazebo.material" />
-        </material>
-      </visual>
-      <collision>
-        <origin rpy="0 0 0" xyz="0 0 0"/>
-        <geometry>
-          <mesh filename="model://mara_description/meshes/MARA_T30.stl" scale="0.001 0.001 0.001"/>
+          <texture filename="package://mara_description/material/gazebo.material" />
+        </material>
+      </visual>
+      <collision>
+        <origin rpy="0 0 0" xyz="0 0 0"/>
+        <geometry>
+          <mesh filename="package://mara_description/meshes/MARA_T30.dae" scale="0.001 0.001 0.001"/>
         </geometry>
       </collision>
@@ -178,15 +178,15 @@
         <origin rpy="0 0 0" xyz="0 0 0"/>
         <geometry>
-          <mesh filename="model://mara_description/meshes/MARA_T30_Black.stl" scale="0.001 0.001 0.001"/>
-        </geometry>
-        <material name="Gazebo/Black">
-          <color rgba="0. 0. 0. 1"/>
-          <texture filename="model://mara_description/material/gazebo.material" />
-        </material>
-      </visual>
-      <collision>
-        <origin rpy="0 0 0" xyz="0 0 0"/>
-        <geometry>
-          <mesh filename="model://mara_description/meshes/MARA_T30_Black.stl" scale="0.001 0.001 0.001"/>
+          <mesh filename="package://mara_description/meshes/MARA_T30_Black.dae" scale="0.001 0.001 0.001"/>
+        </geometry>
+        <material name="Gazebo/Black">
+          <color rgba="0. 0. 0. 1"/>
+          <texture filename="package://mara_description/material/gazebo.material" />
+        </material>
+      </visual>
+      <collision>
+        <origin rpy="0 0 0" xyz="0 0 0"/>
+        <geometry>
+          <mesh filename="package://mara_description/meshes/MARA_T30_Black.dae" scale="0.001 0.001 0.001"/>
         </geometry>
       </collision>
@@ -205,15 +205,15 @@
         <origin rpy="0 0 0" xyz="0 0 0"/>
         <geometry>
-          <mesh filename="model://mara_description/meshes/MARA_Link2.stl" scale="0.001 0.001 0.001"/>
-        </geometry>
-        <material name="Gazebo/Black">
-          <color rgba="0. 0. 0. 1"/>
-          <texture filename="model://mara_description/material/gazebo.material" />
-        </material>
-      </visual>
-      <collision>
-        <origin rpy="0 0 0" xyz="0 0 0"/>
-        <geometry>
-          <mesh filename="model://mara_description/meshes/MARA_Link2.stl" scale="0.001 0.001 0.001"/>
+          <mesh filename="package://mara_description/meshes/MARA_Link2.dae" scale="0.001 0.001 0.001"/>
+        </geometry>
+        <material name="Gazebo/Black">
+          <color rgba="0. 0. 0. 1"/>
+          <texture filename="package://mara_description/material/gazebo.material" />
+        </material>
+      </visual>
+      <collision>
+        <origin rpy="0 0 0" xyz="0 0 0"/>
+        <geometry>
+          <mesh filename="package://mara_description/meshes/MARA_Link2.dae" scale="0.001 0.001 0.001"/>
         </geometry>
       </collision>
@@ -232,15 +232,15 @@
         <origin rpy="0 0 0" xyz="0 0 0"/>
         <geometry>
-          <mesh filename="model://mara_description/meshes/MARA_T5.4.stl" scale="0.001 0.001 0.001"/>
+          <mesh filename="package://mara_description/meshes/MARA_T5.4.dae" scale="0.001 0.001 0.001"/>
         </geometry>
         <material name="Gazebo/White">
           <color rgba="0. 0. 0. 1"/>
-          <texture filename="model://mara_description/material/gazebo.material" />
-        </material>
-      </visual>
-      <collision>
-        <origin rpy="0 0 0" xyz="0 0 0"/>
-        <geometry>
-          <mesh filename="model://mara_description/meshes/MARA_T5.4.stl" scale="0.001 0.001 0.001"/>
+          <texture filename="package://mara_description/material/gazebo.material" />
+        </material>
+      </visual>
+      <collision>
+        <origin rpy="0 0 0" xyz="0 0 0"/>
+        <geometry>
+          <mesh filename="package://mara_description/meshes/MARA_T5.4.dae" scale="0.001 0.001 0.001"/>
         </geometry>
       </collision>
@@ -259,15 +259,15 @@
         <origin rpy="0 0 0" xyz="0 0 0"/>
         <geometry>
-          <mesh filename="model://mara_description/meshes/MARA_T5.4_black.stl" scale="0.001 0.001 0.001"/>
-        </geometry>
-        <material name="Gazebo/Black">
-          <color rgba="0. 0. 0. 1"/>
-          <texture filename="model://mara_description/material/gazebo.material" />
-        </material>
-      </visual>
-      <collision>
-        <origin rpy="0 0 0" xyz="0 0 0"/>
-        <geometry>
-          <mesh filename="model://mara_description/meshes/MARA_T5.4_black.stl" scale="0.001 0.001 0.001"/>
+          <mesh filename="package://mara_description/meshes/MARA_T5.4_black.dae" scale="0.001 0.001 0.001"/>
+        </geometry>
+        <material name="Gazebo/Black">
+          <color rgba="0. 0. 0. 1"/>
+          <texture filename="package://mara_description/material/gazebo.material" />
+        </material>
+      </visual>
+      <collision>
+        <origin rpy="0 0 0" xyz="0 0 0"/>
+        <geometry>
+          <mesh filename="package://mara_description/meshes/MARA_T5.4_black.dae" scale="0.001 0.001 0.001"/>
         </geometry>
       </collision>
@@ -286,9 +286,9 @@
         <origin rpy="0 0 0" xyz="0 0 0"/>
         <geometry>
-          <mesh filename="model://mara_description/meshes/MARA_GripperAdapter.stl" scale="0.001 0.001 0.001"/>
-        </geometry>
-        <material name="Gazebo/Black">
-          <color rgba="0. 0. 0. 1"/>
-          <texture filename="model://mara_description/material/gazebo.material" />
+          <mesh filename="package://mara_description/meshes/MARA_GripperAdapter.dae" scale="0.001 0.001 0.001"/>
+        </geometry>
+        <material name="Gazebo/Black">
+          <color rgba="0. 0. 0. 1"/>
+          <texture filename="package://mara_description/material/gazebo.material" />
       </material>
       </visual>
@@ -296,5 +296,5 @@
         <origin rpy="0 0 0" xyz="0 0 0"/>
         <geometry>
-          <mesh filename="model://mara_description/meshes/MARA_GripperAdapter.stl" scale="0.001 0.001 0.001"/>
+          <mesh filename="package://mara_description/meshes/MARA_GripperAdapter.dae" scale="0.001 0.001 0.001"/>
         </geometry>
       </collision>

File: mara_description/urdf/mara_robot_camera_top.urdf (robot description, URDF)
Before this commit: robot mara, 24 links, 23 joints
Links:
- link base_link: geometry collision mesh filename=package://mara_description/meshes/Base_plancha.dae scale=0.001 0.001 0.001; visual mesh filename=package://mara_description/meshes/Base_plancha.dae scale=0.001 0.001 0.001
- link base_robot: geometry collision mesh filename=package://mara_description/meshes/Base.dae scale=0.001 0.001 0.001; visual mesh filename=package://mara_description/meshes/Base.dae scale=0.001 0.001 0.001
- link motor1_cover: geometry collision mesh filename=package://mara_description/meshes/MARA_T49_Black.dae scale=0.001 0.001 0.001; visual mesh filename=package://mara_description/meshes/MARA_T49_Black.dae scale=0.001 0.001 0.001
- link motor1_link: geometry collision mesh filename=package://mara_description/meshes/MARA_T49.dae scale=0.001 0.001 0.001; visual mesh filename=package://mara_description/meshes/MARA_T49.dae scale=0.001 0.001 0.001
- link motor2_link: geometry collision mesh filename=package://mara_description/meshes/MARA_Link1.dae scale=0.001 0.001 0.001; visual mesh filename=package://mara_description/meshes/MARA_Link1.dae scale=0.001 0.001 0.001
- link motor3_cover: geometry collision mesh filename=package://mara_description/meshes/MARA_T30_Black.dae scale=0.001 0.001 0.001; visual mesh filename=package://mara_description/meshes/MARA_T30_Black.dae scale=0.001 0.001 0.001
- link motor3_link: geometry collision mesh filename=package://mara_description/meshes/MARA_T30.dae scale=0.001 0.001 0.001; visual mesh filename=package://mara_description/meshes/MARA_T30.dae scale=0.001 0.001 0.001
- link motor4_link: geometry collision mesh filename=package://mara_description/meshes/MARA_Link2.dae scale=0.001 0.001 0.001; visual mesh filename=package://mara_description/meshes/MARA_Link2.dae scale=0.001 0.001 0.001
- link motor5_cover: geometry collision mesh filename=package://mara_description/meshes/MARA_T5.4_black.dae scale=0.001 0.001 0.001; visual mesh filename=package://mara_description/meshes/MARA_T5.4_black.dae scale=0.001 0.001 0.001
- link motor5_link: geometry collision mesh filename=package://mara_description/meshes/MARA_T5.4.dae scale=0.001 0.001 0.001; visual mesh filename=package://mara_description/meshes/MARA_T5.4.dae scale=0.001 0.001 0.001
- link motor6_link: geometry collision mesh filename=package://mara_description/meshes/MARA_GripperAdapter.dae scale=0.001 0.001 0.001; visual mesh filename=package://mara_description/meshes/MARA_GripperAdapter.dae scale=0.001 0.001 0.001
- link table: geometry collision box size=1.5 1 0.05; visual mesh filename=package://mara_description/urdf/table.obj scale=0.1 0.1 0.58

Commit message: fixing issues with gripper links

File: mara_description/urdf/mara.urdf.xacro (robot description, xacro)
@@ -45,5 +45,5 @@
           <mesh filename="package://mara_description/meshes/Base.dae" scale="0.001 0.001 0.001"/>
         </geometry>
-        <material name="Gazebo/Grey">
+        <material name="Gazebo/Black">
           <color rgba="0. 0. 0. 1"/>
           <texture filename="package://mara_description/material/gazebo.material" />
@@ -58,5 +58,5 @@
     </link>
     <gazebo reference="${prefix}base_robot">
-      <material>Gazebo/Grey</material>
+      <material>Gazebo/Black</material>
       <selfCollide>True</selfCollide>
     </gazebo>

File: mara_description/urdf/mara_robot_camera_top.urdf (robot description, URDF)
Before this commit: robot mara, 24 links, 23 joints
Links:
- added link robotiq_adapter_link, mass 0.22652; collision mesh filename=package://robotiq_85_gripper_description/meshes/hros_roboti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 scale=0.001 0.001 0.001; visual mesh filename=package://robotiq_85_gripper_description/meshes/hros_roboti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 scale=0.001 0.001 0.001
- link table: geometry collision box size=1.5 1 0.05; visual mesh filename=model://mara_description/urdf/table.obj scale=0.1 0.1 0.58
Joints:
- added joint base_adapter_to_base_robotiq_joint: type fixed, parent robotiq_adapter_link, child robotiq_arg2f_base_link, origin xyz= 0 0 0.03653 rpy=0 0 0
- joint end_effector_adapter_to_robotiq: child robotiq_arg2f_base_link -> robotiq_adapter_link
- joint left_inner_knuckle_joint: limit lower=0 upper=0.87 effort=1000 velocity=2.0 -> lower=0 upper=0.78 effort=1000 velocity=2.0
- joint left_outer_finger_joint: limit lower=0.1 upper=0.875 effort=1000 velocity=2.0 -> lower=-0.875 upper=-0.0075 effort=1000 velocity=2.0
- joint left_outer_knuckle_joint: limit lower=0 upper=0.875 effort=1000 velocity=2.0 -> lower=0 upper=0.78 effort=1000 velocity=2.0
- joint right_inner_knuckle_joint: limit lower=0 upper=0.87 effort=1000 velocity=2.0 -> lower=0 upper=0.78 effort=1000 velocity=2.0
- joint right_outer_finger_joint: limit lower=0.1 upper=0.875 effort=1000 velocity=2.0 -> lower=-0.875 upper=-0.0075 effort=1000 velocity=2.0
- joint right_outer_knuckle_joint: limit lower=0 upper=0.875 effort=1000 velocity=2.0 -> lower=0 upper=0.78 effort=1000 velocity=2.0

File: mara_description/urdf/mara_robot_camera_top.urdf.xacro (robot description, xacro)
@@ -7,10 +7,10 @@
   <xacro:include filename="$(find mara_description)/urdf/mara.urdf.xacro" />
   <!-- robotiq 140 gripper -->
-  <xacro:include filename="$(find robotiq_140_gripper_description)/urdf/robotiq_gripper.urdf.xacro" />
+  <xacro:include filename="$(find robotiq_140_gripper_description)/urdf/robotiq_140.urdf.xacro" />
   <!-- <xacro:include filename="$(find mara_description)/urdf/camera_top.urdf.xacro" /> -->
   <xacro:include filename="$(find mara_description)/urdf/table.urdf.xacro" />
   <!-- arm -->
   <xacro:mara_robot prefix="" joint_limited="false"/>
-  <xacro:robotiq_gripper prefix="" />
+  <xacro:robotiq_gripper prefix="mara" />
   <!-- <xacro:mara_camera_top prefix="" /> -->
   <xacro:table prefix="" />
@@ -19,5 +19,5 @@
     <origin rpy="0 0 1.57" xyz=" 0 0 0.04659"/>
     <parent link="motor6_link"/>
-    <child link="robotiq_arg2f_base_link"/>
+    <child link="robotiq_adapter_link"/>
   </joint>
   <joint name="world_to_table_joint" type="fixed">

File: robotiq_140_gripper_description/urdf/module_gripper.urdf.xacro (robot description, xacro)
@@ -4,5 +4,5 @@
   <!-- robotiq hande_gripper -->
   <xacro:include filename="$(find robotiq_140_gripper_description)/urdf/robotiq_140.urdf.xacro" />
-  <xacro:robotiq_gripper prefix=""/>
+  <xacro:robotiq_gripper prefix="robotiq_140"/>
   <link name="world" />
   <joint name="world_to_hande_joint" type="fixed">

File: robotiq_140_gripper_description/urdf/robotiq_140.urdf.xacro (robot description, xacro)
@@ -362,6 +362,6 @@
       <joint name="left_inner_finger_knuckle_joint" type="revolute">
         <pose frame="">0 0.006 -0.018 0 0 0</pose>
-        <parent>robotiq_140::left_inner_knuckle</parent>
-        <child>robotiq_140::left_inner_finger</child>
+        <parent>${prefix}::left_inner_knuckle</parent>
+        <child>${prefix}::left_inner_finger</child>
         <axis>
           <xyz>1 0 0</xyz>
@@ -376,6 +376,6 @@
       <joint name="right_inner_finger_knuckle_joint" type="revolute">
         <pose frame="">0 0.006 -0.018 0 0 0</pose>
-        <parent>robotiq_140::right_inner_knuckle</parent>
-        <child>robotiq_140::right_inner_finger</child>
+        <parent>${prefix}::right_inner_knuckle</parent>
+        <child>${prefix}::right_inner_finger</child>
         <axis>
           <xyz>-1 0 0</xyz>

File: robotiq_85_gripper_description/urdf/module_gripper.urdf.xacro (robot description, xacro)
@@ -4,5 +4,5 @@
   <!-- robotiq hande_gripper -->
   <xacro:include filename="$(find robotiq_85_gripper_description)/urdf/robotiq_85.urdf.xacro" />
-  <xacro:robotiq_85 prefix=""/>
+  <xacro:robotiq_85 prefix="robotiq85"/>
   <link name="world" />
   <joint name="world_to_hande_joint" type="fixed">

File: robotiq_85_gripper_description/urdf/robotiq_85.urdf.xacro (robot description, xacro)
@@ -332,6 +332,6 @@
       <joint name="left_finger_joint2" type="revolute">
         <pose frame="">0.017901 0 0.00651469 0 0 0</pose>
-        <parent>robotiq85::robotiq_85_left_inner_finger_link</parent>
-        <child>robotiq85::robotiq_85_left_finger_link</child>
+        <parent>${prefix}::robotiq_85_left_inner_finger_link</parent>
+        <child>${prefix}::robotiq_85_left_finger_link</child>
         <axis>
           <xyz>0 -1 0</xyz>
@@ -346,6 +346,6 @@
       <joint name="right_finger_joint2" type="revolute">
         <pose frame="">0.017901 0 0.00651469 0 0 0</pose>
-        <parent>robotiq85::robotiq_85_right_inner_finger_link</parent>
-        <child>robotiq85::robotiq_85_right_finger_link</child>
+        <parent>${prefix}::robotiq_85_right_inner_finger_link</parent>
+        <child>${prefix}::robotiq_85_right_finger_link</child>
         <axis>
           <xyz>0 1 0</xyz>
