Commit message: adding ee_link_distance param

File: mara_description/urdf/mara.urdf.xacro (robot description, xacro)
@@ -6,5 +6,5 @@
   <xacro:include filename="$(find mara_description)/urdf/mara.transmission.xacro" />
   <xacro:include filename="$(find mara_description)/urdf/mara_gazebo.urdf.xacro" />
-  <xacro:macro name="mara_robot"  params="prefix joint_limited">
+  <xacro:macro name="mara_robot"  params="prefix ee_link_distance">
     <link name="${prefix}base_link">
       <inertial>
@@ -379,5 +379,5 @@
     </joint>
     <joint name="${prefix}ee_link" type="fixed">
-      <origin rpy="0 -1.57 0" xyz="0 0.0 0.24"/>
+      <origin rpy="0 -1.57 0" xyz="0 0.0 ${ee_link_distance}"/> <!-- 0.24 -->
       <parent link="${prefix}motor6_link"/>
       <child link="${prefix}ee_link"/>
@@ -385,5 +385,5 @@
     <link name="${prefix}tool0"/>
     <joint name="${prefix}${prefix}motor6_link-tool0_fixed_joint" type="fixed">
-      <origin rpy="0 -1.57 0" xyz="0 0.0 0.24"/>
+      <origin rpy="0 -1.57 0" xyz="0 0.0 ${ee_link_distance}"/>
       <parent link="${prefix}${prefix}motor6_link"/>
       <child link="${prefix}tool0"/>

File: mara_description/urdf/mara_robot_gripper_140.urdf.xacro (robot description, xacro)
@@ -11,5 +11,5 @@
   <xacro:include filename="$(find mara_description)/urdf/table.urdf.xacro" />
   <!-- arm -->
-  <xacro:mara_robot prefix="" joint_limited="false"/>
+  <xacro:mara_robot prefix="" ee_link_distance="0.24"/>
   <xacro:robotiq_gripper prefix="mara" />
   <!-- <xacro:mara_camera_top prefix="" /> -->

File: mara_description/urdf/mara_robot_gripper_85.urdf (robot description, URDF)
Before this commit: robot mara, 24 links, 23 joints
Joints:
- joint ee_link: origin xyz=0 0.0 0.24 rpy=0 -1.57 0 -> xyz=0 0.0 0.165 rpy=0 -1.57 0
- joint motor6_link-tool0_fixed_joint: origin xyz=0 0.0 0.24 rpy=0 -1.57 0 -> xyz=0 0.0 0.165 rpy=0 -1.57 0

File: mara_description/urdf/mara_robot_gripper_85.urdf.xacro (robot description, xacro)
@@ -10,5 +10,5 @@
   <xacro:include filename="$(find mara_description)/urdf/table.urdf.xacro" />
   <!-- arm -->
-  <xacro:mara_robot prefix="" joint_limited="false"/>
+  <xacro:mara_robot prefix="" ee_link_distance="0.165"/>
   <xacro:robotiq_85 prefix="mara" />
   <xacro:table prefix="" />

File: mara_description/urdf/mara_robot_gripper_hande.urdf (robot description, URDF)
Before this commit: robot mara, 18 links, 17 joints
Joints:
- joint ee_link: origin xyz=0 0.0 0.24 rpy=0 -1.57 0 -> xyz=0 0.0 0.18 rpy=0 -1.57 0
- joint motor6_link-tool0_fixed_joint: origin xyz=0 0.0 0.24 rpy=0 -1.57 0 -> xyz=0 0.0 0.18 rpy=0 -1.57 0

File: mara_description/urdf/mara_robot_gripper_hande.urdf.xacro (robot description, xacro)
@@ -10,5 +10,5 @@
   <xacro:include filename="$(find mara_description)/urdf/table.urdf.xacro" />
   <!-- arm -->
-  <xacro:mara_robot prefix="" joint_limited="false"/>
+  <xacro:mara_robot prefix="" ee_link_distance="0.18"/>
   <xacro:robotiq_hande prefix="mara" />
   <xacro:table prefix="" />

Commit message: add blue point

File: mara_description/urdf/mara.urdf.xacro (robot description, xacro)
@@ -305,4 +305,12 @@
     </gazebo>
     <link name="${prefix}ee_link">
+      <visual>
+        <geometry>
+          <sphere radius="0.01"/>
+        </geometry>
+        <material name="Gazebo/Grey">
+          <color rgba="0. 0. 0. 1"/>
+        </material>
+      </visual>
     </link>
     <gazebo reference="${prefix}ee_link">

File: mara_description/urdf/mara_robot_gripper_140.urdf (robot description, URDF)
Before this commit: robot mara, 24 links, 23 joints
Links:
- link ee_link: geometry visual sphere radius=0.01

Commit message: Update URDFs

File: mara_description/urdf/mara.urdf.xacro (robot description, xacro)
@@ -20,5 +20,4 @@
         <material name="Gazebo/Grey">
           <color rgba="0. 0. 0. 1"/>
-          <texture filename="package://mara_description/material/gazebo.material" />
         </material>
       </visual>
@@ -47,5 +46,4 @@
         <material name="Gazebo/Black">
           <color rgba="0. 0. 0. 1"/>
-          <texture filename="package://mara_description/material/gazebo.material" />
       </material>
       </visual>
@@ -74,5 +72,4 @@
         <material name="Gazebo/White">
           <color rgba="0. 0. 0. 1"/>
-          <texture filename="package://mara_description/material/gazebo.material" />
         </material>
       </visual>
@@ -101,5 +98,4 @@
         <material name="Gazebo/Black">
           <color rgba="0. 0. 0. 1"/>
-          <texture filename="package://mara_description/material/gazebo.material" />
         </material>
       </visual>
@@ -128,5 +124,4 @@
         <material name="Gazebo/Black">
           <color rgba="0. 0. 0. 1"/>
-          <texture filename="package://mara_description/material/gazebo.material" />
         </material>
       </visual>
@@ -155,5 +150,4 @@
         <material name="Gazebo/White">
           <color rgba="0. 0. 0. 1"/>
-          <texture filename="package://mara_description/material/gazebo.material" />
         </material>
       </visual>
@@ -182,5 +176,4 @@
         <material name="Gazebo/Black">
           <color rgba="0. 0. 0. 1"/>
-          <texture filename="package://mara_description/material/gazebo.material" />
         </material>
       </visual>
@@ -209,5 +202,4 @@
         <material name="Gazebo/Black">
           <color rgba="0. 0. 0. 1"/>
-          <texture filename="package://mara_description/material/gazebo.material" />
         </material>
       </visual>
@@ -236,5 +228,4 @@
         <material name="Gazebo/White">
           <color rgba="0. 0. 0. 1"/>
-          <texture filename="package://mara_description/material/gazebo.material" />
         </material>
       </visual>
@@ -263,5 +254,4 @@
         <material name="Gazebo/Black">
           <color rgba="0. 0. 0. 1"/>
-          <texture filename="package://mara_description/material/gazebo.material" />
         </material>
       </visual>
@@ -290,5 +280,4 @@
         <material name="Gazebo/Black">
           <color rgba="0. 0. 0. 1"/>
-          <texture filename="package://mara_description/material/gazebo.material" />
       </material>
       </visual>

File: mara_description/urdf/mara_gazebo.urdf.xacro (robot description, xacro)
@@ -14,12 +14,5 @@
     		<joint_name>motor5</joint_name>
         <joint_name>motor6</joint_name>
-        <joint_name>left_inner_knuckle_joint</joint_name>
-        <joint_name>left_outer_knuckle_joint</joint_name>
-        <joint_name>left_outer_finger_joint</joint_name>
-        <joint_name>left_inner_finger_joint</joint_name>
-        <joint_name>right_inner_knuckle_joint</joint_name>
-        <joint_name>right_outer_knuckle_joint</joint_name>
-        <joint_name>right_outer_finger_joint</joint_name>
-        <joint_name>right_inner_finger_joint</joint_name>
+        <joint_name>joint_finger</joint_name>
     	</plugin>
       <plugin name="hros_actuation_servomotor_000000000001" filename="libmara_gazebo_joint_plugin.so">

File: mara_description/urdf/table.urdf.xacro (robot description, xacro)
@@ -14,9 +14,8 @@
         <origin rpy="0 0 0" xyz="0 0 0.6"/>
         <geometry>
-  				<mesh filename="model://mara_description/urdf/table.obj" scale="1.5 1 0.05"/>
+  				<mesh filename="package://mara_description/urdf/table.obj" scale="1.5 1 0.05"/>
         </geometry>
          <material name="brown">
            <color rgba="0.63 0.16 0.16 1"/>
-          <texture filename="model://mara_description/material/gazebo.material" />
         </material>
       </visual>
@@ -30,5 +29,5 @@
         <origin rpy="0 0 0" xyz="-0.65 -0.4 0.29"/>
         <geometry>
-  	    <mesh filename="model://mara_description/urdf/table.obj" scale="0.1 0.1 0.58"/>
+  	    <mesh filename="package://mara_description/urdf/table.obj" scale="0.1 0.1 0.58"/>
         </geometry>
   	  <material name="framemat0"/>
@@ -37,5 +36,5 @@
         <origin rpy="0 0 0" xyz="-0.65 0.4 0.29"/>
         <geometry>
-          <mesh filename="model://mara_description/urdf/table.obj" scale="0.1 0.1 0.58"/>
+          <mesh filename="package://mara_description/urdf/table.obj" scale="0.1 0.1 0.58"/>
         </geometry>
   	  <material name="framemat0"/>
@@ -44,5 +43,5 @@
         <origin rpy="0 0 0" xyz="0.65 -0.4 0.29"/>
         <geometry>
-          <mesh filename="model://mara_description/urdf/table.obj" scale="0.1 0.1 0.58"/>
+          <mesh filename="package://mara_description/urdf/table.obj" scale="0.1 0.1 0.58"/>
         </geometry>
   	  <material name="framemat0"/>
@@ -51,5 +50,5 @@
         <origin rpy="0 0 0" xyz="0.65 0.4 0.29"/>
         <geometry>
-          <mesh filename="model://mara_description/urdf/table.obj" scale="0.1 0.1 0.58"/>
+          <mesh filename="package://mara_description/urdf/table.obj" scale="0.1 0.1 0.58"/>
         </geometry>
       </visual>

Commit message: orient ee_link axes same as motors

File: mara_description/urdf/mara.urdf.xacro (robot description, xacro)
@@ -376,5 +376,5 @@
     </joint>
     <joint name="${prefix}ee_link" type="fixed">
-      <origin rpy="0 -1.57 0" xyz="0 0.0 ${ee_link_distance}"/> <!-- 0.24 -->
+      <origin rpy="0 0 0" xyz="0 0.0 ${ee_link_distance}"/> <!-- 0.24 -->
       <parent link="${prefix}motor6_link"/>
       <child link="${prefix}ee_link"/>
@@ -382,5 +382,5 @@
     <link name="${prefix}tool0"/>
     <joint name="${prefix}${prefix}motor6_link-tool0_fixed_joint" type="fixed">
-      <origin rpy="0 -1.57 0" xyz="0 0.0 ${ee_link_distance}"/>
+      <origin rpy="0 0 0" xyz="0 0.0 ${ee_link_distance}"/>
       <parent link="${prefix}${prefix}motor6_link"/>
       <child link="${prefix}tool0"/>

File: mara_description/urdf/mara_robot_gripper_140.urdf (robot description, URDF)
Before this commit: robot mara, 24 links, 23 joints
Joints:
- joint ee_link: origin xyz=0 0.0 0.24 rpy=0 -1.57 0 -> xyz=0 0.0 0.24 rpy=0 0 0
- joint motor6_link-tool0_fixed_joint: origin xyz=0 0.0 0.24 rpy=0 -1.57 0 -> xyz=0 0.0 0.24 rpy=0 0 0

Commit message: Fixing inertias, center of mass, limits and efforts

File: mara_description/urdf/mara.urdf.xacro (robot description, xacro)
@@ -37,5 +37,5 @@
         <origin rpy="0 0 0" xyz="8.625E-08 -4.6583E-06 0.03145"/>
         <mass value="7.033"/>
-        <inertia ixx="0.1478344" ixy="-0.00001" ixz="0.0" iyy="0.14782335" iyz="0.0" izz="0.29471799"/>
+        <inertia ixx="0.1478344" ixy="0.00001" ixz="0.0" iyy="0.14782335" iyz="0.0" izz="0.29471799"/>
       </inertial>
       <visual>
@@ -45,6 +45,6 @@
         </geometry>
         <material name="Gazebo/Black">
-          <color rgba="0. 0. 0. 1"/>
-      </material>
+          <color rgba="1. 0. 0. 1.0"/>
+        </material>
       </visual>
       <collision>
@@ -61,7 +61,7 @@
     <link name="${prefix}motor1_link">
       <inertial>
-        <origin rpy="0 0 0" xyz="8.625E-08 -4.6583E-06 0.03145"/>
-        <mass value="5.8"/>
-        <inertia ixx="0.10105893" ixy="0.000211" ixz="-0.004" iyy="0.09386624" iyz="-0.01698537" izz="0.01449937"/>
+        <origin rpy="0 0 0" xyz="0.02066 0 0.12051"/>
+        <mass value="5.6"/>
+        <inertia ixx="0.0200769278" ixy="-7.72273E-006" ixz="0.0050158708" iyy="0.0257088151" iyz="5.49229E-006" izz="0.0120821377"/>
       </inertial>
       <visual>
@@ -88,6 +88,6 @@
       <inertial>
         <origin rpy="0 0 0" xyz="8.625E-08 -4.6583E-06 0.03145"/>
-        <mass value="5.8"/>
-        <inertia ixx="0.10105893" ixy="0.000211" ixz="-0.004" iyy="0.09386624" iyz="-0.01698537" izz="0.01449937"/>
+        <mass value="0.0"/>
+        <inertia ixx="0.0" ixy="0.0" ixz="0.0" iyy="0.0" iyz="0.0" izz="0.0"/>
       </inertial>
       <visual>
@@ -113,7 +113,7 @@
     <link name="${prefix}motor2_link">
       <inertial>
-        <origin rpy="0 0 0" xyz="8.625E-08 -4.6583E-06 0.03145"/>
-        <mass value="1.03237"/>
-        <inertia ixx="0.014865226" ixy="0.0" ixz="0.0" iyy="0.01557" iyz="0.00071" izz="0.00092"/>
+        <origin rpy="0 0 0" xyz="-0.01665 0.0 0.09639"/>
+        <mass value="1.236"/>
+        <inertia ixx="0.0079614839" ixy="0.000000037" ixz="-0.0003203013" iyy="0.007135338" iyz="-0.000001062" izz="0.001111114"/>
       </inertial>
       <visual>
@@ -139,7 +139,7 @@
     <link name="${prefix}motor3_link">
       <inertial>
-        <origin rpy="0 0 0" xyz="8.625E-08 -4.6583E-06 0.03145"/>
-        <mass value="3.8"/>
-        <inertia ixx="0.04517" ixy="0.00002" ixz="0.0" iyy="0.01587" iyz="0.01444" izz="0.03303"/>
+        <origin rpy="0 0 0" xyz="-0.08963 0.0 0.0403"/>
+        <mass value="3.95"/>
+        <inertia ixx="0.0115136615" ixy="-1.231046E-005" ixz="-0.003148516" iyy="0.0149841676" iyz="-8.81378E-006" izz="0.0070387807"/>
       </inertial>
       <visual>
@@ -166,6 +166,6 @@
       <inertial>
         <origin rpy="0 0 0" xyz="8.625E-08 -4.6583E-06 0.03145"/>
-        <mass value="3.8"/>
-        <inertia ixx="0.04517" ixy="0.00002" ixz="0.0" iyy="0.01587" iyz="0.01444" izz="0.03303"/>
+        <mass value="0.0"/>
+        <inertia ixx="0.0" ixy="0.0" ixz="0.0" iyy="0.0" iyz="0.0" izz="0.0"/>
       </inertial>
       <visual>
@@ -191,7 +191,7 @@
     <link name="${prefix}motor4_link">
       <inertial>
-        <origin rpy="0 0 0" xyz="8.625E-08 -4.6583E-06 0.03145"/>
-        <mass value="1.1"/>
-        <inertia ixx="0.01464" ixy="0.0" ixz="0.0" iyy="0.00895" iyz="-0.00631" izz="0.00725"/>
+        <origin rpy="0 0 0" xyz="0.06357 0.0 0.05698"/>
+        <mass value="1.258"/>
+        <inertia ixx="0.005919676" ixy="0.000000923" ixz="0.0022280208" iyy="0.0068807393" iyz="6.1373E-007" izz="0.00257485"/>
       </inertial>
       <visual>
@@ -217,7 +217,7 @@
     <link name="${prefix}motor5_link">
       <inertial>
-        <origin rpy="0 0 0" xyz="8.625E-08 -4.6583E-06 0.03145"/>
-        <mass value="2.9"/>
-        <inertia ixx="0.03406" ixy="0.0" ixz="0.0" iyy="0.01066" iyz="0.00989" izz="0.02563"/>
+        <origin rpy="0 0 0" xyz="-0.09105 0.0 0.03676"/>
+        <mass value="2.85"/>
+        <inertia ixx="0.0072829492" ixy="3.77994E-006" ixz="-0.0015682105" iyy="0.0098263499" iyz="2.52745E-006" izz="0.0045615321"/>
       </inertial>
       <visual>
@@ -244,6 +244,6 @@
       <inertial>
         <origin rpy="0 0 0" xyz="8.625E-08 -4.6583E-06 0.03145"/>
-        <mass value="2.9"/>
-        <inertia ixx="0.03406" ixy="0.0" ixz="0.0" iyy="0.01066" iyz="0.00989" izz="0.02563"/>
+        <mass value="0.0"/>
+        <inertia ixx="0.0" ixy="0.0" ixz="0.0" iyy="0.0" iyz="0.0" izz="0.0"/>
       </inertial>
       <visual>
@@ -269,7 +269,7 @@
     <link name="${prefix}motor6_link">
       <inertial>
-        <origin rpy="0 0 0" xyz="8.625E-08 -4.6583E-06 0.03145"/>
-        <mass value="2.9"/>
-        <inertia ixx="0.0005" ixy="0.0" ixz="0.0" iyy="0.0005" iyz="0.0000" izz="0.0003"/>
+        <origin rpy="0 0 0" xyz="0.0 0.0 -0.0173"/>
+        <mass value="0.14"/>
+        <inertia ixx="9.22e-05" ixy="6.35e-7" ixz="2.00e-11" iyy="9.73e-5" iyz="2.36e-9" izz="1.77e-4"/>
       </inertial>
       <visual>
@@ -280,5 +280,5 @@
         <material name="Gazebo/Black">
           <color rgba="0. 0. 0. 1"/>
-      </material>
+        </material>
       </visual>
       <collision>
@@ -309,5 +309,5 @@
       <child link="${prefix}motor1_link"/>
       <axis xyz="0 0 -1"/>
-      <limit effort="330.0" lower="-3.1416" upper="3.1416" velocity="3.1416"/>
+      <limit effort="104.0" lower="-3.1416" upper="3.1416" velocity="1.57"/>
       <dynamics damping="0" friction="0"/>
     </joint>
@@ -322,5 +322,5 @@
       <child link="${prefix}motor2_link"/>
       <axis xyz="-1 0 0"/>
-      <limit effort="330.0" lower="-3.1416" upper="3.1416" velocity="3.1416"/>
+      <limit effort="104.0" lower="-2.35" upper="2.35" velocity="1.57"/>
       <dynamics damping="0" friction="0"/>
     </joint>
@@ -330,5 +330,5 @@
       <child link="${prefix}motor3_link"/>
       <axis xyz="1 0 0"/>
-      <limit effort="330.0" lower="-3.1416" upper="3.1416" velocity="3.1416"/>
+      <limit effort="69" lower="-2.61" upper="2.61" velocity="1.57"/>
       <dynamics damping="0" friction="0"/>
     </joint>
@@ -343,5 +343,5 @@
       <child link="${prefix}motor4_link"/>
       <axis xyz="0 0 -1"/>
-      <limit effort="330.0" lower="-3.1416" upper="3.1416" velocity="3.1416"/>
+      <limit effort="69" lower="-3.14" upper="3.14" velocity="1.57"/>
       <dynamics damping="0" friction="0"/>
     </joint>
@@ -351,5 +351,5 @@
       <child link="${prefix}motor5_link"/>
       <axis xyz="1 0 0"/>
-      <limit effort="330.0" lower="-3.1416" upper="3.1416" velocity="3.1416"/>
+      <limit effort="34" lower="-2.56" upper="2.56" velocity="1.57"/>
       <dynamics damping="0" friction="0"/>
     </joint>
@@ -364,5 +364,5 @@
       <child link="${prefix}motor6_link"/>
       <axis xyz="0 0 -1"/>
-      <limit effort="330.0" lower="-3.1416" upper="3.1416" velocity="3.1416"/>
+      <limit effort="34" lower="-3.14" upper="3.14" velocity="1.57"/>
       <dynamics damping="0" friction="0"/>
     </joint>

File: mara_description/urdf/mara_robot_gripper_140.urdf (robot description, URDF)
Before this commit: robot mara, 25 links, 24 joints
Links:
- link motor1_cover: mass 5.8 -> 0.0
- link motor1_link: mass 5.8 -> 5.6
- link motor2_link: mass 1.03237 -> 1.236
- link motor3_cover: mass 3.8 -> 0.0
- link motor3_link: mass 3.8 -> 3.95
- link motor4_link: mass 1.1 -> 1.258
- link motor5_cover: mass 2.9 -> 0.0
- link motor5_link: mass 2.9 -> 2.85
- link motor6_link: mass 2.9 -> 0.14
Joints:
- joint motor1: limit lower=-3.1416 upper=3.1416 effort=330.0 velocity=3.1416 -> lower=-3.1416 upper=3.1416 effort=104.0 velocity=1.57
- joint motor2: limit lower=-3.1416 upper=3.1416 effort=330.0 velocity=3.1416 -> lower=-2.35 upper=2.35 effort=104.0 velocity=1.57
- joint motor3: limit lower=-3.1416 upper=3.1416 effort=330.0 velocity=3.1416 -> lower=-2.61 upper=2.61 effort=69 velocity=1.57
- joint motor4: limit lower=-3.1416 upper=3.1416 effort=330.0 velocity=3.1416 -> lower=-3.14 upper=3.14 effort=69 velocity=1.57
- joint motor5: limit lower=-3.1416 upper=3.1416 effort=330.0 velocity=3.1416 -> lower=-2.56 upper=2.56 effort=34 velocity=1.57
- joint motor6: limit lower=-3.1416 upper=3.1416 effort=330.0 velocity=3.1416 -> lower=-3.14 upper=3.14 effort=34 velocity=1.57

File: mara_description/urdf/mara_robot_gripper_85.urdf (robot description, URDF)
Before this commit: robot mara, 25 links, 24 joints
Links:
- link motor1_cover: mass 5.8 -> 0.0
- link motor1_link: mass 5.8 -> 5.6
- link motor2_link: mass 1.03237 -> 1.236
- link motor3_cover: mass 3.8 -> 0.0
- link motor3_link: mass 3.8 -> 3.95
- link motor4_link: mass 1.1 -> 1.258
- link motor5_cover: mass 2.9 -> 0.0
- link motor5_link: mass 2.9 -> 2.85
- link motor6_link: mass 2.9 -> 0.14
Joints:
- joint motor1: limit lower=-3.1416 upper=3.1416 effort=330.0 velocity=3.1416 -> lower=-3.1416 upper=3.1416 effort=104.0 velocity=1.57
- joint motor2: limit lower=-3.1416 upper=3.1416 effort=330.0 velocity=3.1416 -> lower=-2.35 upper=2.35 effort=104.0 velocity=1.57
- joint motor3: limit lower=-3.1416 upper=3.1416 effort=330.0 velocity=3.1416 -> lower=-2.61 upper=2.61 effort=69 velocity=1.57
- joint motor4: limit lower=-3.1416 upper=3.1416 effort=330.0 velocity=3.1416 -> lower=-3.14 upper=3.14 effort=69 velocity=1.57
- joint motor5: limit lower=-3.1416 upper=3.1416 effort=330.0 velocity=3.1416 -> lower=-2.56 upper=2.56 effort=34 velocity=1.57
- joint motor6: limit lower=-3.1416 upper=3.1416 effort=330.0 velocity=3.1416 -> lower=-3.14 upper=3.14 effort=34 velocity=1.57

File: mara_description/urdf/mara_robot_gripper_hande.urdf (robot description, URDF)
Before this commit: robot mara, 19 links, 18 joints
Links:
- link motor1_cover: mass 5.8 -> 0.0
- link motor1_link: mass 5.8 -> 5.6
- link motor2_link: mass 1.03237 -> 1.236
- link motor3_cover: mass 3.8 -> 0.0
- link motor3_link: mass 3.8 -> 3.95
- link motor4_link: mass 1.1 -> 1.258
- link motor5_cover: mass 2.9 -> 0.0
- link motor5_link: mass 2.9 -> 2.85
- link motor6_link: mass 2.9 -> 0.14
Joints:
- joint motor1: limit lower=-3.1416 upper=3.1416 effort=330.0 velocity=3.1416 -> lower=-3.1416 upper=3.1416 effort=104.0 velocity=1.57
- joint motor2: limit lower=-3.1416 upper=3.1416 effort=330.0 velocity=3.1416 -> lower=-2.35 upper=2.35 effort=104.0 velocity=1.57
- joint motor3: limit lower=-3.1416 upper=3.1416 effort=330.0 velocity=3.1416 -> lower=-2.61 upper=2.61 effort=69 velocity=1.57
- joint motor4: limit lower=-3.1416 upper=3.1416 effort=330.0 velocity=3.1416 -> lower=-3.14 upper=3.14 effort=69 velocity=1.57
- joint motor5: limit lower=-3.1416 upper=3.1416 effort=330.0 velocity=3.1416 -> lower=-2.56 upper=2.56 effort=34 velocity=1.57
- joint motor6: limit lower=-3.1416 upper=3.1416 effort=330.0 velocity=3.1416 -> lower=-3.14 upper=3.14 effort=34 velocity=1.57

File: mara_description/urdf/mara_robot_gripper_ur_j.urdf (robot description, URDF)
Before this commit: robot mara, 18 links, 17 joints
Links:
- link motor1_cover: mass 5.8 -> 0.0
- link motor1_link: mass 5.8 -> 5.6
- link motor2_link: mass 1.03237 -> 1.236
- link motor3_cover: mass 3.8 -> 0.0
- link motor3_link: mass 3.8 -> 3.95
- link motor4_link: mass 1.1 -> 1.258
- link motor5_cover: mass 2.9 -> 0.0
- link motor5_link: mass 2.9 -> 2.85
- link motor6_link: mass 2.9 -> 0.14
Joints:
- joint motor1: limit lower=-3.1416 upper=3.1416 effort=330.0 velocity=3.1416 -> lower=-3.1416 upper=3.1416 effort=104.0 velocity=1.57
- joint motor2: limit lower=-3.1416 upper=3.1416 effort=330.0 velocity=3.1416 -> lower=-2.35 upper=2.35 effort=104.0 velocity=1.57
- joint motor3: limit lower=-3.1416 upper=3.1416 effort=330.0 velocity=3.1416 -> lower=-2.61 upper=2.61 effort=69 velocity=1.57
- joint motor4: limit lower=-3.1416 upper=3.1416 effort=330.0 velocity=3.1416 -> lower=-3.14 upper=3.14 effort=69 velocity=1.57
- joint motor5: limit lower=-3.1416 upper=3.1416 effort=330.0 velocity=3.1416 -> lower=-2.56 upper=2.56 effort=34 velocity=1.57
- joint motor6: limit lower=-3.1416 upper=3.1416 effort=330.0 velocity=3.1416 -> lower=-3.14 upper=3.14 effort=34 velocity=1.57
