Commit message: Axis according ROS 2 and real one

File: mara_description/urdf/mara.urdf.xacro (robot description, xacro)
@@ -308,5 +308,5 @@
       <parent link="${prefix}base_robot"/>
       <child link="${prefix}motor1_link"/>
-      <axis xyz="0 0 -1"/>
+      <axis xyz="0 0 1"/>
       <limit effort="104.0" lower="-3.1416" upper="3.1416" velocity="1.57"/>
       <dynamics damping="0" friction="0"/>
@@ -321,5 +321,5 @@
       <parent link="${prefix}motor1_link"/>
       <child link="${prefix}motor2_link"/>
-      <axis xyz="-1 0 0"/>
+      <axis xyz="1 0 0"/>
       <limit effort="104.0" lower="-2.35" upper="2.35" velocity="1.57"/>
       <dynamics damping="0" friction="0"/>
@@ -329,5 +329,5 @@
       <parent link="${prefix}motor2_link"/>
       <child link="${prefix}motor3_link"/>
-      <axis xyz="1 0 0"/>
+      <axis xyz="-1 0 0"/>
       <limit effort="69" lower="-2.61" upper="2.61" velocity="1.57"/>
       <dynamics damping="0" friction="0"/>
@@ -342,5 +342,5 @@
       <parent link="${prefix}motor3_link"/>
       <child link="${prefix}motor4_link"/>
-      <axis xyz="0 0 -1"/>
+      <axis xyz="0 0 1"/>
       <limit effort="69" lower="-3.14" upper="3.14" velocity="1.57"/>
       <dynamics damping="0" friction="0"/>
@@ -350,5 +350,5 @@
       <parent link="${prefix}motor4_link"/>
       <child link="${prefix}motor5_link"/>
-      <axis xyz="1 0 0"/>
+      <axis xyz="-1 0 0"/>
       <limit effort="34" lower="-2.56" upper="2.56" velocity="1.57"/>
       <dynamics damping="0" friction="0"/>
@@ -363,5 +363,5 @@
       <parent link="${prefix}motor5_link"/>
       <child link="${prefix}motor6_link"/>
-      <axis xyz="0 0 -1"/>
+      <axis xyz="0 0 1"/>
       <limit effort="34" lower="-3.14" upper="3.14" velocity="1.57"/>
       <dynamics damping="0" friction="0"/>

File: mara_description/urdf/mara_robot_gripper_140.urdf (robot description, URDF)
Before this commit: robot mara, 25 links, 24 joints
Joints:
- joint motor1: axis 0 0 -1 -> 0 0 1
- joint motor2: axis -1 0 0 -> 1 0 0
- joint motor3: axis 1 0 0 -> -1 0 0
- joint motor4: axis 0 0 -1 -> 0 0 1
- joint motor5: axis 1 0 0 -> -1 0 0
- joint motor6: axis 0 0 -1 -> 0 0 1

File: mara_description/urdf/mara_robot_gripper_85.urdf (robot description, URDF)
Before this commit: robot mara, 25 links, 24 joints
Joints:
- joint motor1: axis 0 0 -1 -> 0 0 1
- joint motor2: axis -1 0 0 -> 1 0 0
- joint motor3: axis 1 0 0 -> -1 0 0
- joint motor4: axis 0 0 -1 -> 0 0 1
- joint motor5: axis 1 0 0 -> -1 0 0
- joint motor6: axis 0 0 -1 -> 0 0 1

File: mara_description/urdf/mara_robot_gripper_hande.urdf (robot description, URDF)
Before this commit: robot mara, 19 links, 18 joints
Joints:
- joint motor1: axis 0 0 -1 -> 0 0 1
- joint motor2: axis -1 0 0 -> 1 0 0
- joint motor3: axis 1 0 0 -> -1 0 0
- joint motor4: axis 0 0 -1 -> 0 0 1
- joint motor5: axis 1 0 0 -> -1 0 0
- joint motor6: axis 0 0 -1 -> 0 0 1

File: mara_description/urdf/mara_robot_gripper_ur_j.urdf (robot description, URDF)
Before this commit: robot mara, 18 links, 17 joints
Joints:
- joint motor1: axis 0 0 -1 -> 0 0 1
- joint motor2: axis -1 0 0 -> 1 0 0
- joint motor3: axis 1 0 0 -> -1 0 0
- joint motor4: axis 0 0 -1 -> 0 0 1
- joint motor5: axis 1 0 0 -> -1 0 0
- joint motor6: axis 0 0 -1 -> 0 0 1

Commit message: update adapters in mara_robot.urdf

File: mara_description/urdf/mara.urdf.xacro (robot description, xacro)
@@ -267,36 +267,25 @@
       <selfCollide>True</selfCollide>
     </gazebo>
+    <!-- dummy link with the required tags-->
     <link name="${prefix}motor6_link">
       <inertial>
-        <origin rpy="0 0 0" xyz="0.0 0.0 -0.0173"/>
-        <mass value="0.14"/>
-        <inertia ixx="9.22e-05" ixy="6.35e-7" ixz="2.00e-11" iyy="9.73e-5" iyz="2.36e-9" izz="1.77e-4"/>
-      </inertial>
-      <visual>
-        <origin rpy="0 0 0" xyz="0 0 0"/>
-        <geometry>
-          <mesh filename="package://mara_description/meshes/MARA_GripperAdapter.dae" scale="0.001 0.001 0.001"/>
-        </geometry>
-        <material name="Gazebo/Black">
-          <color rgba="0. 0. 0. 1"/>
-        </material>
-      </visual>
-      <collision>
-        <origin rpy="0 0 0" xyz="0 0 0"/>
-        <geometry>
-          <mesh filename="package://mara_description/meshes/MARA_GripperAdapter.dae" scale="0.001 0.001 0.001"/>
-        </geometry>
-      </collision>
-    </link>
-    <gazebo reference="${prefix}motor6_link">
-      <material>Gazebo/Black</material>
-      <selfCollide>True</selfCollide>
-    </gazebo>
-    <link name="${prefix}ee_link">
-    </link>
-    <gazebo reference="${prefix}ee_link">
-      <material>Gazebo/Blue</material>
-      <selfCollide>False</selfCollide>
-    </gazebo>
+        <origin rpy="0 0 0" xyz="0 0 0"/>
+        <mass value="0.00001"/>
+        <inertia ixx="0" ixy="0" ixz="0" iyy="0" iyz="0" izz="0"/>
+      </inertial>
+      <visual>
+        <origin rpy="0 0 0" xyz="0 0 0"/>
+        <geometry>
+          <sphere radius="0"/>
+        </geometry>
+      </visual>
+      <collision>
+        <origin rpy="0 0 0" xyz="0 0 0"/>
+        <geometry>
+          <sphere radius="0"/>
+        </geometry>
+      </collision>
+    </link>
+    <link name="${prefix}ee_link"/>
     <joint name="${prefix}joint_bases" type="fixed">
       <origin rpy="0 0 0" xyz="0 0 0.04"/>
@@ -368,5 +357,5 @@
     </joint>
     <joint name="${prefix}ee_link" type="fixed">
-      <origin rpy="0 -1.57 0" xyz="0 0.0 ${ee_link_distance}"/> <!-- 0.24 -->
+      <origin rpy="0 -1.57 0" xyz="0 0.0 ${ee_link_distance}"/>
       <parent link="${prefix}motor6_link"/>
       <child link="${prefix}ee_link"/>

File: mara_description/urdf/mara_robot.urdf (robot description, URDF)
Before this commit: robot mara, 14 links, 13 joints
Links:
- link motor6_link: mass 0.14 -> 0.00001; geometry collision sphere radius=0; visual sphere radius=0

Commit message: fix inertial values of the motors

File: mara_description/urdf/mara.urdf.xacro (robot description, xacro)
@@ -63,5 +63,5 @@
         <origin rpy="0 0 0" xyz="0.02066 0 0.12051"/>
         <mass value="5.6"/>
-        <inertia ixx="0.0200769278" ixy="-7.72273E-006" ixz="0.0050158708" iyy="0.0257088151" iyz="5.49229E-006" izz="0.0120821377"/>
+        <inertia ixx="0.0200769278" ixy="-7.72273E-006" ixz="-0.0050158708" iyy="0.0257088151" iyz="5.49229E-006" izz="0.0120821377"/>
       </inertial>
       <visual>
@@ -87,5 +87,5 @@
     <link name="${prefix}motor1_cover">
       <inertial>
-        <origin rpy="0 0 0" xyz="8.625E-08 -4.6583E-06 0.03145"/>
+        <origin rpy="0 0 0" xyz="0 0 0"/>
         <mass value="0.0"/>
         <inertia ixx="0.0" ixy="0.0" ixz="0.0" iyy="0.0" iyz="0.0" izz="0.0"/>
@@ -114,6 +114,6 @@
       <inertial>
         <origin rpy="0 0 0" xyz="-0.01665 0.0 0.09639"/>
-        <mass value="1.236"/>
-        <inertia ixx="0.0079614839" ixy="0.000000037" ixz="-0.0003203013" iyy="0.007135338" iyz="-0.000001062" izz="0.001111114"/>
+        <mass value="1.24"/>
+        <inertia ixx="0.0079614839" ixy="0.000000037" ixz="0.0003203013" iyy="0.007135338" iyz="-0.000001062" izz="0.001111114"/>
       </inertial>
       <visual>
@@ -139,7 +139,7 @@
     <link name="${prefix}motor3_link">
       <inertial>
-        <origin rpy="0 0 0" xyz="-0.08963 0.0 0.0403"/>
+        <origin rpy="0 0 0" xyz="-0.08963 0 0.0403"/>
         <mass value="3.95"/>
-        <inertia ixx="0.0115136615" ixy="-1.231046E-005" ixz="-0.003148516" iyy="0.0149841676" iyz="-8.81378E-006" izz="0.0070387807"/>
+        <inertia ixx="0.0115136615" ixy="-1.231046E-005" ixz="0.003148516" iyy="0.0149841676" iyz="-8.81378E-006" izz="0.0070387807"/>
       </inertial>
       <visual>
@@ -165,5 +165,5 @@
     <link name="${prefix}motor3_cover">
       <inertial>
-        <origin rpy="0 0 0" xyz="8.625E-08 -4.6583E-06 0.03145"/>
+        <origin rpy="0 0 0" xyz="0 0 0"/>
         <mass value="0.0"/>
         <inertia ixx="0.0" ixy="0.0" ixz="0.0" iyy="0.0" iyz="0.0" izz="0.0"/>
@@ -192,6 +192,6 @@
       <inertial>
         <origin rpy="0 0 0" xyz="0.06357 0.0 0.05698"/>
-        <mass value="1.258"/>
-        <inertia ixx="0.005919676" ixy="0.000000923" ixz="0.0022280208" iyy="0.0068807393" iyz="6.1373E-007" izz="0.00257485"/>
+        <mass value="1.26"/>
+        <inertia ixx="0.005919676" ixy="0.000000923" ixz="-0.0022280208" iyy="0.0068807393" iyz="6.1373E-007" izz="0.00257485"/>
       </inertial>
       <visual>
@@ -219,5 +219,5 @@
         <origin rpy="0 0 0" xyz="-0.09105 0.0 0.03676"/>
         <mass value="2.85"/>
-        <inertia ixx="0.0072829492" ixy="3.77994E-006" ixz="-0.0015682105" iyy="0.0098263499" iyz="2.52745E-006" izz="0.0045615321"/>
+        <inertia ixx="0.0072829492" ixy="3.77994E-006" ixz="0.0015682105" iyy="0.0098263499" iyz="2.52745E-006" izz="0.0045615321"/>
       </inertial>
       <visual>
@@ -243,5 +243,5 @@
     <link name="${prefix}motor5_cover">
       <inertial>
-        <origin rpy="0 0 0" xyz="8.625E-08 -4.6583E-06 0.03145"/>
+        <origin rpy="0 0 0" xyz="0 0 0"/>
         <mass value="0.0"/>
         <inertia ixx="0.0" ixy="0.0" ixz="0.0" iyy="0.0" iyz="0.0" izz="0.0"/>

File: mara_description/urdf/mara_robot.urdf (robot description, URDF)
Before this commit: robot mara, 14 links, 13 joints
Links:
- link motor2_link: mass 1.236 -> 1.24
- link motor4_link: mass 1.258 -> 1.26

File: mara_description/urdf/mara_robot_gripper_140.urdf (robot description, URDF)
Before this commit: robot mara, 26 links, 25 joints
Links:
- link motor2_link: mass 1.236 -> 1.24
- link motor4_link: mass 1.258 -> 1.26

File: mara_description/urdf/mara_robot_gripper_140_no_table.urdf (robot description, URDF)
Before this commit: robot mara, 25 links, 24 joints
Links:
- link motor2_link: mass 1.236 -> 1.24
- link motor4_link: mass 1.258 -> 1.26

File: mara_description/urdf/mara_robot_gripper_85.urdf (robot description, URDF)
Before this commit: robot mara, 26 links, 25 joints
Links:
- link motor2_link: mass 1.236 -> 1.24
- link motor4_link: mass 1.258 -> 1.26

File: mara_description/urdf/mara_robot_gripper_hande.urdf (robot description, URDF)
Before this commit: robot mara, 20 links, 19 joints
Links:
- link motor2_link: mass 1.236 -> 1.24
- link motor4_link: mass 1.258 -> 1.26

File: mara_description/urdf/reinforcement_learning/mara_robot_gripper_140_camera_run.urdf (robot description, URDF)
Before this commit: robot mara, 30 links, 29 joints
Links:
- link motor2_link: mass 1.236 -> 1.24
- link motor4_link: mass 1.258 -> 1.26

File: mara_description/urdf/reinforcement_learning/mara_robot_gripper_140_camera_train.urdf (robot description, URDF)
Before this commit: robot mara, 30 links, 29 joints
Links:
- link motor2_link: mass 1.236 -> 1.24
- link motor4_link: mass 1.258 -> 1.26

File: mara_description/urdf/reinforcement_learning/mara_robot_run.urdf (robot description, URDF)
Before this commit: robot mara, 12 links, 11 joints
Links:
- link motor2_link: mass 1.236 -> 1.24
- link motor4_link: mass 1.258 -> 1.26

File: mara_description/urdf/reinforcement_learning/mara_robot_train.urdf (robot description, URDF)
Before this commit: robot mara, 12 links, 11 joints
Links:
- link motor2_link: mass 1.236 -> 1.24
- link motor4_link: mass 1.258 -> 1.26

File: mara_description/urdf/reinforcement_learning/mara_run.urdf.xacro (robot description, xacro)
@@ -8,5 +8,5 @@
         <origin rpy="0 0 0" xyz="0.02066 0 0.12051"/>
         <mass value="5.6"/>
-        <inertia ixx="0.0200769278" ixy="-7.72273E-006" ixz="0.0050158708" iyy="0.0257088151" iyz="5.49229E-006" izz="0.0120821377"/>
+        <inertia ixx="0.0200769278" ixy="-7.72273E-006" ixz="-0.0050158708" iyy="0.0257088151" iyz="5.49229E-006" izz="0.0120821377"/>
       </inertial>
       <visual>
@@ -32,5 +32,5 @@
     <link name="${prefix}motor1_cover">
       <inertial>
-        <origin rpy="0 0 0" xyz="8.625E-08 -4.6583E-06 0.03145"/>
+        <origin rpy="0 0 0" xyz="0 0 0"/>
         <mass value="0.0"/>
         <inertia ixx="0.0" ixy="0.0" ixz="0.0" iyy="0.0" iyz="0.0" izz="0.0"/>
@@ -59,6 +59,6 @@
       <inertial>
         <origin rpy="0 0 0" xyz="-0.01665 0.0 0.09639"/>
-        <mass value="1.236"/>
-        <inertia ixx="0.0079614839" ixy="0.000000037" ixz="-0.0003203013" iyy="0.007135338" iyz="-0.000001062" izz="0.001111114"/>
+        <mass value="1.24"/>
+        <inertia ixx="0.0079614839" ixy="0.000000037" ixz="0.0003203013" iyy="0.007135338" iyz="-0.000001062" izz="0.001111114"/>
       </inertial>
       <visual>
@@ -84,7 +84,7 @@
     <link name="${prefix}motor3_link">
       <inertial>
-        <origin rpy="0 0 0" xyz="-0.08963 0.0 0.0403"/>
+        <origin rpy="0 0 0" xyz="-0.08963 0 0.0403"/>
         <mass value="3.95"/>
-        <inertia ixx="0.0115136615" ixy="-1.231046E-005" ixz="-0.003148516" iyy="0.0149841676" iyz="-8.81378E-006" izz="0.0070387807"/>
+        <inertia ixx="0.0115136615" ixy="-1.231046E-005" ixz="0.003148516" iyy="0.0149841676" iyz="-8.81378E-006" izz="0.0070387807"/>
       </inertial>
       <visual>
@@ -110,5 +110,5 @@
     <link name="${prefix}motor3_cover">
       <inertial>
-        <origin rpy="0 0 0" xyz="8.625E-08 -4.6583E-06 0.03145"/>
+        <origin rpy="0 0 0" xyz="0 0 0"/>
         <mass value="0.0"/>
         <inertia ixx="0.0" ixy="0.0" ixz="0.0" iyy="0.0" iyz="0.0" izz="0.0"/>
@@ -137,6 +137,6 @@
       <inertial>
         <origin rpy="0 0 0" xyz="0.06357 0.0 0.05698"/>
-        <mass value="1.258"/>
-        <inertia ixx="0.005919676" ixy="0.000000923" ixz="0.0022280208" iyy="0.0068807393" iyz="6.1373E-007" izz="0.00257485"/>
+        <mass value="1.26"/>
+        <inertia ixx="0.005919676" ixy="0.000000923" ixz="-0.0022280208" iyy="0.0068807393" iyz="6.1373E-007" izz="0.00257485"/>
       </inertial>
       <visual>
@@ -164,5 +164,5 @@
         <origin rpy="0 0 0" xyz="-0.09105 0.0 0.03676"/>
         <mass value="2.85"/>
-        <inertia ixx="0.0072829492" ixy="3.77994E-006" ixz="-0.0015682105" iyy="0.0098263499" iyz="2.52745E-006" izz="0.0045615321"/>
+        <inertia ixx="0.0072829492" ixy="3.77994E-006" ixz="0.0015682105" iyy="0.0098263499" iyz="2.52745E-006" izz="0.0045615321"/>
       </inertial>
       <visual>
@@ -188,5 +188,5 @@
     <link name="${prefix}motor5_cover">
       <inertial>
-        <origin rpy="0 0 0" xyz="8.625E-08 -4.6583E-06 0.03145"/>
+        <origin rpy="0 0 0" xyz="0 0 0"/>
         <mass value="0.0"/>
         <inertia ixx="0.0" ixy="0.0" ixz="0.0" iyy="0.0" iyz="0.0" izz="0.0"/>

File: mara_description/urdf/reinforcement_learning/mara_train.urdf.xacro (robot description, xacro)
@@ -8,5 +8,5 @@
         <origin rpy="0 0 0" xyz="0.02066 0 0.12051"/>
         <mass value="5.6"/>
-        <inertia ixx="0.0200769278" ixy="-7.72273E-006" ixz="0.0050158708" iyy="0.0257088151" iyz="5.49229E-006" izz="0.0120821377"/>
+        <inertia ixx="0.0200769278" ixy="-7.72273E-006" ixz="-0.0050158708" iyy="0.0257088151" iyz="5.49229E-006" izz="0.0120821377"/>
       </inertial>
       <visual>
@@ -32,5 +32,5 @@
     <link name="${prefix}motor1_cover">
       <inertial>
-        <origin rpy="0 0 0" xyz="8.625E-08 -4.6583E-06 0.03145"/>
+        <origin rpy="0 0 0" xyz="0 0 0"/>
         <mass value="0.0"/>
         <inertia ixx="0.0" ixy="0.0" ixz="0.0" iyy="0.0" iyz="0.0" izz="0.0"/>
@@ -59,6 +59,6 @@
       <inertial>
         <origin rpy="0 0 0" xyz="-0.01665 0.0 0.09639"/>
-        <mass value="1.236"/>
-        <inertia ixx="0.0079614839" ixy="0.000000037" ixz="-0.0003203013" iyy="0.007135338" iyz="-0.000001062" izz="0.001111114"/>
+        <mass value="1.24"/>
+        <inertia ixx="0.0079614839" ixy="0.000000037" ixz="0.0003203013" iyy="0.007135338" iyz="-0.000001062" izz="0.001111114"/>
       </inertial>
       <visual>
@@ -84,7 +84,7 @@
     <link name="${prefix}motor3_link">
       <inertial>
-        <origin rpy="0 0 0" xyz="-0.08963 0.0 0.0403"/>
+        <origin rpy="0 0 0" xyz="-0.08963 0 0.0403"/>
         <mass value="3.95"/>
-        <inertia ixx="0.0115136615" ixy="-1.231046E-005" ixz="-0.003148516" iyy="0.0149841676" iyz="-8.81378E-006" izz="0.0070387807"/>
+        <inertia ixx="0.0115136615" ixy="-1.231046E-005" ixz="0.003148516" iyy="0.0149841676" iyz="-8.81378E-006" izz="0.0070387807"/>
       </inertial>
       <visual>
@@ -110,5 +110,5 @@
     <link name="${prefix}motor3_cover">
       <inertial>
-        <origin rpy="0 0 0" xyz="8.625E-08 -4.6583E-06 0.03145"/>
+        <origin rpy="0 0 0" xyz="0 0 0"/>
         <mass value="0.0"/>
         <inertia ixx="0.0" ixy="0.0" ixz="0.0" iyy="0.0" iyz="0.0" izz="0.0"/>
@@ -137,6 +137,6 @@
       <inertial>
         <origin rpy="0 0 0" xyz="0.06357 0.0 0.05698"/>
-        <mass value="1.258"/>
-        <inertia ixx="0.005919676" ixy="0.000000923" ixz="0.0022280208" iyy="0.0068807393" iyz="6.1373E-007" izz="0.00257485"/>
+        <mass value="1.26"/>
+        <inertia ixx="0.005919676" ixy="0.000000923" ixz="-0.0022280208" iyy="0.0068807393" iyz="6.1373E-007" izz="0.00257485"/>
       </inertial>
       <visual>
@@ -164,5 +164,5 @@
         <origin rpy="0 0 0" xyz="-0.09105 0.0 0.03676"/>
         <mass value="2.85"/>
-        <inertia ixx="0.0072829492" ixy="3.77994E-006" ixz="-0.0015682105" iyy="0.0098263499" iyz="2.52745E-006" izz="0.0045615321"/>
+        <inertia ixx="0.0072829492" ixy="3.77994E-006" ixz="0.0015682105" iyy="0.0098263499" iyz="2.52745E-006" izz="0.0045615321"/>
       </inertial>
       <visual>
@@ -188,5 +188,5 @@
     <link name="${prefix}motor5_cover">
       <inertial>
-        <origin rpy="0 0 0" xyz="8.625E-08 -4.6583E-06 0.03145"/>
+        <origin rpy="0 0 0" xyz="0 0 0"/>
         <mass value="0.0"/>
         <inertia ixx="0.0" ixy="0.0" ixz="0.0" iyy="0.0" iyz="0.0" izz="0.0"/>

Commit message: add two robots urdfs

File: mara_description/urdf/mara.urdf.xacro (robot description, xacro)
@@ -6,5 +6,5 @@
   <xacro:include filename="$(find mara_description)/urdf/mara.transmission.xacro" />
   <xacro:include filename="$(find mara_description)/urdf/mara_gazebo.urdf.xacro" />
-  <xacro:macro name="mara_robot"  params="prefix ee_link_distance">
+  <xacro:macro name="mara_robot"  params="prefix ee_link_distance MAC1 MAC2 MAC3">
     <link name="${prefix}base_link">
       <inertial>
@@ -362,11 +362,11 @@
     </joint>
     <link name="${prefix}tool0"/>
-    <joint name="${prefix}${prefix}motor6_link-tool0_fixed_joint" type="fixed">
+    <joint name="${prefix}motor6_link-tool0_fixed_joint" type="fixed">
       <origin rpy="0 -1.57 0" xyz="0 0.0 ${ee_link_distance}"/>
-      <parent link="${prefix}${prefix}motor6_link"/>
+      <parent link="${prefix}motor6_link"/>
       <child link="${prefix}tool0"/>
     </joint>
     <xacro:mara_transmission prefix="${prefix}"/>
-    <xacro:mara_gazebo prefix="${prefix}"/>
+    <xacro:mara_gazebo prefix="${prefix}" MAC1="${MAC1}" MAC2="${MAC2}" MAC3="${MAC3}"/>
   </xacro:macro>
 </robot>

File: mara_description/urdf/mara_gazebo.urdf.xacro (robot description, xacro)
@@ -1,5 +1,5 @@
 <?xml version="1.0"?>
 <robot xmlns:xacro="http://ros.org/wiki/xacro">
-  <xacro:macro name="mara_gazebo" params="prefix">
+  <xacro:macro name="mara_gazebo" params="prefix MAC1 MAC2 MAC3">
     <gazebo>
       <plugin name="mara_joint_state" filename="libgazebo_ros_joint_state_publisher.so">
@@ -8,28 +8,28 @@
     		</ros>
     		<update_rate>25</update_rate>
-    		<joint_name>motor1</joint_name>
-    		<joint_name>motor2</joint_name>
-    		<joint_name>motor3</joint_name>
-    		<joint_name>motor4</joint_name>
-    		<joint_name>motor5</joint_name>
-        <joint_name>motor6</joint_name>
-        <joint_name>joint_finger</joint_name>
+    		<joint_name>${prefix}motor1</joint_name>
+    		<joint_name>${prefix}motor2</joint_name>
+    		<joint_name>${prefix}motor3</joint_name>
+    		<joint_name>${prefix}motor4</joint_name>
+    		<joint_name>${prefix}motor5</joint_name>
+        <joint_name>${prefix}motor6</joint_name>
+        <joint_name>${prefix}joint_finger</joint_name>
     	</plugin>
-      <plugin name="hrim_actuation_servomotor_000000000001" filename="libmara_gazebo_joint_plugin.so">
+      <plugin name="hrim_actuation_servomotor${MAC1}" filename="libmara_gazebo_joint_plugin.so">
         <ros></ros>
-        <axis1>motor2</axis1>
-        <axis2>motor1</axis2>
+        <axis1>${prefix}motor2</axis1>
+        <axis2>${prefix}motor1</axis2>
         <type>series14</type>
       </plugin>
-      <plugin name="hrim_actuation_servomotor_000000000002" filename="libmara_gazebo_joint_plugin.so">
+      <plugin name="hrim_actuation_servomotor${MAC2}" filename="libmara_gazebo_joint_plugin.so">
         <ros></ros>
-        <axis1>motor3</axis1>
-        <axis2>motor4</axis2>
+        <axis1>${prefix}motor3</axis1>
+        <axis2>${prefix}motor4</axis2>
         <type>series17</type>
       </plugin>
-      <plugin name="hrim_actuation_servomotor_000000000003" filename="libmara_gazebo_joint_plugin.so">
+      <plugin name="hrim_actuation_servomotor${MAC3}" filename="libmara_gazebo_joint_plugin.so">
         <ros></ros>
-        <axis1>motor5</axis1>
-        <axis2>motor6</axis2>
+        <axis1>${prefix}motor5</axis1>
+        <axis2>${prefix}motor6</axis2>
         <type>series20</type>
       </plugin>

File: mara_description/urdf/mara_robot_gripper_140.urdf.xacro (robot description, xacro)
@@ -9,6 +9,6 @@
   <xacro:include filename="$(find mara_description)/urdf/table.urdf.xacro" />
   <!-- arm -->
-  <xacro:mara_robot prefix="" ee_link_distance="0.24497"/>
-  <xacro:robotiq_gripper prefix="mara" />
+  <xacro:mara_robot prefix="" ee_link_distance="0.24497" MAC1="_000000000001" MAC2="_000000000002" MAC3="_000000000003"/>
+  <xacro:robotiq_gripper prefix="" MAC="_000000000004"/>
   <xacro:table prefix="" />
   <link name="world" />

File: mara_description/urdf/mara_robot_gripper_140_no_table.urdf.xacro (robot description, xacro)
@@ -8,6 +8,6 @@
   <xacro:include filename="$(find robotiq_140_gripper_description)/urdf/robotiq_140.urdf.xacro" />
   <!-- arm -->
-  <xacro:mara_robot prefix="" ee_link_distance="0.24497"/>
-  <xacro:robotiq_gripper prefix="mara" />
+  <xacro:mara_robot prefix="" ee_link_distance="0.24497" MAC1="_000000000001" MAC2="_000000000002" MAC3="_000000000003"/>
+  <xacro:robotiq_gripper prefix="" MAC="_000000000004"/>
   <link name="world" />
   <link name="gripper_adapter">

File: mara_description/urdf/mara_robot_gripper_85.urdf.xacro (robot description, xacro)
@@ -9,5 +9,5 @@
   <xacro:include filename="$(find mara_description)/urdf/table.urdf.xacro" />
   <!-- arm -->
-  <xacro:mara_robot prefix="" ee_link_distance="0.18491"/>
+  <xacro:mara_robot prefix="" ee_link_distance="0.18491" MAC1="_000000000001" MAC2="_000000000002" MAC3="_000000000003"/>
   <xacro:robotiq_85 prefix="mara" />
   <xacro:table prefix="" />

File: mara_description/urdf/mara_robot_gripper_hande.urdf.xacro (robot description, xacro)
@@ -9,5 +9,5 @@
   <xacro:include filename="$(find mara_description)/urdf/table.urdf.xacro" />
   <!-- arm -->
-  <xacro:mara_robot prefix="" ee_link_distance="0.18253"/>
+  <xacro:mara_robot prefix="" ee_link_distance="0.18253" MAC1="_000000000001" MAC2="_000000000002" MAC3="_000000000003"/>
   <xacro:robotiq_hande prefix="mara" />
   <xacro:table prefix="" />
