Commit message: minor fixes and changed name of plugin

File: robotiq_140_gripper_description/urdf/robotiq_gripper.urdf.xacro (robot description, xacro)
@@ -242,5 +242,5 @@
     <link name="right_outer_finger">
       <inertial>
-        <origin xyz="-0.0002009,  0.0396149, -0.0161363" rpy="0 0 0" />
+        <origin xyz="-0.0002009  0.0396149 -0.0161363" rpy="0 0 0" />
         <mass value="0.022614240507152" />
         <inertia
@@ -363,5 +363,5 @@
         </axis>
       </joint>
-      <plugin filename="librobotiq_140_gripper_gazebo_plugin.so" name="robotiq_arg2f_gazebo_plugins"/>
+      <plugin filename="librobotiq_140_gripper_gazebo_plugin.so" name="hros_actuation_gripper_000000000004"/>
       <plugin filename="libgazebo_grasp_fix.so" name="gazebo_grasp_fix">
         <arm>

Commit message: Updating robotiq gripper xacro

File: robotiq_140_gripper_description/urdf/robotiq_gripper.urdf.xacro (robot description, xacro)
@@ -58,5 +58,5 @@
     <gazebo reference="left_outer_knuckle">
       <material>Gazebo/Grey</material>
-      <selfCollide>True</selfCollide>
+      <selfCollide>False</selfCollide>
     </gazebo>
     <link name="right_outer_knuckle">
@@ -90,5 +90,5 @@
     <gazebo reference="right_outer_knuckle">
       <material>Gazebo/Grey</material>
-      <selfCollide>True</selfCollide>
+      <selfCollide>False</selfCollide>
     </gazebo>
     <link name="left_inner_knuckle">
@@ -272,36 +272,32 @@
       <selfCollide>True</selfCollide>
     </gazebo>
-<!-- OK -->
     <joint name="left_outer_knuckle_joint" type="revolute">
-      <origin xyz="0 -0.030601 0.054905" rpy="2.29579632679 0 0" />
+      <origin xyz="0 -0.030601 0.054905" rpy="2.31 0 0" />
       <parent link="robotiq_arg2f_base_link" />
       <child link="left_outer_knuckle" />
       <axis xyz="-1 0 0" />
-      <limit lower="-2" upper="2" velocity="2.0" effort="1000" />
-    </joint>
-<!-- OK -->
+      <limit lower="0" upper="0.875"  velocity="2.0" effort="1000" />
+    </joint>
     <joint name="right_outer_knuckle_joint" type="revolute">
-      <origin xyz="0 0.030601 0.054905" rpy="2.29579632679 0 3.14" />
+      <origin xyz="0 0.030601 0.054905" rpy="2.31 0 3.1416" />
       <parent link="robotiq_arg2f_base_link" />
       <child link="right_outer_knuckle" />
       <axis xyz="-1 0 0" />
-      <limit lower="-2" upper="2" velocity="2.0" effort="1000" />
-    </joint>
-<!-- OK -->
+      <limit lower="0" upper="0.875" velocity="2.0" effort="1000" />
+    </joint>
     <joint name="left_inner_knuckle_joint" type="revolute">
-      <origin xyz="0 -0.0127 0.06142" rpy="2.29579632679 0 0" />
+      <origin xyz="0 -0.0127 0.06142" rpy="2.29 0 0" />
       <parent link="robotiq_arg2f_base_link" />
       <child link="left_inner_knuckle" />
       <axis xyz="-1 0 0" />
-      <limit lower="0" upper="0.8757" velocity="2.0" effort="1000" />
+      <limit lower="0" upper="0.87" velocity="2.0" effort="1000" />
       <mimic joint="left_outer_knuckle_joint" multiplier="-1" offset="0" />
     </joint>
-<!-- OK -->
     <joint name="right_inner_knuckle_joint" type="revolute">
-      <origin xyz="0 0.0127 0.06142" rpy="2.29579632679 0  -3.14" />
+      <origin xyz="0 0.0127 0.06142" rpy="2.29 0 -3.1416" />
       <parent link="robotiq_arg2f_base_link" />
       <child link="right_inner_knuckle" />
       <axis xyz="-1 0 0" />
-      <limit lower="0" upper="0.8757" velocity="2.0" effort="1000" />
+      <limit lower="0" upper="0.87" velocity="2.0" effort="1000" />
       <mimic joint="right_outer_knuckle_joint" multiplier="-1" offset="0" />
     </joint>
@@ -310,6 +306,6 @@
       <parent link="left_outer_knuckle" />
       <child link="left_outer_finger" />
-      <axis xyz="1 0 0" />
-      <limit lower="-2" upper="2" velocity="2.0" effort="1000" />
+      <axis xyz="-1 0 0" />
+      <limit lower="0.1" upper="0.875" velocity="2.0" effort="1000" />
     </joint>
     <joint name="right_outer_finger_joint" type="revolute">
@@ -318,5 +314,5 @@
       <child link="right_outer_finger" />
       <axis xyz="-1 0 0" />
-      <limit lower="-2" upper="2" velocity="2.0" effort="1000" />
+      <limit lower="0.1" upper="0.875" velocity="2.0" effort="1000" />
     </joint>
     <joint name="left_inner_finger_joint" type="revolute">
@@ -340,5 +336,5 @@
         <child>mara::left_inner_finger</child>
         <axis>
-          <xyz>0 1 0</xyz>
+          <xyz>1 0 0</xyz>
           <limit>
             <lower>-0.6</lower>
@@ -354,5 +350,5 @@
         <child>mara::right_inner_finger</child>
         <axis>
-          <xyz>0 1 0</xyz>
+          <xyz>-1 0 0</xyz>
           <limit>
             <lower>-0.6</lower>
@@ -364,21 +360,4 @@
       </joint>
       <plugin filename="librobotiq_140_gripper_gazebo_plugin.so" name="hros_actuation_gripper_000000000004"/>
-      <plugin filename="libgazebo_grasp_fix.so" name="gazebo_grasp_fix">
-        <arm>
-          <arm_name>robot</arm_name>
-          <palm_link>left_inner_finger</palm_link>
-          <gripper_link>left_inner_finger</gripper_link>
-          <gripper_link>right_inner_finger</gripper_link>
-          <gripper_link>left_inner_knuckle</gripper_link>
-          <gripper_link>right_inner_knuckle</gripper_link>
-        </arm>
-        <forces_angle_tolerance>100</forces_angle_tolerance>
-        <update_rate>20</update_rate>
-        <grip_count_threshold>4</grip_count_threshold>
-        <max_grip_count>8</max_grip_count>
-        <release_tolerance>0.05</release_tolerance>
-        <disable_collisions_on_attach>false</disable_collisions_on_attach>
-        <contact_topic>__default_topic__</contact_topic>
-     </plugin>
     </gazebo>
   </xacro:macro>
