Commit message: Fix robotiq gripper 140 urdf

File: robotiq_140_gripper_description/urdf/robotiq_140.urdf (robot description, URDF)
Before this commit: robot robotiq_gripper, 10 links, 9 joints
Joints:
- joint left_inner_knuckle_joint: limit lower=0 upper=0.87 effort=1000 velocity=2.0 -> lower=0 upper=0.78 effort=1000 velocity=2.0; origin xyz=0 -0.0127 0.06142 rpy=2.29 0 0 -> xyz=0 -0.0127 0.06142 rpy=2.31 0 0
- joint left_outer_finger_joint: limit lower=0.1 upper=0.875 effort=1000 velocity=2.0 -> lower=-0.875 upper=-0.0075 effort=1000 velocity=2.0
- joint left_outer_knuckle_joint: limit lower=0 upper=0.875 effort=1000 velocity=2.0 -> lower=0 upper=0.78 effort=1000 velocity=2.0
- joint right_inner_knuckle_joint: limit lower=0 upper=0.87 effort=1000 velocity=2.0 -> lower=0 upper=0.78 effort=1000 velocity=2.0; origin xyz=0 0.0127 0.06142 rpy=2.29 0 -3.14159265359 -> xyz=0 0.0127 0.06142 rpy=2.31 0 -3.14159265359
- joint right_outer_finger_joint: limit lower=0.1 upper=0.875 effort=1000 velocity=2.0 -> lower=-0.875 upper=-0.0075 effort=1000 velocity=2.0
- joint right_outer_knuckle_joint: limit lower=0 upper=0.875 effort=1000 velocity=2.0 -> lower=0 upper=0.78 effort=1000 velocity=2.0

File: robotiq_140_gripper_description/urdf/robotiq_140.urdf.xacro (robot description, xacro)
@@ -277,5 +277,5 @@
       <child link="left_outer_knuckle" />
       <axis xyz="-1 0 0" />
-      <limit lower="0" upper="0.875"  velocity="2.0" effort="1000" />
+      <limit lower="0" upper="0.78"  velocity="2.0" effort="1000" />
     </joint>
     <joint name="right_outer_knuckle_joint" type="revolute">
@@ -284,5 +284,5 @@
       <child link="right_outer_knuckle" />
       <axis xyz="-1 0 0" />
-      <limit lower="0" upper="0.875" velocity="2.0" effort="1000" />
+      <limit lower="0" upper="0.78" velocity="2.0" effort="1000" />
     </joint>
     <joint name="left_inner_knuckle_joint" type="revolute">
@@ -291,5 +291,5 @@
       <child link="left_inner_knuckle" />
       <axis xyz="-1 0 0" />
-      <limit lower="0" upper="0.87" velocity="2.0" effort="1000" />
+      <limit lower="0" upper="0.78" velocity="2.0" effort="1000" />
     </joint>
     <joint name="right_inner_knuckle_joint" type="revolute">
@@ -298,5 +298,5 @@
       <child link="right_inner_knuckle" />
       <axis xyz="-1 0 0" />
-      <limit lower="0" upper="0.87" velocity="2.0" effort="1000" />
+      <limit lower="0" upper="0.78" velocity="2.0" effort="1000" />
     </joint>
     <joint name="left_outer_finger_joint" type="revolute">
@@ -305,5 +305,5 @@
       <child link="left_outer_finger" />
       <axis xyz="-1 0 0" />
-      <limit lower="0.1" upper="0.875" velocity="2.0" effort="1000" />
+      <limit lower="-0.875" upper="-0.0075" velocity="2.0" effort="1000" />
     </joint>
     <joint name="right_outer_finger_joint" type="revolute">
@@ -312,5 +312,5 @@
       <child link="right_outer_finger" />
       <axis xyz="-1 0 0" />
-      <limit lower="0.1" upper="0.875" velocity="2.0" effort="1000" />
+      <limit lower="-0.875" upper="-0.0075" velocity="2.0" effort="1000" />
     </joint>
     <joint name="left_inner_finger_joint" type="revolute">
@@ -331,6 +331,6 @@
       <joint name="left_inner_finger_knuckle_joint" type="revolute">
         <pose frame="">0 0.006 -0.018 0 0 0</pose>
-        <parent>mara::left_inner_knuckle</parent>
-        <child>mara::left_inner_finger</child>
+        <parent>robotiq_140::left_inner_knuckle</parent>
+        <child>robotiq_140::left_inner_finger</child>
         <axis>
           <xyz>1 0 0</xyz>
@@ -345,6 +345,6 @@
       <joint name="right_inner_finger_knuckle_joint" type="revolute">
         <pose frame="">0 0.006 -0.018 0 0 0</pose>
-        <parent>mara::right_inner_knuckle</parent>
-        <child>mara::right_inner_finger</child>
+        <parent>robotiq_140::right_inner_knuckle</parent>
+        <child>robotiq_140::right_inner_finger</child>
         <axis>
           <xyz>-1 0 0</xyz>
