Commit message: Adding textures and reducing size

File: robotiq_140_gripper_description/urdf/module_gripper.urdf.xacro (robot description, xacro)
@@ -7,7 +7,7 @@
   <link name="world" />
   <joint name="world_to_hande_joint" type="fixed">
-    <origin rpy="0 0 0" xyz="0 0 0.5"/>
+    <origin rpy="0 0 1.57" xyz="0 0 0.5"/>
     <parent link="world"/>
-    <child link="robotiq_arg2f_base_link"/>
+    <child link="robotiq_adapter_link"/>
   </joint>
 </robot>

File: robotiq_140_gripper_description/urdf/robotiq_140.urdf (robot description, URDF)
Before this commit: robot robotiq_gripper, 10 links, 9 joints
Links:
- added link robotiq_adapter_link, mass 0.22652; collision mesh filename=package://robotiq_85_gripper_description/meshes/hros_roboti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 scale=0.001 0.001 0.001; visual mesh filename=package://robotiq_85_gripper_description/meshes/hros_roboti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 scale=0.001 0.001 0.001
Joints:
- added joint base_adapter_to_base_robotiq_joint: type fixed, parent robotiq_adapter_link, child robotiq_arg2f_base_link, origin xyz= 0 0 0.03653 rpy=0 0 0
- joint left_inner_knuckle_joint: origin xyz=0 -0.0127 0.06142 rpy=2.31 0 0 -> xyz=0 -0.0127 0.06142 rpy=2.29 0 0
- joint right_inner_knuckle_joint: origin xyz=0 0.0127 0.06142 rpy=2.31 0 -3.14159265359 -> xyz=0 0.0127 0.06142 rpy=2.29 0 -3.14159265359
- joint world_to_hande_joint: child robotiq_arg2f_base_link -> robotiq_adapter_link; origin xyz=0 0 0.5 rpy=0 0 0 -> xyz=0 0 0.5 rpy=0 0 1.57

File: robotiq_140_gripper_description/urdf/robotiq_140.urdf.xacro (robot description, xacro)
@@ -2,5 +2,5 @@
 <robot xmlns:xacro="http://ros.org/wiki/xacro">
   <xacro:macro name="robotiq_gripper"  params="prefix">
-    <link name="robotiq_arg2f_base_link">
+    <link name="robotiq_adapter_link">
       <inertial>
         <origin xyz="8.625E-08 -4.6583E-06 0.03145" rpy="0 0 0" />
@@ -9,9 +9,35 @@
       </inertial>
       <visual>
+        <origin xyz="0 0 0" rpy="0 0 0" />
+        <geometry>
+          <mesh filename="package://robotiq_85_gripper_description/meshes/hros_robotiq_adapter.dae" scale="0.001 0.001 0.001"/>
+        </geometry>
+        <material name="Gazebo/Black">
+          <color rgba="0.1 0.1 0.1 1" />
+        </material>
+      </visual>
+      <collision>
+        <origin xyz="0 0 0" rpy="0 0 0" />
+        <geometry>
+          <mesh filename="package://robotiq_85_gripper_description/meshes/hros_robotiq_adapter.dae" scale="0.001 0.001 0.001"/>
+        </geometry>
+      </collision>
+    </link>
+    <gazebo reference="robotiq_adapter_link">
+      <material>Gazebo/Black</material>
+      <selfCollide>True</selfCollide>
+    </gazebo>
+    <link name="robotiq_arg2f_base_link">
+      <inertial>
+        <origin xyz="8.625E-08 -4.6583E-06 0.03145" rpy="0 0 0" />
+        <mass value="0.22652" />
+        <inertia ixx="0.00020005" ixy="0" ixz="0" iyy="0.00017832" iyz="0" izz="0.00013478" />
+      </inertial>
+      <visual>
         <origin xyz="0 0 0" rpy="0 0 1.57" />
         <geometry>
           <mesh filename="package://robotiq_140_gripper_description/meshes/GRIPPER_base_axis.stl" scale="0.001 0.001 0.001"/>
         </geometry>
-        <material name="">
+        <material name="Gazebo/Black">
           <color rgba="0.1 0.1 0.1 1" />
         </material>
@@ -25,5 +51,5 @@
     </link>
     <gazebo reference="robotiq_arg2f_base_link">
-      <material>Gazebo/Grey</material>
+      <material>Gazebo/Black</material>
       <selfCollide>True</selfCollide>
     </gazebo>
@@ -109,5 +135,5 @@
           <mesh filename="package://robotiq_140_gripper_description/meshes/robotiq_140_left_inner_knuckle.stl" />
         </geometry>
-        <material name="">
+        <material name="Gazebo/Black">
           <color rgba="0.1 0.1 0.1 1" />
         </material>
@@ -115,5 +141,5 @@
     </link>
     <gazebo reference="left_inner_knuckle">
-      <material>Gazebo/Grey</material>
+      <material>Gazebo/Black</material>
       <selfCollide>True</selfCollide>
     </gazebo>
@@ -135,5 +161,5 @@
           <mesh filename="package://robotiq_140_gripper_description/meshes/robotiq_140_right_inner_knuckle.stl" />
         </geometry>
-        <material name="">
+        <material name="Gazebo/Black">
           <color rgba="0.1 0.1 0.1 1" />
         </material>
@@ -141,5 +167,5 @@
     </link>
     <gazebo reference="right_inner_knuckle">
-      <material>Gazebo/Grey</material>
+      <material>Gazebo/Black</material>
       <selfCollide>True</selfCollide>
     </gazebo>
@@ -161,5 +187,5 @@
           <mesh filename="package://robotiq_140_gripper_description/meshes/robotiq_140_left_inner_finger.stl" scale="0.001 0.001 0.001" />
         </geometry>
-        <material name="">
+        <material name="Gazebo/Black">
           <color rgba="0.1 0.1 0.1 1" />
         </material>
@@ -173,5 +199,5 @@
     </link>
     <gazebo reference="left_inner_finger">
-      <material>Gazebo/Grey</material>
+      <material>Gazebo/Black</material>
       <selfCollide>True</selfCollide>
     </gazebo>
@@ -193,5 +219,5 @@
           <mesh filename="package://robotiq_140_gripper_description/meshes/robotiq_140_right_inner_finger.stl" scale="0.001 0.001 0.001"/>
         </geometry>
-        <material name="">
+        <material name="Gazebo/Black">
           <color rgba="0.1 0.1 0.1 1" />
         </material>
@@ -205,5 +231,5 @@
     </link>
     <gazebo reference="right_inner_finger">
-      <material>Gazebo/Grey</material>
+      <material>Gazebo/Black</material>
       <selfCollide>True</selfCollide>
     </gazebo>
@@ -225,5 +251,5 @@
           <mesh filename="package://robotiq_140_gripper_description/meshes/robotiq_140_left_outer_finger.stl" />
         </geometry>
-        <material name="">
+        <material name="Gazebo/Black">
           <color rgba="0.1 0.1 0.1 1" />
         </material>
@@ -237,5 +263,5 @@
     </link>
     <gazebo reference="left_outer_finger">
-      <material>Gazebo/Grey</material>
+      <material>Gazebo/Black</material>
       <selfCollide>True</selfCollide>
     </gazebo>
@@ -257,5 +283,5 @@
           <mesh filename="package://robotiq_140_gripper_description/meshes/robotiq_140_right_outer_finger.stl" />
         </geometry>
-        <material name="">
+        <material name="Gazebo/Black">
           <color rgba="0.1 0.1 0.1 1" />
         </material>
@@ -269,7 +295,12 @@
     </link>
     <gazebo reference="right_outer_finger">
-      <material>Gazebo/Grey</material>
-      <selfCollide>True</selfCollide>
-    </gazebo>
+      <material>Gazebo/Black</material>
+      <selfCollide>True</selfCollide>
+    </gazebo>
+    <joint name="base_adapter_to_base_robotiq_joint" type="fixed">
+      <origin rpy="0 0 0" xyz=" 0 0 0.03653"/>
+      <parent link="robotiq_adapter_link" />
+      <child link="robotiq_arg2f_base_link"/>
+    </joint>
     <joint name="left_outer_knuckle_joint" type="revolute">
       <origin xyz="0 -0.030601 0.054905" rpy="2.31 0 0" />
