Commit message: updated urdfs and converted stl to dae robotiq 140

File: robotiq_140_gripper_description/urdf/robotiq_140.urdf.xacro (robot description, xacro)
@@ -11,5 +11,5 @@
         <origin xyz="0 0 0" rpy="0 0 1.57" />
         <geometry>
-          <mesh filename="package://robotiq_140_gripper_description/meshes/GRIPPER_base_axis.stl" scale="0.001 0.001 0.001"/>
+          <mesh filename="package://robotiq_140_gripper_description/meshes/GRIPPER_base_axis.dae" scale="0.001 0.001 0.001"/>
         </geometry>
         <material name="Gazebo/Black">
@@ -20,5 +20,5 @@
         <origin xyz="0 0 0" rpy="0 0 1.57" />
         <geometry>
-          <mesh filename="package://robotiq_140_gripper_description/meshes/GRIPPER_base_axis.stl" scale="0.001 0.001 0.001"/>
+          <mesh filename="package://robotiq_140_gripper_description/meshes/GRIPPER_base_axis.dae" scale="0.001 0.001 0.001"/>
         </geometry>
       </collision>
@@ -43,5 +43,5 @@
         <origin xyz="0 0 0" rpy="0 0 0" />
         <geometry>
-          <mesh filename="package://robotiq_140_gripper_description/meshes/robotiq_140_left_outer_knuckle.stl" />
+          <mesh filename="package://robotiq_140_gripper_description/meshes/robotiq_140_left_outer_knuckle.dae" />
         </geometry>
         <material name="">
@@ -52,5 +52,5 @@
         <origin xyz="0 0 0" rpy="0 0 0" />
         <geometry>
-          <mesh filename="package://robotiq_140_gripper_description/meshes/robotiq_140_left_outer_knuckle.stl" />
+          <mesh filename="package://robotiq_140_gripper_description/meshes/robotiq_140_left_outer_knuckle.dae" />
         </geometry>
       </collision>
@@ -75,5 +75,5 @@
         <origin xyz="0 0 0" rpy="0 0 0" />
         <geometry>
-          <mesh filename="package://robotiq_140_gripper_description/meshes/robotiq_140_right_outer_knuckle.stl" />
+          <mesh filename="package://robotiq_140_gripper_description/meshes/robotiq_140_right_outer_knuckle.dae" />
         </geometry>
         <material name="">
@@ -84,5 +84,5 @@
         <origin xyz="0 0 0" rpy="0 0 0" />
         <geometry>
-          <mesh filename="package://robotiq_140_gripper_description/meshes/robotiq_140_right_outer_knuckle.stl" />
+          <mesh filename="package://robotiq_140_gripper_description/meshes/robotiq_140_right_outer_knuckle.dae" />
         </geometry>
       </collision>
@@ -107,5 +107,5 @@
         <origin xyz="0 0 0" rpy="0 0 0" />
         <geometry>
-          <mesh filename="package://robotiq_140_gripper_description/meshes/robotiq_140_left_inner_knuckle.stl" />
+          <mesh filename="package://robotiq_140_gripper_description/meshes/robotiq_140_left_inner_knuckle.dae" />
         </geometry>
         <material name="Gazebo/Black">
@@ -133,5 +133,5 @@
         <origin xyz="0 0 0" rpy="0 0 0" />
         <geometry>
-          <mesh filename="package://robotiq_140_gripper_description/meshes/robotiq_140_right_inner_knuckle.stl" />
+          <mesh filename="package://robotiq_140_gripper_description/meshes/robotiq_140_right_inner_knuckle.dae" />
         </geometry>
         <material name="Gazebo/Black">
@@ -159,14 +159,14 @@
         <origin xyz="0 0 0" rpy="0 0 0" />
         <geometry>
-          <mesh filename="package://robotiq_140_gripper_description/meshes/robotiq_140_left_inner_finger.stl" scale="0.001 0.001 0.001" />
-        </geometry>
-        <material name="Gazebo/Black">
-          <color rgba="0.1 0.1 0.1 1" />
-        </material>
-      </visual>
-      <collision>
-        <origin xyz="0 0 0" rpy="0 0 0" />
-        <geometry>
-          <mesh filename="package://robotiq_140_gripper_description/meshes/robotiq_140_left_inner_finger.stl" scale="0.001 0.001 0.001" />
+          <mesh filename="package://robotiq_140_gripper_description/meshes/robotiq_140_left_inner_finger.dae" scale="0.001 0.001 0.001" />
+        </geometry>
+        <material name="Gazebo/Black">
+          <color rgba="0.1 0.1 0.1 1" />
+        </material>
+      </visual>
+      <collision>
+        <origin xyz="0 0 0" rpy="0 0 0" />
+        <geometry>
+          <mesh filename="package://robotiq_140_gripper_description/meshes/robotiq_140_left_inner_finger.dae" scale="0.001 0.001 0.001" />
         </geometry>
       </collision>
@@ -191,14 +191,14 @@
         <origin xyz="0 0 0" rpy="0 0 0" />
         <geometry>
-          <mesh filename="package://robotiq_140_gripper_description/meshes/robotiq_140_right_inner_finger.stl" scale="0.001 0.001 0.001"/>
-        </geometry>
-        <material name="Gazebo/Black">
-          <color rgba="0.1 0.1 0.1 1" />
-        </material>
-      </visual>
-      <collision>
-        <origin xyz="0 0 0" rpy="0 0 0" />
-        <geometry>
-          <mesh filename="package://robotiq_140_gripper_description/meshes/robotiq_140_right_inner_finger.stl" scale="0.001 0.001 0.001"/>
+          <mesh filename="package://robotiq_140_gripper_description/meshes/robotiq_140_right_inner_finger.dae" scale="0.001 0.001 0.001"/>
+        </geometry>
+        <material name="Gazebo/Black">
+          <color rgba="0.1 0.1 0.1 1" />
+        </material>
+      </visual>
+      <collision>
+        <origin xyz="0 0 0" rpy="0 0 0" />
+        <geometry>
+          <mesh filename="package://robotiq_140_gripper_description/meshes/robotiq_140_right_inner_finger.dae" scale="0.001 0.001 0.001"/>
         </geometry>
       </collision>
@@ -223,14 +223,14 @@
         <origin xyz="0 0 0" rpy="0 0 0" />
         <geometry>
-          <mesh filename="package://robotiq_140_gripper_description/meshes/robotiq_140_left_outer_finger.stl" />
-        </geometry>
-        <material name="Gazebo/Black">
-          <color rgba="0.1 0.1 0.1 1" />
-        </material>
-      </visual>
-      <collision>
-        <origin xyz="0 0 0" rpy="0 0 0" />
-        <geometry>
-          <mesh filename="package://robotiq_140_gripper_description/meshes/robotiq_140_left_outer_finger.stl" />
+          <mesh filename="package://robotiq_140_gripper_description/meshes/robotiq_140_left_outer_finger.dae" />
+        </geometry>
+        <material name="Gazebo/Black">
+          <color rgba="0.1 0.1 0.1 1" />
+        </material>
+      </visual>
+      <collision>
+        <origin xyz="0 0 0" rpy="0 0 0" />
+        <geometry>
+          <mesh filename="package://robotiq_140_gripper_description/meshes/robotiq_140_left_outer_finger.dae" />
         </geometry>
       </collision>
@@ -255,14 +255,14 @@
         <origin xyz="0 0 0" rpy="0 0 0" />
         <geometry>
-          <mesh filename="package://robotiq_140_gripper_description/meshes/robotiq_140_right_outer_finger.stl" />
-        </geometry>
-        <material name="Gazebo/Black">
-          <color rgba="0.1 0.1 0.1 1" />
-        </material>
-      </visual>
-      <collision>
-        <origin xyz="0 0 0" rpy="0 0 0" />
-        <geometry>
-          <mesh filename="package://robotiq_140_gripper_description/meshes/robotiq_140_right_outer_finger.stl" />
+          <mesh filename="package://robotiq_140_gripper_description/meshes/robotiq_140_right_outer_finger.dae" />
+        </geometry>
+        <material name="Gazebo/Black">
+          <color rgba="0.1 0.1 0.1 1" />
+        </material>
+      </visual>
+      <collision>
+        <origin xyz="0 0 0" rpy="0 0 0" />
+        <geometry>
+          <mesh filename="package://robotiq_140_gripper_description/meshes/robotiq_140_right_outer_finger.dae" />
         </geometry>
       </collision>

File: robotiq_140_gripper_description/urdf/robotiq_140_hros_support.urdf.xacro (robot description, xacro)
@@ -37,5 +37,5 @@
         <origin xyz="0 0 0" rpy="0 0 1.57" />
         <geometry>
-          <mesh filename="package://robotiq_140_gripper_description/meshes/GRIPPER_base_axis.stl" scale="0.001 0.001 0.001"/>
+          <mesh filename="package://robotiq_140_gripper_description/meshes/GRIPPER_base_axis.dae" scale="0.001 0.001 0.001"/>
         </geometry>
         <material name="Gazebo/Black">
@@ -46,5 +46,5 @@
         <origin xyz="0 0 0" rpy="0 0 1.57" />
         <geometry>
-          <mesh filename="package://robotiq_140_gripper_description/meshes/GRIPPER_base_axis.stl" scale="0.001 0.001 0.001"/>
+          <mesh filename="package://robotiq_140_gripper_description/meshes/GRIPPER_base_axis.dae" scale="0.001 0.001 0.001"/>
         </geometry>
       </collision>
@@ -69,5 +69,5 @@
         <origin xyz="0 0 0" rpy="0 0 0" />
         <geometry>
-          <mesh filename="package://robotiq_140_gripper_description/meshes/robotiq_140_left_outer_knuckle.stl" />
+          <mesh filename="package://robotiq_140_gripper_description/meshes/robotiq_140_left_outer_knuckle.dae" />
         </geometry>
         <material name="">
@@ -78,5 +78,5 @@
         <origin xyz="0 0 0" rpy="0 0 0" />
         <geometry>
-          <mesh filename="package://robotiq_140_gripper_description/meshes/robotiq_140_left_outer_knuckle.stl" />
+          <mesh filename="package://robotiq_140_gripper_description/meshes/robotiq_140_left_outer_knuckle.dae" />
         </geometry>
       </collision>
@@ -101,5 +101,5 @@
         <origin xyz="0 0 0" rpy="0 0 0" />
         <geometry>
-          <mesh filename="package://robotiq_140_gripper_description/meshes/robotiq_140_right_outer_knuckle.stl" />
+          <mesh filename="package://robotiq_140_gripper_description/meshes/robotiq_140_right_outer_knuckle.dae" />
         </geometry>
         <material name="">
@@ -110,5 +110,5 @@
         <origin xyz="0 0 0" rpy="0 0 0" />
         <geometry>
-          <mesh filename="package://robotiq_140_gripper_description/meshes/robotiq_140_right_outer_knuckle.stl" />
+          <mesh filename="package://robotiq_140_gripper_description/meshes/robotiq_140_right_outer_knuckle.dae" />
         </geometry>
       </collision>
@@ -133,5 +133,5 @@
         <origin xyz="0 0 0" rpy="0 0 0" />
         <geometry>
-          <mesh filename="package://robotiq_140_gripper_description/meshes/robotiq_140_left_inner_knuckle.stl" />
+          <mesh filename="package://robotiq_140_gripper_description/meshes/robotiq_140_left_inner_knuckle.dae" />
         </geometry>
         <material name="Gazebo/Black">
@@ -159,5 +159,5 @@
         <origin xyz="0 0 0" rpy="0 0 0" />
         <geometry>
-          <mesh filename="package://robotiq_140_gripper_description/meshes/robotiq_140_right_inner_knuckle.stl" />
+          <mesh filename="package://robotiq_140_gripper_description/meshes/robotiq_140_right_inner_knuckle.dae" />
         </geometry>
         <material name="Gazebo/Black">
@@ -185,14 +185,14 @@
         <origin xyz="0 0 0" rpy="0 0 0" />
         <geometry>
-          <mesh filename="package://robotiq_140_gripper_description/meshes/robotiq_140_left_inner_finger.stl" scale="0.001 0.001 0.001" />
-        </geometry>
-        <material name="Gazebo/Black">
-          <color rgba="0.1 0.1 0.1 1" />
-        </material>
-      </visual>
-      <collision>
-        <origin xyz="0 0 0" rpy="0 0 0" />
-        <geometry>
-          <mesh filename="package://robotiq_140_gripper_description/meshes/robotiq_140_left_inner_finger.stl" scale="0.001 0.001 0.001" />
+          <mesh filename="package://robotiq_140_gripper_description/meshes/robotiq_140_left_inner_finger.dae" scale="0.001 0.001 0.001" />
+        </geometry>
+        <material name="Gazebo/Black">
+          <color rgba="0.1 0.1 0.1 1" />
+        </material>
+      </visual>
+      <collision>
+        <origin xyz="0 0 0" rpy="0 0 0" />
+        <geometry>
+          <mesh filename="package://robotiq_140_gripper_description/meshes/robotiq_140_left_inner_finger.dae" scale="0.001 0.001 0.001" />
         </geometry>
       </collision>
@@ -217,14 +217,14 @@
         <origin xyz="0 0 0" rpy="0 0 0" />
         <geometry>
-          <mesh filename="package://robotiq_140_gripper_description/meshes/robotiq_140_right_inner_finger.stl" scale="0.001 0.001 0.001"/>
-        </geometry>
-        <material name="Gazebo/Black">
-          <color rgba="0.1 0.1 0.1 1" />
-        </material>
-      </visual>
-      <collision>
-        <origin xyz="0 0 0" rpy="0 0 0" />
-        <geometry>
-          <mesh filename="package://robotiq_140_gripper_description/meshes/robotiq_140_right_inner_finger.stl" scale="0.001 0.001 0.001"/>
+          <mesh filename="package://robotiq_140_gripper_description/meshes/robotiq_140_right_inner_finger.dae" scale="0.001 0.001 0.001"/>
+        </geometry>
+        <material name="Gazebo/Black">
+          <color rgba="0.1 0.1 0.1 1" />
+        </material>
+      </visual>
+      <collision>
+        <origin xyz="0 0 0" rpy="0 0 0" />
+        <geometry>
+          <mesh filename="package://robotiq_140_gripper_description/meshes/robotiq_140_right_inner_finger.dae" scale="0.001 0.001 0.001"/>
         </geometry>
       </collision>
@@ -249,14 +249,14 @@
         <origin xyz="0 0 0" rpy="0 0 0" />
         <geometry>
-          <mesh filename="package://robotiq_140_gripper_description/meshes/robotiq_140_left_outer_finger.stl" />
-        </geometry>
-        <material name="Gazebo/Black">
-          <color rgba="0.1 0.1 0.1 1" />
-        </material>
-      </visual>
-      <collision>
-        <origin xyz="0 0 0" rpy="0 0 0" />
-        <geometry>
-          <mesh filename="package://robotiq_140_gripper_description/meshes/robotiq_140_left_outer_finger.stl" />
+          <mesh filename="package://robotiq_140_gripper_description/meshes/robotiq_140_left_outer_finger.dae" />
+        </geometry>
+        <material name="Gazebo/Black">
+          <color rgba="0.1 0.1 0.1 1" />
+        </material>
+      </visual>
+      <collision>
+        <origin xyz="0 0 0" rpy="0 0 0" />
+        <geometry>
+          <mesh filename="package://robotiq_140_gripper_description/meshes/robotiq_140_left_outer_finger.dae" />
         </geometry>
       </collision>
@@ -281,14 +281,14 @@
         <origin xyz="0 0 0" rpy="0 0 0" />
         <geometry>
-          <mesh filename="package://robotiq_140_gripper_description/meshes/robotiq_140_right_outer_finger.stl" />
-        </geometry>
-        <material name="Gazebo/Black">
-          <color rgba="0.1 0.1 0.1 1" />
-        </material>
-      </visual>
-      <collision>
-        <origin xyz="0 0 0" rpy="0 0 0" />
-        <geometry>
-          <mesh filename="package://robotiq_140_gripper_description/meshes/robotiq_140_right_outer_finger.stl" />
+          <mesh filename="package://robotiq_140_gripper_description/meshes/robotiq_140_right_outer_finger.dae" />
+        </geometry>
+        <material name="Gazebo/Black">
+          <color rgba="0.1 0.1 0.1 1" />
+        </material>
+      </visual>
+      <collision>
+        <origin xyz="0 0 0" rpy="0 0 0" />
+        <geometry>
+          <mesh filename="package://robotiq_140_gripper_description/meshes/robotiq_140_right_outer_finger.dae" />
         </geometry>
       </collision>
