Commit message: Fix robotiq 85 gripper urdf joint name mispelling

File: robotiq_85_gripper_description/urdf/robotiq_85.urdf (robot description, URDF)
Before this commit: robot robotiq_85, 11 links, 10 joints
Joints:
- removed joint right_inner_knuckler_joint
- added joint right_inner_knuckle_joint: type revolute, parent robotiq_85_base_link, child robotiq_85_right_inner_knuckle_link, origin xyz=0.0306 0 0.05490 rpy=0 0 3.1416, axis 0 1 0, limit lower=0 upper=0.8757 effort=1000 velocity=2.0

File: robotiq_85_gripper_description/urdf/robotiq_85.urdf.xacro (robot description, xacro)
@@ -274,5 +274,5 @@
       <limit lower="0.0" upper="0.8757" velocity="2.0" effort="1000" />
     </joint>
-    <joint name="right_inner_knuckler_joint" type="revolute">
+    <joint name="right_inner_knuckle_joint" type="revolute">
       <origin xyz="0.0306 0 0.05490" rpy="0 0 3.1416" />
       <parent link="robotiq_85_base_link" />

Commit message: Fix robotiq gripper 85 urdf

File: robotiq_85_gripper_description/urdf/robotiq_85.urdf (robot description, URDF)
Before this commit: robot robotiq_85, 11 links, 10 joints
Joints:
- joint left_finger_joint: axis 0 1 0 -> 0 -1 0
- joint left_inner_knuckle_joint: limit lower=0.0 upper=0.8757 effort=1000 velocity=2.0 -> lower=0 upper=0.794 effort=1000 velocity=2.0
- joint left_outer_knuckle_joint: axis 0 1 0 -> 0 -1 0
- joint right_finger_joint: axis 0 1 0 -> 0 -1 0
- joint right_inner_knuckle_joint: limit lower=0 upper=0.8757 effort=1000 velocity=2.0 -> lower=0 upper=0.794 effort=1000 velocity=2.0
- joint right_outer_knuckle_joint: axis 0 1 0 -> 0 -1 0

File: robotiq_85_gripper_description/urdf/robotiq_85.urdf.xacro (robot description, xacro)
@@ -272,5 +272,5 @@
       <child link="robotiq_85_left_inner_knuckle_link" />
       <axis xyz="0 1 0" />
-      <limit lower="0.0" upper="0.8757" velocity="2.0" effort="1000" />
+      <limit lower="0.0" upper="0.794" velocity="2.0" effort="1000" />
     </joint>
     <joint name="right_inner_knuckle_joint" type="revolute">
@@ -279,5 +279,5 @@
       <child link="robotiq_85_right_inner_knuckle_link" />
       <axis xyz="0 1 0" />
-      <limit lower="0" upper="0.8757" velocity="2.0" effort="1000" />
+      <limit lower="0" upper="0.794" velocity="2.0" effort="1000" />
     </joint>
     <joint name="left_outer_knuckle_joint" type="revolute">
@@ -285,5 +285,5 @@
       <parent link="robotiq_85_left_inner_knuckle_link" />
       <child link="robotiq_85_left_outer_knuckle_link" />
-      <axis xyz="0 1 0" />
+      <axis xyz="0 -1 0" />
       <limit lower="0" upper="0.8757" velocity="2.0" effort="1000" />
     </joint>
@@ -292,5 +292,5 @@
       <parent link="robotiq_85_right_inner_knuckle_link" />
       <child link="robotiq_85_right_outer_knuckle_link" />
-      <axis xyz="0 1 0" />
+      <axis xyz="0 -1 0" />
       <limit lower="0" upper="0.8757" velocity="2.0" effort="1000" />
     </joint>
@@ -313,5 +313,5 @@
       <parent link="robotiq_85_left_outer_knuckle_link" />
       <child link="robotiq_85_left_finger_link" />
-      <axis xyz="0 1 0" />
+      <axis xyz="0 -1 0" />
       <limit lower="-0.1" upper="0.8757" velocity="2.0" effort="1000" />
     </joint>
@@ -320,8 +320,9 @@
       <parent link="robotiq_85_right_outer_knuckle_link" />
       <child link="robotiq_85_right_finger_link" />
-      <axis xyz="0 1 0"/>
+      <axis xyz="0 -1 0"/>
       <limit lower="-0.1" upper="0.8757" velocity="2.0" effort="1000" />
     </joint>
     <gazebo>
+      <plugin name='gripper' filename='librobotiq_gripper_gazebo_plugin.so'/>
       <joint name="left_finger_joint2" type="revolute">
         <pose frame="">0.017901 0 0.00651469 0 0 0</pose>
@@ -329,5 +330,5 @@
         <child>robotiq85::robotiq_85_left_finger_link</child>
         <axis>
-          <xyz>0 1 0</xyz>
+          <xyz>0 -1 0</xyz>
           <limit>
             <lower>-0.1</lower>

Commit message: Recuding size and improve textures

File: robotiq_85_gripper_description/urdf/robotiq_85.urdf (robot description, URDF)
Before this commit: robot robotiq_85, 11 links, 10 joints
Joints:
- joint left_inner_knuckle_joint: limit lower=0 upper=0.794 effort=1000 velocity=2.0 -> lower=0.0 upper=0.794 effort=1000 velocity=2.0

File: robotiq_85_gripper_description/urdf/robotiq_85.urdf.xacro (robot description, xacro)
@@ -11,19 +11,19 @@
         <origin xyz="0 0 0" rpy="0 0 0" />
         <geometry>
-          <mesh filename="package://robotiq_85_gripper_description/meshes/hros_robotiq_adapter.stl" scale="0.001 0.001 0.001"/>
-        </geometry>
-        <material name="">
-          <color rgba="0.1 0.1 0.1 1" />
-        </material>
-      </visual>
-      <collision>
-        <origin xyz="0 0 0" rpy="0 0 0" />
-        <geometry>
-          <mesh filename="package://robotiq_85_gripper_description/meshes/hros_robotiq_adapter.stl" scale="0.001 0.001 0.001"/>
+          <mesh filename="package://robotiq_85_gripper_description/meshes/hros_robotiq_adapter.dae" scale="0.001 0.001 0.001"/>
+        </geometry>
+        <material name="Gazebo/Black">
+          <color rgba="0.1 0.1 0.1 1" />
+        </material>
+      </visual>
+      <collision>
+        <origin xyz="0 0 0" rpy="0 0 0" />
+        <geometry>
+          <mesh filename="package://robotiq_85_gripper_description/meshes/hros_robotiq_adapter.dae" scale="0.001 0.001 0.001"/>
         </geometry>
       </collision>
     </link>
     <gazebo reference="robotiq_adapter_link">
-      <material>Gazebo/Grey</material>
+      <material>Gazebo/Black</material>
       <selfCollide>True</selfCollide>
     </gazebo>
@@ -39,5 +39,5 @@
           <mesh filename="package://robotiq_85_gripper_description/meshes/base_gripper.stl" scale="0.001 0.001 0.001"/>
         </geometry>
-        <material name="">
+        <material name="Gazebo/Black">
           <color rgba="0.1 0.1 0.1 1" />
         </material>
@@ -51,5 +51,5 @@
     </link>
     <gazebo reference="robotiq_85_base_link">
-      <material>Gazebo/Grey</material>
+      <material>Gazebo/Black</material>
       <selfCollide>True</selfCollide>
     </gazebo>
@@ -65,5 +65,5 @@
           <mesh filename="package://robotiq_85_gripper_description/meshes/2-F-85_1_l.stl" scale="0.001 0.001 0.001"/>
         </geometry>
-        <material name="">
+        <material name="Gazebo/Grey">
           <color rgba="0.1 0.1 0.1 1" />
         </material>
@@ -91,5 +91,5 @@
           <mesh filename="package://robotiq_85_gripper_description/meshes/2-F-85_1_r.stl" scale="0.001 0.001 0.001"/>
         </geometry>
-        <material name="">
+        <material name="Gazebo/Grey">
           <color rgba="0.1 0.1 0.1 1" />
         </material>
@@ -117,5 +117,5 @@
           <mesh filename="package://robotiq_85_gripper_description/meshes/2-F-85_3_l.stl" scale="0.001 0.001 0.001"/>
         </geometry>
-        <material name="">
+        <material name="Gazebo/Black">
           <color rgba="0.1 0.1 0.1 1" />
         </material>
@@ -129,5 +129,5 @@
     </link>
     <gazebo reference="robotiq_85_left_outer_knuckle_link">
-      <material>Gazebo/Grey</material>
+      <material>Gazebo/Black</material>
       <selfCollide>True</selfCollide>
     </gazebo>
@@ -143,5 +143,5 @@
           <mesh filename="package://robotiq_85_gripper_description/meshes/2-F-85_3_r.stl" scale="0.001 0.001 0.001"/>
         </geometry>
-        <material name="">
+        <material name="Gazebo/Black">
           <color rgba="0.1 0.1 0.1 1" />
         </material>
@@ -155,5 +155,5 @@
     </link>
     <gazebo reference="robotiq_85_right_outer_knuckle_link">
-      <material>Gazebo/Grey</material>
+      <material>Gazebo/Black</material>
       <selfCollide>True</selfCollide>
     </gazebo>
@@ -169,5 +169,5 @@
           <mesh filename="package://robotiq_85_gripper_description/meshes/2-F-85_2_l.stl" scale="0.001 0.001 0.001"/>
         </geometry>
-        <material name="">
+        <material name="Gazebo/Black">
           <color rgba="0.1 0.1 0.1 1" />
         </material>
@@ -181,5 +181,5 @@
     </link>
     <gazebo reference="robotiq_85_left_inner_finger_link">
-      <material>Gazebo/Grey</material>
+      <material>Gazebo/Black</material>
       <selfCollide>True</selfCollide>
     </gazebo>
@@ -195,5 +195,5 @@
           <mesh filename="package://robotiq_85_gripper_description/meshes/2-F-85_2_r.stl" scale="0.001 0.001 0.001"/>
         </geometry>
-        <material name="">
+        <material name="Gazebo/Black">
           <color rgba="0.1 0.1 0.1 1" />
         </material>
@@ -207,5 +207,5 @@
     </link>
     <gazebo reference="robotiq_85_right_inner_finger_link">
-      <material>Gazebo/Grey</material>
+      <material>Gazebo/Black</material>
       <selfCollide>True</selfCollide>
     </gazebo>
@@ -221,5 +221,5 @@
           <mesh filename="package://robotiq_85_gripper_description/meshes/2-F-85_4_l.stl" scale="0.001 0.001 0.001"/>
         </geometry>
-        <material name="">
+        <material name="Gazebo/Black">
           <color rgba="0.1 0.1 0.1 1" />
         </material>
@@ -233,5 +233,5 @@
     </link>
     <gazebo reference="robotiq_85_left_finger_link">
-      <material>Gazebo/Grey</material>
+      <material>Gazebo/Black</material>
       <selfCollide>True</selfCollide>
     </gazebo>
@@ -247,5 +247,5 @@
           <mesh filename="package://robotiq_85_gripper_description/meshes/2-F-85_4_r.stl" scale="0.001 0.001 0.001"/>
         </geometry>
-        <material name="">
+        <material name="Gazebo/Black">
           <color rgba="0.1 0.1 0.1 1" />
         </material>
@@ -259,5 +259,5 @@
     </link>
     <gazebo reference="robotiq_85_right_finger_link">
-      <material>Gazebo/Grey</material>
+      <material>Gazebo/Black</material>
       <selfCollide>True</selfCollide>
     </gazebo>
