Commit message: updated urdfs and converted stl to dae

File: robotiq_85_gripper_description/urdf/robotiq_85.urdf.xacro (robot description, xacro)
@@ -11,14 +11,14 @@
         <origin xyz="0 0 0" rpy="0 0 0" />
         <geometry>
-          <mesh filename="package://robotiq_85_gripper_description/meshes/base_gripper.stl" scale="0.001 0.001 0.001"/>
-        </geometry>
-        <material name="Gazebo/Black">
-          <color rgba="0.1 0.1 0.1 1" />
-        </material>
-      </visual>
-      <collision>
-        <origin xyz="0 0 0" rpy="0 0 0" />
-        <geometry>
-          <mesh filename="package://robotiq_85_gripper_description/meshes/base_gripper.stl" scale="0.001 0.001 0.001"/>
+          <mesh filename="package://robotiq_85_gripper_description/meshes/base_gripper.dae" scale="0.001 0.001 0.001"/>
+        </geometry>
+        <material name="Gazebo/Black">
+          <color rgba="0.1 0.1 0.1 1" />
+        </material>
+      </visual>
+      <collision>
+        <origin xyz="0 0 0" rpy="0 0 0" />
+        <geometry>
+          <mesh filename="package://robotiq_85_gripper_description/meshes/base_gripper.dae" scale="0.001 0.001 0.001"/>
         </geometry>
       </collision>
@@ -37,5 +37,5 @@
         <origin xyz="0 0 0" rpy="0 0 0" />
         <geometry>
-          <mesh filename="package://robotiq_85_gripper_description/meshes/2-F-85_1_l.stl" scale="0.001 0.001 0.001"/>
+          <mesh filename="package://robotiq_85_gripper_description/meshes/2-F-85_1_l.dae" scale="0.001 0.001 0.001"/>
         </geometry>
         <material name="Gazebo/Grey">
@@ -46,5 +46,5 @@
         <origin xyz="0 0 0" rpy="0 0 0" />
         <geometry>
-          <mesh filename="package://robotiq_85_gripper_description/meshes/2-F-85_1_l.stl" scale="0.001 0.001 0.001"/>
+          <mesh filename="package://robotiq_85_gripper_description/meshes/2-F-85_1_l.dae" scale="0.001 0.001 0.001"/>
         </geometry>
       </collision>
@@ -63,5 +63,5 @@
         <origin xyz="0 0 0" rpy="0 0 0" />
         <geometry>
-          <mesh filename="package://robotiq_85_gripper_description/meshes/2-F-85_1_r.stl" scale="0.001 0.001 0.001"/>
+          <mesh filename="package://robotiq_85_gripper_description/meshes/2-F-85_1_r.dae" scale="0.001 0.001 0.001"/>
         </geometry>
         <material name="Gazebo/Grey">
@@ -72,5 +72,5 @@
         <origin xyz="0 0 0" rpy="0 0 0" />
         <geometry>
-          <mesh filename="package://robotiq_85_gripper_description/meshes/2-F-85_1_r.stl" scale="0.001 0.001 0.001"/>
+          <mesh filename="package://robotiq_85_gripper_description/meshes/2-F-85_1_r.dae" scale="0.001 0.001 0.001"/>
         </geometry>
       </collision>
@@ -89,14 +89,14 @@
         <origin xyz="0 0 0" rpy="0 0 0" />
         <geometry>
-          <mesh filename="package://robotiq_85_gripper_description/meshes/2-F-85_3_l.stl" scale="0.001 0.001 0.001"/>
-        </geometry>
-        <material name="Gazebo/Black">
-          <color rgba="0.1 0.1 0.1 1" />
-        </material>
-      </visual>
-      <collision>
-        <origin xyz="0 0 0" rpy="0 0 0" />
-        <geometry>
-          <mesh filename="package://robotiq_85_gripper_description/meshes/2-F-85_3_l.stl" scale="0.001 0.001 0.001"/>
+          <mesh filename="package://robotiq_85_gripper_description/meshes/2-F-85_3_l.dae" scale="0.001 0.001 0.001"/>
+        </geometry>
+        <material name="Gazebo/Black">
+          <color rgba="0.1 0.1 0.1 1" />
+        </material>
+      </visual>
+      <collision>
+        <origin xyz="0 0 0" rpy="0 0 0" />
+        <geometry>
+          <mesh filename="package://robotiq_85_gripper_description/meshes/2-F-85_3_l.dae" scale="0.001 0.001 0.001"/>
         </geometry>
       </collision>
@@ -115,14 +115,14 @@
         <origin xyz="0 0 0" rpy="0 0 0" />
         <geometry>
-          <mesh filename="package://robotiq_85_gripper_description/meshes/2-F-85_3_r.stl" scale="0.001 0.001 0.001"/>
-        </geometry>
-        <material name="Gazebo/Black">
-          <color rgba="0.1 0.1 0.1 1" />
-        </material>
-      </visual>
-      <collision>
-        <origin xyz="0 0 0" rpy="0 0 0" />
-        <geometry>
-          <mesh filename="package://robotiq_85_gripper_description/meshes/2-F-85_3_r.stl" scale="0.001 0.001 0.001"/>
+          <mesh filename="package://robotiq_85_gripper_description/meshes/2-F-85_3_r.dae" scale="0.001 0.001 0.001"/>
+        </geometry>
+        <material name="Gazebo/Black">
+          <color rgba="0.1 0.1 0.1 1" />
+        </material>
+      </visual>
+      <collision>
+        <origin xyz="0 0 0" rpy="0 0 0" />
+        <geometry>
+          <mesh filename="package://robotiq_85_gripper_description/meshes/2-F-85_3_r.dae" scale="0.001 0.001 0.001"/>
         </geometry>
       </collision>
@@ -141,14 +141,14 @@
         <origin xyz="0 0 0" rpy="0 0 0" />
         <geometry>
-          <mesh filename="package://robotiq_85_gripper_description/meshes/2-F-85_2_l.stl" scale="0.001 0.001 0.001"/>
-        </geometry>
-        <material name="Gazebo/Black">
-          <color rgba="0.1 0.1 0.1 1" />
-        </material>
-      </visual>
-      <collision>
-        <origin xyz="0 0 0" rpy="0 0 0" />
-        <geometry>
-          <mesh filename="package://robotiq_85_gripper_description/meshes/2-F-85_2_l.stl" scale="0.001 0.001 0.001"/>
+          <mesh filename="package://robotiq_85_gripper_description/meshes/2-F-85_2_l.dae" scale="0.001 0.001 0.001"/>
+        </geometry>
+        <material name="Gazebo/Black">
+          <color rgba="0.1 0.1 0.1 1" />
+        </material>
+      </visual>
+      <collision>
+        <origin xyz="0 0 0" rpy="0 0 0" />
+        <geometry>
+          <mesh filename="package://robotiq_85_gripper_description/meshes/2-F-85_2_l.dae" scale="0.001 0.001 0.001"/>
         </geometry>
       </collision>
@@ -167,14 +167,14 @@
         <origin xyz="0 0 0" rpy="0 0 0" />
         <geometry>
-          <mesh filename="package://robotiq_85_gripper_description/meshes/2-F-85_2_r.stl" scale="0.001 0.001 0.001"/>
-        </geometry>
-        <material name="Gazebo/Black">
-          <color rgba="0.1 0.1 0.1 1" />
-        </material>
-      </visual>
-      <collision>
-        <origin xyz="0 0 0" rpy="0 0 0" />
-        <geometry>
-          <mesh filename="package://robotiq_85_gripper_description/meshes/2-F-85_2_r.stl" scale="0.001 0.001 0.001"/>
+          <mesh filename="package://robotiq_85_gripper_description/meshes/2-F-85_2_r.dae" scale="0.001 0.001 0.001"/>
+        </geometry>
+        <material name="Gazebo/Black">
+          <color rgba="0.1 0.1 0.1 1" />
+        </material>
+      </visual>
+      <collision>
+        <origin xyz="0 0 0" rpy="0 0 0" />
+        <geometry>
+          <mesh filename="package://robotiq_85_gripper_description/meshes/2-F-85_2_r.dae" scale="0.001 0.001 0.001"/>
         </geometry>
       </collision>
@@ -193,14 +193,14 @@
         <origin xyz="0 0 0" rpy="0 0 0" />
         <geometry>
-          <mesh filename="package://robotiq_85_gripper_description/meshes/2-F-85_4_l.stl" scale="0.001 0.001 0.001"/>
-        </geometry>
-        <material name="Gazebo/Black">
-          <color rgba="0.1 0.1 0.1 1" />
-        </material>
-      </visual>
-      <collision>
-        <origin xyz="0 0 0" rpy="0 0 0" />
-        <geometry>
-          <mesh filename="package://robotiq_85_gripper_description/meshes/2-F-85_4_l.stl" scale="0.001 0.001 0.001"/>
+          <mesh filename="package://robotiq_85_gripper_description/meshes/2-F-85_4_l.dae" scale="0.001 0.001 0.001"/>
+        </geometry>
+        <material name="Gazebo/Black">
+          <color rgba="0.1 0.1 0.1 1" />
+        </material>
+      </visual>
+      <collision>
+        <origin xyz="0 0 0" rpy="0 0 0" />
+        <geometry>
+          <mesh filename="package://robotiq_85_gripper_description/meshes/2-F-85_4_l.dae" scale="0.001 0.001 0.001"/>
         </geometry>
       </collision>
@@ -219,14 +219,14 @@
         <origin xyz="0 0 0" rpy="0 0 0" />
         <geometry>
-          <mesh filename="package://robotiq_85_gripper_description/meshes/2-F-85_4_r.stl" scale="0.001 0.001 0.001"/>
-        </geometry>
-        <material name="Gazebo/Black">
-          <color rgba="0.1 0.1 0.1 1" />
-        </material>
-      </visual>
-      <collision>
-        <origin xyz="0 0 0" rpy="0 0 0" />
-        <geometry>
-          <mesh filename="package://robotiq_85_gripper_description/meshes/2-F-85_4_r.stl" scale="0.001 0.001 0.001"/>
+          <mesh filename="package://robotiq_85_gripper_description/meshes/2-F-85_4_r.dae" scale="0.001 0.001 0.001"/>
+        </geometry>
+        <material name="Gazebo/Black">
+          <color rgba="0.1 0.1 0.1 1" />
+        </material>
+      </visual>
+      <collision>
+        <origin xyz="0 0 0" rpy="0 0 0" />
+        <geometry>
+          <mesh filename="package://robotiq_85_gripper_description/meshes/2-F-85_4_r.dae" scale="0.001 0.001 0.001"/>
         </geometry>
       </collision>

File: robotiq_85_gripper_description/urdf/robotiq_85_hros_support.urdf.xacro (robot description, xacro)
@@ -37,14 +37,14 @@
         <origin xyz="0 0 0" rpy="0 0 0" />
         <geometry>
-          <mesh filename="package://robotiq_85_gripper_description/meshes/base_gripper.stl" scale="0.001 0.001 0.001"/>
-        </geometry>
-        <material name="Gazebo/Black">
-          <color rgba="0.1 0.1 0.1 1" />
-        </material>
-      </visual>
-      <collision>
-        <origin xyz="0 0 0" rpy="0 0 0" />
-        <geometry>
-          <mesh filename="package://robotiq_85_gripper_description/meshes/base_gripper.stl" scale="0.001 0.001 0.001"/>
+          <mesh filename="package://robotiq_85_gripper_description/meshes/base_gripper.dae" scale="0.001 0.001 0.001"/>
+        </geometry>
+        <material name="Gazebo/Black">
+          <color rgba="0.1 0.1 0.1 1" />
+        </material>
+      </visual>
+      <collision>
+        <origin xyz="0 0 0" rpy="0 0 0" />
+        <geometry>
+          <mesh filename="package://robotiq_85_gripper_description/meshes/base_gripper.dae" scale="0.001 0.001 0.001"/>
         </geometry>
       </collision>
@@ -63,5 +63,5 @@
         <origin xyz="0 0 0" rpy="0 0 0" />
         <geometry>
-          <mesh filename="package://robotiq_85_gripper_description/meshes/2-F-85_1_l.stl" scale="0.001 0.001 0.001"/>
+          <mesh filename="package://robotiq_85_gripper_description/meshes/2-F-85_1_l.dae" scale="0.001 0.001 0.001"/>
         </geometry>
         <material name="Gazebo/Grey">
@@ -72,5 +72,5 @@
         <origin xyz="0 0 0" rpy="0 0 0" />
         <geometry>
-          <mesh filename="package://robotiq_85_gripper_description/meshes/2-F-85_1_l.stl" scale="0.001 0.001 0.001"/>
+          <mesh filename="package://robotiq_85_gripper_description/meshes/2-F-85_1_l.dae" scale="0.001 0.001 0.001"/>
         </geometry>
       </collision>
@@ -89,5 +89,5 @@
         <origin xyz="0 0 0" rpy="0 0 0" />
         <geometry>
-          <mesh filename="package://robotiq_85_gripper_description/meshes/2-F-85_1_r.stl" scale="0.001 0.001 0.001"/>
+          <mesh filename="package://robotiq_85_gripper_description/meshes/2-F-85_1_r.dae" scale="0.001 0.001 0.001"/>
         </geometry>
         <material name="Gazebo/Grey">
@@ -98,5 +98,5 @@
         <origin xyz="0 0 0" rpy="0 0 0" />
         <geometry>
-          <mesh filename="package://robotiq_85_gripper_description/meshes/2-F-85_1_r.stl" scale="0.001 0.001 0.001"/>
+          <mesh filename="package://robotiq_85_gripper_description/meshes/2-F-85_1_r.dae" scale="0.001 0.001 0.001"/>
         </geometry>
       </collision>
@@ -115,14 +115,14 @@
         <origin xyz="0 0 0" rpy="0 0 0" />
         <geometry>
-          <mesh filename="package://robotiq_85_gripper_description/meshes/2-F-85_3_l.stl" scale="0.001 0.001 0.001"/>
-        </geometry>
-        <material name="Gazebo/Black">
-          <color rgba="0.1 0.1 0.1 1" />
-        </material>
-      </visual>
-      <collision>
-        <origin xyz="0 0 0" rpy="0 0 0" />
-        <geometry>
-          <mesh filename="package://robotiq_85_gripper_description/meshes/2-F-85_3_l.stl" scale="0.001 0.001 0.001"/>
+          <mesh filename="package://robotiq_85_gripper_description/meshes/2-F-85_3_l.dae" scale="0.001 0.001 0.001"/>
+        </geometry>
+        <material name="Gazebo/Black">
+          <color rgba="0.1 0.1 0.1 1" />
+        </material>
+      </visual>
+      <collision>
+        <origin xyz="0 0 0" rpy="0 0 0" />
+        <geometry>
+          <mesh filename="package://robotiq_85_gripper_description/meshes/2-F-85_3_l.dae" scale="0.001 0.001 0.001"/>
         </geometry>
       </collision>
@@ -141,14 +141,14 @@
         <origin xyz="0 0 0" rpy="0 0 0" />
         <geometry>
-          <mesh filename="package://robotiq_85_gripper_description/meshes/2-F-85_3_r.stl" scale="0.001 0.001 0.001"/>
-        </geometry>
-        <material name="Gazebo/Black">
-          <color rgba="0.1 0.1 0.1 1" />
-        </material>
-      </visual>
-      <collision>
-        <origin xyz="0 0 0" rpy="0 0 0" />
-        <geometry>
-          <mesh filename="package://robotiq_85_gripper_description/meshes/2-F-85_3_r.stl" scale="0.001 0.001 0.001"/>
+          <mesh filename="package://robotiq_85_gripper_description/meshes/2-F-85_3_r.dae" scale="0.001 0.001 0.001"/>
+        </geometry>
+        <material name="Gazebo/Black">
+          <color rgba="0.1 0.1 0.1 1" />
+        </material>
+      </visual>
+      <collision>
+        <origin xyz="0 0 0" rpy="0 0 0" />
+        <geometry>
+          <mesh filename="package://robotiq_85_gripper_description/meshes/2-F-85_3_r.dae" scale="0.001 0.001 0.001"/>
         </geometry>
       </collision>
@@ -167,14 +167,14 @@
         <origin xyz="0 0 0" rpy="0 0 0" />
         <geometry>
-          <mesh filename="package://robotiq_85_gripper_description/meshes/2-F-85_2_l.stl" scale="0.001 0.001 0.001"/>
-        </geometry>
-        <material name="Gazebo/Black">
-          <color rgba="0.1 0.1 0.1 1" />
-        </material>
-      </visual>
-      <collision>
-        <origin xyz="0 0 0" rpy="0 0 0" />
-        <geometry>
-          <mesh filename="package://robotiq_85_gripper_description/meshes/2-F-85_2_l.stl" scale="0.001 0.001 0.001"/>
+          <mesh filename="package://robotiq_85_gripper_description/meshes/2-F-85_2_l.dae" scale="0.001 0.001 0.001"/>
+        </geometry>
+        <material name="Gazebo/Black">
+          <color rgba="0.1 0.1 0.1 1" />
+        </material>
+      </visual>
+      <collision>
+        <origin xyz="0 0 0" rpy="0 0 0" />
+        <geometry>
+          <mesh filename="package://robotiq_85_gripper_description/meshes/2-F-85_2_l.dae" scale="0.001 0.001 0.001"/>
         </geometry>
       </collision>
@@ -193,14 +193,14 @@
         <origin xyz="0 0 0" rpy="0 0 0" />
         <geometry>
-          <mesh filename="package://robotiq_85_gripper_description/meshes/2-F-85_2_r.stl" scale="0.001 0.001 0.001"/>
-        </geometry>
-        <material name="Gazebo/Black">
-          <color rgba="0.1 0.1 0.1 1" />
-        </material>
-      </visual>
-      <collision>
-        <origin xyz="0 0 0" rpy="0 0 0" />
-        <geometry>
-          <mesh filename="package://robotiq_85_gripper_description/meshes/2-F-85_2_r.stl" scale="0.001 0.001 0.001"/>
+          <mesh filename="package://robotiq_85_gripper_description/meshes/2-F-85_2_r.dae" scale="0.001 0.001 0.001"/>
+        </geometry>
+        <material name="Gazebo/Black">
+          <color rgba="0.1 0.1 0.1 1" />
+        </material>
+      </visual>
+      <collision>
+        <origin xyz="0 0 0" rpy="0 0 0" />
+        <geometry>
+          <mesh filename="package://robotiq_85_gripper_description/meshes/2-F-85_2_r.dae" scale="0.001 0.001 0.001"/>
         </geometry>
       </collision>
@@ -219,14 +219,14 @@
         <origin xyz="0 0 0" rpy="0 0 0" />
         <geometry>
-          <mesh filename="package://robotiq_85_gripper_description/meshes/2-F-85_4_l.stl" scale="0.001 0.001 0.001"/>
-        </geometry>
-        <material name="Gazebo/Black">
-          <color rgba="0.1 0.1 0.1 1" />
-        </material>
-      </visual>
-      <collision>
-        <origin xyz="0 0 0" rpy="0 0 0" />
-        <geometry>
-          <mesh filename="package://robotiq_85_gripper_description/meshes/2-F-85_4_l.stl" scale="0.001 0.001 0.001"/>
+          <mesh filename="package://robotiq_85_gripper_description/meshes/2-F-85_4_l.dae" scale="0.001 0.001 0.001"/>
+        </geometry>
+        <material name="Gazebo/Black">
+          <color rgba="0.1 0.1 0.1 1" />
+        </material>
+      </visual>
+      <collision>
+        <origin xyz="0 0 0" rpy="0 0 0" />
+        <geometry>
+          <mesh filename="package://robotiq_85_gripper_description/meshes/2-F-85_4_l.dae" scale="0.001 0.001 0.001"/>
         </geometry>
       </collision>
@@ -245,14 +245,14 @@
         <origin xyz="0 0 0" rpy="0 0 0" />
         <geometry>
-          <mesh filename="package://robotiq_85_gripper_description/meshes/2-F-85_4_r.stl" scale="0.001 0.001 0.001"/>
-        </geometry>
-        <material name="Gazebo/Black">
-          <color rgba="0.1 0.1 0.1 1" />
-        </material>
-      </visual>
-      <collision>
-        <origin xyz="0 0 0" rpy="0 0 0" />
-        <geometry>
-          <mesh filename="package://robotiq_85_gripper_description/meshes/2-F-85_4_r.stl" scale="0.001 0.001 0.001"/>
+          <mesh filename="package://robotiq_85_gripper_description/meshes/2-F-85_4_r.dae" scale="0.001 0.001 0.001"/>
+        </geometry>
+        <material name="Gazebo/Black">
+          <color rgba="0.1 0.1 0.1 1" />
+        </material>
+      </visual>
+      <collision>
+        <origin xyz="0 0 0" rpy="0 0 0" />
+        <geometry>
+          <mesh filename="package://robotiq_85_gripper_description/meshes/2-F-85_4_r.dae" scale="0.001 0.001 0.001"/>
         </geometry>
       </collision>
