Commit message: Fix robotiq hand-e gripper urdf & include plugin

File: robotiq_hande_gripper_description/urdf/hande_gripper.urdf.xacro (robot description, xacro)
@@ -80,13 +80,23 @@
       <selfCollide>True</selfCollide>
     </gazebo>
-    <joint name="finger1_joint" type="fixed">
+    <gazebo>
+      <plugin filename="librobotiq_linear_gripper_gazebo_plugin.so" name="robotiq_hande_gripper">
+        <left_joint>finger1_joint</left_joint>
+        <right_joint>finger2_joint</right_joint>
+      </plugin>
+    </gazebo>
+    <joint name="finger1_joint" type="prismatic">
       <origin rpy="0 0 0" xyz="0 0 0.0"/>
       <parent link="robotiq_hande_base_link"/>
       <child link="finger1"/>
+      <axis xyz="0 0 -1"/>
+      <limit effort="1000" lower="0" upper="0.024858" velocity="2.0"/>
     </joint>
-    <joint name="finger2_joint" type="fixed">
+    <joint name="finger2_joint" type="prismatic">
       <origin rpy="0 0 0" xyz="0 0 0.0"/>
       <parent link="robotiq_hande_base_link"/>
       <child link="finger2"/>
+      <axis xyz="0 0 1"/>
+      <limit effort="1000" lower="0" upper="0.024858" velocity="2.0"/>
     </joint>
   </xacro:macro>

File: robotiq_hande_gripper_description/urdf/robotiq_hande.urdf (robot description, URDF)
Before this commit: robot robotiq_hande, 4 links, 3 joints
Joints:
- joint finger1_joint: axis (none) -> 0 0 -1; limit (none) -> lower=0 upper=0.024858 effort=1000 velocity=2.0; type fixed -> prismatic
- joint finger2_joint: axis (none) -> 0 0 1; limit (none) -> lower=0 upper=0.024858 effort=1000 velocity=2.0; type fixed -> prismatic
