Commit message: add blue point to RL urdfs

File: mara_description/urdf/reinforcement_learning/mara_robot_gripper_140_run.urdf (robot description, URDF)
Before this commit: robot mara, 25 links, 24 joints
Links:
- link ee_link: geometry visual sphere radius=0.01

File: mara_description/urdf/reinforcement_learning/mara_robot_gripper_140_train.urdf (robot description, URDF)
Before this commit: robot mara, 25 links, 24 joints
Links:
- link ee_link: geometry visual sphere radius=0.01

Commit message: Fix gripper. DONT MERGE

File: mara_description/urdf/reinforcement_learning/mara_robot_gripper_140_run.urdf (robot description, URDF)
Before this commit: robot mara, 24 links, 23 joints
Links:
- added link base_robot, mass 7.033; collision mesh filename=package://mara_description/meshes/Base.dae scale=0.001 0.001 0.001; visual mesh filename=package://mara_description/meshes/Base.dae scale=0.001 0.001 0.001
- link motor1_cover: mass 0.0 -> 5.8
- link motor1_link: mass 5.6 -> 5.8
- link motor2_link: mass 1.236 -> 1.03237
- link motor3_cover: mass 0.0 -> 3.8
- link motor3_link: mass 3.95 -> 3.8
- link motor4_link: mass 1.258 -> 1.1
- link motor5_cover: mass 0.0 -> 2.9
- link motor5_link: mass 2.85 -> 2.9
- link motor6_link: mass 0.14 -> 2.9
Joints:
- added joint joint_bases: type fixed, parent base_link, child base_robot, origin xyz=0 0 0.04 rpy=0 0 0
- joint end_effector_adapter_to_robotiq: origin xyz= 0 0 0.0 rpy=0 0 1.57 -> xyz= 0 0 0 rpy=0 0 1.57
- joint motor1: axis 0 0 1 -> 0 0 -1; limit lower=-3.1416 upper=3.1416 effort=104.0 velocity=1.57 -> lower=-3.1416 upper=3.1416 effort=330.0 velocity=3.1416; origin xyz=0 0 0.02125 rpy=0 0 0 -> xyz=0 0 0.05122 rpy=0 0 0; parent base_link -> base_robot
- joint motor2: axis 1 0 0 -> -1 0 0; limit lower=-2.35 upper=2.35 effort=104.0 velocity=1.57 -> lower=-3.1416 upper=3.1416 effort=330.0 velocity=3.1416
- joint motor3: axis -1 0 0 -> 1 0 0; limit lower=-2.61 upper=2.61 effort=69 velocity=1.57 -> lower=-3.1416 upper=3.1416 effort=330.0 velocity=3.1416
- joint motor4: axis 0 0 1 -> 0 0 -1; limit lower=-3.14 upper=3.14 effort=69 velocity=1.57 -> lower=-3.1416 upper=3.1416 effort=330.0 velocity=3.1416
- joint motor5: axis -1 0 0 -> 1 0 0; limit lower=-2.56 upper=2.56 effort=34 velocity=1.57 -> lower=-3.1416 upper=3.1416 effort=330.0 velocity=3.1416
- joint motor6: axis 0 0 1 -> 0 0 -1; limit lower=-3.14 upper=3.14 effort=34 velocity=1.57 -> lower=-3.1416 upper=3.1416 effort=330.0 velocity=3.1416
- joint table_to_base_joint: origin xyz=0 0 0.62 rpy=0 0 0 -> xyz=0 0 0.62 rpy=0 0 1.57
