Commit message: add new mara models
without the robot_base and, with/without camera + train and run plugin

File: mara_description/urdf/reinforcement_learning/mara_robot_gripper_140_camera_run.urdf (robot description, URDF)
Before this commit: robot mara, 33 links, 32 joints
Links:
- removed link base_robot
- link ee_link: geometry visual sphere radius=0.01
Joints:
- removed joint joint_bases
- joint motor1: origin xyz=0 0 0.05122 rpy=0 0 0 -> xyz=0 0 0.02125 rpy=0 0 0; parent base_robot -> base_link

File: mara_description/urdf/reinforcement_learning/mara_robot_gripper_140_camera_train.urdf (robot description, URDF)
Before this commit: robot mara, 24 links, 23 joints
Links:
- added link camera_color
- added link camera_ir_projector
- added link camera_left_depth
- added link camera_link, mass 0.564; collision mesh filename=package://mara_description/meshes/Intel_RealSense_Depth_Cam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 scale=0.001 0.001 0.001; visual mesh filename=package://mara_description/meshes/Intel_RealSense_Depth_Cam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 scale=0.001 0.001 0.001
- added link camera_right_depth
- added link mara_camera_support1_link, mass 0.1; collision mesh filename=package://mara_description/meshes/Camera_Support_1.dae scale=0.001 0.001 0.001; visual mesh filename=package://mara_description/meshes/Camera_Support_1.dae scale=0.001 0.001 0.001
- added link mara_camera_support2_link, mass 0.1; collision mesh filename=package://mara_description/meshes/Camera_Support_2.dae scale=0.001 0.001 0.001; visual mesh filename=package://mara_description/meshes/Camera_Support_2.dae scale=0.001 0.001 0.001
- added link mara_gripper_adapter, mass 0.1; collision mesh filename=package://mara_description/meshes/ROBOTIQ_Gripper_Adapter.d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 scale=0.001 0.001 0.001; visual mesh filename=package://mara_description/meshes/ROBOTIQ_Gripper_Adapter.d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 scale=0.001 0.001 0.001
Joints:
- removed joint end_effector_adapter_to_robotiq
- added joint camera_support1_to_support2: type fixed, parent mara_camera_support1_link, child mara_camera_support2_link, origin xyz=0 0.01029 -0.0128 rpy=0 0 0
- added joint camera_support2_to_camera: type fixed, parent mara_camera_support2_link, child camera_link, origin xyz=0 0.018 0.012 rpy=0 0 0
- added joint camera_to_color: type fixed, parent camera_link, child camera_color, origin xyz=-0.0325 0.0214 0.0 rpy=0.0 0.0 1.57
- added joint camera_to_ir_projector: type fixed, parent camera_link, child camera_ir_projector, origin xyz=0.0115 0.0214 0.0 rpy=0 0 0
- added joint camera_to_left_depth: type fixed, parent camera_link, child camera_left_depth, origin xyz=-0.0175 0.024 0.0 rpy=0 0 0
- added joint camera_to_right_depth: type fixed, parent camera_link, child camera_right_depth, origin xyz=0.0325 0.024 0.0 rpy=1.57 0 0
- added joint gripper_adapter_to_camera_support1: type fixed, parent mara_gripper_adapter, child mara_camera_support1_link, origin xyz=0 0.03956 -0.0213 rpy=0 0 0
- added joint gripper_adapter_to_robotiq_adapter: type fixed, parent mara_gripper_adapter, child robotiq_adapter_link, origin xyz= 0 0 0 rpy=0 0 1.57
- added joint motor6_to_gripper_adapter: type fixed, parent motor6_link, child mara_gripper_adapter, origin xyz=0 0 0.002026 rpy=0 0 0

File: mara_description/urdf/reinforcement_learning/mara_robot_gripper_140_camera_train.urdf.xacro (robot description, xacro)
@@ -3,7 +3,7 @@
        name="mara" >
   <!-- common stuff -->
-  <xacro:include filename="$(find mara_description)/urdf/mara_gazebo.urdf.xacro" />
+  <xacro:include filename="$(find mara_description)/urdf/reinforcement_learning/mara_gazebo_train.urdf.xacro" />
   <!-- mara -->
-  <xacro:include filename="$(find mara_description)/urdf/mara.urdf.xacro" />
+  <xacro:include filename="$(find mara_description)/urdf/reinforcement_learning/mara_train.urdf.xacro" />
   <xacro:include filename="$(find mara_description)/urdf/camera_gripper_support.urdf.xacro" />
   <xacro:include filename="$(find mara_description)/urdf/rs_d435.urdf.xacro" />
@@ -12,5 +12,5 @@
   <xacro:include filename="$(find mara_description)/urdf/table.urdf.xacro" />
   <!-- arm -->
-  <xacro:mara_robot prefix="" ee_link_distance="0.24"/>
+  <xacro:mara_robot_train prefix="" ee_link_distance="0.24"/>
   <xacro:mara_camera_gripper_support prefix="" />
   <xacro:rs_d435_camera prefix="" />

File: mara_description/urdf/reinforcement_learning/mara_robot_gripper_140_train.urdf (robot description, URDF)
Before this commit: robot mara, 25 links, 24 joints
Links:
- removed link base_robot
Joints:
- removed joint joint_bases
- joint motor1: origin xyz=0 0 0.05122 rpy=0 0 0 -> xyz=0 0 0.02125 rpy=0 0 0; parent base_robot -> base_link

File: mara_description/urdf/reinforcement_learning/mara_train.urdf.xacro (robot description, xacro)
@@ -1,10 +1,7 @@
 <?xml version="1.0"?>
 <robot xmlns:xacro="http://ros.org/wiki/xacro">
-<!--
-  Author: Alejandro  Hernandez
--->
   <xacro:include filename="$(find mara_description)/urdf/mara.transmission.xacro" />
-  <xacro:include filename="$(find mara_description)/urdf/mara_gazebo.urdf.xacro" />
-  <xacro:macro name="mara_robot"  params="prefix ee_link_distance">
+  <xacro:include filename="$(find mara_description)/urdf/reinforcement_learning/mara_gazebo_train.urdf.xacro" />
+  <xacro:macro name="mara_robot_train"  params="prefix ee_link_distance">
     <link name="${prefix}base_link">
       <inertial>
@@ -33,30 +30,4 @@
       <selfCollide>True</selfCollide>
     </gazebo>
-    <link name="${prefix}base_robot">
-      <inertial>
-        <origin rpy="0 0 0" xyz="8.625E-08 -4.6583E-06 0.03145"/>
-        <mass value="7.033"/>
-        <inertia ixx="0.1478344" ixy="0.00001" ixz="0.0" iyy="0.14782335" iyz="0.0" izz="0.29471799"/>
-      </inertial>
-      <visual>
-        <origin rpy="0 0 0" xyz="0 0 0"/>
-        <geometry>
-          <mesh filename="package://mara_description/meshes/Base.dae" scale="0.001 0.001 0.001"/>
-        </geometry>
-        <material name="Gazebo/Black">
-          <color rgba="1. 0. 0. 1.0"/>
-        </material>
-      </visual>
-      <collision>
-        <origin rpy="0 0 0" xyz="0 0 0"/>
-        <geometry>
-          <mesh filename="package://mara_description/meshes/Base.dae" scale="0.001 0.001 0.001"/>
-        </geometry>
-      </collision>
-    </link>
-    <gazebo reference="${prefix}base_robot">
-      <material>Gazebo/Black</material>
-      <selfCollide>True</selfCollide>
-    </gazebo>
     <link name="${prefix}motor1_link">
       <inertial>
@@ -302,16 +273,12 @@
         </material>
       </visual>
+    </link>
     <gazebo reference="${prefix}ee_link">
       <material>Gazebo/Blue</material>
       <selfCollide>False</selfCollide>
     </gazebo>
-    <joint name="${prefix}joint_bases" type="fixed">
-      <origin rpy="0 0 0" xyz="0 0 0.04"/>
+    <joint name="${prefix}motor1" type="revolute">
+      <origin rpy="0 0 0" xyz="0 0 0.02125"/>
       <parent link="${prefix}base_link"/>
-      <child link="${prefix}base_robot"/>
-    </joint>
-    <joint name="${prefix}motor1" type="revolute">
-      <origin rpy="0 0 0" xyz="0 0 0.05122"/>
-      <parent link="${prefix}base_robot"/>
       <child link="${prefix}motor1_link"/>
       <axis xyz="0 0 1"/>
@@ -386,5 +353,5 @@
     </joint>
     <xacro:mara_transmission prefix="${prefix}"/>
-    <xacro:mara_gazebo prefix="${prefix}"/>
+    <xacro:mara_gazebo_train prefix="${prefix}"/>
   </xacro:macro>
 </robot>

Commit message: camera_right_depth roll 0

File: mara_description/urdf/reinforcement_learning/mara_robot_gripper_140_camera_run.urdf (robot description, URDF)
Before this commit: robot mara, 32 links, 31 joints
Joints:
- joint camera_to_right_depth: origin xyz=0.0325 0.024 0.0 rpy=1.57 0 0 -> xyz=0.0325 0.024 0.0 rpy=0 0 0

File: mara_description/urdf/reinforcement_learning/mara_robot_gripper_140_camera_train.urdf (robot description, URDF)
Before this commit: robot mara, 32 links, 31 joints
Joints:
- joint camera_to_right_depth: origin xyz=0.0325 0.024 0.0 rpy=1.57 0 0 -> xyz=0.0325 0.024 0.0 rpy=0 0 0

File: mara_description/urdf/rs_d435.urdf.xacro (robot description, xacro)
@@ -56,5 +56,5 @@
     </gazebo>
     <joint name="camera_to_right_depth" type="fixed">
-      <origin rpy="1.57 0 0" xyz="0.0325 0.024 0.0"/>
+      <origin rpy="0 0 0" xyz="0.0325 0.024 0.0"/>
       <parent link="${prefix}camera_link"/>
       <child link="${prefix}camera_right_depth" />

Commit message: update ee_link distance in rl

File: mara_description/urdf/reinforcement_learning/mara_robot_gripper_140_camera_run.urdf (robot description, URDF)
Before this commit: robot mara, 30 links, 29 joints
Joints:
- joint ee_link: origin xyz=0 0.0 0.24 rpy=0 0 0 -> xyz=0 0.0 0.24497 rpy=0 0 0

File: mara_description/urdf/reinforcement_learning/mara_robot_gripper_140_camera_run.urdf.xacro (robot description, xacro)
@@ -10,5 +10,5 @@
   <xacro:include filename="$(find robotiq_140_gripper_description)/urdf/robotiq_140.urdf.xacro" />
   <!-- arm -->
-  <xacro:mara_robot_run prefix="" ee_link_distance="0.24"/>
+  <xacro:mara_robot_run prefix="" ee_link_distance="0.24497"/>
   <xacro:camera_gripper_support prefix="" />
   <xacro:rs_d435_camera prefix="" />

File: mara_description/urdf/reinforcement_learning/mara_robot_gripper_140_camera_train.urdf (robot description, URDF)
Before this commit: robot mara, 30 links, 29 joints
Joints:
- joint ee_link: origin xyz=0 0.0 0.24 rpy=0 0 0 -> xyz=0 0.0 0.24497 rpy=0 0 0

File: mara_description/urdf/reinforcement_learning/mara_robot_gripper_140_camera_train.urdf.xacro (robot description, xacro)
@@ -10,5 +10,5 @@
   <xacro:include filename="$(find robotiq_140_gripper_description)/urdf/robotiq_140.urdf.xacro" />
   <!-- arm -->
-  <xacro:mara_robot_train prefix="" ee_link_distance="0.24"/>
+  <xacro:mara_robot_train prefix="" ee_link_distance="0.24497"/>
   <xacro:camera_gripper_support prefix="" />
   <xacro:rs_d435_camera prefix="" />
