Commit message: update models  - remove mara1_ prefix  - remove duplicated plugin  - enable multiple robots in rl

File: mara_description/urdf/reinforcement_learning/mara_gazebo_run.urdf.xacro (robot description, xacro)
@@ -1,35 +1,35 @@
 <?xml version="1.0"?>
 <robot xmlns:xacro="http://ros.org/wiki/xacro">
-  <xacro:macro name="mara_gazebo_run" params="prefix">
+  <xacro:macro name="mara_gazebo_run" params="prefix MAC1 MAC2 MAC3">
     <gazebo>
-      <plugin filename="libgazebo_ros_joint_state_publisher.so" name="mara_joint_state">
+      <plugin filename="libgazebo_ros_joint_state_publisher.so" name="${prefix}joint_state">
         <ros>
-          <argument>~/out:=joint_states</argument>
+          <argument>~/out:=${prefix}joint_states</argument>
         </ros>
         <update_rate>25</update_rate>
-        <joint_name>motor1</joint_name>
-        <joint_name>motor2</joint_name>
-        <joint_name>motor3</joint_name>
-        <joint_name>motor4</joint_name>
-        <joint_name>motor5</joint_name>
-        <joint_name>motor6</joint_name>
-        <joint_name>joint_finger</joint_name>
+        <joint_name>${prefix}motor1</joint_name>
+        <joint_name>${prefix}motor2</joint_name>
+        <joint_name>${prefix}motor3</joint_name>
+        <joint_name>${prefix}motor4</joint_name>
+        <joint_name>${prefix}motor5</joint_name>
+        <joint_name>${prefix}motor6</joint_name>
+        <joint_name>${prefix}joint_finger</joint_name>
       </plugin>
-      <plugin filename="libmara_gazebo_joint_plugin.so" name="hrim_actuation_servomotor_000000000001">
+      <plugin filename="libmara_gazebo_joint_plugin.so" name="hrim_actuation_servomotor${MAC1}">
         <ros/>
-        <axis1>motor2</axis1>
-        <axis2>motor1</axis2>
+        <axis1>${prefix}motor2</axis1>
+        <axis2>${prefix}motor1</axis2>
         <type>series14</type>
       </plugin>
-      <plugin filename="libmara_gazebo_joint_plugin.so" name="hrim_actuation_servomotor_000000000002">
+      <plugin filename="libmara_gazebo_joint_plugin.so" name="hrim_actuation_servomotor${MAC2}">
         <ros/>
-        <axis1>motor3</axis1>
-        <axis2>motor4</axis2>
+        <axis1>${prefix}motor3</axis1>
+        <axis2>${prefix}motor4</axis2>
         <type>series17</type>
       </plugin>
-      <plugin filename="libmara_gazebo_joint_plugin.so" name="hrim_actuation_servomotor_000000000003">
+      <plugin filename="libmara_gazebo_joint_plugin.so" name="hrim_actuation_servomotor${MAC3}">
         <ros/>
-        <axis1>motor5</axis1>
-        <axis2>motor6</axis2>
+        <axis1>${prefix}motor5</axis1>
+        <axis2>${prefix}motor6</axis2>
         <type>series20</type>
       </plugin>

File: mara_description/urdf/reinforcement_learning/mara_gazebo_train.urdf.xacro (robot description, xacro)
@@ -1,14 +1,14 @@
 <?xml version="1.0"?>
 <robot xmlns:xacro="http://ros.org/wiki/xacro">
-  <xacro:macro name="mara_gazebo_train" params="prefix">
+  <xacro:macro name="mara_gazebo_train" params="prefix MAC0">
     <gazebo>
-      <plugin filename="libmara_gazebo_joint_training_plugin.so" name="hrim_actuation_servomotor_00000000000">
+      <plugin filename="libmara_gazebo_joint_training_plugin.so" name="hrim_actuation_servomotor${MAC0}">
         <ros/>
-        <axis1>motor2</axis1>
-        <axis2>motor1</axis2>
-        <axis3>motor3</axis3>
-        <axis4>motor4</axis4>
-        <axis5>motor5</axis5>
-        <axis6>motor6</axis6>
+        <axis1>${prefix}motor2</axis1>
+        <axis2>${prefix}motor1</axis2>
+        <axis3>${prefix}motor3</axis3>
+        <axis4>${prefix}motor4</axis4>
+        <axis5>${prefix}motor5</axis5>
+        <axis6>${prefix}motor6</axis6>
       </plugin>
     </gazebo>

File: mara_description/urdf/reinforcement_learning/mara_robot_gripper_140_camera_run.urdf.xacro (robot description, xacro)
@@ -10,8 +10,8 @@
   <xacro:include filename="$(find robotiq_140_gripper_description)/urdf/robotiq_140.urdf.xacro" />
   <!-- arm -->
-  <xacro:mara_robot_run prefix="" ee_link_distance="0.24497"/>
+  <xacro:mara_robot_run prefix="" ee_link_distance="0.24497" MAC1="_000000000001" MAC2="_000000000002" MAC3="_000000000003"/>
   <xacro:camera_gripper_support prefix="" />
   <xacro:rs_d435_camera prefix="" />
-  <xacro:robotiq_gripper prefix="mara" />
+  <xacro:robotiq_gripper prefix="" MAC="_000000000004"/>
   <link name="world"/>
   <link name="base_robot">

File: mara_description/urdf/reinforcement_learning/mara_robot_gripper_140_camera_train.urdf.xacro (robot description, xacro)
@@ -10,8 +10,8 @@
   <xacro:include filename="$(find robotiq_140_gripper_description)/urdf/robotiq_140.urdf.xacro" />
   <!-- arm -->
-  <xacro:mara_robot_train prefix="" ee_link_distance="0.24497"/>
+  <xacro:mara_robot_train prefix="" ee_link_distance="0.24497"  MAC0="_00000000000"/>
   <xacro:camera_gripper_support prefix="" />
   <xacro:rs_d435_camera prefix="" />
-  <xacro:robotiq_gripper prefix="mara" />
+  <xacro:robotiq_gripper prefix="" MAC="_000000000004"/>
   <link name="world"/>
   <link name="base_robot">

File: mara_description/urdf/reinforcement_learning/mara_robot_run.urdf.xacro (robot description, xacro)
@@ -6,5 +6,5 @@
   <xacro:include filename="$(find mara_description)/urdf/reinforcement_learning/mara_run.urdf.xacro"/>
   <!-- arm -->
-  <xacro:mara_robot_run prefix="" ee_link_distance="0.0"/>
+  <xacro:mara_robot_run prefix="" ee_link_distance="0.0" MAC1="_000000000001" MAC2="_000000000002" MAC3="_000000000003"/>
   <link name="world"/>
   <link name="base_robot">

File: mara_description/urdf/reinforcement_learning/mara_robot_train.urdf.xacro (robot description, xacro)
@@ -6,5 +6,5 @@
   <xacro:include filename="$(find mara_description)/urdf/reinforcement_learning/mara_train.urdf.xacro"/>
   <!-- arm -->
-  <xacro:mara_robot_train prefix="" ee_link_distance="0.0"/>
+  <xacro:mara_robot_train prefix="" ee_link_distance="0.0" MAC0="_00000000000"/>
   <link name="world"/>
   <link name="base_robot">

File: mara_description/urdf/reinforcement_learning/mara_run.urdf.xacro (robot description, xacro)
@@ -3,5 +3,5 @@
   <xacro:include filename="$(find mara_description)/urdf/mara.transmission.xacro" />
   <xacro:include filename="$(find mara_description)/urdf/reinforcement_learning/mara_gazebo_run.urdf.xacro" />
-  <xacro:macro name="mara_robot_run"  params="prefix ee_link_distance">
+  <xacro:macro name="mara_robot_run"  params="prefix ee_link_distance MAC1 MAC2 MAC3">
     <link name="${prefix}motor1_link">
       <inertial>
@@ -307,5 +307,5 @@
     </joint>
     <xacro:mara_transmission prefix="${prefix}"/>
-    <xacro:mara_gazebo_run prefix="${prefix}"/>
+    <xacro:mara_gazebo_run prefix="${prefix}" MAC1="${MAC1}" MAC2="${MAC2}" MAC3="${MAC3}"/>
   </xacro:macro>
 </robot>

File: mara_description/urdf/reinforcement_learning/mara_train.urdf.xacro (robot description, xacro)
@@ -3,5 +3,5 @@
   <xacro:include filename="$(find mara_description)/urdf/mara.transmission.xacro" />
   <xacro:include filename="$(find mara_description)/urdf/reinforcement_learning/mara_gazebo_train.urdf.xacro" />
-  <xacro:macro name="mara_robot_train"  params="prefix ee_link_distance">
+  <xacro:macro name="mara_robot_train"  params="prefix ee_link_distance MAC0">
     <link name="${prefix}motor1_link">
       <inertial>
@@ -307,5 +307,5 @@
     </joint>
     <xacro:mara_transmission prefix="${prefix}"/>
-    <xacro:mara_gazebo_train prefix="${prefix}"/>
+    <xacro:mara_gazebo_train prefix="${prefix}" MAC0="${MAC0}"/>
   </xacro:macro>
 </robot>

File: mara_description/urdf/two_mara_robots.urdf (robot description, URDF)
Before this commit: robot mara, 27 links, 26 joints
Links:
- removed link mara1_base_link
- removed link mara1_base_robot
- removed link mara1_ee_link
- removed link mara1_motor1_cover
- removed link mara1_motor1_link
- removed link mara1_motor2_link
- removed link mara1_motor3_cover
- removed link mara1_motor3_link
- removed link mara1_motor4_link
- removed link mara1_motor5_cover
- removed link mara1_motor5_link
- removed link mara1_motor6_link
- removed link mara1_tool0
- added link base_link, mass 7.033; collision mesh filename=package://mara_description/meshes/Base_plancha.dae scale=0.001 0.001 0.001; visual mesh filename=package://mara_description/meshes/Base_plancha.dae scale=0.001 0.001 0.001
- added link base_robot, mass 7.033; collision mesh filename=package://mara_description/meshes/Base.dae scale=0.001 0.001 0.001; visual mesh filename=package://mara_description/meshes/Base.dae scale=0.001 0.001 0.001
- added link ee_link
- added link motor1_cover, mass 0.0; collision mesh filename=package://mara_description/meshes/MARA_T49_Black.dae scale=0.001 0.001 0.001; visual mesh filename=package://mara_description/meshes/MARA_T49_Black.dae scale=0.001 0.001 0.001
- added link motor1_link, mass 5.6; collision mesh filename=package://mara_description/meshes/MARA_T49.dae scale=0.001 0.001 0.001; visual mesh filename=package://mara_description/meshes/MARA_T49.dae scale=0.001 0.001 0.001
- added link motor2_link, mass 1.24; collision mesh filename=package://mara_description/meshes/MARA_Link1.dae scale=0.001 0.001 0.001; visual mesh filename=package://mara_description/meshes/MARA_Link1.dae scale=0.001 0.001 0.001
- added link motor3_cover, mass 0.0; collision mesh filename=package://mara_description/meshes/MARA_T30_Black.dae scale=0.001 0.001 0.001; visual mesh filename=package://mara_description/meshes/MARA_T30_Black.dae scale=0.001 0.001 0.001
- added link motor3_link, mass 3.95; collision mesh filename=package://mara_description/meshes/MARA_T30.dae scale=0.001 0.001 0.001; visual mesh filename=package://mara_description/meshes/MARA_T30.dae scale=0.001 0.001 0.001
- added link motor4_link, mass 1.26; collision mesh filename=package://mara_description/meshes/MARA_Link2.dae scale=0.001 0.001 0.001; visual mesh filename=package://mara_description/meshes/MARA_Link2.dae scale=0.001 0.001 0.001
- added link motor5_cover, mass 0.0; collision mesh filename=package://mara_description/meshes/MARA_T5.4_black.dae scale=0.001 0.001 0.001; visual mesh filename=package://mara_description/meshes/MARA_T5.4_black.dae scale=0.001 0.001 0.001
- added link motor5_link, mass 2.85; collision mesh filename=package://mara_description/meshes/MARA_T5.4.dae scale=0.001 0.001 0.001; visual mesh filename=package://mara_description/meshes/MARA_T5.4.dae scale=0.001 0.001 0.001
- added link motor6_link, mass 0.00001; collision sphere radius=0; visual sphere radius=0
- added link tool0
Joints:
- removed joint mara1_ee_link
- removed joint mara1_joint_bases
- removed joint mara1_motor1
- removed joint mara1_motor1_cover_joint
- removed joint mara1_motor2
- removed joint mara1_motor3
- removed joint mara1_motor3_cover_joint
- removed joint mara1_motor4
- removed joint mara1_motor5
- removed joint mara1_motor5_cover_joint
- removed joint mara1_motor6
- removed joint mara1_motor6_link-tool0_fixed_joint
- added joint ee_link: type fixed, parent motor6_link, child ee_link, origin xyz=0 0.0 0.0 rpy=0 -1.57 0
- added joint joint_bases: type fixed, parent base_link, child base_robot, origin xyz=0 0 0.04 rpy=0 0 0
- added joint motor1: type revolute, parent base_robot, child motor1_link, origin xyz=0 0 0.05122 rpy=0 0 0, axis 0 0 1, limit lower=-3.1416 upper=3.1416 effort=104.0 velocity=1.57
- added joint motor1_cover_joint: type fixed, parent motor1_link, child motor1_cover, origin xyz=0 0 0.0 rpy=0 0 0
- added joint motor2: type revolute, parent motor1_link, child motor2_link, origin xyz=0.118 0 0.1637 rpy=0 0 0, axis 1 0 0, limit lower=-2.35 upper=2.35 effort=104.0 velocity=1.57
- added joint motor3: type revolute, parent motor2_link, child motor3_link, origin xyz=-0.009 0 0.2 rpy=0 0 0, axis -1 0 0, limit lower=-2.61 upper=2.61 effort=69 velocity=1.57
- added joint motor3_cover_joint: type fixed, parent motor3_link, child motor3_cover, origin xyz=0 0 0.0 rpy=0 0 0
- added joint motor4: type revolute, parent motor3_link, child motor4_link, origin xyz=-0.109255 0 0.149255 rpy=0 0 0, axis 0 0 1, limit lower=-3.14 upper=3.14 effort=69 velocity=1.57
- added joint motor5: type revolute, parent motor4_link, child motor5_link, origin xyz=0.1054570 0 0.16074 rpy=0 0 0, axis -1 0 0, limit lower=-2.56 upper=2.56 effort=34 velocity=1.57
- added joint motor5_cover_joint: type fixed, parent motor5_link, child motor5_cover, origin xyz=0 0 0.0 rpy=0 0 0
- added joint motor6: type revolute, parent motor5_link, child motor6_link, origin xyz=-0.10625569 0 0.14675569 rpy=0 0 0, axis 0 0 1, limit lower=-3.14 upper=3.14 effort=34 velocity=1.57
- added joint motor6_link-tool0_fixed_joint: type fixed, parent motor6_link, child tool0, origin xyz=0 0.0 0.0 rpy=0 -1.57 0
- joint world_to_base1_joint: child mara1_base_link -> base_link
