Commit message: update models  - remove mara1_ prefix  - remove duplicated plugin  - enable multiple robots in rl

File: mara_description/urdf/two_mara_robots_gripper_140_no_table.urdf (robot description, URDF)
Before this commit: robot mara, 49 links, 48 joints
Links:
- removed link mara1_base_link
- removed link mara1_base_robot
- removed link mara1_ee_link
- removed link mara1_gripper_adapter
- removed link mara1_left_inner_finger
- removed link mara1_left_inner_knuckle
- removed link mara1_left_outer_finger
- removed link mara1_left_outer_knuckle
- removed link mara1_motor1_cover
- removed link mara1_motor1_link
- removed link mara1_motor2_link
- removed link mara1_motor3_cover
- removed link mara1_motor3_link
- removed link mara1_motor4_link
- removed link mara1_motor5_cover
- removed link mara1_motor5_link
- removed link mara1_motor6_link
- removed link mara1_right_inner_finger
- removed link mara1_right_inner_knuckle
- removed link mara1_right_outer_finger
- removed link mara1_right_outer_knuckle
- removed link mara1_robotiq_adapter_link
- removed link mara1_robotiq_arg2f_base_link
- removed link mara1_tool0
- added link base_link, mass 7.033; collision mesh filename=package://mara_description/meshes/Base_plancha.dae scale=0.001 0.001 0.001; visual mesh filename=package://mara_description/meshes/Base_plancha.dae scale=0.001 0.001 0.001
- added link base_robot, mass 7.033; collision mesh filename=package://mara_description/meshes/Base.dae scale=0.001 0.001 0.001; visual mesh filename=package://mara_description/meshes/Base.dae scale=0.001 0.001 0.001
- added link ee_link
- added link gripper_adapter, mass 0.13969; collision mesh filename=package://mara_description/meshes/gripper_adapter.dae scale=0.001 0.001 0.001; visual mesh filename=package://mara_description/meshes/gripper_adapter.dae scale=0.001 0.001 0.001
- added link left_inner_finger, mass 0.045; collision mesh filename=package://robotiq_140_gripper_description/meshes/robotiq_14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 scale=0.001 0.001 0.001; visual mesh filename=package://robotiq_140_gripper_description/meshes/robotiq_14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 scale=0.001 0.001 0.001
- added link left_inner_knuckle, mass 0.04476; collision mesh filename=package://robotiq_140_gripper_description/meshes/robotiq_14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 scale=0.001 0.001 0.001; visual mesh filename=package://robotiq_140_gripper_description/meshes/robotiq_14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 scale=0.001 0.001 0.001
- added link left_outer_finger, mass 0.07637; collision mesh filename=package://robotiq_140_gripper_description/meshes/robotiq_14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 scale=0.001 0.001 0.001; visual mesh filename=package://robotiq_140_gripper_description/meshes/robotiq_14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 scale=0.001 0.001 0.001
- added link left_outer_knuckle, mass 0.0131; collision mesh filename=package://robotiq_140_gripper_description/meshes/robotiq_14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 scale=0.001 0.001 0.001; visual mesh filename=package://robotiq_140_gripper_description/meshes/robotiq_14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 scale=0.001 0.001 0.001
- added link motor1_cover, mass 0.0; collision mesh filename=package://mara_description/meshes/MARA_T49_Black.dae scale=0.001 0.001 0.001; visual mesh filename=package://mara_description/meshes/MARA_T49_Black.dae scale=0.001 0.001 0.001
- added link motor1_link, mass 5.6; collision mesh filename=package://mara_description/meshes/MARA_T49.dae scale=0.001 0.001 0.001; visual mesh filename=package://mara_description/meshes/MARA_T49.dae scale=0.001 0.001 0.001
- added link motor2_link, mass 1.24; collision mesh filename=package://mara_description/meshes/MARA_Link1.dae scale=0.001 0.001 0.001; visual mesh filename=package://mara_description/meshes/MARA_Link1.dae scale=0.001 0.001 0.001
- added link motor3_cover, mass 0.0; collision mesh filename=package://mara_description/meshes/MARA_T30_Black.dae scale=0.001 0.001 0.001; visual mesh filename=package://mara_description/meshes/MARA_T30_Black.dae scale=0.001 0.001 0.001
- added link motor3_link, mass 3.95; collision mesh filename=package://mara_description/meshes/MARA_T30.dae scale=0.001 0.001 0.001; visual mesh filename=package://mara_description/meshes/MARA_T30.dae scale=0.001 0.001 0.001
- added link motor4_link, mass 1.26; collision mesh filename=package://mara_description/meshes/MARA_Link2.dae scale=0.001 0.001 0.001; visual mesh filename=package://mara_description/meshes/MARA_Link2.dae scale=0.001 0.001 0.001
- added link motor5_cover, mass 0.0; collision mesh filename=package://mara_description/meshes/MARA_T5.4_black.dae scale=0.001 0.001 0.001; visual mesh filename=package://mara_description/meshes/MARA_T5.4_black.dae scale=0.001 0.001 0.001
- added link motor5_link, mass 2.85; collision mesh filename=package://mara_description/meshes/MARA_T5.4.dae scale=0.001 0.001 0.001; visual mesh filename=package://mara_description/meshes/MARA_T5.4.dae scale=0.001 0.001 0.001
- added link motor6_link, mass 0.00001; collision sphere radius=0; visual sphere radius=0
- added link right_inner_finger, mass 0.045; collision mesh filename=package://robotiq_140_gripper_description/meshes/robotiq_14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 scale=0.001 0.001 0.001; visual mesh filename=package://robotiq_140_gripper_description/meshes/robotiq_14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 scale=0.001 0.001 0.001
- added link right_inner_knuckle, mass 0.04476; collision mesh filename=package://robotiq_140_gripper_description/meshes/robotiq_14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 scale=0.001 0.001 0.001; visual mesh filename=package://robotiq_140_gripper_description/meshes/robotiq_14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 scale=0.001 0.001 0.001
- added link right_outer_finger, mass 0.07637; collision mesh filename=package://robotiq_140_gripper_description/meshes/robotiq_14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 scale=0.001 0.001 0.001; visual mesh filename=package://robotiq_140_gripper_description/meshes/robotiq_14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 scale=0.001 0.001 0.001
- added link right_outer_knuckle, mass 0.0131; collision mesh filename=package://robotiq_140_gripper_description/meshes/robotiq_14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 scale=0.001 0.001 0.001; visual mesh filename=package://robotiq_140_gripper_description/meshes/robotiq_14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 scale=0.001 0.001 0.001
- added link robotiq_adapter_link, mass 0.22652; collision mesh filename=package://mara_description/meshes/robotiq_adapter.dae scale=0.001 0.001 0.001; visual mesh filename=package://mara_description/meshes/robotiq_adapter.dae scale=0.001 0.001 0.001
- added link robotiq_arg2f_base_link, mass 0.52954; collision mesh filename=package://robotiq_140_gripper_description/meshes/GRIPPER_ba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 scale=0.001 0.001 0.001; visual mesh filename=package://robotiq_140_gripper_description/meshes/GRIPPER_ba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 scale=0.001 0.001 0.001
- added link tool0
Joints:
- removed joint mara1_ee_link
- removed joint mara1_joint_bases
- removed joint mara1_joint_finger
- removed joint mara1_left_outer_finger_to_inner
- removed joint mara1_left_outer_knuckle_to_finger
- removed joint mara1_motor1
- removed joint mara1_motor1_cover_joint
- removed joint mara1_motor2
- removed joint mara1_motor3
- removed joint mara1_motor3_cover_joint
- removed joint mara1_motor4
- removed joint mara1_motor5
- removed joint mara1_motor5_cover_joint
- removed joint mara1_motor6
- removed joint mara1_motor6_link-tool0_fixed_joint
- removed joint mara1_right_outer_finger_to_inner
- removed joint mara1_right_outer_knuckle_to_finger
- removed joint robotiq_arg2f_base_to_mara1_left_inner_knuckle
- removed joint robotiq_arg2f_base_to_mara1_left_outer_knuckle
- removed joint robotiq_arg2f_base_to_mara1_right_inner_knuckle
- added joint ee_link: type fixed, parent motor6_link, child ee_link, origin xyz=0 0.0 0.24497 rpy=0 -1.57 0
- added joint joint_bases: type fixed, parent base_link, child base_robot, origin xyz=0 0 0.04 rpy=0 0 0
- added joint joint_finger: type revolute, parent robotiq_arg2f_base_link, child right_outer_knuckle, origin xyz=-0.0306 0 0.05466 rpy=0 0 0, axis 0 1 0, limit lower=0 upper=0.78574722925 effort=18.65 velocity=3.54
- added joint left_outer_finger_to_inner: type revolute, parent left_outer_finger, child left_inner_finger, origin xyz=0.03543 0 0.0789 rpy=0 0 0, axis 0 1 0, limit lower=0 upper=0.78574722925 effort=18.65 velocity=3.54, mimic joint=joint_finger multiplier=1 offset=0
- added joint left_outer_knuckle_to_finger: type fixed, parent left_outer_knuckle, child left_outer_finger, origin xyz=0.03142 0 -0.00453 rpy=0 0 0
- added joint motor1: type revolute, parent base_robot, child motor1_link, origin xyz=0 0 0.05122 rpy=0 0 0, axis 0 0 1, limit lower=-3.1416 upper=3.1416 effort=104.0 velocity=1.57
- added joint motor1_cover_joint: type fixed, parent motor1_link, child motor1_cover, origin xyz=0 0 0.0 rpy=0 0 0
- added joint motor2: type revolute, parent motor1_link, child motor2_link, origin xyz=0.118 0 0.1637 rpy=0 0 0, axis 1 0 0, limit lower=-2.35 upper=2.35 effort=104.0 velocity=1.57
- added joint motor3: type revolute, parent motor2_link, child motor3_link, origin xyz=-0.009 0 0.2 rpy=0 0 0, axis -1 0 0, limit lower=-2.61 upper=2.61 effort=69 velocity=1.57
- added joint motor3_cover_joint: type fixed, parent motor3_link, child motor3_cover, origin xyz=0 0 0.0 rpy=0 0 0
- added joint motor4: type revolute, parent motor3_link, child motor4_link, origin xyz=-0.109255 0 0.149255 rpy=0 0 0, axis 0 0 1, limit lower=-3.14 upper=3.14 effort=69 velocity=1.57
- added joint motor5: type revolute, parent motor4_link, child motor5_link, origin xyz=0.1054570 0 0.16074 rpy=0 0 0, axis -1 0 0, limit lower=-2.56 upper=2.56 effort=34 velocity=1.57
- added joint motor5_cover_joint: type fixed, parent motor5_link, child motor5_cover, origin xyz=0 0 0.0 rpy=0 0 0
- added joint motor6: type revolute, parent motor5_link, child motor6_link, origin xyz=-0.10625569 0 0.14675569 rpy=0 0 0, axis 0 0 1, limit lower=-3.14 upper=3.14 effort=34 velocity=1.57
- added joint motor6_link-tool0_fixed_joint: type fixed, parent motor6_link, child tool0, origin xyz=0 0.0 0.24497 rpy=0 -1.57 0
- added joint right_outer_finger_to_inner: type revolute, parent right_outer_finger, child right_inner_finger, origin xyz=-0.03543 0 0.0789 rpy=0 0 0, axis 0 -1 0, limit lower=0 upper=0.78574722925 effort=18.65 velocity=3.54, mimic joint=joint_finger multiplier=1 offset=0
- added joint right_outer_knuckle_to_finger: type fixed, parent right_outer_knuckle, child right_outer_finger, origin xyz=-0.03142 0 -0.00453 rpy=0 0 0
- added joint robotiq_arg2f_base_to_left_inner_knuckle: type revolute, parent robotiq_arg2f_base_link, child left_inner_knuckle, origin xyz=0.0127 0 0.06118 rpy=0 0 0, axis 0 -1 0, limit lower=0 upper=0.78574722925 effort=18.65 velocity=3.54, mimic joint=joint_finger multiplier=1 offset=0
- added joint robotiq_arg2f_base_to_left_outer_knuckle: type revolute, parent robotiq_arg2f_base_link, child left_outer_knuckle, origin xyz=0.0306 0 0.05466 rpy=0 0 0, axis 0 -1 0, limit lower=0 upper=0.78574722925 effort=18.65 velocity=2.0, mimic joint=joint_finger multiplier=1 offset=0
- added joint robotiq_arg2f_base_to_right_inner_knuckle: type revolute, parent robotiq_arg2f_base_link, child right_inner_knuckle, origin xyz=-0.0127 0 0.06118 rpy=0 0 0, axis 0 1 0, limit lower=0 upper=0.78574722925 effort=18.65 velocity=3.54, mimic joint=joint_finger multiplier=1 offset=0
- joint gripper_adapter_to_robotiq_adapter1: child mara1_robotiq_adapter_link -> robotiq_adapter_link; parent mara1_gripper_adapter -> gripper_adapter
- joint motor6_to_gripper_adapter1: child mara1_gripper_adapter -> gripper_adapter; parent mara1_motor6_link -> motor6_link
- joint robotiq_adapter_to_arg2f_base1: child mara1_robotiq_arg2f_base_link -> robotiq_arg2f_base_link; parent mara1_robotiq_adapter_link -> robotiq_adapter_link
- joint world_to_base1: child mara1_base_link -> base_link
