Commit message: update mara robot run and train according to real robot

File: mara_description/urdf/reinforcement_learning/mara_robot_run.urdf (robot description, URDF)
Before this commit: robot mara, 14 links, 13 joints
Links:
- removed link base_link
- link base_robot: geometry collision mesh filename=package://mara_description/meshes/v8_MARA_Base.dae scale=0.001 0.001 0.001; visual mesh filename=package://mara_description/meshes/v8_MARA_Base.dae scale=0.001 0.001 0.001
- link ee_link: geometry visual sphere radius=0.01
- link motor6_link: mass 0.14 -> 0.00001; geometry collision sphere radius=0; visual sphere radius=0
Joints:
- removed joint joint_bases
- removed joint world_to_base_joint
- added joint world_to_base_robot: type fixed, parent world, child base_robot, origin xyz=0 0 0 rpy=0 0 0
- joint ee_link: origin xyz=0 0.0 0.0 rpy=0 -1.57 0 -> xyz=0 0.0 0.0 rpy=0 0 0
- joint motor1: origin xyz=0 0 0.05122 rpy=0 0 0 -> xyz=0 0 0.06874 rpy=0 0 0
- joint motor6_link-tool0_fixed_joint: origin xyz=0 0.0 0.0 rpy=0 -1.57 0 -> xyz=0 0.0 0.0 rpy=0 0 0

File: mara_description/urdf/reinforcement_learning/mara_robot_run.urdf.xacro (robot description, xacro)
@@ -1,16 +1,49 @@
 <?xml version="1.0"?>
-<robot xmlns:xacro="http://ros.org/wiki/xacro"
-       name="mara" >
+<robot xmlns:xacro="http://ros.org/wiki/xacro" name="mara">
   <!-- common stuff -->
-  <xacro:include filename="$(find mara_description)/urdf/mara_gazebo_run.urdf.xacro" />
+  <xacro:include filename="$(find mara_description)/urdf/reinforcement_learning/mara_gazebo_run.urdf.xacro"/>
   <!-- mara -->
-  <xacro:include filename="$(find mara_description)/urdf/mara_run.urdf.xacro" />
+  <xacro:include filename="$(find mara_description)/urdf/reinforcement_learning/mara_run.urdf.xacro"/>
   <!-- arm -->
   <xacro:mara_robot_run prefix="" ee_link_distance="0.0"/>
-  <link name="world" />
-  <joint name="world_to_base_joint" type="fixed">
+  <link name="world"/>
+  <link name="base_robot">
+    <inertial>
+      <origin rpy="0 0 0" xyz="8.625E-08 -4.6583E-06 0.03145"/>
+      <mass value="7.033"/>
+      <inertia ixx="0.1478344" ixy="0.00001" ixz="0.0" iyy="0.14782335" iyz="0.0" izz="0.29471799"/>
+    </inertial>
+    <visual>
+      <origin rpy="0 0 0" xyz="0 0 0"/>
+      <geometry>
+        <mesh filename="package://mara_description/meshes/v8_MARA_Base.dae" scale="0.001 0.001 0.001"/>
+      </geometry>
+      <material name="Gazebo/Black">
+        <color rgba="1. 0. 0. 1.0"/>
+      </material>
+    </visual>
+    <collision>
+      <origin rpy="0 0 0" xyz="0 0 0"/>
+      <geometry>
+        <mesh filename="package://mara_description/meshes/v8_MARA_Base.dae" scale="0.001 0.001 0.001"/>
+      </geometry>
+    </collision>
+  </link>
+  <gazebo reference="base_robot">
+    <material>Gazebo/Black</material>
+    <selfCollide>True</selfCollide>
+  </gazebo>
+  <joint name="world_to_base_robot" type="fixed">
     <origin rpy="0 0 0" xyz="0 0 0"/>
     <parent link="world"/>
-    <child link="base_link"/>
+    <child link="base_robot"/>
+  </joint>
+  <joint name="motor1" type="revolute">
+    <origin rpy="0 0 0" xyz="0 0 0.06874"/>
+    <parent link="base_robot"/>
+    <child link="motor1_link"/>
+    <axis xyz="0 0 1"/>
+    <limit effort="104.0" lower="-3.1416" upper="3.1416" velocity="1.57"/>
+    <dynamics damping="0" friction="0"/>
   </joint>
 </robot>

File: mara_description/urdf/reinforcement_learning/mara_robot_train.urdf (robot description, URDF)
Before this commit: robot mara, 14 links, 13 joints
Links:
- removed link base_link
- link base_robot: geometry collision mesh filename=package://mara_description/meshes/v8_MARA_Base.dae scale=0.001 0.001 0.001; visual mesh filename=package://mara_description/meshes/v8_MARA_Base.dae scale=0.001 0.001 0.001
- link ee_link: geometry visual sphere radius=0.01
- link motor6_link: mass 0.14 -> 0.00001; geometry collision sphere radius=0; visual sphere radius=0
Joints:
- removed joint joint_bases
- removed joint world_to_base_joint
- added joint world_to_base_robot: type fixed, parent world, child base_robot, origin xyz=0 0 0 rpy=0 0 0
- joint ee_link: origin xyz=0 0.0 0.0 rpy=0 -1.57 0 -> xyz=0 0.0 0.0 rpy=0 0 0
- joint motor1: origin xyz=0 0 0.05122 rpy=0 0 0 -> xyz=0 0 0.06874 rpy=0 0 0
- joint motor6_link-tool0_fixed_joint: origin xyz=0 0.0 0.0 rpy=0 -1.57 0 -> xyz=0 0.0 0.0 rpy=0 0 0

File: mara_description/urdf/reinforcement_learning/mara_robot_train.urdf.xacro (robot description, xacro)
@@ -1,16 +1,49 @@
 <?xml version="1.0"?>
-<robot xmlns:xacro="http://ros.org/wiki/xacro"
-       name="mara" >
+<robot xmlns:xacro="http://ros.org/wiki/xacro" name="mara">
   <!-- common stuff -->
-  <xacro:include filename="$(find mara_description)/urdf/mara_gazebo_train.urdf.xacro" />
+  <xacro:include filename="$(find mara_description)/urdf/reinforcement_learning/mara_gazebo_train.urdf.xacro"/>
   <!-- mara -->
-  <xacro:include filename="$(find mara_description)/urdf/mara_train.urdf.xacro" />
+  <xacro:include filename="$(find mara_description)/urdf/reinforcement_learning/mara_train.urdf.xacro"/>
   <!-- arm -->
   <xacro:mara_robot_train prefix="" ee_link_distance="0.0"/>
-  <link name="world" />
-  <joint name="world_to_base_joint" type="fixed">
+  <link name="world"/>
+  <link name="base_robot">
+    <inertial>
+      <origin rpy="0 0 0" xyz="8.625E-08 -4.6583E-06 0.03145"/>
+      <mass value="7.033"/>
+      <inertia ixx="0.1478344" ixy="0.00001" ixz="0.0" iyy="0.14782335" iyz="0.0" izz="0.29471799"/>
+    </inertial>
+    <visual>
+      <origin rpy="0 0 0" xyz="0 0 0"/>
+      <geometry>
+        <mesh filename="package://mara_description/meshes/v8_MARA_Base.dae" scale="0.001 0.001 0.001"/>
+      </geometry>
+      <material name="Gazebo/Black">
+        <color rgba="1. 0. 0. 1.0"/>
+      </material>
+    </visual>
+    <collision>
+      <origin rpy="0 0 0" xyz="0 0 0"/>
+      <geometry>
+        <mesh filename="package://mara_description/meshes/v8_MARA_Base.dae" scale="0.001 0.001 0.001"/>
+      </geometry>
+    </collision>
+  </link>
+  <gazebo reference="base_robot">
+    <material>Gazebo/Black</material>
+    <selfCollide>True</selfCollide>
+  </gazebo>
+  <joint name="world_to_base_robot" type="fixed">
     <origin rpy="0 0 0" xyz="0 0 0"/>
     <parent link="world"/>
-    <child link="base_link"/>
+    <child link="base_robot"/>
+  </joint>
+  <joint name="motor1" type="revolute">
+    <origin rpy="0 0 0" xyz="0 0 0.06874"/>
+    <parent link="base_robot"/>
+    <child link="motor1_link"/>
+    <axis xyz="0 0 1"/>
+    <limit effort="104.0" lower="-3.1416" upper="3.1416" velocity="1.57"/>
+    <dynamics damping="0" friction="0"/>
   </joint>
 </robot>

File: mara_description/urdf/reinforcement_learning/mara_run.urdf.xacro (robot description, xacro)
@@ -4,30 +4,4 @@
   <xacro:include filename="$(find mara_description)/urdf/reinforcement_learning/mara_gazebo_run.urdf.xacro" />
   <xacro:macro name="mara_robot_run"  params="prefix ee_link_distance">
-    <link name="${prefix}base_link">
-      <inertial>
-        <origin rpy="0 0 0" xyz="8.625E-08 -4.6583E-06 0.03145"/>
-        <mass value="7.033"/>
-        <inertia ixx="0.1478344" ixy="-0.00001" ixz="0.0" iyy="0.14782335" iyz="0.0" izz="0.29471799"/>
-      </inertial>
-      <visual>
-        <origin rpy="0 0 0" xyz="0 0 0"/>
-        <geometry>
-          <mesh filename="package://mara_description/meshes/Base_plancha.dae" scale="0.001 0.001 0.001"/>
-        </geometry>
-        <material name="Gazebo/Grey">
-          <color rgba="0. 0. 0. 1"/>
-        </material>
-      </visual>
-      <collision>
-        <origin rpy="0 0 0" xyz="0 0 0"/>
-        <geometry>
-          <mesh filename="package://mara_description/meshes/Base_plancha.dae" scale="0.001 0.001 0.001"/>
-        </geometry>
-      </collision>
-    </link>
-    <gazebo reference="${prefix}base_link">
-      <material>Gazebo/Grey</material>
-      <selfCollide>True</selfCollide>
-    </gazebo>
     <link name="${prefix}motor1_link">
       <inertial>
@@ -238,30 +212,24 @@
       <selfCollide>True</selfCollide>
     </gazebo>
+    <!-- dummy link with the required tags-->
     <link name="${prefix}motor6_link">
       <inertial>
-        <origin rpy="0 0 0" xyz="0.0 0.0 -0.0173"/>
-        <mass value="0.14"/>
-        <inertia ixx="9.22e-05" ixy="6.35e-7" ixz="2.00e-11" iyy="9.73e-5" iyz="2.36e-9" izz="1.77e-4"/>
-      </inertial>
-      <visual>
-        <origin rpy="0 0 0" xyz="0 0 0"/>
-        <geometry>
-          <mesh filename="package://mara_description/meshes/MARA_GripperAdapter.dae" scale="0.001 0.001 0.001"/>
-        </geometry>
-        <material name="Gazebo/Black">
-          <color rgba="0. 0. 0. 1"/>
-        </material>
-      </visual>
-      <collision>
-        <origin rpy="0 0 0" xyz="0 0 0"/>
-        <geometry>
-          <mesh filename="package://mara_description/meshes/MARA_GripperAdapter.dae" scale="0.001 0.001 0.001"/>
-        </geometry>
-      </collision>
-    </link>
-    <gazebo reference="${prefix}motor6_link">
-      <material>Gazebo/Black</material>
-      <selfCollide>True</selfCollide>
-    </gazebo>
+        <origin rpy="0 0 0" xyz="0 0 0"/>
+        <mass value="0.00001"/>
+        <inertia ixx="0" ixy="0" ixz="0" iyy="0" iyz="0" izz="0"/>
+      </inertial>
+      <visual>
+        <origin rpy="0 0 0" xyz="0 0 0"/>
+        <geometry>
+          <sphere radius="0"/>
+        </geometry>
+      </visual>
+      <collision>
+        <origin rpy="0 0 0" xyz="0 0 0"/>
+        <geometry>
+          <sphere radius="0"/>
+        </geometry>
+      </collision>
+    </link>
     <link name="${prefix}ee_link">
       <visual>
@@ -278,12 +246,4 @@
       <selfCollide>False</selfCollide>
     </gazebo>
-    <joint name="${prefix}motor1" type="revolute">
-      <origin rpy="0 0 0" xyz="0 0 0.02125"/>
-      <parent link="${prefix}base_link"/>
-      <child link="${prefix}motor1_link"/>
-      <axis xyz="0 0 1"/>
-      <limit effort="104.0" lower="-3.1416" upper="3.1416" velocity="1.57"/>
-      <dynamics damping="0" friction="0"/>
-    </joint>
     <joint name="${prefix}motor1_cover_joint" type="fixed">
       <origin rpy="0 0 0" xyz="0 0 0.0"/>
@@ -342,5 +302,5 @@
     </joint>
     <joint name="${prefix}ee_link" type="fixed">
-      <origin rpy="0 -1.57 0" xyz="0 0.0 ${ee_link_distance}"/> <!-- 0.24 -->
+      <origin rpy="0 0 0" xyz="0 0.0 ${ee_link_distance}"/> <!-- 0.24 -->
       <parent link="${prefix}motor6_link"/>
       <child link="${prefix}ee_link"/>
@@ -348,5 +308,5 @@
     <link name="${prefix}tool0"/>
     <joint name="${prefix}${prefix}motor6_link-tool0_fixed_joint" type="fixed">
-      <origin rpy="0 -1.57 0" xyz="0 0.0 ${ee_link_distance}"/>
+      <origin rpy="0 0 0" xyz="0 0.0 ${ee_link_distance}"/>
       <parent link="${prefix}${prefix}motor6_link"/>
       <child link="${prefix}tool0"/>

File: mara_description/urdf/reinforcement_learning/mara_train.urdf.xacro (robot description, xacro)
@@ -4,30 +4,4 @@
   <xacro:include filename="$(find mara_description)/urdf/reinforcement_learning/mara_gazebo_train.urdf.xacro" />
   <xacro:macro name="mara_robot_train"  params="prefix ee_link_distance">
-    <link name="${prefix}base_link">
-      <inertial>
-        <origin rpy="0 0 0" xyz="8.625E-08 -4.6583E-06 0.03145"/>
-        <mass value="7.033"/>
-        <inertia ixx="0.1478344" ixy="-0.00001" ixz="0.0" iyy="0.14782335" iyz="0.0" izz="0.29471799"/>
-      </inertial>
-      <visual>
-        <origin rpy="0 0 0" xyz="0 0 0"/>
-        <geometry>
-          <mesh filename="package://mara_description/meshes/Base_plancha.dae" scale="0.001 0.001 0.001"/>
-        </geometry>
-        <material name="Gazebo/Grey">
-          <color rgba="0. 0. 0. 1"/>
-        </material>
-      </visual>
-      <collision>
-        <origin rpy="0 0 0" xyz="0 0 0"/>
-        <geometry>
-          <mesh filename="package://mara_description/meshes/Base_plancha.dae" scale="0.001 0.001 0.001"/>
-        </geometry>
-      </collision>
-    </link>
-    <gazebo reference="${prefix}base_link">
-      <material>Gazebo/Grey</material>
-      <selfCollide>True</selfCollide>
-    </gazebo>
     <link name="${prefix}motor1_link">
       <inertial>
@@ -238,30 +212,24 @@
       <selfCollide>True</selfCollide>
     </gazebo>
+    <!-- dummy link with the required tags-->
     <link name="${prefix}motor6_link">
       <inertial>
-        <origin rpy="0 0 0" xyz="0.0 0.0 -0.0173"/>
-        <mass value="0.14"/>
-        <inertia ixx="9.22e-05" ixy="6.35e-7" ixz="2.00e-11" iyy="9.73e-5" iyz="2.36e-9" izz="1.77e-4"/>
-      </inertial>
-      <visual>
-        <origin rpy="0 0 0" xyz="0 0 0"/>
-        <geometry>
-          <mesh filename="package://mara_description/meshes/MARA_GripperAdapter.dae" scale="0.001 0.001 0.001"/>
-        </geometry>
-        <material name="Gazebo/Black">
-          <color rgba="0. 0. 0. 1"/>
-        </material>
-      </visual>
-      <collision>
-        <origin rpy="0 0 0" xyz="0 0 0"/>
-        <geometry>
-          <mesh filename="package://mara_description/meshes/MARA_GripperAdapter.dae" scale="0.001 0.001 0.001"/>
-        </geometry>
-      </collision>
-    </link>
-    <gazebo reference="${prefix}motor6_link">
-      <material>Gazebo/Black</material>
-      <selfCollide>True</selfCollide>
-    </gazebo>
+        <origin rpy="0 0 0" xyz="0 0 0"/>
+        <mass value="0.00001"/>
+        <inertia ixx="0" ixy="0" ixz="0" iyy="0" iyz="0" izz="0"/>
+      </inertial>
+      <visual>
+        <origin rpy="0 0 0" xyz="0 0 0"/>
+        <geometry>
+          <sphere radius="0"/>
+        </geometry>
+      </visual>
+      <collision>
+        <origin rpy="0 0 0" xyz="0 0 0"/>
+        <geometry>
+          <sphere radius="0"/>
+        </geometry>
+      </collision>
+    </link>
     <link name="${prefix}ee_link">
       <visual>
@@ -278,12 +246,4 @@
       <selfCollide>False</selfCollide>
     </gazebo>
-    <joint name="${prefix}motor1" type="revolute">
-      <origin rpy="0 0 0" xyz="0 0 0.02125"/>
-      <parent link="${prefix}base_link"/>
-      <child link="${prefix}motor1_link"/>
-      <axis xyz="0 0 1"/>
-      <limit effort="104.0" lower="-3.1416" upper="3.1416" velocity="1.57"/>
-      <dynamics damping="0" friction="0"/>
-    </joint>
     <joint name="${prefix}motor1_cover_joint" type="fixed">
       <origin rpy="0 0 0" xyz="0 0 0.0"/>
@@ -342,5 +302,5 @@
     </joint>
     <joint name="${prefix}ee_link" type="fixed">
-      <origin rpy="0 -1.57 0" xyz="0 0.0 ${ee_link_distance}"/> <!-- 0.24 -->
+      <origin rpy="0 0 0" xyz="0 0.0 ${ee_link_distance}"/> <!-- 0.24 -->
       <parent link="${prefix}motor6_link"/>
       <child link="${prefix}ee_link"/>
@@ -348,5 +308,5 @@
     <link name="${prefix}tool0"/>
     <joint name="${prefix}${prefix}motor6_link-tool0_fixed_joint" type="fixed">
-      <origin rpy="0 -1.57 0" xyz="0 0.0 ${ee_link_distance}"/>
+      <origin rpy="0 0 0" xyz="0 0.0 ${ee_link_distance}"/>
       <parent link="${prefix}${prefix}motor6_link"/>
       <child link="${prefix}tool0"/>

Commit message: adapt for demo

File: mara_description/urdf/reinforcement_learning/mara_robot_run.urdf (robot description, URDF)
Before this commit: robot mara, 12 links, 11 joints
Links:
- link ee_link: geometry 
Joints:
- joint ee_link: origin xyz=0 0.0 0.0 rpy=0 0 0 -> xyz=0 0.0 0.24497 rpy=0 0 0
